File: design-files/pg09-system-clk-rst.kicad_sch (KiCad schematic)
At the start: 13 parts, among them J201 Clock Source, J202 Reset Connector, Q201 2N7000, SW201 SW_Push, U201 CD74ACT109, U202 CD74ACT163, U203 DS1813, X201 ACO-32.000MHz

Commit message: Updates to Clock / Reset generator: - Add 100 ohm series resistors omn E and Q to tamp down signal reflections.   Values may need adjustment in the future. - Add a 3rd bypass cap.
Parts:
- added C203: 0.1µF, symbol Device:C_Small
- added R204, R205: 100, symbol Device:R_Small
Connections:
- net +5V: now also C203.1
- net E: now also R205.2; no longer U201.10 (Q)
- net GND: now also C203.2
- net Q: now also R204.2; no longer U201.13 (~{K}), U201.14 (J), U201.6 (Q)
- new net: R205.1, U201.10 (Q)
- new net: R204.1, U201.13 (~{K}), U201.14 (J), U201.6 (Q)
Other:
- note added: "Series resistors to tamp down over- and under-shoot of E and Q signals. Values may need adjustment."
Changed lines of the file:
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@@
   (junction (at 114.935 79.375) (diameter 0) (color 0 0 0 0)
   )
+  (junction (at 204.47 113.03) (diameter 0) (color 0 0 0 0)
+  )
   (junction (at 83.185 79.375) (diameter 0) (color 0 0 0 0)
   )
@@
   )
   (junction (at 83.185 76.835) (diameter 0) (color 0 0 0 0)
+  )
+  (junction (at 204.47 107.95) (diameter 0) (color 0 0 0 0)
   )
   (junction (at 116.205 81.915) (diameter 0) (color 0 0 0 0)
@@
     (stroke (width 0) (type default) (color 0 0 0 0))
   )
+  (wire (pts (xy 213.995 76.835) (xy 213.995 66.675))
+    (stroke (width 0) (type default) (color 0 0 0 0))
+  )
   (wire (pts (xy 184.785 81.915) (xy 188.595 81.915))
     (stroke (width 0) (type default) (color 0 0 0 0))
@@
     (stroke (width 0) (type default) (color 0 0 0 0))
   )
+  (wire (pts (xy 213.995 66.675) (xy 216.535 66.675))
+    (stroke (width 0) (type default) (color 0 0 0 0))
+  )
+  (wire (pts (xy 221.615 59.69) (xy 229.235 59.69))
+    (stroke (width 0) (type default) (color 0 0 0 0))
+  )
   (wire (pts (xy 184.785 76.835) (xy 188.595 76.835))
     (stroke (width 0) (type default) (color 0 0 0 0))
@@
     (stroke (width 0) (type default) (color 0 0 0 0))
   )
+  (wire (pts (xy 221.615 66.675) (xy 229.235 66.675))
+    (stroke (width 0) (type default) (color 0 0 0 0))
+  )
   (wire (pts (xy 114.935 62.865) (xy 114.935 79.375))
     (stroke (width 0) (type default) (color 0 0 0 0))
@@
     (stroke (width 0) (type default) (color 0 0 0 0))
   )
+  (wire (pts (xy 204.47 113.03) (xy 214.63 113.03))
+    (stroke (width 0) (type default) (color 0 0 0 0))
+  )
   (wire (pts (xy 108.585 81.915) (xy 116.205 81.915))
     (stroke (width 0) (type default) (color 0 0 0 0))
@@
     (stroke (width 0) (type default) (color 0 0 0 0))
   )
-  (wire (pts (xy 184.785 65.405) (xy 213.995 65.405))
-    (stroke (width 0) (type default) (color 0 0 0 0))
-  )
   (wire (pts (xy 106.045 172.085) (xy 106.045 168.275))
     (stroke (width 0) (type default) (color 0 0 0 0))
@@
     (stroke (width 0) (type default) (color 0 0 0 0))
   )
+  (wire (pts (xy 204.47 107.95) (xy 214.63 107.95))
+    (stroke (width 0) (type default) (color 0 0 0 0))
+  )
   (wire (pts (xy 203.835 94.615) (xy 159.385 94.615))
     (stroke (width 0) (type default) (color 0 0 0 0))
@@
     (stroke (width 0) (type default) (color 0 0 0 0))
   )
+  (wire (pts (xy 184.785 59.69) (xy 216.535 59.69))
+    (stroke (width 0) (type default) (color 0 0 0 0))
+  )
   (wire (pts (xy 203.835 76.835) (xy 213.995 76.835))
     (stroke (width 0) (type default) (color 0 0 0 0))
@@
     (stroke (width 0) (type default) (color 0 0 0 0))
   )
-  (wire (pts (xy 184.785 76.835) (xy 184.785 65.405))
+  (wire (pts (xy 184.785 76.835) (xy 184.785 59.69))
     (stroke (width 0) (type default) (color 0 0 0 0))
   )
@@
   (wire (pts (xy 106.045 149.225) (xy 106.045 168.275))
     (stroke (width 0) (type default) (color 0 0 0 0))
+  )
+  (text "Series resistors to tamp down over- and under-shoot\nof E and Q signals.  Values may need adjustment."
+    (at 193.04 52.705 0)
+    (effects (font (size 1.27 1.27)) (justify left bottom))
   )
   (text "Clock Generator" (at 129.54 56.515 0)
@@
     )
   )
-  (global_label "E" (shape output) (at 213.995 76.835 0) (fields_autoplaced)
+  (global_label "E" (shape output) (at 229.235 66.675 0) (fields_autoplaced)
     (effects (font (size 1.27 1.27)) (justify left))
-    (property "Intersheet References" "${INTERSHEET_REFS}" (id 0) (at 217.5571 76.7556 0)
+    (property "Intersheet References" "${INTERSHEET_REFS}" (id 0) (at 232.7971 66.5956 0)
       (effects (font (size 1.27 1.27)) (justify left) hide)
     )
   )
-  (global_label "Q" (shape output) (at 213.995 65.405 0) (fields_autoplaced)
+  (global_label "Q" (shape output) (at 229.235 59.69 0) (fields_autoplaced)
     (effects (font (size 1.27 1.27)) (justify left))
-    (property "Intersheet References" "${INTERSHEET_REFS}" (id 0) (at 217.7386 65.3256 0)
+    (property "Intersheet References" "${INTERSHEET_REFS}" (id 0) (at 232.9786 59.6106 0)
       (effects (font (size 1.27 1.27)) (justify left) hide)
     )
@@
     (pin "2")
   )
+  (symbol (lib_id "Device:C_Small") (at 214.63 110.49 0) (unit 1)
+    (in_bom yes) (on_board yes) (fields_autoplaced)
+    (property "Reference" "C203" (id 0) (at 216.9541 109.6616 0)
+      (effects (font (size 1.27 1.27)) (justify left))
+    )
+    (property "Value" "0.1µF" (id 1) (at 216.9541 112.1985 0)
+      (effects (font (size 1.27 1.27)) (justify left))
+    )
+    (property "Footprint" "" (id 2) (at 214.63 110.49 0)
+      (effects (font (size 1.27 1.27)) hide)
+    )
+    (property "Datasheet" "~" (id 3) (at 214.63 110.49 0)
+      (effects (font (size 1.27 1.27)) hide)
+    )
+    (pin "1")
+    (pin "2")
+  )
   (symbol (lib_id "power:+5V") (at 169.545 100.965 0) (unit 1)
     (in_bom yes) (on_board yes) (fields_autoplaced)
@@
     )
     (pin "1")
+  )
+  (symbol (lib_id "Device:R_Small") (at 219.075 59.69 90) (unit 1)
+    (in_bom yes) (on_board yes)
+    (property "Reference" "R204" (id 0) (at 219.075 55.2536 90))
+    (property "Value" "100" (id 1) (at 219.075 57.7905 90))
+    (property "Footprint" "" (id 2) (at 219.075 59.69 0)
+      (effects (font (size 1.27 1.27)) hide)
+    )
+    (property "Datasheet" "~" (id 3) (at 219.075 59.69 0)
+      (effects (font (size 1.27 1.27)) hide)
+    )
+    (pin "1")
+    (pin "2")
   )
   (symbol (lib_id "74xx:74LS109") (at 169.545 111.125 0) (unit 3)
@@
     (pin "1")
   )
+  (symbol (lib_id "Device:R_Small") (at 219.075 66.675 90) (unit 1)
+    (in_bom yes) (on_board yes)
+    (property "Reference" "R205" (id 0) (at 219.075 62.2386 90))
+    (property "Value" "100" (id 1) (at 219.075 64.7755 90))
+    (property "Footprint" "" (id 2) (at 219.075 66.675 0)
+      (effects (font (size 1.27 1.27)) hide)
+    )
+    (property "Datasheet" "~" (id 3) (at 219.075 66.675 0)
+      (effects (font (size 1.27 1.27)) hide)
+    )
+    (pin "1")
+    (pin "2")
+  )
   (symbol (lib_id "74xx:74LS163") (at 95.885 89.535 0) (unit 1)
