File: design-files/pg09-system-clk-rst.kicad_sch (KiCad schematic)
At the start: 16 parts, among them J201 Clock Source, J202 Reset Connector, Q201 2N7000, SW201 SW_Push, U201 CD74ACT109, U202 CD74ACT163, U203 DS1813, X201 ACO-32.000MHz

Commit message: Assign a bunch of footprints.
Parts:
- C201, C202, C203: footprint (none) -> Capacitor_THT:C_Disc_D6.0mm_W4.4mm_P5.00mm
- U201, U202: footprint (none) -> Package_DIP:DIP-16_W7.62mm_Socket
Changed lines of the file:
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@@
       (effects (font (size 1.27 1.27)) (justify left))
     )
-    (property "Footprint" "" (at 196.215 79.375 0)
+    (property "Footprint" "Package_DIP:DIP-16_W7.62mm_Socket" (at 196.215 79.375 0)
       (effects (font (size 1.27 1.27)) hide)
     )
@@
       (effects (font (size 1.27 1.27)) (justify left))
     )
-    (property "Footprint" "" (at 214.63 110.49 0)
+    (property "Footprint" "Capacitor_THT:C_Disc_D6.0mm_W4.4mm_P5.00mm" (at 214.63 110.49 0)
       (effects (font (size 1.27 1.27)) hide)
     )
@@
       (effects (font (size 1.27 1.27)) (justify left))
     )
-    (property "Footprint" "" (at 204.47 110.49 0)
+    (property "Footprint" "Capacitor_THT:C_Disc_D6.0mm_W4.4mm_P5.00mm" (at 204.47 110.49 0)
       (effects (font (size 1.27 1.27)) hide)
     )
@@
       (effects (font (size 1.27 1.27)) (justify left))
     )
-    (property "Footprint" "" (at 194.31 110.49 0)
+    (property "Footprint" "Capacitor_THT:C_Disc_D6.0mm_W4.4mm_P5.00mm" (at 194.31 110.49 0)
       (effects (font (size 1.27 1.27)) hide)
     )
@@
       (effects (font (size 1.27 1.27)) (justify left))
     )
-    (property "Footprint" "" (at 169.545 111.125 0)
+    (property "Footprint" "Package_DIP:DIP-16_W7.62mm_Socket" (at 169.545 111.125 0)
       (effects (font (size 1.27 1.27)) hide)
     )
@@
       (effects (font (size 1.27 1.27)) (justify left))
     )
-    (property "Footprint" "" (at 169.545 79.375 0)
+    (property "Footprint" "Package_DIP:DIP-16_W7.62mm_Socket" (at 169.545 79.375 0)
       (effects (font (size 1.27 1.27)) hide)
     )
@@
       (effects (font (size 1.27 1.27)) (justify left))
     )
-    (property "Footprint" "" (at 95.885 89.535 0)
-      (effects (font (size 1.27 1.27)) hide)
-    )
+    (property "Footprint" "Package_DIP:DIP-16_W7.62mm_Socket" (at 95.885 89.535 0)
+      (effects (font (size 1.27 1.27)) hide)
+    )

Commit message: Finish assigning footprints.
Parts:
- R201, R202, R203, R204, R205: footprint (none) -> Resistor_THT:R_Axial_DIN0207_L6.3mm_D2.5mm_P7.62mm_Horizontal
- SW201: footprint (none) -> Button_Switch_THT:SW_PUSH_6mm
Changed lines of the file:
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@@
       (effects (font (size 1.27 1.27)) (justify left))
     )
-    (property "Footprint" "" (at 220.345 76.835 0)
+    (property "Footprint" "Resistor_THT:R_Axial_DIN0207_L6.3mm_D2.5mm_P7.62mm_Horizontal" (at 220.345 76.835 0)
       (effects (font (size 1.27 1.27)) hide)
     )
@@
       (effects (font (size 1.27 1.27)) (justify right))
     )
-    (property "Footprint" "" (at 212.725 88.265 0)
+    (property "Footprint" "Resistor_THT:R_Axial_DIN0207_L6.3mm_D2.5mm_P7.62mm_Horizontal" (at 212.725 88.265 0)
       (effects (font (size 1.27 1.27)) hide)
     )
@@
       (effects (font (size 1.27 1.27)))
     )
-    (property "Footprint" "" (at 100.965 163.195 0)
+    (property "Footprint" "Button_Switch_THT:SW_PUSH_6mm" (at 100.965 163.195 0)
       (effects (font (size 1.27 1.27)) hide)
     )
@@
       (effects (font (size 1.27 1.27)) (justify right))
     )
-    (property "Footprint" "" (at 84.455 151.765 0)
+    (property "Footprint" "Resistor_THT:R_Axial_DIN0207_L6.3mm_D2.5mm_P7.62mm_Horizontal" (at 84.455 151.765 0)
       (effects (font (size 1.27 1.27)) hide)
     )
@@
       (effects (font (size 1.27 1.27)))
     )
-    (property "Footprint" "" (at 219.075 59.69 0)
+    (property "Footprint" "Resistor_THT:R_Axial_DIN0207_L6.3mm_D2.5mm_P7.62mm_Horizontal" (at 219.075 59.69 0)
       (effects (font (size 1.27 1.27)) hide)
     )
@@
       (effects (font (size 1.27 1.27)))
     )
-    (property "Footprint" "" (at 219.075 66.675 0)
-      (effects (font (size 1.27 1.27)) hide)
-    )
+    (property "Footprint" "Resistor_THT:R_Axial_DIN0207_L6.3mm_D2.5mm_P7.62mm_Horizontal" (at 219.075 66.675 0)
+      (effects (font (size 1.27 1.27)) hide)
+    )

Commit message: Fix various errors and omissions discovered while working on the first cut of the PCB layout.
Connections:
- net GND: now also J202.2 (Pin_2); no longer J202.1 (Pin_1)
- net ~{RESET}: now also J202.1 (Pin_1); no longer J202.2 (Pin_2)
Other:
- moved on the sheet: J202, R203, SW201, U203

Commit message: Specify a physically smaller bypass cap.
Parts:
- C201, C202, C203: footprint Capacitor_THT:C_Disc_D6.0mm_W4.4mm_P5.00mm -> Capacitor_THT:C_Disc_D3.8mm_W2.6mm_P2.50mm
Changed lines of the file:
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@@
       (effects (font (size 1.27 1.27)) (justify left))
     )
-    (property "Footprint" "Capacitor_THT:C_Disc_D6.0mm_W4.4mm_P5.00mm" (at 214.63 110.49 0)
+    (property "Footprint" "Capacitor_THT:C_Disc_D3.8mm_W2.6mm_P2.50mm" (at 214.63 110.49 0)
       (effects (font (size 1.27 1.27)) hide)
     )
@@
       (effects (font (size 1.27 1.27)) (justify left))
     )
-    (property "Footprint" "Capacitor_THT:C_Disc_D6.0mm_W4.4mm_P5.00mm" (at 204.47 110.49 0)
+    (property "Footprint" "Capacitor_THT:C_Disc_D3.8mm_W2.6mm_P2.50mm" (at 204.47 110.49 0)
       (effects (font (size 1.27 1.27)) hide)
     )
@@
       (effects (font (size 1.27 1.27)) (justify left))
     )
-    (property "Footprint" "Capacitor_THT:C_Disc_D6.0mm_W4.4mm_P5.00mm" (at 194.31 110.49 0)
-      (effects (font (size 1.27 1.27)) hide)
-    )
+    (property "Footprint" "Capacitor_THT:C_Disc_D3.8mm_W2.6mm_P2.50mm" (at 194.31 110.49 0)
+      (effects (font (size 1.27 1.27)) hide)
+    )

Commit message: Name the Reset button.
Parts:
- SW201: value SW_Push -> Reset
Changed lines of the file:
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@@
       (effects (font (size 1.27 1.27)))
     )
-    (property "Value" "SW_Push" (at 101.6 163.5561 0)
+    (property "Value" "Reset" (at 101.6 163.5561 0)
       (effects (font (size 1.27 1.27)))
     )

Commit message: Add the CLKSEL GAL and wire up the Clock Speed register into the IO0SEL memory map.
Parts:
- added C204: 0.1µF, Capacitor_THT:C_Disc_D3.8mm_W2.6mm_P2.50mm, symbol Device:C_Small
- added R206, R207, R208: 10K, Resistor_THT:R_Axial_DIN0207_L6.3mm_D2.5mm_P7.62mm_Horizontal, symbol Device:R_Small
- added U204: GAL22V10, Package_DIP:DIP-24_W7.62mm_Socket, symbol jrt-ICs:GAL22V10
- J201: value Clock Source -> Clock Speed
Connections:
- net +5V: now also C204.1, R206.2, R207.2, R208.2, U204.24 (VCC)
- net CLK_16MHz: now also U204.2 (I2); no longer J201.1 (Pin_1)
- net CLK_4MHz: now also U204.4 (I4); no longer J201.5 (Pin_5)
- net CLK_8MHz: now also U204.3 (I3); no longer J201.3 (Pin_3)
- net E: now also U204.1 (I1/CLK)
- net GND: now also J201.1 (Pin_1), J201.3 (Pin_3), J201.5 (Pin_5), C204.2, U204.12 (GND)
- new net: U201.12 (C), U201.4 (C), U204.14 (IO1)
- new net: J201.2 (Pin_2), R206.1, U204.5 (I5)
- new net: J201.4 (Pin_4), R207.1, U204.6 (I6)
- new net: J201.6 (Pin_6), R208.1, U204.7 (I7)
- new net A4: U204.8 (I8)
- new net D0: U204.23 (IO10)
- new net D1: U204.22 (IO9)
- new net D2: U204.21 (IO8)
- new net D3: U204.20 (IO7)
- new net D4: U204.19 (IO6)
- new net D5: U204.18 (IO5)
- new net D6: U204.17 (IO4)
- new net D7: U204.16 (IO3)
- new net R/~{W}: U204.11 (I11)
- new net nA0: U204.9 (I9)
- new net ~{IO0SEL}: U204.10 (I10)
- no-connect marks 3 -> 5
Other:
- note added: "1MHz"
- note added: "2MHz"
- note added: "4MHz"
- note added: "clksel.chp"
- moved on the sheet: C201, C202, C203, J201, J202, Q201, R201, R202, R203, R204, R205, SW201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

Commit message: Checkpoint with new layout.
Parts:
- removed R206, R207, R208: 10K, Resistor_THT:R_Axial_DIN0207_L6.3mm_D2.5mm_P7.62mm_Horizontal, symbol Device:R_Small
- added RN201: 10K, Resistor_THT:R_Array_SIP9, symbol Device:R_Network08
Connections:
- net +5V: now also RN201.1 (common)
- net GND: now also J201.2 (Pin_2), J201.4 (Pin_4), J201.6 (Pin_6); no longer J201.1 (Pin_1), J201.3 (Pin_3), J201.5 (Pin_5)
- net at U204.5 (I5): now also J201.1 (Pin_1), RN201.7 (R6); no longer J201.2 (Pin_2)
- net at U204.6 (I6): now also J201.3 (Pin_3), RN201.8 (R7); no longer J201.4 (Pin_4)
- net at U204.7 (I7): now also J201.5 (Pin_5), RN201.9 (R8); no longer J201.6 (Pin_6)
- new net ~{FIRQ}: RN201.3 (R2)
- new net ~{HALT}: RN201.4 (R3)
- new net ~{NMI}: RN201.2 (R1)
- no-connect marks 5 -> 7
Other:
- moved on the sheet: J201

Commit message: Move the reset connector to the front panel header.
Parts:
- removed J202: Reset Connector, Connector_PinHeader_2.54mm:PinHeader_1x02_P2.54mm_Vertical, symbol Connector_Generic:Conn_01x02
Changed lines of the file:
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@@
-    (stroke (width 0) (type default))
-  )
-  (wire (pts (xy 69.85 173.355) (xy 69.85 168.275))
     (stroke (width 0) (type default))
   )
@@
     (stroke (width 0) (type default))
   )
-  (wire (pts (xy 73.66 173.355) (xy 69.85 173.355))
-    (stroke (width 0) (type default))
-  )
   (wire (pts (xy 108.585 76.835) (xy 113.665 76.835))
     (stroke (width 0) (type default))
@@
     (stroke (width 0) (type default))
   )
-  (wire (pts (xy 80.01 173.355) (xy 80.01 168.275))
-    (stroke (width 0) (type default))
-  )
   (wire (pts (xy 172.72 74.295) (xy 172.72 79.375))
     (stroke (width 0) (type default))
@@
   )
   (wire (pts (xy 229.235 113.03) (xy 239.395 113.03))
-    (stroke (width 0) (type default))
-  )
-  (wire (pts (xy 76.2 173.355) (xy 80.01 173.355))
     (stroke (width 0) (type default))
   )
@@
         )
       )
-    )
-  )
-  (symbol (lib_id "Connector_Generic:Conn_01x02") (at 73.66 178.435 90) (mirror x) (unit 1)
-    (in_bom yes) (on_board yes) (dnp no)
-    (property "Reference" "J202" (at 71.628 177.6003 90)
-      (effects (font (size 1.27 1.27)) (justify left))
-    )
-    (property "Value" "Reset Connector" (at 71.628 180.1372 90)
-      (effects (font (size 1.27 1.27)) (justify left))
-    )
-    (property "Footprint" "Connector_PinHeader_2.54mm:PinHeader_1x02_P2.54mm_Vertical" (at 73.66 178.435 0)
-      (effects (font (size 1.27 1.27)) hide)
-    )
-    (property "Datasheet" "~" (at 73.66 178.435 0)
-      (effects (font (size 1.27 1.27)) hide)
-    )
-    (pin "1")
-    (pin "2")
-    (instances
-      (project "pg09-system"
-        (path "/44572023-3621-4b3a-bd53-c3b2b3f42871/4db01e9b-9f77-42a7-9351-8914253ebfe9"
-          (reference "J202") (unit 1)
-        )
-      )
