File: design-files/pg09-system.kicad_sch (KiCad schematic)
At the start: 10 parts, among them U101 MC6809E, U102 GAL22V10, U103 74AHCT245, U104 74AHCT245, U105 74AHCT245

Commit message: Add UART interface schematic sheet.
Other:
- added sheet UARTs (pg09-system-uarts.kicad_sch)
Changed lines of the file:
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@@
+    )
+  )
+  (sheet (at 201.93 16.51) (size 34.29 15.24) (fields_autoplaced)
+    (stroke (width 0.1524) (type solid))
+    (fill (color 0 0 0 0.0000))
+    (property "Sheetname" "UARTs" (at 201.93 15.7984 0)
+      (effects (font (size 1.27 1.27)) (justify left bottom))
+    )
+    (property "Sheetfile" "pg09-system-uarts.kicad_sch" (at 201.93 32.3346 0)
+      (effects (font (size 1.27 1.27)) (justify left top))
+    )
+    (instances
+      (project "pg09-system"
+        (path "/44572023-3621-4b3a-bd53-c3b2b3f42871" (page "7"))
+      )
     )
   )

Commit message: Connect the A5-A15 outputs of the 6809 directly to the inputs of the GALs that implement the address decoding logic.
Connections:
- net dA8: now reaches U101.16 (A8), U105.2 (A0)
- net dA9: now reaches U101.17 (A9), U105.3 (A1)
- net dA10: now reaches U101.18 (A10), U105.4 (A2)
- net dA11: now reaches U101.19 (A11), U105.5 (A3)
- net dA12: now reaches U101.20 (A12), U105.6 (A4)
- net dA13: now reaches U101.21 (A13), U105.7 (A5)
- net dA14: now reaches U101.22 (A14), U105.8 (A6)
- net dA15: now reaches U101.23 (A15), U105.9 (A7)
- net dA5: now reaches U101.13 (A5), U104.7 (A5)
- net dA6: now reaches U101.14 (A6), U104.8 (A6)
- net dA7: now reaches U101.15 (A7), U104.9 (A7)
Other:
- note added: "Address Decoder Inputs"
- moved on the sheet: U104, U105

Commit message: Connect the data bus buffer's A/B input to the CPU's R/W output, not the global R/W signal.
Connections:
- net R/~{W}: no longer U103.1 (A->B)
- net at U101.32 (R/~{W}), U102.2 (I2): now also U103.1 (A->B)
Changed lines of the file:
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@@
   (junction (at 110.49 120.65) (diameter 0) (color 0 0 0 0)
+  )
+  (junction (at 100.33 153.67) (diameter 0) (color 0 0 0 0)
   )
   (junction (at 106.68 113.03) (diameter 0) (color 0 0 0 0)
@@
     (stroke (width 0) (type default))
   )
+  (wire (pts (xy 104.14 179.07) (xy 26.67 179.07))
+    (stroke (width 0) (type default))
+  )
   (wire (pts (xy 93.98 105.41) (xy 135.89 105.41))
     (stroke (width 0) (type default))
@@
     (stroke (width 0) (type default))
   )
+  (wire (pts (xy 100.33 153.67) (xy 104.14 153.67))
+    (stroke (width 0) (type default))
+  )
+  (wire (pts (xy 26.67 128.27) (xy 31.75 128.27))
+    (stroke (width 0) (type default))
+  )
   (wire (pts (xy 100.33 156.21) (xy 100.33 171.45))
     (stroke (width 0) (type default))
@@
     (stroke (width 0) (type default))
   )
+  (wire (pts (xy 26.67 179.07) (xy 26.67 128.27))
+    (stroke (width 0) (type default))
+  )
   (wire (pts (xy 57.15 107.95) (xy 68.58 107.95))
     (stroke (width 0) (type default))
@@
   )
   (wire (pts (xy 104.14 87.63) (xy 104.14 107.95))
+    (stroke (width 0) (type default))
+  )
+  (wire (pts (xy 104.14 153.67) (xy 104.14 179.07))
     (stroke (width 0) (type default))
   )
@@
       (effects (font (size 1.27 1.27)) (justify right) hide)
     )
-  )
-  (global_label "R{slash}~{W}" (shape input) (at 31.75 128.27 180) (fields_autoplaced)
-    (effects (font (size 1.27 1.27)) (justify right))
-    (property "Intersheetrefs" "${INTERSHEET_REFS}" (at 24.7923 128.27 0)
-      (effects (font (size 1.27 1.27)) (justify right) hide)
-    )

Commit message: Re-arrange the outputs on the MEMINTF GAL, and drop the IRQF and FIRQF signals, since they're not going to be used at any point in the forseeable future.  Leave the comments that describe decoding them, though, for posterity.
Connections:
- net FIRQF is gone; now on net nA3: U102.18 (IO5)
- net IRQF is gone; now on net nA4: U102.17 (IO4)
- net HALTED: now also U102.21 (IO8); no longer U102.16 (IO3)
- net R/~{W}: now also U102.23 (IO10); no longer U102.20 (IO7)
- net nA2: now also U102.19 (IO6); no longer U102.23 (IO10)
- net nA3: no longer U102.22 (IO9)
- net nA4: no longer U102.21 (IO8)
- net ~{FLASHWR}: now also U102.16 (IO3); no longer U102.19 (IO6)
- no-connect marks 6 -> 8
Changed lines of the file:
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@@
   )
   (no_connect (at 191.77 128.27))
+  (no_connect (at 217.17 120.65))
   (no_connect (at 93.98 151.13))
   (no_connect (at 191.77 133.35))
   (no_connect (at 93.98 148.59))
+  (no_connect (at 217.17 125.73))
   (no_connect (at 93.98 163.83))
   (no_connect (at 191.77 130.81))
@@
     (stroke (width 0) (type default))
   )
-  (wire (pts (xy 217.17 107.95) (xy 226.06 107.95))
+  (wire (pts (xy 217.17 107.95) (xy 228.6 107.95))
     (stroke (width 0) (type default))
   )
@@
     (stroke (width 0) (type default))
   )
-  (wire (pts (xy 217.17 128.27) (xy 226.06 128.27))
-    (stroke (width 0) (type default))
-  )
   (wire (pts (xy 93.98 140.97) (xy 113.03 140.97))
     (stroke (width 0) (type default))
@@
     (stroke (width 0) (type default))
   )
-  (wire (pts (xy 217.17 123.19) (xy 226.06 123.19))
-    (stroke (width 0) (type default))
-  )
   (wire (pts (xy 135.89 138.43) (xy 148.59 138.43))
     (stroke (width 0) (type default))
@@
     (stroke (width 0) (type default))
   )
-  (wire (pts (xy 217.17 113.03) (xy 226.06 113.03))
+  (wire (pts (xy 217.17 113.03) (xy 228.6 113.03))
     (stroke (width 0) (type default))
   )
@@
     (stroke (width 0) (type default))
   )
-  (wire (pts (xy 217.17 118.11) (xy 226.06 118.11))
+  (wire (pts (xy 217.17 118.11) (xy 223.52 118.11))
     (stroke (width 0) (type default))
   )
@@
     )
   )
-  (global_label "nA4" (shape output) (at 226.06 123.19 0) (fields_autoplaced)
-    (effects (font (size 1.27 1.27)) (justify left))
-    (property "Intersheetrefs" "${INTERSHEET_REFS}" (at 232.4129 123.19 0)
+  (global_label "nA4" (shape output) (at 228.6 113.03 0) (fields_autoplaced)
+    (effects (font (size 1.27 1.27)) (justify left))
+    (property "Intersheetrefs" "${INTERSHEET_REFS}" (at 234.9529 113.03 0)
       (effects (font (size 1.27 1.27)) (justify left) hide)
     )
@@
     )
   )
-  (global_label "nA2" (shape output) (at 226.06 128.27 0) (fields_autoplaced)
-    (effects (font (size 1.27 1.27)) (justify left))
-    (property "Intersheetrefs" "${INTERSHEET_REFS}" (at 232.4129 128.27 0)
+  (global_label "nA2" (shape output) (at 223.52 118.11 0) (fields_autoplaced)
+    (effects (font (size 1.27 1.27)) (justify left))
+    (property "Intersheetrefs" "${INTERSHEET_REFS}" (at 229.8729 118.11 0)
       (effects (font (size 1.27 1.27)) (justify left) hide)
     )
@@
     )
   )
-  (global_label "~{WR}" (shape output) (at 226.06 107.95 0) (fields_autoplaced)
-    (effects (font (size 1.27 1.27)) (justify left))
-    (property "Intersheetrefs" "${INTERSHEET_REFS}" (at 231.6872 107.95 0)
+  (global_label "~{WR}" (shape output) (at 228.6 107.95 0) (fields_autoplaced)
+    (effects (font (size 1.27 1.27)) (justify left))
+    (property "Intersheetrefs" "${INTERSHEET_REFS}" (at 234.2272 107.95 0)
       (effects (font (size 1.27 1.27)) (justify left) hide)
     )
@@
     )
   )
-  (global_label "HALTED" (shape output) (at 217.17 110.49 0) (fields_autoplaced)
-    (effects (font (size 1.27 1.27)) (justify left))
-    (property "Intersheetrefs" "${INTERSHEET_REFS}" (at 226.9096 110.49 0)
+  (global_label "HALTED" (shape output) (at 217.17 123.19 0) (fields_autoplaced)
+    (effects (font (size 1.27 1.27)) (justify left))
+    (property "Intersheetrefs" "${INTERSHEET_REFS}" (at 226.9096 123.19 0)
       (effects (font (size 1.27 1.27)) (justify left) hide)
     )
@@
     )
   )
-  (global_label "IRQF" (shape output) (at 226.06 113.03 0) (fields_autoplaced)
-    (effects (font (size 1.27 1.27)) (justify left))
-    (property "Intersheetrefs" "${INTERSHEET_REFS}" (at 233.2597 113.03 0)
-      (effects (font (size 1.27 1.27)) (justify left) hide)
-    )
-  )
   (global_label "dA7" (shape output) (at 128.27 46.99 0) (fields_autoplaced)
     (effects (font (size 1.27 1.27)) (justify left))
@@
     )
   )
-  (global_label "R{slash}~{W}" (shape output) (at 217.17 120.65 0) (fields_autoplaced)
-    (effects (font (size 1.27 1.27)) (justify left))
-    (property "Intersheetrefs" "${INTERSHEET_REFS}" (at 224.1277 120.65 0)
-      (effects (font (size 1.27 1.27)) (justify left) hide)
-    )
-  )
-  (global_label "FIRQF" (shape output) (at 217.17 115.57 0) (fields_autoplaced)
-    (effects (font (size 1.27 1.27)) (justify left))
-    (property "Intersheetrefs" "${INTERSHEET_REFS}" (at 225.4583 115.57 0)
+  (global_label "R{slash}~{W}" (shape output) (at 217.17 128.27 0) (fields_autoplaced)
+    (effects (font (size 1.27 1.27)) (justify left))
+    (property "Intersheetrefs" "${INTERSHEET_REFS}" (at 224.1277 128.27 0)
       (effects (font (size 1.27 1.27)) (justify left) hide)
     )
@@
     )
   )
-  (global_label "~{FLASHWR}" (shape output) (at 226.06 118.11 0) (fields_autoplaced)
-    (effects (font (size 1.27 1.27)) (justify left))
-    (property "Intersheetrefs" "${INTERSHEET_REFS}" (at 237.4325 118.11 0)
+  (global_label "~{FLASHWR}" (shape output) (at 217.17 110.49 0) (fields_autoplaced)
+    (effects (font (size 1.27 1.27)) (justify left))
+    (property "Intersheetrefs" "${INTERSHEET_REFS}" (at 228.5425 110.49 0)
       (effects (font (size 1.27 1.27)) (justify left) hide)
     )
@@
     )
   )
-  (global_label "nA3" (shape output) (at 217.17 125.73 0) (fields_autoplaced)
-    (effects (font (size 1.27 1.27)) (justify left))
-    (property "Intersheetrefs" "${INTERSHEET_REFS}" (at 223.5229 125.73 0)
-      (effects (font (size 1.27 1.27)) (justify left) hide)
-    )
+  (global_label "nA3" (shape output) (at 217.17 115.57 0) (fields_autoplaced)
+    (effects (font (size 1.27 1.27)) (justify left))
+    (property "Intersheetrefs" "${INTERSHEET_REFS}" (at 223.5229 115.57 0)
+      (effects (font (size 1.27 1.27)) (justify left) hide)
+    )

Commit message: Put pull-ups on the outputs of the MEMINTF GAL.
Parts:
- added RN401: 10K, Resistor_THT:R_Array_SIP9, symbol Device:R_Network08
Connections:
- net +5V: now also RN401.1 (common)
- net HALTED: now also RN401.8 (R7)
- net R/~{W}: now also RN401.9 (R8)
- net nA2: now also RN401.7 (R6)
- net nA3: now also RN401.6 (R5)
- net nA4: now also RN401.5 (R4)
- net ~{FLASHWR}: now also RN401.4 (R3)
- net ~{RD}: now also RN401.2 (R1)
- net ~{WR}: now also RN401.3 (R2)
Changed lines of the file:
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@@
+    (stroke (width 0) (type default))
+  )
+  (wire (pts (xy 250.19 114.3) (xy 256.54 114.3))
     (stroke (width 0) (type default))
   )
@@
     (stroke (width 0) (type default))
   )
+  (wire (pts (xy 251.46 109.22) (xy 256.54 109.22))
+    (stroke (width 0) (type default))
+  )
   (wire (pts (xy 31.75 130.81) (xy 31.75 138.43))
     (stroke (width 0) (type default))
@@
     (stroke (width 0) (type default))
   )
+  (wire (pts (xy 250.19 119.38) (xy 256.54 119.38))
+    (stroke (width 0) (type default))
+  )
   (wire (pts (xy 100.33 83.82) (xy 186.69 83.82))
     (stroke (width 0) (type default))
@@
   )
   (wire (pts (xy 161.29 123.19) (xy 167.64 123.19))
+    (stroke (width 0) (type default))
+  )
+  (wire (pts (xy 251.46 104.14) (xy 256.54 104.14))
     (stroke (width 0) (type default))
   )
@@
     )
   )
+  (global_label "R{slash}~{W}" (shape input) (at 256.54 121.92 180) (fields_autoplaced)
+    (effects (font (size 1.27 1.27)) (justify right))
+    (property "Intersheetrefs" "${INTERSHEET_REFS}" (at 249.5823 121.92 0)
+      (effects (font (size 1.27 1.27)) (justify right) hide)
+    )
+  )
   (global_label "A15" (shape output) (at 167.64 175.26 0) (fields_autoplaced)
     (effects (font (size 1.27 1.27)) (justify left))
@@
     )
   )
+  (global_label "nA3" (shape input) (at 250.19 114.3 180) (fields_autoplaced)
+    (effects (font (size 1.27 1.27)) (justify right))
+    (property "Intersheetrefs" "${INTERSHEET_REFS}" (at 243.8371 114.3 0)
+      (effects (font (size 1.27 1.27)) (justify right) hide)
+    )
+  )
+  (global_label "~{WR}" (shape input) (at 256.54 106.68 180) (fields_autoplaced)
+    (effects (font (size 1.27 1.27)) (justify right))
+    (property "Intersheetrefs" "${INTERSHEET_REFS}" (at 250.9128 106.68 0)
+      (effects (font (size 1.27 1.27)) (justify right) hide)
+    )
+  )
   (global_label "D6" (shape bidirectional) (at 31.75 120.65 180) (fields_autoplaced)
     (effects (font (size 1.27 1.27)) (justify right))
@@
     )
   )
+  (global_label "~{RD}" (shape input) (at 251.46 104.14 180) (fields_autoplaced)
+    (effects (font (size 1.27 1.27)) (justify right))
+    (property "Intersheetrefs" "${INTERSHEET_REFS}" (at 246.0142 104.14 0)
+      (effects (font (size 1.27 1.27)) (justify right) hide)
+    )
+  )
+  (global_label "HALTED" (shape input) (at 250.19 119.38 180) (fields_autoplaced)
+    (effects (font (size 1.27 1.27)) (justify right))
+    (property "Intersheetrefs" "${INTERSHEET_REFS}" (at 240.4504 119.38 0)
+      (effects (font (size 1.27 1.27)) (justify right) hide)
+    )
+  )
   (global_label "~{FIRQ}" (shape input) (at 60.96 135.89 180) (fields_autoplaced)
     (effects (font (size 1.27 1.27)) (justify right))
@@
     )
   )
+  (global_label "nA4" (shape input) (at 256.54 111.76 180) (fields_autoplaced)
+    (effects (font (size 1.27 1.27)) (justify right))
+    (property "Intersheetrefs" "${INTERSHEET_REFS}" (at 250.1871 111.76 0)
+      (effects (font (size 1.27 1.27)) (justify right) hide)
+    )
+  )
   (global_label "D2" (shape bidirectional) (at 31.75 110.49 180) (fields_autoplaced)
     (effects (font (size 1.27 1.27)) (justify right))
@@
     )
   )
+  (global_label "nA2" (shape input) (at 256.54 116.84 180) (fields_autoplaced)
+    (effects (font (size 1.27 1.27)) (justify right))
+    (property "Intersheetrefs" "${INTERSHEET_REFS}" (at 250.1871 116.84 0)
+      (effects (font (size 1.27 1.27)) (justify right) hide)
+    )
+  )
   (global_label "A2" (shape output) (at 161.29 110.49 0) (fields_autoplaced)
     (effects (font (size 1.27 1.27)) (justify left))
@@
     (effects (font (size 1.27 1.27)) (justify right))
     (property "Intersheetrefs" "${INTERSHEET_REFS}" (at 177.918 125.73 0)
+      (effects (font (size 1.27 1.27)) (justify right) hide)
+    )
+  )
+  (global_label "~{FLASHWR}" (shape input) (at 251.46 109.22 180) (fields_autoplaced)
+    (effects (font (size 1.27 1.27)) (justify right))
+    (property "Intersheetrefs" "${INTERSHEET_REFS}" (at 240.0875 109.22 0)
       (effects (font (size 1.27 1.27)) (justify right) hide)
     )
@@
     )
   )
+  (symbol (lib_id "Device:R_Network08") (at 261.62 114.3 270) (unit 1)
+    (in_bom yes) (on_board yes) (dnp no) (fields_autoplaced)
+    (property "Reference" "RN401" (at 261.366 99.06 90)
+      (effects (font (size 1.27 1.27)))
+    )
+    (property "Value" "10K" (at 261.366 101.6 90)
+      (effects (font (size 1.27 1.27)))
+    )
+    (property "Footprint" "Resistor_THT:R_Array_SIP9" (at 261.62 126.365 90)
+      (effects (font (size 1.27 1.27)) hide)
+    )
+    (property "Datasheet" "http://www.vishay.com/docs/31509/csc.pdf" (at 261.62 114.3 0)
+      (effects (font (size 1.27 1.27)) hide)
+    )
+    (pin "1")
+    (pin "2")
+    (pin "3")
+    (pin "4")
+    (pin "5")
+    (pin "6")
+    (pin "7")
+    (pin "8")
+    (pin "9")
+    (instances
+      (project "pg09-system"
+        (path "/44572023-3621-4b3a-bd53-c3b2b3f42871/7138fc46-10d4-4cc4-afd5-54717dbe5db7"
+          (reference "RN401") (unit 1)
+        )
+        (path "/44572023-3621-4b3a-bd53-c3b2b3f42871"
+          (reference "RN101") (unit 1)
+        )
+      )
+    )
+  )
   (symbol (lib_id "74xx:74HC245") (at 148.59 118.11 0) (unit 1)
     (in_bom yes) (on_board yes) (dnp no) (fields_autoplaced)
@@
         )
       )
+    )
+  )
+  (symbol (lib_id "power:+5V") (at 266.7 104.14 0) (unit 1)
+    (in_bom yes) (on_board yes) (dnp no) (fields_autoplaced)
+    (property "Reference" "#PWR0115" (at 266.7 107.95 0)
+      (effects (font (size 1.27 1.27)) hide)
+    )
+    (property "Value" "+5V" (at 266.7 100.33 0)
+      (effects (font (size 1.27 1.27)))
+    )
+    (property "Footprint" "" (at 266.7 104.14 0)
+      (effects (font (size 1.27 1.27)) hide)
+    )
+    (property "Datasheet" "" (at 266.7 104.14 0)
+      (effects (font (size 1.27 1.27)) hide)
+    )
+    (pin "1")
+    (instances
+      (project "pg09-system"
+        (path "/44572023-3621-4b3a-bd53-c3b2b3f42871"
+          (reference "#PWR0115") (unit 1)
+        )
+      )

Commit message: Re-arrange outputs on the MEMINTF GAL to make PCB layout easier.
Connections:
- net HALTED: now also RN401.3 (R2), U102.22 (IO9); no longer RN401.8 (R7), U102.21 (IO8)
- net R/~{W}: now also RN401.2 (R1); no longer RN401.9 (R8)
- net nA2: now also RN401.4 (R3), U102.21 (IO8); no longer RN401.7 (R6), U102.19 (IO6)
- net nA3: now also RN401.5 (R4), U102.20 (IO7); no longer RN401.6 (R5), U102.18 (IO5)
- net nA4: now also RN401.6 (R5), U102.19 (IO6); no longer RN401.5 (R4), U102.17 (IO4)
- net ~{FLASHWR}: now also RN401.9 (R8); no longer RN401.4 (R3)
- net ~{RD}: now also RN401.8 (R7), U102.17 (IO4); no longer RN401.2 (R1), U102.14 (IO1)
- net ~{WR}: now also RN401.7 (R6), U102.18 (IO5); no longer RN401.3 (R2), U102.15 (IO2)
Other:
- moved on the sheet: RN401

Commit message: Add pull-ups to all of the address decoder outputs.  Also connect pull-ups to /NMI, /IRQ, /FIRQ, and /HALT (using 4 spares in a resistor network on the address decoder).
Other:
- note added: "~{NMI}, ~{IRQ}, ~{FIRQ}, and ~{HALT} are pulled-up on the Address Decoder sheet."
Changed lines of the file:
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@@
     (stroke (width 0) (type default))
+  )
+  (text "~{NMI}, ~{IRQ}, ~{FIRQ}, and ~{HALT}\nare pulled-up on the Address\nDecoder sheet."
+    (at 34.29 158.75 0)
+    (effects (font (size 1.27 1.27)) (justify left bottom))
   )
   (text "mem_intf.chp" (at 198.12 93.98 0)

Commit message: Assign a bunch of footprints.
Parts:
- C201, C202, C203: footprint (none) -> Capacitor_THT:C_Disc_D6.0mm_W4.4mm_P5.00mm
- U101: footprint Package_DIP:DIP-40_W15.24mm -> Package_DIP:DIP-40_W15.24mm_Socket
- U102: footprint (none) -> Package_DIP:DIP-24_W7.62mm_Socket
- U103, U104, U105: footprint (none) -> Package_DIP:DIP-20_W7.62mm_Socket
Changed lines of the file:
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@@
       (effects (font (size 1.27 1.27)) (justify left))
     )
-    (property "Footprint" "" (at 148.59 170.18 0)
+    (property "Footprint" "Package_DIP:DIP-20_W7.62mm_Socket" (at 148.59 170.18 0)
       (effects (font (size 1.27 1.27)) hide)
     )
@@
       (effects (font (size 1.27 1.27)) (justify left))
     )
-    (property "Footprint" "Package_DIP:DIP-40_W15.24mm" (at 81.28 173.99 0)
+    (property "Footprint" "Package_DIP:DIP-40_W15.24mm_Socket" (at 81.28 173.99 0)
       (effects (font (size 1.27 1.27)) hide)
     )
@@
       (effects (font (size 1.27 1.27)) (justify left))
     )
-    (property "Footprint" "" (at 148.59 118.11 0)
+    (property "Footprint" "Package_DIP:DIP-20_W7.62mm_Socket" (at 148.59 118.11 0)
       (effects (font (size 1.27 1.27)) hide)
     )
@@
       (effects (font (size 1.27 1.27)) (justify left))
     )
-    (property "Footprint" "" (at 220.98 154.94 0)
+    (property "Footprint" "Capacitor_THT:C_Disc_D6.0mm_W4.4mm_P5.00mm" (at 220.98 154.94 0)
       (effects (font (size 1.27 1.27)) hide)
     )
@@
       (effects (font (size 1.27 1.27)) (justify left))
     )
-    (property "Footprint" "" (at 180.34 154.94 0)
+    (property "Footprint" "Capacitor_THT:C_Disc_D6.0mm_W4.4mm_P5.00mm" (at 180.34 154.94 0)
       (effects (font (size 1.27 1.27)) hide)
     )
@@
       (effects (font (size 1.27 1.27)) (justify left))
     )
-    (property "Footprint" "" (at 44.45 118.11 0)
+    (property "Footprint" "Package_DIP:DIP-20_W7.62mm_Socket" (at 44.45 118.11 0)
       (effects (font (size 1.27 1.27)) hide)
     )
@@
       (effects (font (size 1.27 1.27)) (justify left))
     )
-    (property "Footprint" "" (at 210.82 154.94 0)
+    (property "Footprint" "Capacitor_THT:C_Disc_D6.0mm_W4.4mm_P5.00mm" (at 210.82 154.94 0)
       (effects (font (size 1.27 1.27)) hide)
     )
@@
       (effects (font (size 1.27 1.27)) (justify left))
     )
-    (property "Footprint" "" (at 190.5 154.94 0)
+    (property "Footprint" "Capacitor_THT:C_Disc_D6.0mm_W4.4mm_P5.00mm" (at 190.5 154.94 0)
       (effects (font (size 1.27 1.27)) hide)
     )
@@
       (effects (font (size 1.27 1.27)) (justify left))
     )
-    (property "Footprint" "" (at 200.66 154.94 0)
+    (property "Footprint" "Capacitor_THT:C_Disc_D6.0mm_W4.4mm_P5.00mm" (at 200.66 154.94 0)
       (effects (font (size 1.27 1.27)) hide)
     )
@@
       (effects (font (size 1.27 1.27)) (justify left))
     )
-    (property "Footprint" "" (at 204.47 119.38 0)
-      (effects (font (size 1.27 1.27)) hide)
-    )
+    (property "Footprint" "Package_DIP:DIP-24_W7.62mm_Socket" (at 204.47 119.38 0)
+      (effects (font (size 1.27 1.27)) hide)
+    )
