File: design-files/pg09-system.kicad_sch (KiCad schematic)
At the start: 11 parts, among them U101 MC6809E, U102 GAL22V10, U103 74AHCT245, U104 74AHCT245, U105 74AHCT245

Commit message: Add a PSU interface sheet.  Super simple for now.
Connections:
- net +5V: no longer U104.1 (A->B), U105.1 (A->B)
- net A0: now also U104.2 (A0); no longer U104.18 (B0)
- net A1: now also U104.3 (A1); no longer U104.17 (B1)
- net A10: now also U105.4 (A2); no longer U105.16 (B2)
- net A11: now also U105.5 (A3); no longer U105.15 (B3)
- net A12: now also U105.6 (A4); no longer U105.14 (B4)
- net A13: now also U105.7 (A5); no longer U105.13 (B5)
- net A14: now also U105.8 (A6); no longer U105.12 (B6)
- net A15: now also U105.9 (A7); no longer U105.11 (B7)
- net A2: now also U104.4 (A2); no longer U104.16 (B2)
- net A3: now also U104.5 (A3); no longer U104.15 (B3)
- net A4: now also U104.6 (A4); no longer U104.14 (B4)
- net A5: now also U104.7 (A5); no longer U104.13 (B5)
- net A6: now also U104.8 (A6); no longer U104.12 (B6)
- net A7: now also U104.9 (A7); no longer U104.11 (B7)
- net A8: now also U105.2 (A0); no longer U105.18 (B0)
- net A9: now also U105.3 (A1); no longer U105.17 (B1)
- net GND: now also U104.1 (A->B), U105.1 (A->B)
- net dA10: now also U105.16 (B2); no longer U105.4 (A2)
- net dA11: now also U105.15 (B3); no longer U105.5 (A3)
- net dA12: now also U105.14 (B4); no longer U105.6 (A4)
- net dA13: now also U105.13 (B5); no longer U105.7 (A5)
- net dA14: now also U105.12 (B6); no longer U105.8 (A6)
- net dA15: now also U105.11 (B7); no longer U105.9 (A7)
- net dA5: now also U104.13 (B5); no longer U104.7 (A5)
- net dA6: now also U104.12 (B6); no longer U104.8 (A6)
- net dA7: now also U104.11 (B7); no longer U104.9 (A7)
- net dA8: now also U105.18 (B0); no longer U105.2 (A0)
- net dA9: now also U105.17 (B1); no longer U105.3 (A1)
- net at U101.10 (A2), U102.6 (I6): now also U104.16 (B2); no longer U104.4 (A2)
- net at U101.11 (A3), U102.7 (I7): now also U104.15 (B3); no longer U104.5 (A3)
- net at U101.12 (A4), U102.8 (I8): now also U104.14 (B4); no longer U104.6 (A4)
- net at U101.8 (A0): now also U104.18 (B0); no longer U104.2 (A0)
- net at U101.9 (A1), U102.5 (I5): now also U104.17 (B1); no longer U104.3 (A1)
Other:
- added sheet Power Supply (pg09-system-psu.kicad_sch)
Changed lines of the file:
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@@
   (junction (at 190.5 157.48) (diameter 0) (color 0 0 0 0)
   )
+  (junction (at 161.29 130.81) (diameter 0) (color 0 0 0 0)
+  )
   (junction (at 210.82 152.4) (diameter 0) (color 0 0 0 0)
   )
@@
   )
   (junction (at 190.5 152.4) (diameter 0) (color 0 0 0 0)
+  )
+  (junction (at 161.29 182.88) (diameter 0) (color 0 0 0 0)
   )
   (junction (at 104.14 107.95) (diameter 0) (color 0 0 0 0)
@@
     (stroke (width 0) (type default))
   )
+  (wire (pts (xy 161.29 180.34) (xy 161.29 182.88))
+    (stroke (width 0) (type default))
+  )
   (wire (pts (xy 93.98 113.03) (xy 106.68 113.03))
     (stroke (width 0) (type default))
@@
     (stroke (width 0) (type default))
   )
+  (wire (pts (xy 161.29 128.27) (xy 161.29 130.81))
+    (stroke (width 0) (type default))
+  )
   (wire (pts (xy 115.57 130.81) (xy 118.11 130.81))
     (stroke (width 0) (type default))
@@
     (stroke (width 0) (type default))
   )
+  (wire (pts (xy 161.29 182.88) (xy 161.29 190.5))
+    (stroke (width 0) (type default))
+  )
   (wire (pts (xy 185.42 85.09) (xy 185.42 110.49))
     (stroke (width 0) (type default))
@@
     (stroke (width 0) (type default))
   )
+  (wire (pts (xy 161.29 190.5) (xy 148.59 190.5))
+    (stroke (width 0) (type default))
+  )
   (wire (pts (xy 93.98 125.73) (xy 113.03 125.73))
     (stroke (width 0) (type default))
@@
     (stroke (width 0) (type default))
   )
-  (wire (pts (xy 135.89 190.5) (xy 148.59 190.5))
-    (stroke (width 0) (type default))
-  )
   (wire (pts (xy 114.3 54.61) (xy 114.3 128.27))
     (stroke (width 0) (type default))
@@
     (stroke (width 0) (type default))
   )
-  (wire (pts (xy 135.89 138.43) (xy 148.59 138.43))
-    (stroke (width 0) (type default))
-  )
   (wire (pts (xy 184.15 86.36) (xy 184.15 113.03))
     (stroke (width 0) (type default))
@@
     (stroke (width 0) (type default))
   )
+  (wire (pts (xy 161.29 138.43) (xy 148.59 138.43))
+    (stroke (width 0) (type default))
+  )
   (wire (pts (xy 217.17 120.65) (xy 223.52 120.65))
     (stroke (width 0) (type default))
@@
     (stroke (width 0) (type default))
   )
+  (wire (pts (xy 161.29 130.81) (xy 161.29 138.43))
+    (stroke (width 0) (type default))
+  )
   (wire (pts (xy 125.73 175.26) (xy 135.89 175.26))
     (stroke (width 0) (type default))
   )
-  (wire (pts (xy 135.89 130.81) (xy 135.89 138.43))
-    (stroke (width 0) (type default))
-  )
   (wire (pts (xy 210.82 157.48) (xy 220.98 157.48))
     (stroke (width 0) (type default))
@@
   )
   (wire (pts (xy 93.98 138.43) (xy 114.3 138.43))
-    (stroke (width 0) (type default))
-  )
-  (wire (pts (xy 135.89 182.88) (xy 135.89 190.5))
     (stroke (width 0) (type default))
   )
@@
     )
   )
-  (symbol (lib_id "74xx:74HC245") (at 148.59 170.18 0) (unit 1)
-    (in_bom yes) (on_board yes) (dnp no) (fields_autoplaced)
-    (property "Reference" "U105" (at 150.5459 151.13 0)
-      (effects (font (size 1.27 1.27)) (justify left))
-    )
-    (property "Value" "74AHCT245" (at 150.5459 153.67 0)
+  (symbol (lib_id "74xx:74HC245") (at 148.59 170.18 0) (mirror y) (unit 1)
+    (in_bom yes) (on_board yes) (dnp no)
+    (property "Reference" "U105" (at 146.6341 151.13 0)
+      (effects (font (size 1.27 1.27)) (justify left))
+    )
+    (property "Value" "74AHCT245" (at 146.6341 153.67 0)
       (effects (font (size 1.27 1.27)) (justify left))
     )
@@
     )
   )
-  (symbol (lib_id "74xx:74HC245") (at 148.59 118.11 0) (unit 1)
-    (in_bom yes) (on_board yes) (dnp no) (fields_autoplaced)
-    (property "Reference" "U104" (at 150.5459 99.06 0)
-      (effects (font (size 1.27 1.27)) (justify left))
-    )
-    (property "Value" "74AHCT245" (at 150.5459 101.6 0)
+  (symbol (lib_id "74xx:74HC245") (at 148.59 118.11 0) (mirror y) (unit 1)
+    (in_bom yes) (on_board yes) (dnp no)
+    (property "Reference" "U104" (at 146.6341 99.06 0)
+      (effects (font (size 1.27 1.27)) (justify left))
+    )
+    (property "Value" "74AHCT245" (at 146.6341 101.6 0)
       (effects (font (size 1.27 1.27)) (justify left))
     )
@@
     )
   )
-  (symbol (lib_id "power:+5V") (at 135.89 180.34 90) (unit 1)
-    (in_bom yes) (on_board yes) (dnp no) (fields_autoplaced)
-    (property "Reference" "#PWR0109" (at 139.7 180.34 0)
-      (effects (font (size 1.27 1.27)) hide)
-    )
-    (property "Value" "+5V" (at 132.08 180.975 90)
-      (effects (font (size 1.27 1.27)) (justify left))
-    )
-    (property "Footprint" "" (at 135.89 180.34 0)
-      (effects (font (size 1.27 1.27)) hide)
-    )
-    (property "Datasheet" "" (at 135.89 180.34 0)
-      (effects (font (size 1.27 1.27)) hide)
-    )
-    (pin "1")
-    (instances
-      (project "pg09-system"
-        (path "/44572023-3621-4b3a-bd53-c3b2b3f42871"
-          (reference "#PWR0109") (unit 1)
-        )
-      )
-    )
-  )
   (symbol (lib_id "power:+5V") (at 148.59 97.79 0) (unit 1)
     (in_bom yes) (on_board yes) (dnp no) (fields_autoplaced)
@@
         (path "/44572023-3621-4b3a-bd53-c3b2b3f42871"
           (reference "C103") (unit 1)
-        )
-      )
-    )
-  )
-  (symbol (lib_id "power:+5V") (at 135.89 128.27 90) (unit 1)
-    (in_bom yes) (on_board yes) (dnp no) (fields_autoplaced)
-    (property "Reference" "#PWR0108" (at 139.7 128.27 0)
-      (effects (font (size 1.27 1.27)) hide)
-    )
-    (property "Value" "+5V" (at 132.08 128.905 90)
-      (effects (font (size 1.27 1.27)) (justify left))
-    )
-    (property "Footprint" "" (at 135.89 128.27 0)
-      (effects (font (size 1.27 1.27)) hide)
-    )
-    (property "Datasheet" "" (at 135.89 128.27 0)
-      (effects (font (size 1.27 1.27)) hide)
-    )
-    (pin "1")
-    (instances
-      (project "pg09-system"
-        (path "/44572023-3621-4b3a-bd53-c3b2b3f42871"
-          (reference "#PWR0108") (unit 1)
         )
       )
@@
       )
     )
+  )
+  (sheet (at 237.49 16.51) (size 33.02 15.24) (fields_autoplaced)
+    (stroke (width 0.1524) (type solid))
+    (fill (color 0 0 0 0.0000))
+    (property "Sheetname" "Power Supply" (at 237.49 15.7984 0)
+      (effects (font (size 1.27 1.27)) (justify left bottom))
+    )
+    (property "Sheetfile" "pg09-system-psu.kicad_sch" (at 237.49 32.3346 0)
+      (effects (font (size 1.27 1.27)) (justify left top))
+    )
+    (property "Field2" "" (at 237.49 16.51 0)
+      (effects (font (size 1.27 1.27)) hide)
+    )
+    (instances
+      (project "pg09-system"
+        (path "/44572023-3621-4b3a-bd53-c3b2b3f42871" (page "8"))
+      )
+    )

Commit message: Specify a physically smaller bypass cap.
Parts:
- C201: footprint Capacitor_THT:C_Disc_D6.0mm_W4.4mm_P5.00mm -> Capacitor_THT:C_Disc_D3.8mm_W2.6mm_P2.50mm; Mouser (none) -> 80-C315C104M5U-TR
- C202, C203: footprint Capacitor_THT:C_Disc_D6.0mm_W4.4mm_P5.00mm -> Capacitor_THT:C_Disc_D3.8mm_W2.6mm_P2.50mm
Changed lines of the file:
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@@
       (effects (font (size 1.27 1.27)) (justify left))
     )
-    (property "Footprint" "Capacitor_THT:C_Disc_D6.0mm_W4.4mm_P5.00mm" (at 220.98 154.94 0)
+    (property "Footprint" "Capacitor_THT:C_Disc_D3.8mm_W2.6mm_P2.50mm" (at 220.98 154.94 0)
       (effects (font (size 1.27 1.27)) hide)
     )
@@
       (effects (font (size 1.27 1.27)) (justify left))
     )
-    (property "Footprint" "Capacitor_THT:C_Disc_D6.0mm_W4.4mm_P5.00mm" (at 180.34 154.94 0)
+    (property "Footprint" "Capacitor_THT:C_Disc_D3.8mm_W2.6mm_P2.50mm" (at 180.34 154.94 0)
       (effects (font (size 1.27 1.27)) hide)
     )
     (property "Datasheet" "~" (at 180.34 154.94 0)
+      (effects (font (size 1.27 1.27)) hide)
+    )
+    (property "Mouser" "80-C315C104M5U-TR" (at 180.34 154.94 0)
       (effects (font (size 1.27 1.27)) hide)
     )
@@
       (effects (font (size 1.27 1.27)) (justify left))
     )
-    (property "Footprint" "Capacitor_THT:C_Disc_D6.0mm_W4.4mm_P5.00mm" (at 210.82 154.94 0)
+    (property "Footprint" "Capacitor_THT:C_Disc_D3.8mm_W2.6mm_P2.50mm" (at 210.82 154.94 0)
       (effects (font (size 1.27 1.27)) hide)
     )
@@
       (effects (font (size 1.27 1.27)) (justify left))
     )
-    (property "Footprint" "Capacitor_THT:C_Disc_D6.0mm_W4.4mm_P5.00mm" (at 190.5 154.94 0)
+    (property "Footprint" "Capacitor_THT:C_Disc_D3.8mm_W2.6mm_P2.50mm" (at 190.5 154.94 0)
       (effects (font (size 1.27 1.27)) hide)
     )
@@
       (effects (font (size 1.27 1.27)) (justify left))
     )
-    (property "Footprint" "Capacitor_THT:C_Disc_D6.0mm_W4.4mm_P5.00mm" (at 200.66 154.94 0)
-      (effects (font (size 1.27 1.27)) hide)
-    )
+    (property "Footprint" "Capacitor_THT:C_Disc_D3.8mm_W2.6mm_P2.50mm" (at 200.66 154.94 0)
+      (effects (font (size 1.27 1.27)) hide)
+    )

Commit message: Start work on the expansion interface.  Need to spend more time thinking about this one.
Other:
- added sheet Expansion Interface (pg09-system-expansion.kicad_sch)
Changed lines of the file:
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@@
+    )
+  )
+  (sheet (at 12.7 38.1) (size 39.37 15.24) (fields_autoplaced)
+    (stroke (width 0.1524) (type solid))
+    (fill (color 0 0 0 0.0000))
+    (property "Sheetname" "Expansion Interface" (at 12.7 37.3884 0)
+      (effects (font (size 1.27 1.27)) (justify left bottom))
+    )
+    (property "Sheetfile" "pg09-system-expansion.kicad_sch" (at 12.7 53.9246 0)
+      (effects (font (size 1.27 1.27)) (justify left top))
+    )
+    (instances
+      (project "pg09-system"
+        (path "/44572023-3621-4b3a-bd53-c3b2b3f42871" (page "9"))
+      )
     )
   )

Commit message: Integrate the auto-vectoring interrupt controller.
Parts:
- added C203: 0.1µF, Capacitor_THT:C_Disc_D3.8mm_W2.6mm_P2.50mm, symbol Device:C_Small
- added R101: 10K, symbol Device:R_Small
- added U106: GAL22V10, Package_DIP:DIP-24_W7.62mm_Socket, symbol jrt-ICs:GAL22V10
Connections:
- net +5V: now also C203.1, R101.2, U106.24 (VCC)
- net FLASHWREN: now also U102.10 (I10); no longer U102.9 (I9)
- net GND: now also C203.2, U106.12 (GND); no longer U104.19 (CE), U105.19 (CE)
- net nA2: now also RN401.5 (R4), U102.20 (IO7); no longer RN401.4 (R3), U102.21 (IO8)
- net nA3: now also RN401.6 (R5), U102.19 (IO6); no longer RN401.5 (R4), U102.20 (IO7)
- net nA4: now also RN401.7 (R6), U102.18 (IO5); no longer RN401.6 (R5), U102.19 (IO6)
- net ~{FLASHWR}: now also U102.15 (IO2), R101.1; no longer RN401.9 (R8), U102.16 (IO3)
- net ~{RD}: now also RN401.9 (R8); no longer RN401.8 (R7)
- net ~{WR}: now also RN401.8 (R7), U102.16 (IO3); no longer RN401.7 (R6), U102.18 (IO5)
- net dA2: now reaches U101.10 (A2), U104.16 (B2)
- net dA2: now also U102.5 (I5), U106.5 (I5); no longer U102.6 (I6)
- net dA3: now reaches U101.11 (A3), U104.15 (B3)
- net dA3: now also U102.6 (I6), U106.6 (I6); no longer U102.7 (I7)
- net dA4: now reaches U101.12 (A4), U104.14 (B4)
- net dA4: now also U102.7 (I7); no longer U102.8 (I8)
- net at U101.32 (R/~{W}), U102.2 (I2), U103.1 (A->B): now also U106.3 (I3)
- net BS: now reaches U101.5 (BS)
- net BS: now also U106.2 (I2); no longer U102.4 (I4)
- net BA: now reaches U101.6 (BA)
- net BA: now also U106.1 (I1/CLK); no longer U102.3 (I3)
- net dA0: now reaches U101.8 (A0), U104.18 (B0)
- net dA0: now also U102.3 (I3)
- net dA1: now reaches U101.9 (A1), U104.17 (B1)
- net dA1: now also U102.4 (I4), U106.4 (I4); no longer U102.5 (I5)
- net HALTED renamed nA0
- new net IVV: U106.11 (I11)
- new net nA1: RN401.4 (R3), U102.21 (IO8)
- new net ~{HALTACK}: U106.14 (IO1)
- new net ~{INTCACK}: U106.16 (IO3)
- new net ~{NORMAL}: U106.17 (IO4)
- new net ~{SYNCACK}: U106.15 (IO2)
- new net ~{aCPU}: U104.19 (CE), U105.19 (CE), U106.18 (IO5)
- new net ~{aINTC}: U106.23 (IO10)
- no-connect marks 8 -> 17
Other:
- note added: "abus_sel.chp"
- note removed: "Address Decoder Inputs"
- moved on the sheet: C201, C202, C203, RN401, U101, U102, U103, U104, U105

Commit message: Add pull-up resistors to the data bus.
Parts:
- added RN102: 10K, Resistor_THT:R_Array_SIP9, symbol Device:R_Network08
Connections:
- net +5V: now also RN102.1 (common)
- net D0: now also RN102.2 (R1)
- net D1: now also RN102.3 (R2)
- net D2: now also RN102.4 (R3)
- net D3: now also RN102.5 (R4)
- net D4: now also RN102.6 (R5)
- net D5: now also RN102.7 (R6)
- net D6: now also RN102.8 (R7)
- net D7: now also RN102.9 (R8)
Changed lines of the file:
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@@
   (junction (at 116.84 183.515) (diameter 0) (color 0 0 0 0)
   )
+  (junction (at 242.57 127.635) (diameter 0) (color 0 0 0 0)
+  )
+  (junction (at 179.07 198.755) (diameter 0) (color 0 0 0 0)
+  )
   (junction (at 118.745 231.14) (diameter 0) (color 0 0 0 0)
   )
@@
   (junction (at 78.105 236.22) (diameter 0) (color 0 0 0 0)
   )
-  (junction (at 73.66 173.355) (diameter 0) (color 0 0 0 0)
-  )
   (junction (at 108.585 236.22) (diameter 0) (color 0 0 0 0)
   )
@@
   )
   (junction (at 98.425 236.22) (diameter 0) (color 0 0 0 0)
-  )
-  (junction (at 242.57 127.635) (diameter 0) (color 0 0 0 0)
   )
   (no_connect (at 258.445 200.025))
@@
     (stroke (width 0) (type default))
   )
-  (wire (pts (xy 73.66 173.355) (xy 73.66 127.635))
-    (stroke (width 0) (type default))
-  )
   (wire (pts (xy 222.25 205.105) (xy 228.6 205.105))
     (stroke (width 0) (type default))
@@
     (stroke (width 0) (type default))
   )
-  (wire (pts (xy 179.07 224.155) (xy 73.66 224.155))
+  (wire (pts (xy 179.07 224.155) (xy 66.675 224.155))
     (stroke (width 0) (type default))
   )
@@
     (stroke (width 0) (type default))
   )
+  (wire (pts (xy 79.375 163.195) (xy 84.455 163.195))
+    (stroke (width 0) (type default))
+  )
   (wire (pts (xy 173.355 188.595) (xy 166.37 188.595))
     (stroke (width 0) (type default))
@@
     (stroke (width 0) (type default))
   )
-  (wire (pts (xy 73.66 127.635) (xy 242.57 127.635))
-    (stroke (width 0) (type default))
-  )
   (wire (pts (xy 222.25 215.265) (xy 228.6 215.265))
     (stroke (width 0) (type default))
@@
     (stroke (width 0) (type default))
   )
+  (wire (pts (xy 181.61 127.635) (xy 242.57 127.635))
+    (stroke (width 0) (type default))
+  )
   (wire (pts (xy 99.06 158.115) (xy 104.14 158.115))
     (stroke (width 0) (type default))
@@
     (stroke (width 0) (type default))
   )
-  (wire (pts (xy 73.66 173.355) (xy 104.14 173.355))
+  (wire (pts (xy 79.375 158.115) (xy 84.455 158.115))
+    (stroke (width 0) (type default))
+  )
+  (wire (pts (xy 66.675 173.355) (xy 104.14 173.355))
     (stroke (width 0) (type default))
   )
@@
     (stroke (width 0) (type default))
   )
-  (wire (pts (xy 73.66 224.155) (xy 73.66 173.355))
+  (wire (pts (xy 66.675 224.155) (xy 66.675 173.355))
+    (stroke (width 0) (type default))
+  )
+  (wire (pts (xy 179.07 198.755) (xy 181.61 198.755))
     (stroke (width 0) (type default))
   )
@@
     (stroke (width 0) (type default))
   )
+  (wire (pts (xy 79.375 153.035) (xy 84.455 153.035))
+    (stroke (width 0) (type default))
+  )
   (wire (pts (xy 251.46 132.715) (xy 258.445 132.715))
     (stroke (width 0) (type default))
@@
     (stroke (width 0) (type default))
   )
+  (wire (pts (xy 79.375 168.275) (xy 84.455 168.275))
+    (stroke (width 0) (type default))
+  )
   (wire (pts (xy 129.54 155.575) (xy 140.97 155.575))
     (stroke (width 0) (type default))
@@
   )
   (wire (pts (xy 189.865 168.275) (xy 196.85 168.275))
+    (stroke (width 0) (type default))
+  )
+  (wire (pts (xy 181.61 198.755) (xy 181.61 127.635))
     (stroke (width 0) (type default))
   )
@@
     )
   )
+  (global_label "D0" (shape bidirectional) (at 79.375 150.495 0) (fields_autoplaced)
+    (effects (font (size 1.27 1.27)) (justify left))
+    (property "Intersheetrefs" "${INTERSHEET_REFS}" (at 85.8716 150.495 0)
+      (effects (font (size 1.27 1.27)) (justify left) hide)
+    )
+  )
   (global_label "D7" (shape bidirectional) (at 99.06 168.275 180) (fields_autoplaced)
     (effects (font (size 1.27 1.27)) (justify right))
@@
     )
   )
+  (global_label "D3" (shape bidirectional) (at 84.455 158.115 0) (fields_autoplaced)
+    (effects (font (size 1.27 1.27)) (justify left))
+    (property "Intersheetrefs" "${INTERSHEET_REFS}" (at 90.9516 158.115 0)
+      (effects (font (size 1.27 1.27)) (justify left) hide)
+    )
+  )
   (global_label "~{HALT}" (shape input) (at 140.97 193.675 180) (fields_autoplaced)
     (effects (font (size 1.27 1.27)) (justify right))
@@
     )
   )
+  (global_label "D5" (shape bidirectional) (at 84.455 163.195 0) (fields_autoplaced)
+    (effects (font (size 1.27 1.27)) (justify left))
+    (property "Intersheetrefs" "${INTERSHEET_REFS}" (at 90.9516 163.195 0)
+      (effects (font (size 1.27 1.27)) (justify left) hide)
+    )
+  )
   (global_label "R{slash}~{W}" (shape input) (at 309.88 130.175 180) (fields_autoplaced)
     (effects (font (size 1.27 1.27)) (justify right))
@@
     )
   )
+  (global_label "D6" (shape bidirectional) (at 79.375 165.735 0) (fields_autoplaced)
+    (effects (font (size 1.27 1.27)) (justify left))
+    (property "Intersheetrefs" "${INTERSHEET_REFS}" (at 85.8716 165.735 0)
+      (effects (font (size 1.27 1.27)) (justify left) hide)
+    )
+  )
+  (global_label "D2" (shape bidirectional) (at 79.375 155.575 0) (fields_autoplaced)
+    (effects (font (size 1.27 1.27)) (justify left))
+    (property "Intersheetrefs" "${INTERSHEET_REFS}" (at 85.8716 155.575 0)
+      (effects (font (size 1.27 1.27)) (justify left) hide)
+    )
+  )
   (global_label "A10" (shape output) (at 222.25 207.645 0) (fields_autoplaced)
     (effects (font (size 1.27 1.27)) (justify left))
@@
     )
   )
+  (global_label "D7" (shape bidirectional) (at 84.455 168.275 0) (fields_autoplaced)
+    (effects (font (size 1.27 1.27)) (justify left))
+    (property "Intersheetrefs" "${INTERSHEET_REFS}" (at 90.9516 168.275 0)
+      (effects (font (size 1.27 1.27)) (justify left) hide)
+    )
+  )
   (global_label "~{RESET}" (shape input) (at 140.97 173.355 180) (fields_autoplaced)
     (effects (font (size 1.27 1.27)) (justify right))
@@
     )
   )
+  (global_label "D1" (shape bidirectional) (at 84.455 153.035 0) (fields_autoplaced)
+    (effects (font (size 1.27 1.27)) (justify left))
+    (property "Intersheetrefs" "${INTERSHEET_REFS}" (at 90.9516 153.035 0)
+      (effects (font (size 1.27 1.27)) (justify left) hide)
+    )
+  )
   (global_label "~{aINTC}" (shape output) (at 283.845 200.025 0) (fields_autoplaced)
     (effects (font (size 1.27 1.27)) (justify left))
@@
     (effects (font (size 1.27 1.27)) (justify left))
     (property "Intersheetrefs" "${INTERSHEET_REFS}" (at 289.2908 132.715 0)
+      (effects (font (size 1.27 1.27)) (justify left) hide)
+    )
+  )
+  (global_label "D4" (shape bidirectional) (at 79.375 160.655 0) (fields_autoplaced)
+    (effects (font (size 1.27 1.27)) (justify left))
+    (property "Intersheetrefs" "${INTERSHEET_REFS}" (at 85.8716 160.655 0)
       (effects (font (size 1.27 1.27)) (justify left) hide)
     )
@@
         (path "/44572023-3621-4b3a-bd53-c3b2b3f42871"
           (reference "U105") (unit 1)
+        )
+      )
+    )
+  )
+  (symbol (lib_id "Device:R_Network08") (at 74.295 160.655 90) (mirror x) (unit 1)
+    (in_bom yes) (on_board yes) (dnp no)
+    (property "Reference" "RN102" (at 74.549 145.415 90)
+      (effects (font (size 1.27 1.27)))
+    )
+    (property "Value" "10K" (at 74.549 147.955 90)
+      (effects (font (size 1.27 1.27)))
+    )
+    (property "Footprint" "Resistor_THT:R_Array_SIP9" (at 74.295 172.72 90)
+      (effects (font (size 1.27 1.27)) hide)
+    )
+    (property "Datasheet" "http://www.vishay.com/docs/31509/csc.pdf" (at 74.295 160.655 0)
+      (effects (font (size 1.27 1.27)) hide)
+    )
+    (pin "1")
+    (pin "2")
+    (pin "3")
+    (pin "4")
+    (pin "5")
+    (pin "6")
+    (pin "7")
+    (pin "8")
+    (pin "9")
+    (instances
+      (project "pg09-system"
+        (path "/44572023-3621-4b3a-bd53-c3b2b3f42871"
+          (reference "RN102") (unit 1)
         )
       )
@@
         )
       )
+    )
+  )
+  (symbol (lib_id "power:+5V") (at 69.215 150.495 0) (unit 1)
+    (in_bom yes) (on_board yes) (dnp no) (fields_autoplaced)
+    (property "Reference" "#PWR0120" (at 69.215 154.305 0)
+      (effects (font (size 1.27 1.27)) hide)
+    )
+    (property "Value" "+5V" (at 69.215 146.685 0)
+      (effects (font (size 1.27 1.27)))
+    )
+    (property "Footprint" "" (at 69.215 150.495 0)
+      (effects (font (size 1.27 1.27)) hide)
+    )
+    (property "Datasheet" "" (at 69.215 150.495 0)
+      (effects (font (size 1.27 1.27)) hide)
+    )
+    (pin "1")
+    (instances
+      (project "pg09-system"
+        (path "/44572023-3621-4b3a-bd53-c3b2b3f42871"
+          (reference "#PWR0120") (unit 1)
+        )
+      )
