File: design-files/pg09-system.kicad_sch (KiCad schematic)
At the start: 15 parts, among them U101 MC6809E, U102 GAL22V10, U103 74AHCT245, U104 74AHCT245, U105 74AHCT245, U106 GAL22V10

Commit message: WIP re-laying out PCB.
Parts:
- R101: footprint (none) -> Resistor_THT:R_Axial_DIN0207_L6.3mm_D2.5mm_P7.62mm_Horizontal
Connections:
- net ~{RD}: now also RN401.8 (R7); no longer RN401.9 (R8)
- net ~{WR}: now also RN401.9 (R8); no longer RN401.8 (R7)
Changed lines of the file:
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@@
     )
   )
-  (global_label "~{WR}" (shape input) (at 308.61 145.415 180) (fields_autoplaced)
-    (effects (font (size 1.27 1.27)) (justify right))
-    (property "Intersheetrefs" "${INTERSHEET_REFS}" (at 302.9828 145.415 0)
+  (global_label "~{WR}" (shape input) (at 318.77 147.955 180) (fields_autoplaced)
+    (effects (font (size 1.27 1.27)) (justify right))
+    (property "Intersheetrefs" "${INTERSHEET_REFS}" (at 313.1428 147.955 0)
       (effects (font (size 1.27 1.27)) (justify right) hide)
     )
@@
     )
   )
-  (global_label "~{RD}" (shape input) (at 318.77 147.955 180) (fields_autoplaced)
-    (effects (font (size 1.27 1.27)) (justify right))
-    (property "Intersheetrefs" "${INTERSHEET_REFS}" (at 313.3242 147.955 0)
+  (global_label "~{RD}" (shape input) (at 308.61 145.415 180) (fields_autoplaced)
+    (effects (font (size 1.27 1.27)) (justify right))
+    (property "Intersheetrefs" "${INTERSHEET_REFS}" (at 303.1642 145.415 0)
       (effects (font (size 1.27 1.27)) (justify right) hide)
     )
@@
       (effects (font (size 1.27 1.27)))
     )
-    (property "Footprint" "" (at 323.85 156.21 0)
-      (effects (font (size 1.27 1.27)) hide)
-    )
+    (property "Footprint" "Resistor_THT:R_Axial_DIN0207_L6.3mm_D2.5mm_P7.62mm_Horizontal" (at 323.85 156.21 0)
+      (effects (font (size 1.27 1.27)) hide)
+    )

Commit message: Checkpoint WIP new PCB layout.
Parts:
- added H101, H102, H103, H104, H105, H106, H107, H108, H109, H110: MountingHole_Pad, MountingHole:MountingHole_4.3mm_M4_Pad_Via, symbol Mechanical:MountingHole_Pad
Connections:
- net GND: now also H101.1, H102.1, H103.1, H104.1, H105.1, H106.1, H107.1, H108.1, H109.1, H110.1

Commit message: Add a 10uF tantalum capacitor for the CPU.
Parts:
- added C107: 10µF 50V, Capacitor_THT:CP_Radial_D8.0mm_P2.50mm, symbol Device:C_Polarized_Small
Connections:
- net +5V: now also C107.1
- net GND: now also C107.2
Other:
- note added: "Tantalum"
Changed lines of the file:
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@@
   (junction (at 98.425 231.14) (diameter 0) (color 0 0 0 0)
+  )
+  (junction (at 158.115 130.175) (diameter 0) (color 0 0 0 0)
   )
   (junction (at 15.875 238.125) (diameter 0) (color 0 0 0 0)
@@
     (stroke (width 0) (type default))
   )
+  (wire (pts (xy 153.67 145.415) (xy 153.67 130.175))
+    (stroke (width 0) (type default))
+  )
   (wire (pts (xy 222.25 158.115) (xy 228.6 158.115))
     (stroke (width 0) (type default))
@@
   )
   (wire (pts (xy 108.585 236.22) (xy 118.745 236.22))
+    (stroke (width 0) (type default))
+  )
+  (wire (pts (xy 153.67 130.175) (xy 158.115 130.175))
     (stroke (width 0) (type default))
   )
@@
   (text "Data Bus Buffer" (at 100.33 193.675 0)
     (effects (font (size 2.54 2.54) (thickness 0.254) bold italic) (justify left bottom))
+  )
+  (text "Tantalum" (at 160.655 137.16 0)
+    (effects (font (size 1.27 1.27)) (justify left bottom))
   )
   (global_label "dA7" (shape input) (at 189.865 168.275 180) (fields_autoplaced)
@@
     )
   )
+  (symbol (lib_id "power:GND") (at 158.115 135.255 0) (unit 1)
+    (in_bom yes) (on_board yes) (dnp no) (fields_autoplaced)
+    (property "Reference" "#PWR0122" (at 158.115 141.605 0)
+      (effects (font (size 1.27 1.27)) hide)
+    )
+    (property "Value" "GND" (at 158.115 140.335 0)
+      (effects (font (size 1.27 1.27)))
+    )
+    (property "Footprint" "" (at 158.115 135.255 0)
+      (effects (font (size 1.27 1.27)) hide)
+    )
+    (property "Datasheet" "" (at 158.115 135.255 0)
+      (effects (font (size 1.27 1.27)) hide)
+    )
+    (pin "1")
+    (instances
+      (project "pg09-system"
+        (path "/44572023-3621-4b3a-bd53-c3b2b3f42871"
+          (reference "#PWR0122") (unit 1)
+        )
+      )
+    )
+  )
   (symbol (lib_id "Device:R_Network08") (at 323.85 140.335 270) (unit 1)
     (in_bom yes) (on_board yes) (dnp no) (fields_autoplaced)
@@
         (path "/44572023-3621-4b3a-bd53-c3b2b3f42871"
           (reference "#PWR0120") (unit 1)
+        )
+      )
+    )
+  )
+  (symbol (lib_id "Device:C_Polarized_Small") (at 158.115 132.715 0) (unit 1)
+    (in_bom yes) (on_board yes) (dnp no) (fields_autoplaced)
+    (property "Reference" "C107" (at 160.655 131.5339 0)
+      (effects (font (size 1.27 1.27)) (justify left))
+    )
+    (property "Value" "10µF 50V" (at 160.655 134.0739 0)
+      (effects (font (size 1.27 1.27)) (justify left))
+    )
+    (property "Footprint" "Capacitor_THT:CP_Radial_D8.0mm_P2.50mm" (at 158.115 132.715 0)
+      (effects (font (size 1.27 1.27)) hide)
+    )
+    (property "Datasheet" "~" (at 158.115 132.715 0)
+      (effects (font (size 1.27 1.27)) hide)
+    )
+    (pin "1")
+    (pin "2")
+    (instances
+      (project "pg09-system"
+        (path "/44572023-3621-4b3a-bd53-c3b2b3f42871"
+          (reference "C107") (unit 1)
         )
       )
@@
     )
   )
-  (symbol (lib_id "power:+5V") (at 153.67 145.415 0) (unit 1)
-    (in_bom yes) (on_board yes) (dnp no) (fields_autoplaced)
-    (property "Reference" "#PWR0101" (at 153.67 149.225 0)
-      (effects (font (size 1.27 1.27)) hide)
-    )
-    (property "Value" "+5V" (at 153.67 141.605 0)
-      (effects (font (size 1.27 1.27)))
-    )
-    (property "Footprint" "" (at 153.67 145.415 0)
-      (effects (font (size 1.27 1.27)) hide)
-    )
-    (property "Datasheet" "" (at 153.67 145.415 0)
-      (effects (font (size 1.27 1.27)) hide)
-    )
+  (symbol (lib_id "power:+5V") (at 158.115 130.175 0) (unit 1)
+    (in_bom yes) (on_board yes) (dnp no) (fields_autoplaced)
+    (property "Reference" "#PWR0101" (at 158.115 133.985 0)
+      (effects (font (size 1.27 1.27)) hide)
+    )
+    (property "Value" "+5V" (at 158.115 126.365 0)
+      (effects (font (size 1.27 1.27)))
+    )
+    (property "Footprint" "" (at 158.115 130.175 0)
+      (effects (font (size 1.27 1.27)) hide)
+    )
+    (property "Datasheet" "" (at 158.115 130.175 0)
+      (effects (font (size 1.27 1.27)) hide)
+    )
