File: design-files/pg09-system.kicad_sch (KiCad schematic)
At the start: 33 parts, among them J101 Front Panel, SW201 NMI, SW201 Reset, U101 MC6809E, U102 GAL22V10, U103 74AHCT245, U104 74AHCT245, U105 74AHCT245, U106 GAL22V10, U203 DS1813

Commit message: Remove resistor associated with NMI button -- NMI is already pulled-up.
Parts:
- removed R203: 3K3, Resistor_THT:R_Axial_DIN0207_L6.3mm_D2.5mm_P7.62mm_Horizontal, symbol Device:R_Small
Changed lines of the file:
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@@
   (junction (at 360.045 245.745) (diameter 0) (color 0 0 0 0)
   )
-  (junction (at 337.185 226.695) (diameter 0) (color 0 0 0 0)
-  )
   (junction (at 15.875 259.08) (diameter 0) (color 0 0 0 0)
-  )
-  (junction (at 349.885 235.585) (diameter 0) (color 0 0 0 0)
   )
   (no_connect (at 258.445 200.025))
@@
     (stroke (width 0) (type default))
   )
-  (wire (pts (xy 337.185 231.775) (xy 337.185 235.585))
-    (stroke (width 0) (type default))
-  )
   (wire (pts (xy 299.085 226.06) (xy 304.165 226.06))
     (stroke (width 0) (type default))
@@
   )
   (wire (pts (xy 15.875 224.155) (xy 20.955 224.155))
-    (stroke (width 0) (type default))
-  )
-  (wire (pts (xy 337.185 235.585) (xy 349.885 235.585))
     (stroke (width 0) (type default))
   )
@@
         )
       )
-    )
-  )
-  (symbol (lib_id "Device:R_Small") (at 337.185 229.235 180) (unit 1)
-    (in_bom yes) (on_board yes) (dnp no)
-    (property "Reference" "R203" (at 330.835 227.965 0)
-      (effects (font (size 1.27 1.27)) (justify right))
-    )
-    (property "Value" "3K3" (at 332.105 230.505 0)
-      (effects (font (size 1.27 1.27)) (justify right))
-    )
-    (property "Footprint" "Resistor_THT:R_Axial_DIN0207_L6.3mm_D2.5mm_P7.62mm_Horizontal" (at 337.185 229.235 0)
-      (effects (font (size 1.27 1.27)) hide)
-    )
-    (property "Datasheet" "~" (at 337.185 229.235 0)
-      (effects (font (size 1.27 1.27)) hide)
-    )
-    (pin "1")
-    (pin "2")
-    (instances
-      (project "pg09-system"
-        (path "/44572023-3621-4b3a-bd53-c3b2b3f42871/4db01e9b-9f77-42a7-9351-8914253ebfe9"
-          (reference "R203") (unit 1)
-        )
-        (path "/44572023-3621-4b3a-bd53-c3b2b3f42871"
-          (reference "R103") (unit 1)
-        )
-      )

Commit message: Pull-up /RESET on RN201.
Parts:
- removed R203: 3K3, Resistor_THT:R_Axial_DIN0207_L6.3mm_D2.5mm_P7.62mm_Horizontal, symbol Device:R_Small
Other:
- note added: "~{NMI} and ~{RESET} are pulled-up on the clock generator sheet (RN201)."
- moved on the sheet: SW201, U203

Commit message: Use an R-C circuit in front of the Vcc on /RESET's DS1813 in order to delay power-on-reset by ~0.75 seconds.
Parts:
- added C804: 470µF 50V, Capacitor_THT:CP_Radial_D12.5mm_P5.00mm, symbol Device:C_Polarized_US
- added D101: 1N4448, Diode_THT:D_DO-35_SOD27_P7.62mm_Horizontal, symbol Diode:1N4448
- added R102: 1K, Resistor_THT:R_Axial_DIN0207_L6.3mm_D2.5mm_P7.62mm_Horizontal, symbol Device:R_Small
Connections:
- net +5V: now also D101.1 (K), R102.2; no longer U203.2 (Vcc)
- net GND: now also C804.2
- new net: C804.1, D101.2 (A), R102.1, U203.2 (Vcc)
Other:
- note added: "Delay power-on reset by ~0.75 seconds."
- moved on the sheet: SW201, U203

Commit message: Tweak the reset and NMI circuits -- no pull-ups on those signals needed; the DS1813 has us covered.  Add power-on-reset delay of ~0.5 seconds.
Parts:
- C804: value 470µF 50V -> 100µF 16V; footprint Capacitor_THT:CP_Radial_D12.5mm_P5.00mm -> Capacitor_THT:CP_Radial_D6.3mm_P2.50mm; Mouser 871-B41888C6477M -> 661-E-160L101MF11D
- D101: value 1N4448 -> 1N4001; footprint Diode_THT:D_DO-35_SOD27_P7.62mm_Horizontal -> Diode_THT:D_DO-41_SOD81_P10.16mm_Horizontal; symbol Diode:1N4448 -> Diode:1N4001
- R102: value 1K -> 3K3
Other:
- note removed: "Delay power-on reset by ~0.75 seconds."
- note removed: "~{NMI} and ~{RESET} are pulled-up on the clock generator sheet (RN201)."
- moved on the sheet: C804, D101, R102, SW201, U203

Commit message: Make the RESET diode a 1N4148.  Put the resistor VALUE on the F.Silk layer inside the footprint.
Parts:
- D101: value 1N4001 -> 1N4148; footprint Diode_THT:D_DO-41_SOD81_P10.16mm_Horizontal -> Diode_THT:D_DO-35_SOD27_P7.62mm_Horizontal; symbol Diode:1N4001 -> Diode:1N4148
Changed lines of the file:
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@@
     )
   )
-  (symbol (lib_id "Diode:1N4001") (at 337.312 217.424 270) (unit 1)
+  (symbol (lib_id "Diode:1N4148") (at 337.312 217.424 270) (unit 1)
     (in_bom yes) (on_board yes) (dnp no)
     (property "Reference" "D101" (at 328.422 216.916 90)
       (effects (font (size 1.27 1.27)) (justify left))
     )
-    (property "Value" "1N4001" (at 331.978 218.948 90)
+    (property "Value" "1N4148" (at 331.978 218.948 90)
       (effects (font (size 1.27 1.27)))
     )
-    (property "Footprint" "Diode_THT:D_DO-41_SOD81_P10.16mm_Horizontal" (at 337.312 217.424 0)
+    (property "Footprint" "Diode_THT:D_DO-35_SOD27_P7.62mm_Horizontal" (at 337.312 217.424 0)
       (effects (font (size 1.27 1.27)) hide)
     )
-    (property "Datasheet" "http://www.vishay.com/docs/88503/1n4001.pdf" (at 337.312 217.424 0)
+    (property "Datasheet" "https://assets.nexperia.com/documents/data-sheet/1N4148_1N4448.pdf" (at 337.312 217.424 0)
       (effects (font (size 1.27 1.27)) hide)
     )

Commit message: Make sure FLASHWREN always has a valid value by pulling it to GND.
Parts:
- added R103: 10K, Resistor_THT:R_Axial_DIN0207_L6.3mm_D2.5mm_P7.62mm_Horizontal, symbol Device:R_Small
Connections:
- net FLASHWREN: now also R103.1
- net GND: now also R103.2
Changed lines of the file:
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@@
+    )
+  )
+  (global_label "FLASHWREN" (shape input) (at 321.31 163.83 180) (fields_autoplaced)
+    (effects (font (size 1.27 1.27)) (justify right))
+    (property "Intersheetrefs" "${INTERSHEET_REFS}" (at 307.458 163.83 0)
+      (effects (font (size 1.27 1.27)) (justify right) hide)
     )
   )
@@
     )
   )
+  (symbol (lib_id "power:GND") (at 326.39 163.83 90) (unit 1)
+    (in_bom yes) (on_board yes) (dnp no) (fields_autoplaced)
+    (property "Reference" "#PWR0131" (at 332.74 163.83 0)
+      (effects (font (size 1.27 1.27)) hide)
+    )
+    (property "Value" "GND" (at 330.2 164.465 90)
+      (effects (font (size 1.27 1.27)) (justify right))
+    )
+    (property "Footprint" "" (at 326.39 163.83 0)
+      (effects (font (size 1.27 1.27)) hide)
+    )
+    (property "Datasheet" "" (at 326.39 163.83 0)
+      (effects (font (size 1.27 1.27)) hide)
+    )
+    (pin "1")
+    (instances
+      (project "pg09-system"
+        (path "/44572023-3621-4b3a-bd53-c3b2b3f42871"
+          (reference "#PWR0131") (unit 1)
+        )
+      )
+    )
+  )
   (symbol (lib_id "power:GND") (at 116.84 183.388 0) (unit 1)
     (in_bom yes) (on_board yes) (dnp no) (fields_autoplaced)
@@
         )
       )
+    )
+  )
+  (symbol (lib_id "Device:R_Small") (at 323.85 163.83 90) (unit 1)
+    (in_bom yes) (on_board yes) (dnp no) (fields_autoplaced)
+    (property "Reference" "R103" (at 323.85 159.385 90)
+      (effects (font (size 1.27 1.27)))
+    )
+    (property "Value" "10K" (at 323.85 161.925 90)
+      (effects (font (size 1.27 1.27)))
+    )
+    (property "Footprint" "Resistor_THT:R_Axial_DIN0207_L6.3mm_D2.5mm_P7.62mm_Horizontal" (at 323.85 163.83 0)
+      (effects (font (size 1.27 1.27)) hide)
+    )
+    (property "Datasheet" "~" (at 323.85 163.83 0)
+      (effects (font (size 1.27 1.27)) hide)
+    )
+    (pin "1")
+    (pin "2")
+    (instances
+      (project "pg09-system"
+        (path "/44572023-3621-4b3a-bd53-c3b2b3f42871"
+          (reference "R103") (unit 1)
+        )
+      )

Commit message: Revert "Make sure FLASHWREN always has a valid value by pulling it to GND."
This is actually counter-productive due to the internal pull-up on the
GAL inputs.

This reverts commit e5d063032c780da183b0786b1f57988b4be9d05e.
Parts:
- removed R103: 10K, Resistor_THT:R_Axial_DIN0207_L6.3mm_D2.5mm_P7.62mm_Horizontal, symbol Device:R_Small
Changed lines of the file:
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@@
-    )
-  )
-  (global_label "FLASHWREN" (shape input) (at 321.31 163.83 180) (fields_autoplaced)
-    (effects (font (size 1.27 1.27)) (justify right))
-    (property "Intersheetrefs" "${INTERSHEET_REFS}" (at 307.458 163.83 0)
-      (effects (font (size 1.27 1.27)) (justify right) hide)
     )
   )
@@
     )
   )
-  (symbol (lib_id "power:GND") (at 326.39 163.83 90) (unit 1)
-    (in_bom yes) (on_board yes) (dnp no) (fields_autoplaced)
-    (property "Reference" "#PWR0131" (at 332.74 163.83 0)
-      (effects (font (size 1.27 1.27)) hide)
-    )
-    (property "Value" "GND" (at 330.2 164.465 90)
-      (effects (font (size 1.27 1.27)) (justify right))
-    )
-    (property "Footprint" "" (at 326.39 163.83 0)
-      (effects (font (size 1.27 1.27)) hide)
-    )
-    (property "Datasheet" "" (at 326.39 163.83 0)
-      (effects (font (size 1.27 1.27)) hide)
-    )
-    (pin "1")
-    (instances
-      (project "pg09-system"
-        (path "/44572023-3621-4b3a-bd53-c3b2b3f42871"
-          (reference "#PWR0131") (unit 1)
-        )
-      )
-    )
-  )
   (symbol (lib_id "power:GND") (at 116.84 183.388 0) (unit 1)
     (in_bom yes) (on_board yes) (dnp no) (fields_autoplaced)
@@
         )
       )
-    )
-  )
-  (symbol (lib_id "Device:R_Small") (at 323.85 163.83 90) (unit 1)
-    (in_bom yes) (on_board yes) (dnp no) (fields_autoplaced)
-    (property "Reference" "R103" (at 323.85 159.385 90)
-      (effects (font (size 1.27 1.27)))
-    )
-    (property "Value" "10K" (at 323.85 161.925 90)
-      (effects (font (size 1.27 1.27)))
-    )
-    (property "Footprint" "Resistor_THT:R_Axial_DIN0207_L6.3mm_D2.5mm_P7.62mm_Horizontal" (at 323.85 163.83 0)
-      (effects (font (size 1.27 1.27)) hide)
-    )
-    (property "Datasheet" "~" (at 323.85 163.83 0)
-      (effects (font (size 1.27 1.27)) hide)
-    )
-    (pin "1")
-    (pin "2")
-    (instances
-      (project "pg09-system"
-        (path "/44572023-3621-4b3a-bd53-c3b2b3f42871"
-          (reference "R103") (unit 1)
-        )
-      )
