File: design-files/pg09-system.kicad_pcb (KiCad board)
At the start: 2 copper layers, 0 parts

Commit message: First cut at layout of the PCB.
Parts:
- added C101: 0.1µF, Capacitor_THT:C_Disc_D6.0mm_W4.4mm_P5.00mm, F.Cu at (281.4, 237.5)
- added C102: 0.1µF, Capacitor_THT:C_Disc_D6.0mm_W4.4mm_P5.00mm, F.Cu at (259.8, 240.0)
- added C103: 0.1µF, Capacitor_THT:C_Disc_D6.0mm_W4.4mm_P5.00mm, F.Cu at (276.3, 245.0)
- added C104: 0.1µF, Capacitor_THT:C_Disc_D6.0mm_W4.4mm_P5.00mm, F.Cu at (313.2, 245.1)
- added C105: 0.1µF, Capacitor_THT:C_Disc_D6.0mm_W4.4mm_P5.00mm, F.Cu at (324.6, 245.1)
- added C201: 0.1µF, Capacitor_THT:C_Disc_D6.0mm_W4.4mm_P5.00mm, F.Cu at (324.6, 213.3)
- added C202: 0.1µF, Capacitor_THT:C_Disc_D6.0mm_W4.4mm_P5.00mm, F.Cu at (348.7, 213.3)
- added C203: 0.1µF, Capacitor_THT:C_Disc_D6.0mm_W4.4mm_P5.00mm, F.Cu at (352.5, 237.6)
- added C301: 0.1µF, Capacitor_THT:C_Disc_D6.0mm_W4.4mm_P5.00mm, F.Cu at (205.2, 190.5)
- added C302: 0.1µF, Capacitor_THT:C_Disc_D6.0mm_W4.4mm_P5.00mm, F.Cu at (247.1, 190.5)
- added C303: 0.1µF, Capacitor_THT:C_Disc_D6.0mm_W4.4mm_P5.00mm, F.Cu at (289.0, 190.5)
- added C304: 0.1µF, Capacitor_THT:C_Disc_D6.0mm_W4.4mm_P5.00mm, F.Cu at (330.9, 190.5)
- added C401: 0.1µF, Capacitor_THT:C_Disc_D6.0mm_W4.4mm_P5.00mm, F.Cu at (408.9, 265.4)
- added C402: 0.1µF, Capacitor_THT:C_Disc_D6.0mm_W4.4mm_P5.00mm, F.Cu at (391.2, 191.7)
- added C403: 0.1µF, Capacitor_THT:C_Disc_D6.0mm_W4.4mm_P5.00mm, F.Cu at (408.9, 191.7)
- added C404: 0.1µF, Capacitor_THT:C_Disc_D6.0mm_W4.4mm_P5.00mm, F.Cu at (377.9, 228.6)
- added C501: 0.1µF, Capacitor_THT:C_Disc_D6.0mm_W4.4mm_P5.00mm, F.Cu at (183.6, 270.4)
- added C502: 0.1µF, Capacitor_THT:C_Disc_D6.0mm_W4.4mm_P5.00mm, F.Cu at (248.4, 224.8)
- added C503: 0.1µF, Capacitor_THT:C_Disc_D6.0mm_W4.4mm_P5.00mm, F.Cu at (221.7, 219.7)
- added C601: 0.1µF, Capacitor_THT:C_Disc_D6.0mm_W4.4mm_P5.00mm, F.Cu at (188.7, 335.2)
- added C602: 0.1µF, Capacitor_THT:C_Disc_D6.0mm_W4.4mm_P5.00mm, F.Cu at (323.3, 284.4)
- added C603: 0.1µF, Capacitor_THT:C_Disc_D6.0mm_W4.4mm_P5.00mm, F.Cu at (219.2, 266.7)
- added C604: 0.1µF, Capacitor_THT:C_Disc_D6.0mm_W4.4mm_P5.00mm, F.Cu at (227.1, 284.4)
- added C605: 0.1µF, Capacitor_THT:C_Disc_D6.0mm_W4.4mm_P5.00mm, F.Cu at (246.4, 284.4)
- added C606: 0.1µF, Capacitor_THT:C_Disc_D6.0mm_W4.4mm_P5.00mm, F.Cu at (265.8, 284.4)
- added C607: 0.1µF, Capacitor_THT:C_Disc_D6.0mm_W4.4mm_P5.00mm, F.Cu at (285.2, 284.4)
- added C608: 0.1µF, Capacitor_THT:C_Disc_D6.0mm_W4.4mm_P5.00mm, F.Cu at (304.3, 289.5)
- added C701: 0.1µF, Capacitor_THT:C_Disc_D6.0mm_W4.4mm_P5.00mm, F.Cu at (408.4, 162.6)
- added C702: 0.1µF, Capacitor_THT:C_Disc_D6.0mm_W4.4mm_P5.00mm, F.Cu at (317.5, 166.4)
- added C703: 0.1µF, Capacitor_THT:C_Disc_D6.0mm_W4.4mm_P5.00mm, F.Cu at (292.1, 167.6)
- added C704: 0.1µF, Capacitor_THT:C_Disc_D6.0mm_W4.4mm_P5.00mm, F.Cu at (354.3, 148.6)
- added J201: Clock Source, Connector_PinHeader_2.54mm:PinHeader_2x03_P2.54mm_Vertical, F.Cu at (331.6, 221.0)
- added J202: Reset Connector, Connector_PinHeader_2.54mm:PinHeader_1x02_P2.54mm_Vertical, F.Cu at (353.8, 321.3)
- added Q201: 2N7000, Package_TO_SOT_THT:TO-92_Inline, F.Cu at (305.5, 232.0)
- added Q401: 2N7000, Package_TO_SOT_THT:TO-92_Inline, F.Cu at (367.8, 221.0)
- added Q701: 2N7000, Package_TO_SOT_THT:TO-92_Inline, F.Cu at (368.3, 188.0)
- added R201: 150, Resistor_THT:R_Axial_DIN0207_L6.3mm_D2.5mm_P7.62mm_Horizontal, F.Cu at (303.0, 223.5)
- added R202: 3K3, Resistor_THT:R_Axial_DIN0207_L6.3mm_D2.5mm_P7.62mm_Horizontal, F.Cu at (304.3, 245.1)
- added R203: 3K3, Resistor_THT:R_Axial_DIN0207_L6.3mm_D2.5mm_P7.62mm_Horizontal, F.Cu at (334.8, 320.0)
- added R204: 100, Resistor_THT:R_Axial_DIN0207_L6.3mm_D2.5mm_P7.62mm_Horizontal, F.Cu at (310.6, 228.6)
- added R205: 100, Resistor_THT:R_Axial_DIN0207_L6.3mm_D2.5mm_P7.62mm_Horizontal, F.Cu at (328.4, 215.9)
- added R401: 10K, Resistor_THT:R_Axial_DIN0207_L6.3mm_D2.5mm_P7.62mm_Horizontal, F.Cu at (367.8, 233.7)
- added R701: 10K, Resistor_THT:R_Axial_DIN0207_L6.3mm_D2.5mm_P7.62mm_Horizontal, F.Cu at (367.0, 191.8)
- added R702: 10K, Resistor_THT:R_Axial_DIN0207_L6.3mm_D2.5mm_P7.62mm_Horizontal, F.Cu at (372.1, 191.8)
- added RN101: 10K, Resistor_THT:R_Array_SIP9, F.Cu at (262.4, 242.6)
- added RN301: 10K, Resistor_THT:R_Array_SIP9, F.Cu at (207.8, 187.5)
- added RN302: 10K, Resistor_THT:R_Array_SIP9, F.Cu at (249.7, 187.5)
- added RN303: 10K, Resistor_THT:R_Array_SIP9, F.Cu at (291.6, 187.5)
- added RN304: 10K, Resistor_THT:R_Array_SIP9, F.Cu at (333.5, 187.5)
- added RN305: 10K, Resistor_THT:R_Array_SIP9, F.Cu at (280.1, 212.1)
- added RN401: 10K, Resistor_THT:R_Array_SIP9, F.Cu at (378.5, 191.8)
- added RN402: 10K, Resistor_THT:R_Array_SIP9, F.Cu at (396.2, 191.8)
- added SW201: SW_Push, Button_Switch_THT:SW_PUSH_6mm, F.Cu at (339.1, 320.3)
- added U101: MC6809E, Package_DIP:DIP-40_W15.24mm_Socket, F.Cu at (285.2, 222.3)
- added U102: GAL22V10, Package_DIP:DIP-24_W7.62mm_Socket, F.Cu at (250.9, 242.6)
- added U103: 74AHCT245, Package_DIP:DIP-20_W7.62mm_Socket, F.Cu at (267.4, 247.7)
- added U104: 74AHCT245, Package_DIP:DIP-20_W7.62mm_Socket, F.Cu at (304.3, 247.7)
- added U105: 74AHCT245, Package_DIP:DIP-20_W7.62mm_Socket, F.Cu at (315.7, 247.7)
- added U201: CD74ACT109, Package_DIP:DIP-16_W7.62mm_Socket, F.Cu at (315.7, 215.9)
- added U202: CD74ACT163, Package_DIP:DIP-16_W7.62mm_Socket, F.Cu at (339.8, 215.9)
- added U203: DS1813, Package_TO_SOT_THT:TO-92_Inline, F.Cu at (341.1, 313.7)
- added U301: GAL22V10, Package_DIP:DIP-24_W7.62mm_Socket, F.Cu at (207.8, 199.0)
- added U302: GAL22V10, Package_DIP:DIP-24_W7.62mm_Socket, F.Cu at (249.7, 199.0)
- added U303: GAL22V10, Package_DIP:DIP-24_W7.62mm_Socket, F.Cu at (291.6, 199.0)
- added U304: GAL22V10, Package_DIP:DIP-24_W7.62mm_Socket, F.Cu at (333.5, 199.0)
- added U401: W65C21, Package_DIP:DIP-40_W15.24mm_Socket, F.Cu at (360.7, 261.6)
- added U402: GAL22V10, Package_DIP:DIP-24_W7.62mm_Socket, F.Cu at (382.3, 194.3)
- added U403: GAL22V10, Package_DIP:DIP-24_W7.62mm_Socket, F.Cu at (400.1, 194.3)
- added U404: GAL22V10, Package_DIP:DIP-24_W7.62mm_Socket, F.Cu at (381.0, 237.5)
- added U501: W65C21, Package_DIP:DIP-40_W15.24mm_Socket, F.Cu at (187.4, 222.3)
- added U502: AT28C64, Socket:DIP_Socket-28_W6.9_W7.62_W10.16_W12.7_W13.5_3M_228-4817-00-0602J, F.Cu at (231.9, 224.8)
- added U503: SST39SF040, Package_DIP:DIP-32_W15.24mm_Socket, F.Cu at (206.5, 222.2)
- added U601: W65C21, Package_DIP:DIP-40_W15.24mm_Socket, F.Cu at (192.5, 287.0)
- added U602: AS6C4008-55PCN, Package_DIP:DIP-32_W15.24mm_Socket, F.Cu at (308.1, 287.0)
- added U603: 74AHC138, Package_DIP:DIP-16_W7.62mm_Socket, F.Cu at (221.7, 275.6)
- added U604: AS6C4008-55PCN, Package_DIP:DIP-32_W15.24mm_Socket, F.Cu at (211.8, 287.0)
- added U605: AS6C4008-55PCN, Package_DIP:DIP-32_W15.24mm_Socket, F.Cu at (231.2, 287.0)
- added U606: AS6C4008-55PCN, Package_DIP:DIP-32_W15.24mm_Socket, F.Cu at (250.6, 287.0)
- added U607: AS6C4008-55PCN, Package_DIP:DIP-32_W15.24mm_Socket, F.Cu at (270.0, 287.0)
- added U608: AS6C6264-55PCN, Package_DIP:DIP-28_W15.24mm_Socket, F.Cu at (289.0, 292.1)
- added U701: W65C51, Package_DIP:DIP-28_W15.24mm_Socket, F.Cu at (375.4, 181.6)
- added U702: 16550, Package_DIP:DIP-40_W15.24mm_Socket, F.Cu at (320.0, 181.6)
- added U703: 74HC04, Package_DIP:DIP-14_W7.62mm_Socket, F.Cu at (294.6, 176.5)
- added U704: Ali_Express_FTDI_Breakout, jrt-Connectors:DIP-18_W10.16mm_Socket, F.Cu at (394.5, 134.6)
- added U705: Adafruit_FTDI_Friend, Connector_PinHeader_2.54mm:PinHeader_1x06_P2.54mm_Horizontal, F.Cu at (341.1, 137.7)
- added U706: Ali_Express_FTDI_Breakout, jrt-Connectors:DIP-18_W10.16mm_Socket, F.Cu at (324.6, 134.6)
- added X201: ACO-32.000MHz, Oscillator:Oscillator_DIP-14, F.Cu at (360.1, 232.4)
- added X701: 1.8432MHz, Oscillator:Oscillator_DIP-14, F.Cu at (358.9, 156.2)
Other:
- copper layers 2 -> 4
- board text added: "1"
- board text added: "1MHz"
- board text added: "2"
- board text added: "2MHz"
- board text added: "3"
- board text added: "4"
- board text added: "4MHz"
- board text added: "ADDRDEC0"
- board text added: "ADDRDEC1"
- board text added: "ADDRDEC2"
- board text added: "ADDRDEC3"
- board text added: "Fixed RAM"
- board text added: "High Banked RAM"
- board text added: "INTENC"
- board text added: "INTMUX"
- board text added: "Interrupt Controller"
- board text added: "Low Banked RAM"
- board text added: "MEMINTF"
- board text added: "Reset"

Commit message: Additional PCB tweaks before I start drawing traces.
Parts:
- U704, U706: footprint jrt-Connectors:DIP-18_W10.16mm_Socket -> jrt-Connectors:Ali_Express_FTDI_Breakout
- moved U705 8.15 mm to (349.2, 137.7)
- moved C703 6.52 mm to (298.4, 166.4), turned to 0 degrees
- moved C702 4.60 mm to (320.1, 162.6), turned to 0 degrees
- moved U704 4.55 mm to (389.9, 134.6)
- moved U703 4.02 mm to (298.4, 177.8)
- moved U706 1.80 mm to (326.4, 134.6)
- moved RN305 1.29 mm to (281.4, 212.1)
Other:
- board outline added: 242.6 x 208.3 mm

Commit message: Checkpoint: Lots of traces for the RAM.
Routing:
- net A0: track 0.00 -> 101.6 mm
- net D2: track 0.00 -> 101.6 mm
- net A3: track 0.00 -> 101.6 mm
- net A12: track 0.00 -> 101.6 mm
- net D3: track 0.00 -> 101.6 mm
- net D1: track 0.00 -> 101.6 mm
- net A4: track 0.00 -> 101.6 mm
- net A2: track 0.00 -> 101.6 mm
- net A1: track 0.00 -> 101.6 mm
- net A5: track 0.00 -> 101.6 mm
- net D0: track 0.00 -> 101.6 mm
- net A7: track 0.00 -> 101.6 mm
- net A6: track 0.00 -> 101.6 mm
- net ~{RD}: track 0.00 -> 101.5 mm
- net D6: track 0.00 -> 101.5 mm
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
Commit message: Checkpoint: Route D0-D7 to the RAM.
Routing:
- net D3: track 101.6 -> 201.5 mm, vias 0 -> 1
- net D1: track 101.6 -> 192.9 mm, vias 0 -> 2
- net D2: track 101.6 -> 192.5 mm, vias 0 -> 1
- net D0: track 101.6 -> 192.2 mm, vias 0 -> 2
- net D4: track 101.5 -> 191.6 mm, vias 0 -> 2
- net D5: track 101.3 -> 181.1 mm
- net D6: track 101.5 -> 179.7 mm, vias 0 -> 2
- net D7: track 101.3 -> 177.8 mm, vias 0 -> 2
- net A0: track 101.6 -> 124.2 mm, vias 0 -> 1
- net A1: track 101.6 -> 121.8 mm, vias 0 -> 2

Commit message: Checkpoint: Several ROM traces.
Routing:
- net D3: track 201.5 -> 255.2 mm, vias 1 -> 3
- net D0: track 192.2 -> 240.2 mm, vias 2 -> 4
- net D4: track 191.6 -> 239.5 mm, vias 2 -> 3
- net D7: track 177.8 -> 225.4 mm, vias 2 -> 3
- net D2: track 192.5 -> 239.1 mm, vias 1 -> 3
- net D1: track 192.9 -> 239.2 mm, vias 2 -> 4
- net D5: track 181.1 -> 225.6 mm, vias 0 -> 2
- net D6: track 179.7 -> 221.2 mm
- net Net-(U501-PA0): track 0.00 -> 40.5 mm, vias 0 -> 1
- net Net-(U501-PA4): track 0.00 -> 40.2 mm, vias 0 -> 2
- net Net-(U501-PA5): track 0.00 -> 33.9 mm, vias 0 -> 1
- net Net-(U501-PA3): track 0.00 -> 27.4 mm, vias 0 -> 2
- net A1: track 121.8 -> 148.9 mm
- net A4: track 101.6 -> 128.7 mm
- net A6: track 101.6 -> 128.0 mm
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
Commit message: Checkpoint: Address decoder connections.
Routing:
- net dA9: track 0.00 -> 145.5 mm, vias 0 -> 3
- net dA10: track 0.00 -> 142.9 mm, vias 0 -> 3
- net dA11: track 0.00 -> 140.3 mm, vias 0 -> 3
- net dA12: track 0.00 -> 137.7 mm, vias 0 -> 3
- net dA13: track 0.00 -> 135.0 mm, vias 0 -> 3
- net dA5: track 0.00 -> 134.4 mm, vias 0 -> 3
- net dA6: track 0.00 -> 132.8 mm, vias 0 -> 3
- net dA14: track 0.00 -> 132.4 mm, vias 0 -> 3
- net dA7: track 0.00 -> 130.9 mm, vias 0 -> 3
- net dA8: track 0.00 -> 128.5 mm
- net dA15: track 0.00 -> 128.5 mm

Commit message: Checkpoint: CPU connected to A and D buffers.
Routing:
- net dA9: track 145.5 -> 287.2 mm, vias 3 -> 6
- net dA8: track 128.5 -> 268.9 mm, vias 0 -> 3
- net dA10: track 142.9 -> 278.5 mm, vias 3 -> 6
- net dA11: track 140.3 -> 269.8 mm, vias 3 -> 6
- net dA12: track 137.7 -> 260.1 mm, vias 3 -> 5
- net dA13: track 135.0 -> 237.9 mm, vias 3 -> 5
- net dA14: track 132.4 -> 226.3 mm, vias 3 -> 5
- net dA7: track 130.9 -> 217.5 mm, vias 3 -> 6
- net dA15: track 128.5 -> 213.4 mm, vias 0 -> 1
- net dA6: track 132.8 -> 216.5 mm, vias 3 -> 6
- net dA5: track 134.4 -> 215.5 mm, vias 3 -> 6
- net Net-(U101-D7): track 0.00 -> 43.0 mm, vias 0 -> 2
- net Net-(U101-D6): track 0.00 -> 36.2 mm, vias 0 -> 1
- net Net-(U101-D2): track 0.00 -> 36.1 mm, vias 0 -> 2
- net Net-(U101-D4): track 0.00 -> 34.9 mm, vias 0 -> 2
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
Commit message: Checkpoint: Address bus buffers connected to RAM.
Routing:
- net A0: track 150.7 -> 216.2 mm
- net A1: track 148.9 -> 208.9 mm
- net A2: track 128.0 -> 182.6 mm
- net A10: track 122.6 -> 176.9 mm
- net A8: track 122.8 -> 175.0 mm, vias 0 -> 1
- net A9: track 122.8 -> 174.4 mm, vias 0 -> 1
- net A12: track 128.0 -> 178.8 mm, vias 0 -> 1
- net A3: track 128.0 -> 178.7 mm
- net A11: track 122.7 -> 169.1 mm
- net A4: track 128.7 -> 173.9 mm
- net A15: track 0.00 -> 42.8 mm
- net A5: track 128.0 -> 167.7 mm
- net A14: track 0.00 -> 38.3 mm, vias 0 -> 1
- net A6: track 128.0 -> 162.3 mm
- net A13: track 0.00 -> 32.7 mm
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