File: design-files/pg09-system.kicad_pcb (KiCad board)
At the start: 4 copper layers, 306 x 244 mm, 124 parts, among them J101 Front Panel, J201 Clock Speed, J801 ATX-24, J802 #PS_ON, J803 PSU-CTRL console, J901 Expansion 1, J902 Expansion 1 ext, J903 Expansion 2, J904 Expansion 2 ext, J905 Expansion 3, J906 Expansion 3 ext, J907 Expansion 4, J908 Expansion 4 ext, Q201 2N7000, Q701 2N7000, SW101 NMI, SW201 Reset, SW801 Power, U101 MC6809E, U102 GAL22V10, U103 74AHCT245, U104 74AHCT245, U105 74AHCT245, U106 GAL22V10, U107 DS1813, U201 CD74ACT109, U202 CD74ACT163, U203 DS1813, U204 GAL22V10, U301 GAL22V10, U302 GAL22V10, U401 W65C21, U402 GAL22V10, U403 GAL22V10, U404 GAL22V10, U405 74AHC374, U406 74AHC374, U407 74AHC138, U501 W65C21, U502 AT28C64, U503 SST39SF040, U601 W65C21, U602 AS6C4008-55PCN, U603 74AHC138, U604 AS6C4008-55PCN, U605 AS6C4008-55PCN, U606 AS6C4008-55PCN, U607 AS6C4008-55PCN, U608 AS6C6264-55PCN, U701 W65C51, U702 16550, U703 74HC04, U704 Ali_Express_FTDI_Breakout, U705 Adafruit_FTDI_Friend, U706 Ali_Express_FTDI_Breakout, U801 Adafruit_Metro_Mini, X201 ACO-32.000MHz, X701 1.8432MHz

Commit message: Tweaks to the expansion interface.
Connections:
- J901 pad 17: GND -> E
- J901 pad 19: E -> ~{RESET}
- J901 pad 21: GND -> ~{HALT}
- J901 pad 39: ~{RESET} -> GND
- J902 pad 1: GND -> EXP1_AUDIO_L
- J902 pad 2: GND -> EXP1_AUDIO_R
- J902 pad 3: EXP1_AUDIO_L -> unconnected-(J902-Pin_3-Pad3)
- J902 pad 4: EXP1_AUDIO_R -> unconnected-(J902-Pin_4-Pad4)
- J902 pad 5: GND -> unconnected-(J902-Pin_5-Pad5)
- J902 pad 6: GND -> unconnected-(J902-Pin_6-Pad6)
- J903 pad 17: GND -> E
- J903 pad 19: E -> ~{RESET}
- J903 pad 21: GND -> ~{HALT}
- J903 pad 39: ~{RESET} -> GND
- J904 pad 1: GND -> EXP2_AUDIO_L
- J904 pad 2: GND -> EXP2_AUDIO_R
- J904 pad 3: EXP2_AUDIO_L -> unconnected-(J904-Pin_3-Pad3)
- J904 pad 4: EXP2_AUDIO_R -> unconnected-(J904-Pin_4-Pad4)
- J904 pad 5: GND -> unconnected-(J904-Pin_5-Pad5)
- J904 pad 6: GND -> unconnected-(J904-Pin_6-Pad6)
- J905 pad 17: GND -> E
- J905 pad 19: E -> ~{RESET}
- J905 pad 21: GND -> ~{HALT}
- J905 pad 39: ~{RESET} -> GND
- J906 pad 1: GND -> EXP3_AUDIO_L
- J906 pad 2: GND -> EXP3_AUDIO_R
- J906 pad 3: EXP3_AUDIO_L -> unconnected-(J906-Pin_3-Pad3)
- J906 pad 4: EXP3_AUDIO_R -> unconnected-(J906-Pin_4-Pad4)
- J906 pad 5: GND -> unconnected-(J906-Pin_5-Pad5)
- J906 pad 6: GND -> unconnected-(J906-Pin_6-Pad6)
- J907 pad 17: GND -> E
- J907 pad 19: E -> ~{RESET}
- J907 pad 21: GND -> ~{HALT}
- J907 pad 39: ~{RESET} -> GND
- J908 pad 1: GND -> EXP4_AUDIO_L
- J908 pad 2: GND -> EXP4_AUDIO_R
- J908 pad 3: EXP4_AUDIO_L -> unconnected-(J908-Pin_3-Pad3)
- J908 pad 4: EXP4_AUDIO_R -> unconnected-(J908-Pin_4-Pad4)
- J908 pad 5: GND -> unconnected-(J908-Pin_5-Pad5)
- J908 pad 6: GND -> unconnected-(J908-Pin_6-Pad6)

Commit message: Move Reset to the main sheet.  Checkpoint SD Card SPI interface.
Parts:
- removed R203: 3K3, Resistor_THT:R_Axial_DIN0207_L6.3mm_D2.5mm_P7.62mm_Horizontal
- removed SW201: Reset, Button_Switch_THT:SW_PUSH_6mm
- removed U203: DS1813, Package_TO_SOT_THT:TO-92_Inline
- added C1001: 0.1µF, Capacitor_THT:C_Disc_D3.8mm_W2.6mm_P2.50mm, F.Cu at (426.2, 132.6)
- added C1002: 0.1µF, Capacitor_THT:C_Disc_D3.8mm_W2.6mm_P2.50mm, F.Cu at (404.9, 135.8)
- added C1003: 0.1µF, Capacitor_THT:C_Disc_D3.8mm_W2.6mm_P2.50mm, F.Cu at (379.5, 135.8)
- added J1001: Adafruit MicroSD Card Breakout Board+, Connector_PinHeader_2.54mm:PinHeader_1x08_P2.54mm_Vertical, F.Cu at (353.1, 109.2)
- added Q1001: 2N7000, Package_TO_SOT_THT:TO-92_Inline, F.Cu at (368.8, 117.5)
- added R1001: 10K, Resistor_THT:R_Axial_DIN0207_L6.3mm_D2.5mm_P7.62mm_Horizontal, F.Cu at (358.0, 115.1)
- added R1002: 10K, Resistor_THT:R_Axial_DIN0207_L6.3mm_D2.5mm_P7.62mm_Horizontal, F.Cu at (358.0, 118.2)
- added R1003: 10K, Resistor_THT:R_Axial_DIN0207_L6.3mm_D2.5mm_P7.62mm_Horizontal, F.Cu at (358.0, 121.4)
- added R103: 3K3, Resistor_THT:R_Axial_DIN0207_L6.3mm_D2.5mm_P7.62mm_Horizontal, F.Cu at (428.6, 271.6)
- added SW102: Reset, Button_Switch_THT:SW_PUSH_6mm, F.Cu at (314.4, 324.2)
- added U1001: W65C22, Package_DIP:DIP-40_W15.24mm_Socket, F.Cu at (374.7, 132.6)
- added U1002: 74HC86, Package_DIP:DIP-14_W7.62mm_Socket, F.Cu at (407.7, 143.4)
- added U1003: 74HC164, Package_DIP:DIP-14_W7.62mm_Socket, F.Cu at (382.3, 143.4)
- added U108: DS1813, Package_TO_SOT_THT:TO-92_Inline, F.Cu at (420.9, 271.6)

Commit message: Checkpoint SD card interface.  Need to add activity LED.
Parts:
- added H1001: MountingHole_Pad, MountingHole:MountingHole_2.2mm_M2_Pad_Via, F.Cu at (346.7, 92.2)
- added H1002: MountingHole_Pad, MountingHole:MountingHole_2.2mm_M2_Pad_Via, F.Cu at (367.0, 92.2)
- added H1003: MountingHole_Pad, MountingHole:MountingHole_2.2mm_M2_Pad_Via, F.Cu at (346.7, 112.5)
- added H1004: MountingHole_Pad, MountingHole:MountingHole_2.2mm_M2_Pad_Via, F.Cu at (367.0, 112.5)
- moved R1003 27.0 mm to (374.4, 142.9), turned to 90 degrees
- moved Q1001 21.5 mm to (373.6, 96.5)
- moved R1002 20.9 mm to (376.7, 109.0), turned to 90 degrees
- moved R1001 20.8 mm to (373.6, 101.4), turned to -90 degrees
- moved J1001 11.9 mm to (348.0, 120.0)

Commit message: Add SD Card activity LED.
Parts:
- added D1001: SD Card, LED_THT:LED_D3.0mm, F.Cu at (386.1, 326.4)
- added R1004: 1K, Resistor_THT:R_Axial_DIN0207_L6.3mm_D2.5mm_P7.62mm_Horizontal, F.Cu at (400.8, 306.3)
Connections:
- J1001 pad 7: /SPI SD Card Interface/SD_CS -> SD_LED-
- J101 pad 7: unconnected-(J101-Pin_7-Pad7) -> SD_LED+
- J101 pad 9: unconnected-(J101-Pin_9-Pad9) -> SD_LED-
- Q1001 pad 3: /SPI SD Card Interface/SD_CS -> SD_LED-
- R1002 pad 2: /SPI SD Card Interface/SD_CS -> SD_LED-
- U1002 pad 10: GND -> /SPI SD Card Interface/SD_SCK
- U1002 pad 8: unconnected-(U1002-Pad8) -> SD_LED+
Other:
- board text added: "SD LED+"
- board text added: "SD LED-"

Commit message: Correct footprint for fixed ROM ZIF socket.
Parts:
- U502: footprint Socket:DIP_Socket-28_W6.9_W7.62_W10.16_W12.7_W13.5_3M_228-4817-00-0602J -> Socket:DIP_Socket-28_W11.9_W12.7_W15.24_W17.78_W18.5_3M_228-1277-00-0602J
- moved C501 9.72 mm to (171.5, 317.1)
- moved C503 9.72 mm to (208.4, 266.0)
- moved R101 9.72 mm to (204.7, 313.1)
- moved U501 9.72 mm to (174.7, 268.8)
- moved U503 9.72 mm to (193.2, 268.8)
- moved U502 5.00 mm to (222.8, 273.8)

Commit message: A ZIF socket also for the banked ROM.
Parts:
- U503: footprint Package_DIP:DIP-32_W15.24mm_Socket -> Socket:DIP_Socket-32_W11.9_W12.7_W15.24_W17.78_W18.5_3M_232-1285-00-0602J
- moved C503 10.1 mm to (217.9, 269.2), turned to -90 degrees
- moved R101 7.15 mm to (208.0, 319.5)
- moved C501 5.10 mm to (167.2, 319.9)
- moved U501 5.10 mm to (170.4, 271.6)
- moved U503 3.45 mm to (196.6, 269.0)
- moved U502 2.81 mm to (225.6, 274.1)
- moved C502 2.60 mm to (246.9, 274.1), turned to -90 degrees

Commit message: Give the front panel LED its own current-limiting resistor.
Parts:
- added R1005: 1K, Resistor_THT:R_Axial_DIN0207_L6.3mm_D2.5mm_P7.62mm_Horizontal, F.Cu at (400.8, 303.3)
Connections:
- J1001 pad 7: SD_LED- -> /SPI SD Card Interface/SD_CS
- Q1001 pad 3: SD_LED- -> /SPI SD Card Interface/SD_CS
- R1002 pad 2: SD_LED- -> /SPI SD Card Interface/SD_CS
- R1004 pad 1: Net-(D1001-K) -> /SPI SD Card Interface/SD_CS
- R1004 pad 2: SD_LED- -> Net-(D1001-K)
Changed lines of the file:
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@@
   (net 434 "Net-(U1001-CB1)")
   (net 435 "Net-(U1001-CB2)")
-  (net 436 "unconnected-(U1002-Pad11)")
+  (net 436 "/SPI SD Card Interface/SD_CS")
+  (net 437 "unconnected-(U1002-Pad11)")
   (footprint "Package_DIP:DIP-24_W7.62mm_Socket" (layer "F.Cu")
     (at 245.3748 212.819)
@@
       (net 420 "/SPI SD Card Interface/SD_MOSI") (pinfunction "Pin_6") (pintype "passive"))
     (pad "7" thru_hole oval (at 0 15.24 90) (size 1.7 1.7) (drill 1) (layers "*.Cu" "*.Mask")
-      (net 421 "SD_LED-") (pinfunction "Pin_7") (pintype "passive"))
+      (net 436 "/SPI SD Card Interface/SD_CS") (pinfunction "Pin_7") (pintype "passive"))
     (pad "8" thru_hole oval (at 0 17.78 90) (size 1.7 1.7) (drill 1) (layers "*.Cu" "*.Mask")
       (net 422 "/SPI SD Card Interface/SD_CD") (pinfunction "Pin_8") (pintype "passive"))
@@
       (net 424 "Net-(Q1001-G)") (pinfunction "G") (pintype "input"))
     (pad "3" thru_hole oval (at 2.54 0) (size 1.05 1.5) (drill 0.75) (layers "*.Cu" "*.Mask")
-      (net 421 "SD_LED-") (pinfunction "D") (pintype "passive"))
+      (net 436 "/SPI SD Card Interface/SD_CS") (pinfunction "D") (pintype "passive"))
     (model "${KICAD6_3DMODEL_DIR}/Package_TO_SOT_THT.3dshapes/TO-92_Inline.wrl"
       (offset (xyz 0 0 0))
@@
     )
   )
+  (footprint "Resistor_THT:R_Axial_DIN0207_L6.3mm_D2.5mm_P7.62mm_Horizontal" (layer "F.Cu")
+    (at 400.812 303.276)
+    (descr "Resistor, Axial_DIN0207 series, Axial, Horizontal, pin pitch=7.62mm, 0.25W = 1/4W, length*diameter=6.3*2.5mm^2, http://cdn-reichelt.de/documents/datenblatt/B400/1_4W%23YAG.pdf")
+    (tags "Resistor Axial_DIN0207 series Axial Horizontal pin pitch 7.62mm 0.25W = 1/4W length 6.3mm diameter 2.5mm")
+    (property "Field2" "")
+    (property "Sheetfile" "pg09-system-spi-sdcard.kicad_sch")
+    (property "Sheetname" "SPI SD Card Interface")
+    (property "ki_description" "Resistor, small symbol")
+    (property "ki_keywords" "R resistor")
+    (attr through_hole)
+    (fp_text reference "R1005" (at 11.176 0) (layer "F.SilkS")
+        (effects (font (size 1 1) (thickness 0.15)))
+    )
+    (fp_text value "1K" (at 3.81 2.37) (layer "F.Fab") hide
+        (effects (font (size 1 1) (thickness 0.15)))
+    )
+    (fp_text user "${REFERENCE}" (at 3.81 0) (layer "F.Fab")
+        (effects (font (size 1 1) (thickness 0.15)))
+    )
+    (fp_line (start 0.54 -1.37) (end 7.08 -1.37)
+      (stroke (width 0.12) (type solid)) (layer "F.SilkS"))
+    (fp_line (start 0.54 -1.04) (end 0.54 -1.37)
+      (stroke (width 0.12) (type solid)) (layer "F.SilkS"))
+    (fp_line (start 0.54 1.04) (end 0.54 1.37)
+      (stroke (width 0.12) (type solid)) (layer "F.SilkS"))
+    (fp_line (start 0.54 1.37) (end 7.08 1.37)
+      (stroke (width 0.12) (type solid)) (layer "F.SilkS"))
+    (fp_line (start 7.08 -1.37) (end 7.08 -1.04)
+      (stroke (width 0.12) (type solid)) (layer "F.SilkS"))
+    (fp_line (start 7.08 1.37) (end 7.08 1.04)
+      (stroke (width 0.12) (type solid)) (layer "F.SilkS"))
+    (fp_line (start -1.05 -1.5) (end -1.05 1.5)
+      (stroke (width 0.05) (type solid)) (layer "F.CrtYd"))
+    (fp_line (start -1.05 1.5) (end 8.67 1.5)
+      (stroke (width 0.05) (type solid)) (layer "F.CrtYd"))
+    (fp_line (start 8.67 -1.5) (end -1.05 -1.5)
+      (stroke (width 0.05) (type solid)) (layer "F.CrtYd"))
+    (fp_line (start 8.67 1.5) (end 8.67 -1.5)
+      (stroke (width 0.05) (type solid)) (layer "F.CrtYd"))
+    (fp_line (start 0 0) (end 0.66 0)
+      (stroke (width 0.1) (type solid)) (layer "F.Fab"))
+    (fp_line (start 0.66 -1.25) (end 0.66 1.25)
+      (stroke (width 0.1) (type solid)) (layer "F.Fab"))
+    (fp_line (start 0.66 1.25) (end 6.96 1.25)
+      (stroke (width 0.1) (type solid)) (layer "F.Fab"))
+    (fp_line (start 6.96 -1.25) (end 0.66 -1.25)
+      (stroke (width 0.1) (type solid)) (layer "F.Fab"))
+    (fp_line (start 6.96 1.25) (end 6.96 -1.25)
+      (stroke (width 0.1) (type solid)) (layer "F.Fab"))
+    (fp_line (start 7.62 0) (end 6.96 0)
+      (stroke (width 0.1) (type solid)) (layer "F.Fab"))
+    (pad "1" thru_hole circle (at 0 0) (size 1.6 1.6) (drill 0.8) (layers "*.Cu" "*.Mask")
+      (net 436 "/SPI SD Card Interface/SD_CS") (pintype "passive"))
+    (pad "2" thru_hole oval (at 7.62 0) (size 1.6 1.6) (drill 0.8) (layers "*.Cu" "*.Mask")
+      (net 421 "SD_LED-") (pintype "passive"))
+    (model "${KICAD6_3DMODEL_DIR}/Resistor_THT.3dshapes/R_Axial_DIN0207_L6.3mm_D2.5mm_P7.62mm_Horizontal.wrl"
+      (offset (xyz 0 0 0))
+      (scale (xyz 1 1 1))
+      (rotate (xyz 0 0 0))
+    )
+  )
   (footprint "Package_DIP:DIP-40_W15.24mm_Socket" (layer "F.Cu")
     (at 250.3092 262.822)
@@
     (property "ki_keywords" "R resistor")
     (attr through_hole)
-    (fp_text reference "R1004" (at 3.81 -2.37) (layer "F.SilkS")
+    (fp_text reference "R1004" (at 11.176 0) (layer "F.SilkS")
         (effects (font (size 1 1) (thickness 0.15)))
     )
@@
       (stroke (width 0.1) (type solid)) (layer "F.Fab"))
     (pad "1" thru_hole circle (at 0 0) (size 1.6 1.6) (drill 0.8) (layers "*.Cu" "*.Mask")
-      (net 386 "Net-(D1001-K)") (pintype "passive"))
+      (net 436 "/SPI SD Card Interface/SD_CS") (pintype "passive"))
     (pad "2" thru_hole oval (at 7.62 0) (size 1.6 1.6) (drill 0.8) (layers "*.Cu" "*.Mask")
-      (net 421 "SD_LED-") (pintype "passive"))
+      (net 386 "Net-(D1001-K)") (pintype "passive"))
     (model "${KICAD6_3DMODEL_DIR}/Resistor_THT.3dshapes/R_Axial_DIN0207_L6.3mm_D2.5mm_P7.62mm_Horizontal.wrl"
       (offset (xyz 0 0 0))
@@
       (net 418 "/SPI SD Card Interface/SD_SCK") (pintype "input"))
     (pad "11" thru_hole oval (at 7.62 7.62 90) (size 1.6 1.6) (drill 0.8) (layers "*.Cu" "*.Mask")
-      (net 436 "unconnected-(U1002-Pad11)") (pintype "output+no_connect"))
+      (net 437 "unconnected-(U1002-Pad11)") (pintype "output+no_connect"))
     (pad "12" thru_hole oval (at 7.62 5.08 90) (size 1.6 1.6) (drill 0.8) (layers "*.Cu" "*.Mask")
       (net 2 "GND") (pintype "input"))
@@
       (net 1 "+5V") (pintype "passive"))
     (pad "2" thru_hole oval (at 7.62 0 90) (size 1.6 1.6) (drill 0.8) (layers "*.Cu" "*.Mask")
-      (net 421 "SD_LED-") (pintype "passive"))
+      (net 436 "/SPI SD Card Interface/SD_CS") (pintype "passive"))
     (model "${KICAD6_3DMODEL_DIR}/Resistor_THT.3dshapes/R_Axial_DIN0207_L6.3mm_D2.5mm_P7.62mm_Horizontal.wrl"
       (offset (xyz 0 0 0))

Commit message: Assign IRQ0 to the SD Card interface.
Connections:
- U1001 pad 21: unconnected-(U1001-~{IRQ}-Pad21) -> ~{IRQ0}
