File: design-files/pg09-system.kicad_pcb (KiCad board)
At the start: 4 copper layers, 306 x 244 mm, 142 parts, among them J1001 Adafruit MicroSD Card Breakou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, J101 Front Panel, J1101 PS/2 Keyboard, J1102 SNES-Controller-Socket, J1103 SNES-Controller-Socket, J201 Clock Speed, J801 ATX-24, J802 #PS_ON, J803 PSU-CTRL console, J901 Expansion 1, J902 Expansion 1 ext, J903 Expansion 2, J904 Expansion 2 ext, J905 Expansion 3, J906 Expansion 3 ext, J907 Expansion 4, J908 Expansion 4 ext, Q1001 2N7000, Q701 2N7000, SW101 NMI, SW102 Reset, SW801 Power, U1001 W65C22, U1002 74HC86, U1003 74HC164, U101 MC6809E, U102 GAL22V10, U103 74AHCT245, U104 74AHCT245, U105 74AHCT245, U106 GAL22V10, U107 DS1813, U108 DS1813, U201 CD74ACT109, U202 CD74ACT163, U204 GAL22V10, U301 GAL22V10, U302 GAL22V10, U401 W65C21, U402 GAL22V10, U403 GAL22V10, U404 GAL22V10, U405 74AHC374, U406 74AHC374, U407 74AHC138, U501 W65C21, U502 AT28C64, U503 SST39SF040, U601 W65C21, U602 AS6C4008-55PCN, U603 74AHC138, U604 AS6C4008-55PCN, U605 AS6C4008-55PCN, U606 AS6C4008-55PCN, U607 AS6C4008-55PCN, U608 AS6C6264-55PCN, U701 W65C51, U702 16550, U703 74HC04, U704 Ali_Express_FTDI_Breakout, U705 Adafruit_FTDI_Friend, U801 Adafruit_Metro_Mini, X201 ACO-32.000MHz, X701 1.8432MHz

Commit message: Orient both SNES connectors properly.
Parts:
- moved J1103 26.2 mm to (366.0, 99.8), turned to 180 degrees
Changed lines of the file:
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@@
   )
   (footprint "jrt-SNES:SNES-Connector_Vertical" (layer "F.Cu")
-    (at 339.852 99.822)
+    (at 366.014 99.822 180)
     (property "Sheetfile" "pg09-system-hid.kicad_sch")
     (property "Sheetname" "Human Interface Devices")
     (attr through_hole)
-    (fp_text reference "J1103" (at -9 0 270) (layer "F.Fab")
+    (fp_text reference "J1103" (at -9 0 90) (layer "F.Fab")
         (effects (font (size 1 1) (thickness 0.15)))
     )
@@
     (fp_circle (center 26.5 0) (end 28.15 0)
       (stroke (width 0.12) (type solid)) (fill none) (layer "F.Fab"))
-    (pad "1" thru_hole circle (at 0 0) (size 3 3) (drill 2) (layers "*.Cu" "*.Mask")
+    (pad "1" thru_hole circle (at 0 0 180) (size 3 3) (drill 2) (layers "*.Cu" "*.Mask")
       (net 440 "unconnected-(J1103-5V-Pad1)") (pinfunction "5V") (pintype "power_in+no_connect"))
-    (pad "2" thru_hole circle (at 4 0) (size 3 3) (drill 2) (layers "*.Cu" "*.Mask")
+    (pad "2" thru_hole circle (at 4 0 180) (size 3 3) (drill 2) (layers "*.Cu" "*.Mask")
       (net 441 "unconnected-(J1103-Clock-Pad2)") (pinfunction "Clock") (pintype "input+no_connect"))
-    (pad "3" thru_hole circle (at 8 0) (size 3 3) (drill 2) (layers "*.Cu" "*.Mask")
+    (pad "3" thru_hole circle (at 8 0 180) (size 3 3) (drill 2) (layers "*.Cu" "*.Mask")
       (net 442 "unconnected-(J1103-Latch-Pad3)") (pinfunction "Latch") (pintype "input+no_connect"))
-    (pad "4" thru_hole circle (at 12 0) (size 3 3) (drill 2) (layers "*.Cu" "*.Mask")
+    (pad "4" thru_hole circle (at 12 0 180) (size 3 3) (drill 2) (layers "*.Cu" "*.Mask")
       (net 443 "unconnected-(J1103-Data-Pad4)") (pinfunction "Data") (pintype "output+no_connect"))
-    (pad "5" thru_hole circle (at 18.5 0) (size 3 3) (drill 2) (layers "*.Cu" "*.Mask")
+    (pad "5" thru_hole circle (at 18.5 0 180) (size 3 3) (drill 2) (layers "*.Cu" "*.Mask")
       (net 444 "unconnected-(J1103-N{slash}C-Pad5)") (pinfunction "N/C") (pintype "bidirectional+no_connect"))
-    (pad "6" thru_hole circle (at 22.5 0) (size 3 3) (drill 2) (layers "*.Cu" "*.Mask")
+    (pad "6" thru_hole circle (at 22.5 0 180) (size 3 3) (drill 2) (layers "*.Cu" "*.Mask")
       (net 445 "unconnected-(J1103-N{slash}C-Pad6)") (pinfunction "N/C") (pintype "bidirectional+no_connect"))
-    (pad "7" thru_hole circle (at 26.5 0) (size 3 3) (drill 2) (layers "*.Cu" "*.Mask")
+    (pad "7" thru_hole circle (at 26.5 0 180) (size 3 3) (drill 2) (layers "*.Cu" "*.Mask")
       (net 446 "unconnected-(J1103-GND-Pad7)") (pinfunction "GND") (pintype "power_in+no_connect"))
     (model "${KIPRJMOD}/${PKL_REL_DIR}/packages3d/pkl_connectors.3dshapes/SNES.stp"

Commit message: Re-arrange CLKSEL pins for board layout reasons.
Parts:
- J201: value Clock Speed -> CPU Speed
Connections:
- U204 pad 1: E -> unconnected-(U204-I1/CLK-Pad1)
- U204 pad 13: unconnected-(U204-I12-Pad13) -> E
- U204 pad 14: Net-(U201A-C) -> D7
- U204 pad 15: unconnected-(U204-IO2-Pad15) -> D6
- U204 pad 16: D7 -> D5
- U204 pad 17: D6 -> D4
- U204 pad 18: D5 -> D3
- U204 pad 19: D4 -> D2
- U204 pad 20: D3 -> D1
- U204 pad 21: D2 -> D0
- U204 pad 22: D1 -> unconnected-(U204-IO9-Pad22)
- U204 pad 23: D0 -> Net-(U201A-C)
Changed lines of the file:
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@@
   (net 48 "Net-(J201-Pin_5)")
   (net 49 "Net-(U201A-C)")
-  (net 50 "unconnected-(U204-I12-Pad13)")
-  (net 51 "unconnected-(U204-IO2-Pad15)")
+  (net 50 "unconnected-(U204-I1{slash}CLK-Pad1)")
+  (net 51 "unconnected-(U204-IO9-Pad22)")
   (net 52 "EXP3_AUDIO_L")
   (net 53 "EXP3_AUDIO_R")
@@
       (stroke (width 0.1) (type solid)) (layer "F.Fab"))
     (pad "1" thru_hole rect (at 0 0) (size 1.6 1.6) (drill 0.8) (layers "*.Cu" "*.Mask")
-      (net 14 "E") (pinfunction "I1/CLK") (pintype "input"))
+      (net 50 "unconnected-(U204-I1{slash}CLK-Pad1)") (pinfunction "I1/CLK") (pintype "input+no_connect"))
     (pad "2" thru_hole oval (at 0 2.54) (size 1.6 1.6) (drill 0.8) (layers "*.Cu" "*.Mask")
       (net 3 "CLK_16MHz") (pinfunction "I2") (pintype "input"))
@@
       (net 2 "GND") (pinfunction "GND") (pintype "power_in"))
     (pad "13" thru_hole oval (at 7.62 27.94) (size 1.6 1.6) (drill 0.8) (layers "*.Cu" "*.Mask")
-      (net 50 "unconnected-(U204-I12-Pad13)") (pinfunction "I12") (pintype "input+no_connect"))
+      (net 14 "E") (pinfunction "I12") (pintype "input"))
     (pad "14" thru_hole oval (at 7.62 25.4) (size 1.6 1.6) (drill 0.8) (layers "*.Cu" "*.Mask")
-      (net 49 "Net-(U201A-C)") (pinfunction "IO1") (pintype "tri_state"))
+      (net 103 "D7") (pinfunction "IO1") (pintype "tri_state"))
     (pad "15" thru_hole oval (at 7.62 22.86) (size 1.6 1.6) (drill 0.8) (layers "*.Cu" "*.Mask")
-      (net 51 "unconnected-(U204-IO2-Pad15)") (pinfunction "IO2") (pintype "tri_state+no_connect"))
+      (net 102 "D6") (pinfunction "IO2") (pintype "tri_state"))
     (pad "16" thru_hole oval (at 7.62 20.32) (size 1.6 1.6) (drill 0.8) (layers "*.Cu" "*.Mask")
-      (net 103 "D7") (pinfunction "IO3") (pintype "tri_state"))
+      (net 101 "D5") (pinfunction "IO3") (pintype "tri_state"))
     (pad "17" thru_hole oval (at 7.62 17.78) (size 1.6 1.6) (drill 0.8) (layers "*.Cu" "*.Mask")
-      (net 102 "D6") (pinfunction "IO4") (pintype "tri_state"))
+      (net 100 "D4") (pinfunction "IO4") (pintype "tri_state"))
     (pad "18" thru_hole oval (at 7.62 15.24) (size 1.6 1.6) (drill 0.8) (layers "*.Cu" "*.Mask")
-      (net 101 "D5") (pinfunction "IO5") (pintype "tri_state"))
+      (net 99 "D3") (pinfunction "IO5") (pintype "tri_state"))
     (pad "19" thru_hole oval (at 7.62 12.7) (size 1.6 1.6) (drill 0.8) (layers "*.Cu" "*.Mask")
-      (net 100 "D4") (pinfunction "IO6") (pintype "tri_state"))
+      (net 98 "D2") (pinfunction "IO6") (pintype "tri_state"))
     (pad "20" thru_hole oval (at 7.62 10.16) (size 1.6 1.6) (drill 0.8) (layers "*.Cu" "*.Mask")
-      (net 99 "D3") (pinfunction "IO7") (pintype "tri_state"))
+      (net 97 "D1") (pinfunction "IO7") (pintype "tri_state"))
     (pad "21" thru_hole oval (at 7.62 7.62) (size 1.6 1.6) (drill 0.8) (layers "*.Cu" "*.Mask")
-      (net 98 "D2") (pinfunction "IO8") (pintype "tri_state"))
+      (net 96 "D0") (pinfunction "IO8") (pintype "tri_state"))
     (pad "22" thru_hole oval (at 7.62 5.08) (size 1.6 1.6) (drill 0.8) (layers "*.Cu" "*.Mask")
-      (net 97 "D1") (pinfunction "IO9") (pintype "tri_state"))
+      (net 51 "unconnected-(U204-IO9-Pad22)") (pinfunction "IO9") (pintype "tri_state+no_connect"))
     (pad "23" thru_hole oval (at 7.62 2.54) (size 1.6 1.6) (drill 0.8) (layers "*.Cu" "*.Mask")
-      (net 96 "D0") (pinfunction "IO10") (pintype "tri_state"))
+      (net 49 "Net-(U201A-C)") (pinfunction "IO10") (pintype "tri_state"))
     (pad "24" thru_hole oval (at 7.62 0) (size 1.6 1.6) (drill 0.8) (layers "*.Cu" "*.Mask")
       (net 1 "+5V") (pinfunction "VCC") (pintype "power_in"))
@@
         (effects (font (size 1 1) (thickness 0.15)))
     )
-    (fp_text value "Clock Speed" (at 1.27 7.41) (layer "F.SilkS")
+    (fp_text value "CPU Speed" (at 1.27 7.41) (layer "F.SilkS")
         (effects (font (size 1 1) (thickness 0.15)))
     )

Commit message: Update PCB rats nest for recent changes.
Parts:
- J201: value CPU Speed -> Clock Speed
Connections:
- U204 pad 13: E -> unconnected-(U204-I12-Pad13)
- U204 pad 22: unconnected-(U204-IO9-Pad22) -> E

Commit message: R102 and R103 are gone.
Parts:
- removed R102, R103: 3K3, Resistor_THT:R_Axial_DIN0207_L6.3mm_D2.5mm_P7.62mm_Horizontal
Connections:
- RN201 pad 5: unconnected-(RN201-R4-Pad5) -> ~{RESET}

Commit message: Use an R-C circuit in front of the Vcc on /RESET's DS1813 in order to delay power-on-reset by ~0.75 seconds.
Parts:
- added C108: 470µF 50V, Capacitor_THT:CP_Radial_D12.5mm_P5.00mm, F.Cu at (431.9, 221.0)
- added D101: 1N4448, Diode_THT:D_DO-35_SOD27_P7.62mm_Horizontal, F.Cu at (424.4, 207.3)
- added R102: 1K, Resistor_THT:R_Axial_DIN0207_L6.3mm_D2.5mm_P7.62mm_Horizontal, F.Cu at (424.4, 217.2)
- moved J802 20.6 mm to (433.6, 267.5)
- moved C801 15.7 mm to (427.8, 239.3)
Connections:
- U108 pad 2: +5V -> Net-(D101-A)
Routing:
- net Net-(D101-A): track 0.00 -> 54.6 mm

Commit message: Tweak the reset and NMI circuits -- no pull-ups on those signals needed; the DS1813 has us covered.  Add power-on-reset delay of ~0.5 seconds.
Parts:
- C108: value 470µF 50V -> 100µF 16V; footprint Capacitor_THT:CP_Radial_D12.5mm_P5.00mm -> Capacitor_THT:CP_Radial_D6.3mm_P2.50mm
- D101: value 1N4448 -> 1N4001; footprint Diode_THT:D_DO-35_SOD27_P7.62mm_Horizontal -> Diode_THT:D_DO-41_SOD81_P10.16mm_Horizontal
- R102: value 1K -> 3K3
- moved R102 43.8 mm to (427.7, 260.9)
- moved C108 43.7 mm to (433.4, 264.7)
- moved D101 41.0 mm to (426.7, 248.2)
- moved C801 15.0 mm to (427.8, 224.3)
- moved J802 3.81 mm to (433.6, 271.3)
Connections:
- RN201 pad 2: ~{NMI} -> ~{FIRQ}
- RN201 pad 3: ~{FIRQ} -> ~{HALT}
- RN201 pad 4: ~{HALT} -> unconnected-(RN201-R3-Pad4)
- RN201 pad 5: ~{RESET} -> unconnected-(RN201-R4-Pad5)
Routing:
- net Net-(D101-A): track 54.6 -> 0.00 mm

Commit message: Use physically smaller caps in the PSU.
Parts:
- C801: value 2700µF 50V -> 4700µF 16V; footprint Capacitor_THT:CP_Radial_D18.0mm_P7.50mm -> Capacitor_THT:CP_Radial_D12.5mm_P5.00mm
- C802, C803, C804: value 470µF 50V -> 470µF 25V; footprint Capacitor_THT:CP_Radial_D12.5mm_P5.00mm -> Capacitor_THT:CP_Radial_D10.0mm_P5.00mm
- moved C801 8.86 mm to (431.9, 216.4)
- moved C804 3.56 mm to (431.9, 202.2)
- moved C803 1.27 mm to (431.9, 189.5)
Routing:
- net +3V3: track 81.8 -> 79.0 mm
- net -12V: track 255.9 -> 254.6 mm

Commit message: Make the RESET diode a 1N4148.  Put the resistor VALUE on the F.Silk layer inside the footprint.
Parts:
- D101: value 1N4001 -> 1N4148; footprint Diode_THT:D_DO-41_SOD81_P10.16mm_Horizontal -> Diode_THT:D_DO-35_SOD27_P7.62mm_Horizontal
- moved D101 10.3 mm to (421.1, 256.8), turned to 0 degrees
Changed lines of the file:
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@@
         (effects (font (size 1 1) (thickness 0.15)))
     )
-    (fp_text user "${REFERENCE}" (at 3.81 0) (layer "F.Fab")
+    (fp_text user "${VALUE}" (at 3.81 0) (layer "F.SilkS")
         (effects (font (size 1 1) (thickness 0.15)))
     )
@@
         (effects (font (size 1 1) (thickness 0.15)))
     )
-    (fp_text user "${REFERENCE}" (at 3.81 0 90) (layer "F.Fab")
+    (fp_text user "${VALUE}" (at 3.81 0 90) (layer "F.SilkS")
         (effects (font (size 1 1) (thickness 0.15)))
     )
@@
         (effects (font (size 1 1) (thickness 0.15)))
     )
-    (fp_text user "${REFERENCE}" (at 3.81 0) (layer "F.Fab")
+    (fp_text user "${VALUE}" (at 3.81 0) (layer "F.SilkS")
         (effects (font (size 1 1) (thickness 0.15)))
     )
@@
         (effects (font (size 1 1) (thickness 0.15)))
     )
-    (fp_text user "${REFERENCE}" (at 3.81 0) (layer "F.Fab")
+    (fp_text user "${VALUE}" (at 3.81 0) (layer "F.SilkS")
         (effects (font (size 1 1) (thickness 0.15)))
     )
@@
         (effects (font (size 1 1) (thickness 0.15)))
     )
-    (fp_text user "${REFERENCE}" (at 3.81 0) (layer "F.Fab")
+    (fp_text user "${VALUE}" (at 3.81 0) (layer "F.SilkS")
         (effects (font (size 1 1) (thickness 0.15)))
     )
@@
         (effects (font (size 1 1) (thickness 0.15)))
     )
-    (fp_text user "${REFERENCE}" (at 3.81 0 90) (layer "F.Fab")
+    (fp_text user "${VALUE}" (at 3.81 0 90) (layer "F.SilkS")
         (effects (font (size 1 1) (thickness 0.15)))
     )
@@
     )
   )
-  (footprint "Diode_THT:D_DO-41_SOD81_P10.16mm_Horizontal" (layer "F.Cu")
-    (at 426.72 248.158 -90)
-    (descr "Diode, DO-41_SOD81 series, Axial, Horizontal, pin pitch=10.16mm, , length*diameter=5.2*2.7mm^2, , http://www.diodes.com/_files/packages/DO-41%20(Plastic).pdf")
-    (tags "Diode DO-41_SOD81 series Axial Horizontal pin pitch 10.16mm  length 5.2mm diameter 2.7mm")
+  (footprint "Diode_THT:D_DO-35_SOD27_P7.62mm_Horizontal" (layer "F.Cu")
+    (at 421.132 256.794)
+    (descr "Diode, DO-35_SOD27 series, Axial, Horizontal, pin pitch=7.62mm, , length*diameter=4*2mm^2, , http://www.diodes.com/_files/packages/DO-35.pdf")
+    (tags "Diode DO-35_SOD27 series Axial Horizontal pin pitch 7.62mm  length 4mm diameter 2mm")
     (property "Sheetfile" "pg09-system.kicad_sch")
     (property "Sheetname" "")
     (property "Sim.Device" "D")
     (property "Sim.Pins" "1=K 2=A")
-    (property "ki_description" "50V 1A General Purpose Rectifier Diode, DO-41")
+    (property "ki_description" "100V 0.15A standard switching diode, DO-35")
     (property "ki_keywords" "diode")
     (attr through_hole)
-    (fp_text reference "D101" (at 5.08 -2.47 -90) (layer "F.SilkS")
+    (fp_text reference "D101" (at 3.81 -2.12) (layer "F.SilkS")
         (effects (font (size 1 1) (thickness 0.15)))
     )
-    (fp_text value "1N4001" (at 5.08 2.47 -90) (layer "F.SilkS")
+    (fp_text value "1N4148" (at 3.81 2.12) (layer "F.SilkS")
         (effects (font (size 1 1) (thickness 0.15)))
     )
-    (fp_text user "K" (at 0 -2.1 -90) (layer "F.SilkS")
+    (fp_text user "K" (at 0 -1.8) (layer "F.SilkS")
         (effects (font (size 1 1) (thickness 0.15)))
     )
-    (fp_text user "K" (at 0 -2.1 -90) (layer "F.Fab")
-        (effects (font (size 1 1) (thickness 0.15)))
+    (fp_text user "${REFERENCE}" (at 4.11 0) (layer "F.Fab")
+        (effects (font (size 0.8 0.8) (thickness 0.12)))
     )
-    (fp_text user "${REFERENCE}" (at 5.47 0 -90) (layer "F.Fab")
+    (fp_text user "K" (at 0 -1.8) (layer "F.Fab")
         (effects (font (size 1 1) (thickness 0.15)))
     )
-    (fp_line (start 1.34 0) (end 2.36 0)
+    (fp_line (start 1.04 0) (end 1.69 0)
       (stroke (width 0.12) (type solid)) (layer "F.SilkS"))
-    (fp_line (start 2.36 -1.47) (end 2.36 1.47)
+    (fp_line (start 1.69 -1.12) (end 1.69 1.12)
       (stroke (width 0.12) (type solid)) (layer "F.SilkS"))
-    (fp_line (start 2.36 1.47) (end 7.8 1.47)
+    (fp_line (start 1.69 1.12) (end 5.93 1.12)
       (stroke (width 0.12) (type solid)) (layer "F.SilkS"))
-    (fp_line (start 3.14 -1.47) (end 3.14 1.47)
+    (fp_line (start 2.29 -1.12) (end 2.29 1.12)
       (stroke (width 0.12) (type solid)) (layer "F.SilkS"))
-    (fp_line (start 3.26 -1.47) (end 3.26 1.47)
+    (fp_line (start 2.41 -1.12) (end 2.41 1.12)
       (stroke (width 0.12) (type solid)) (layer "F.SilkS"))
-    (fp_line (start 3.38 -1.47) (end 3.38 1.47)
+    (fp_line (start 2.53 -1.12) (end 2.53 1.12)
       (stroke (width 0.12) (type solid)) (layer "F.SilkS"))
-    (fp_line (start 7.8 -1.47) (end 2.36 -1.47)
+    (fp_line (start 5.93 -1.12) (end 1.69 -1.12)
       (stroke (width 0.12) (type solid)) (layer "F.SilkS"))
-    (fp_line (start 7.8 1.47) (end 7.8 -1.47)
+    (fp_line (start 5.93 1.12) (end 5.93 -1.12)
       (stroke (width 0.12) (type solid)) (layer "F.SilkS"))
-    (fp_line (start 8.82 0) (end 7.8 0)
+    (fp_line (start 6.58 0) (end 5.93 0)
       (stroke (width 0.12) (type solid)) (layer "F.SilkS"))
-    (fp_line (start -1.35 -1.6) (end -1.35 1.6)
+    (fp_line (start -1.05 -1.25) (end -1.05 1.25)
       (stroke (width 0.05) (type solid)) (layer "F.CrtYd"))
-    (fp_line (start -1.35 1.6) (end 11.51 1.6)
+    (fp_line (start -1.05 1.25) (end 8.67 1.25)
       (stroke (width 0.05) (type solid)) (layer "F.CrtYd"))
-    (fp_line (start 11.51 -1.6) (end -1.35 -1.6)
+    (fp_line (start 8.67 -1.25) (end -1.05 -1.25)
       (stroke (width 0.05) (type solid)) (layer "F.CrtYd"))
-    (fp_line (start 11.51 1.6) (end 11.51 -1.6)
+    (fp_line (start 8.67 1.25) (end 8.67 -1.25)
       (stroke (width 0.05) (type solid)) (layer "F.CrtYd"))
-    (fp_line (start 0 0) (end 2.48 0)
+    (fp_line (start 0 0) (end 1.81 0)
       (stroke (width 0.1) (type solid)) (layer "F.Fab"))
-    (fp_line (start 2.48 -1.35) (end 2.48 1.35)
+    (fp_line (start 1.81 -1) (end 1.81 1)
       (stroke (width 0.1) (type solid)) (layer "F.Fab"))
-    (fp_line (start 2.48 1.35) (end 7.68 1.35)
+    (fp_line (start 1.81 1) (end 5.81 1)
       (stroke (width 0.1) (type solid)) (layer "F.Fab"))
-    (fp_line (start 3.16 -1.35) (end 3.16 1.35)
+    (fp_line (start 2.31 -1) (end 2.31 1)
       (stroke (width 0.1) (type solid)) (layer "F.Fab"))
-    (fp_line (start 3.26 -1.35) (end 3.26 1.35)
+    (fp_line (start 2.41 -1) (end 2.41 1)
       (stroke (width 0.1) (type solid)) (layer "F.Fab"))
-    (fp_line (start 3.36 -1.35) (end 3.36 1.35)
+    (fp_line (start 2.51 -1) (end 2.51 1)
       (stroke (width 0.1) (type solid)) (layer "F.Fab"))
-    (fp_line (start 7.68 -1.35) (end 2.48 -1.35)
+    (fp_line (start 5.81 -1) (end 1.81 -1)
       (stroke (width 0.1) (type solid)) (layer "F.Fab"))
-    (fp_line (start 7.68 1.35) (end 7.68 -1.35)
+    (fp_line (start 5.81 1) (end 5.81 -1)
       (stroke (width 0.1) (type solid)) (layer "F.Fab"))
-    (fp_line (start 10.16 0) (end 7.68 0)
+    (fp_line (start 7.62 0) (end 5.81 0)
       (stroke (width 0.1) (type solid)) (layer "F.Fab"))
-    (pad "1" thru_hole rect (at 0 0 270) (size 2.2 2.2) (drill 1.1) (layers "*.Cu" "*.Mask")
+    (pad "1" thru_hole rect (at 0 0) (size 1.6 1.6) (drill 0.8) (layers "*.Cu" "*.Mask")
       (net 1 "+5V") (pinfunction "K") (pintype "passive"))
-    (pad "2" thru_hole oval (at 10.16 0 270) (size 2.2 2.2) (drill 1.1) (layers "*.Cu" "*.Mask")
+    (pad "2" thru_hole oval (at 7.62 0) (size 1.6 1.6) (drill 0.8) (layers "*.Cu" "*.Mask")
       (net 361 "Net-(D101-A)") (pinfunction "A") (pintype "passive"))
-    (model "${KICAD6_3DMODEL_DIR}/Diode_THT.3dshapes/D_DO-41_SOD81_P10.16mm_Horizontal.wrl"
+    (model "${KICAD6_3DMODEL_DIR}/Diode_THT.3dshapes/D_DO-35_SOD27_P7.62mm_Horizontal.wrl"
       (offset (xyz 0 0 0))
       (scale (xyz 1 1 1))
@@
         (effects (font (size 1 1) (thickness 0.15)))
     )
-    (fp_text user "${REFERENCE}" (at 3.81 0) (layer "F.Fab")
+    (fp_text user "${VALUE}" (at 3.81 0) (layer "F.SilkS")
         (effects (font (size 1 1) (thickness 0.15)))
     )
@@
         (effects (font (size 1 1) (thickness 0.15)))
     )
-    (fp_text user "${REFERENCE}" (at 3.81 0 90) (layer "F.Fab")
+    (fp_text user "${VALUE}" (at 3.81 0 90) (layer "F.SilkS")
         (effects (font (size 1 1) (thickness 0.15)))
     )
@@
         (effects (font (size 1 1) (thickness 0.15)))
     )
-    (fp_text user "${REFERENCE}" (at 3.81 0) (layer "F.Fab")
+    (fp_text user "${VALUE}" (at 3.81 0) (layer "F.SilkS")
         (effects (font (size 1 1) (thickness 0.15)))
     )
