File: design-files/pg09-system-rom.kicad_sch (KiCad schematic)
At the start: 6 parts, among them U501 W65C21, U502 AT28C64, U503 SST39SF040

Commit message: Assign a bunch of footprints.
Parts:
- C201, C202, C203: footprint (none) -> Capacitor_THT:C_Disc_D6.0mm_W4.4mm_P5.00mm
- U501: footprint Package_DIP:DIP-40_W15.24mm -> Package_DIP:DIP-40_W15.24mm_Socket
- U502: footprint (none) -> Package_DIP:DIP-28_W15.24mm_Socket
- U503: footprint (none) -> Package_DIP:DIP-32_W15.24mm_Socket
Changed lines of the file:
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@@
       (effects (font (size 1.27 1.27)) (justify left))
     )
-    (property "Footprint" "" (at 198.12 147.32 0)
+    (property "Footprint" "Capacitor_THT:C_Disc_D6.0mm_W4.4mm_P5.00mm" (at 198.12 147.32 0)
       (effects (font (size 1.27 1.27)) hide)
     )
@@
       (effects (font (size 1.27 1.27)) (justify left))
     )
-    (property "Footprint" "Package_DIP:DIP-40_W15.24mm" (at 87.63 151.13 0)
+    (property "Footprint" "Package_DIP:DIP-40_W15.24mm_Socket" (at 87.63 151.13 0)
       (effects (font (size 1.27 1.27)) hide)
     )
@@
       (effects (font (size 1.27 1.27)) (justify left))
     )
-    (property "Footprint" "" (at 218.44 147.32 0)
+    (property "Footprint" "Capacitor_THT:C_Disc_D6.0mm_W4.4mm_P5.00mm" (at 218.44 147.32 0)
       (effects (font (size 1.27 1.27)) hide)
     )
@@
       (effects (font (size 1.27 1.27)) (justify left))
     )
-    (property "Footprint" "" (at 208.28 147.32 0)
+    (property "Footprint" "Capacitor_THT:C_Disc_D6.0mm_W4.4mm_P5.00mm" (at 208.28 147.32 0)
       (effects (font (size 1.27 1.27)) hide)
     )
@@
       (effects (font (size 1.27 1.27)) (justify left))
     )
-    (property "Footprint" "" (at 151.13 22.86 0)
+    (property "Footprint" "Package_DIP:DIP-28_W15.24mm_Socket" (at 151.13 22.86 0)
       (effects (font (size 1.27 1.27)) hide)
     )
@@
       (effects (font (size 1.27 1.27)) (justify left))
     )
-    (property "Footprint" "" (at 151.13 111.76 0)
-      (effects (font (size 1.27 1.27)) hide)
-    )
+    (property "Footprint" "Package_DIP:DIP-32_W15.24mm_Socket" (at 151.13 111.76 0)
+      (effects (font (size 1.27 1.27)) hide)
+    )

Commit message: Fix various errors and omissions discovered while working on the first cut of the PCB layout.
Parts:
- U502: footprint Package_DIP:DIP-28_W15.24mm_Socket -> Socket:DIP_Socket-28_W6.9_W7.62_W10.16_W12.7_W13.5_3M_228-4817-00-0602J
Changed lines of the file:
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@@
       (effects (font (size 1.27 1.27)) (justify left))
     )
-    (property "Footprint" "Package_DIP:DIP-28_W15.24mm_Socket" (at 151.13 22.86 0)
+    (property "Footprint" "Socket:DIP_Socket-28_W6.9_W7.62_W10.16_W12.7_W13.5_3M_228-4817-00-0602J" (at 151.13 22.86 0)
       (effects (font (size 1.27 1.27)) hide)
     )

Commit message: Specify a physically smaller bypass cap.
Parts:
- C201, C202, C203: footprint Capacitor_THT:C_Disc_D6.0mm_W4.4mm_P5.00mm -> Capacitor_THT:C_Disc_D3.8mm_W2.6mm_P2.50mm
Changed lines of the file:
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@@
       (effects (font (size 1.27 1.27)) (justify left))
     )
-    (property "Footprint" "Capacitor_THT:C_Disc_D6.0mm_W4.4mm_P5.00mm" (at 198.12 147.32 0)
+    (property "Footprint" "Capacitor_THT:C_Disc_D3.8mm_W2.6mm_P2.50mm" (at 198.12 147.32 0)
       (effects (font (size 1.27 1.27)) hide)
     )
@@
       (effects (font (size 1.27 1.27)) (justify left))
     )
-    (property "Footprint" "Capacitor_THT:C_Disc_D6.0mm_W4.4mm_P5.00mm" (at 218.44 147.32 0)
+    (property "Footprint" "Capacitor_THT:C_Disc_D3.8mm_W2.6mm_P2.50mm" (at 218.44 147.32 0)
       (effects (font (size 1.27 1.27)) hide)
     )
@@
       (effects (font (size 1.27 1.27)) (justify left))
     )
-    (property "Footprint" "Capacitor_THT:C_Disc_D6.0mm_W4.4mm_P5.00mm" (at 208.28 147.32 0)
+    (property "Footprint" "Capacitor_THT:C_Disc_D3.8mm_W2.6mm_P2.50mm" (at 208.28 147.32 0)
       (effects (font (size 1.27 1.27)) hide)
     )
