File: design-files/pg09-system-rom.kicad_sch (KiCad schematic)
At the start: 6 parts, among them U501 W65C21, U502 AT28C64, U503 SST39SF040

Commit message: Correct footprint for fixed ROM ZIF socket.
Parts:
- U502: footprint Socket:DIP_Socket-28_W6.9_W7.62_W10.16_W12.7_W13.5_3M_228-4817-00-0602J -> Socket:DIP_Socket-28_W11.9_W12.7_W15.24_W17.78_W18.5_3M_228-1277-00-0602J
Changed lines of the file:
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@@
       (effects (font (size 1.27 1.27)) (justify left))
     )
-    (property "Footprint" "Socket:DIP_Socket-28_W6.9_W7.62_W10.16_W12.7_W13.5_3M_228-4817-00-0602J" (at 151.13 22.86 0)
+    (property "Footprint" "Socket:DIP_Socket-28_W11.9_W12.7_W15.24_W17.78_W18.5_3M_228-1277-00-0602J" (at 151.13 22.86 0)
       (effects (font (size 1.27 1.27)) hide)
     )

Commit message: A ZIF socket also for the banked ROM.
Parts:
- U503: footprint Package_DIP:DIP-32_W15.24mm_Socket -> Socket:DIP_Socket-32_W11.9_W12.7_W15.24_W17.78_W18.5_3M_232-1285-00-0602J
Changed lines of the file:
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@@
       (effects (font (size 1.27 1.27)) (justify left))
     )
-    (property "Footprint" "Package_DIP:DIP-32_W15.24mm_Socket" (at 151.13 111.76 0)
+    (property "Footprint" "Socket:DIP_Socket-32_W11.9_W12.7_W15.24_W17.78_W18.5_3M_232-1285-00-0602J" (at 151.13 111.76 0)
       (effects (font (size 1.27 1.27)) hide)
     )

Commit message: Disconnect the PSU controller from the ROM banker PIA and instead give it its own register (offset $11) in IO0SEL.  Use a '138 to decode the address and generate the write strobe for it.
Connections:
- net PSU_CTRL_D0: no longer names the net of U501.10 (PB0)
- net PSU_CTRL_D1: no longer names the net of U501.11 (PB1)
- net ~{PSU_CTRL_WR}: no longer names the net of U501.19 (CB2)
- no-connect marks 12 -> 15
Changed lines of the file:
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@@
   (junction (at 129.54 101.6) (diameter 0) (color 0 0 0 0)
   )
+  (no_connect (at 102.87 172.72))
   (no_connect (at 102.87 137.16))
   (no_connect (at 102.87 157.48))
@@
   (no_connect (at 102.87 160.02))
   (no_connect (at 77.47 180.34))
+  (no_connect (at 102.87 152.4))
   (no_connect (at 102.87 162.56))
   (no_connect (at 102.87 170.18))
   (no_connect (at 102.87 142.24))
-  (wire (pts (xy 102.87 152.4) (xy 118.11 152.4))
-    (stroke (width 0) (type default))
-  )
+  (no_connect (at 102.87 149.86))
   (wire (pts (xy 102.87 129.54) (xy 135.89 129.54))
     (stroke (width 0) (type default))
@@
   )
   (wire (pts (xy 208.28 149.86) (xy 218.44 149.86))
-    (stroke (width 0) (type default))
-  )
-  (wire (pts (xy 102.87 172.72) (xy 118.11 172.72))
     (stroke (width 0) (type default))
   )
@@
     )
   )
-  (global_label "PSU_CTRL_D0" (shape output) (at 102.87 149.86 0) (fields_autoplaced)
-    (effects (font (size 1.27 1.27)) (justify left))
-    (property "Intersheetrefs" "${INTERSHEET_REFS}" (at 118.5362 149.86 0)
-      (effects (font (size 1.27 1.27)) (justify left) hide)
-    )
-  )
   (global_label "R{slash}~{W}" (shape input) (at 77.47 160.02 180) (fields_autoplaced)
     (effects (font (size 1.27 1.27)) (justify right))
@@
     )
   )
-  (global_label "~{PSU_CTRL_WR}" (shape output) (at 118.11 172.72 0) (fields_autoplaced)
-    (effects (font (size 1.27 1.27)) (justify left))
-    (property "Intersheetrefs" "${INTERSHEET_REFS}" (at 134.0181 172.72 0)
-      (effects (font (size 1.27 1.27)) (justify left) hide)
-    )
-  )
   (global_label "E" (shape input) (at 68.58 147.32 180) (fields_autoplaced)
     (effects (font (size 1.27 1.27)) (justify right))
@@
     )
   )
-  (global_label "PSU_CTRL_D1" (shape output) (at 118.11 152.4 0) (fields_autoplaced)
-    (effects (font (size 1.27 1.27)) (justify left))
-    (property "Intersheetrefs" "${INTERSHEET_REFS}" (at 133.7762 152.4 0)
-      (effects (font (size 1.27 1.27)) (justify left) hide)
-    )
-  )

Commit message: Move the ROM banker to the Address Decoder sheet and change its designation to U303.
Parts:
- removed C203: 0.1µF, Capacitor_THT:C_Disc_D3.8mm_W2.6mm_P2.50mm, symbol Device:C_Small
- removed U501: W65C21, Package_DIP:DIP-40_W15.24mm_Socket, symbol jrt-ICs:W65C21
Connections:
- net RB0: now reaches U503.28 (A13)
- net RB1: now reaches U503.29 (A14)
- net RB2: now reaches U503.3 (A15)
- net RB3: now reaches U503.2 (A16)
- net RB4: now reaches U503.30 (A17)
- net RB5: now reaches U503.1 (A18)
- no-connect marks 15 -> 0

Commit message: Fix up the banker capacitors.
Parts:
- renumbered U502 to U501, U503 to U502
Changed lines of the file:
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@@
   (symbol (lib_id "jrt-ICs:AT28C64") (at 151.13 49.53 0) (unit 1)
     (in_bom yes) (on_board yes) (dnp no) (fields_autoplaced)
-    (property "Reference" "U502" (at 153.0859 24.13 0)
+    (property "Reference" "U501" (at 153.0859 24.13 0)
       (effects (font (size 1.27 1.27)) (justify left))
     )
@@
       (project "pg09-system"
         (path "/44572023-3621-4b3a-bd53-c3b2b3f42871/29ccfefd-4ecb-4886-be07-d9fca15abc34"
-          (reference "U502") (unit 1)
+          (reference "U501") (unit 1)
         )
       )
@@
   (symbol (lib_id "Memory_Flash:SST39SF040") (at 151.13 119.38 0) (unit 1)
     (in_bom yes) (on_board yes) (dnp no) (fields_autoplaced)
-    (property "Reference" "U503" (at 153.0859 83.82 0)
+    (property "Reference" "U502" (at 153.0859 83.82 0)
       (effects (font (size 1.27 1.27)) (justify left))
     )
@@
       (project "pg09-system"
         (path "/44572023-3621-4b3a-bd53-c3b2b3f42871/29ccfefd-4ecb-4886-be07-d9fca15abc34"
-          (reference "U503") (unit 1)
+          (reference "U502") (unit 1)
         )
       )

Commit message: Eliminate the AT28C64 EEPROM, and instead use a MUX to force bank 0 of the flash ROM when the fixed ROM region is selected.  Bank 0 is now the fixed ROM image always, and will now be accessible in the banked ROM region if bank 0 is selected.
Parts:
- removed U501: AT28C64, Socket:DIP_Socket-28_W11.9_W12.7_W15.24_W17.78_W18.5_3M_228-1277-00-0602J, symbol jrt-ICs:AT28C64
- added C202: 0.1µF, Capacitor_THT:C_Disc_D3.8mm_W2.6mm_P2.50mm, symbol Device:C_Small
- added U502, U503: 74AHC157, Package_DIP:DIP-16_W7.62mm_Socket, symbol 74xx:74LS157
- renumbered U502 to U501
Connections:
- net +5V: now also C202.1, U502.16 (VCC), U503.16 (VCC)
- net GND: now also C202.2, U502.10 (I1c), U502.13 (I1d), U502.15 (E), U502.3 (I1a), U502.6 (I1b), U502.8 (GND), U503.10 (I1c), U503.11 (I0c), U503.13 (I1d), U503.14 (I0d), U503.15 (E), U503.3 (I1a), U503.6 (I1b), U503.8 (GND)
- net RB0: now also U502.2 (I0a); no longer U501.28 (A13)
- net RB1: now also U502.5 (I0b); no longer U501.29 (A14)
- net RB2: now also U502.11 (I0c); no longer U501.3 (A15)
- net RB3: now also U502.14 (I0d); no longer U501.2 (A16)
- net RB4: now also U503.2 (I0a); no longer U501.30 (A17)
- net RB5: now also U503.5 (I0b); no longer U501.1 (A18)
- net ~{BROMSEL}: now also U502.1 (S), U503.1 (S); no longer U501.22 (CE)
- net ~{FROMSEL}: now also U501.22 (CE)
- new net: U501.30 (A17), U503.4 (Za)
- new net: U501.1 (A18), U503.7 (Zb)
- new net: U501.2 (A16), U502.12 (Zd)
- new net: U501.28 (A13), U502.4 (Za)
- new net: U501.29 (A14), U502.7 (Zb)
- new net: U501.3 (A15), U502.9 (Zc)
- no-connect marks 0 -> 2
Other:
- note added: "When ~{BROMSEL} is not asserted, the bank is forced to 0. When ~{BROMSEL} is asserted, the bank is selected from the ROM bank register."
- note removed: "Fixed ROM"
- moved on the sheet: C201, C202, U501
