File: design-files/pg09-system-addr-decode.kicad_sch (KiCad schematic)
At the start: 13 parts, among them U301 GAL22V10, U302 GAL22V10, U303 GAL22V10, U304 GAL22V10

Commit message: Minor tweaks.
Connections:
- net ~{BROMSEL}: now also RN401.6 (R5); no longer RN401.2 (R1)
- net ~{FIRQ}: now also RN401.4 (R3); no longer RN401.8 (R7)
- net ~{FRAMSEL}: now also RN401.8 (R7); no longer RN401.4 (R3)
- net ~{FROMSEL}: now also RN401.7 (R6); no longer RN401.3 (R2)
- net ~{HALT}: now also RN401.5 (R4); no longer RN401.9 (R8)
- net ~{HBRAMSEL}: now also RN401.9 (R8); no longer RN401.5 (R4)
- net ~{IRQ}: now also RN401.3 (R2); no longer RN401.7 (R6)
- net ~{NMI}: now also RN401.2 (R1); no longer RN401.6 (R5)
Changed lines of the file:
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@@
     (stroke (width 0) (type default))
   )
-  (wire (pts (xy 224.79 151.13) (xy 234.95 151.13))
+  (wire (pts (xy 223.52 151.13) (xy 234.95 151.13))
     (stroke (width 0) (type default))
   )
@@
     (stroke (width 0) (type default))
   )
-  (wire (pts (xy 224.79 146.05) (xy 234.95 146.05))
+  (wire (pts (xy 223.52 146.05) (xy 234.95 146.05))
     (stroke (width 0) (type default))
   )
@@
     )
   )
-  (global_label "~{HALT}" (shape input) (at 224.79 151.13 180) (fields_autoplaced)
-    (effects (font (size 1.27 1.27)) (justify right))
-    (property "Intersheetrefs" "${INTERSHEET_REFS}" (at 217.4694 151.13 0)
+  (global_label "~{HALT}" (shape input) (at 223.52 140.97 180) (fields_autoplaced)
+    (effects (font (size 1.27 1.27)) (justify right))
+    (property "Intersheetrefs" "${INTERSHEET_REFS}" (at 216.1994 140.97 0)
       (effects (font (size 1.27 1.27)) (justify right) hide)
     )
@@
     )
   )
-  (global_label "~{BROMSEL}" (shape input) (at 234.95 133.35 180) (fields_autoplaced)
-    (effects (font (size 1.27 1.27)) (justify right))
-    (property "Intersheetrefs" "${INTERSHEET_REFS}" (at 223.3357 133.35 0)
+  (global_label "~{BROMSEL}" (shape input) (at 234.95 143.51 180) (fields_autoplaced)
+    (effects (font (size 1.27 1.27)) (justify right))
+    (property "Intersheetrefs" "${INTERSHEET_REFS}" (at 223.3357 143.51 0)
       (effects (font (size 1.27 1.27)) (justify right) hide)
     )
@@
     )
   )
-  (global_label "~{FROMSEL}" (shape input) (at 223.52 135.89 180) (fields_autoplaced)
-    (effects (font (size 1.27 1.27)) (justify right))
-    (property "Intersheetrefs" "${INTERSHEET_REFS}" (at 212.0871 135.89 0)
+  (global_label "~{FROMSEL}" (shape input) (at 223.52 146.05 180) (fields_autoplaced)
+    (effects (font (size 1.27 1.27)) (justify right))
+    (property "Intersheetrefs" "${INTERSHEET_REFS}" (at 212.0871 146.05 0)
       (effects (font (size 1.27 1.27)) (justify right) hide)
     )
@@
     )
   )
-  (global_label "~{FRAMSEL}" (shape input) (at 234.95 138.43 180) (fields_autoplaced)
-    (effects (font (size 1.27 1.27)) (justify right))
-    (property "Intersheetrefs" "${INTERSHEET_REFS}" (at 223.759 138.43 0)
+  (global_label "~{FRAMSEL}" (shape input) (at 234.95 148.59 180) (fields_autoplaced)
+    (effects (font (size 1.27 1.27)) (justify right))
+    (property "Intersheetrefs" "${INTERSHEET_REFS}" (at 223.759 148.59 0)
       (effects (font (size 1.27 1.27)) (justify right) hide)
     )
@@
     )
   )
-  (global_label "~{FIRQ}" (shape input) (at 234.95 148.59 180) (fields_autoplaced)
-    (effects (font (size 1.27 1.27)) (justify right))
-    (property "Intersheetrefs" "${INTERSHEET_REFS}" (at 227.7503 148.59 0)
+  (global_label "~{FIRQ}" (shape input) (at 234.95 138.43 180) (fields_autoplaced)
+    (effects (font (size 1.27 1.27)) (justify right))
+    (property "Intersheetrefs" "${INTERSHEET_REFS}" (at 227.7503 138.43 0)
       (effects (font (size 1.27 1.27)) (justify right) hide)
     )
@@
     )
   )
-  (global_label "~{IRQ}" (shape input) (at 224.79 146.05 180) (fields_autoplaced)
-    (effects (font (size 1.27 1.27)) (justify right))
-    (property "Intersheetrefs" "${INTERSHEET_REFS}" (at 218.6789 146.05 0)
+  (global_label "~{IRQ}" (shape input) (at 223.52 135.89 180) (fields_autoplaced)
+    (effects (font (size 1.27 1.27)) (justify right))
+    (property "Intersheetrefs" "${INTERSHEET_REFS}" (at 217.4089 135.89 0)
       (effects (font (size 1.27 1.27)) (justify right) hide)
     )
@@
     )
   )
-  (global_label "~{HBRAMSEL}" (shape input) (at 223.52 140.97 180) (fields_autoplaced)
-    (effects (font (size 1.27 1.27)) (justify right))
-    (property "Intersheetrefs" "${INTERSHEET_REFS}" (at 210.8171 140.97 0)
+  (global_label "~{HBRAMSEL}" (shape input) (at 223.52 151.13 180) (fields_autoplaced)
+    (effects (font (size 1.27 1.27)) (justify right))
+    (property "Intersheetrefs" "${INTERSHEET_REFS}" (at 210.8171 151.13 0)
       (effects (font (size 1.27 1.27)) (justify right) hide)
     )
@@
     )
   )
-  (global_label "~{NMI}" (shape input) (at 234.95 143.51 180) (fields_autoplaced)
-    (effects (font (size 1.27 1.27)) (justify right))
-    (property "Intersheetrefs" "${INTERSHEET_REFS}" (at 228.6575 143.51 0)
-      (effects (font (size 1.27 1.27)) (justify right) hide)
-    )
+  (global_label "~{NMI}" (shape input) (at 234.95 133.35 180) (fields_autoplaced)
+    (effects (font (size 1.27 1.27)) (justify right))
+    (property "Intersheetrefs" "${INTERSHEET_REFS}" (at 228.6575 133.35 0)
+      (effects (font (size 1.27 1.27)) (justify right) hide)
+    )
