File: design-files/pg09-system-addr-decode.kicad_sch (KiCad schematic)
At the start: 13 parts, among them U301 GAL22V10, U302 GAL22V10, U303 GAL22V10, U304 GAL22V10

Commit message: Remove ADDRDEC2 and ADDRDEC3.
Parts:
- removed C203 (x2): 0.1µF, Capacitor_THT:C_Disc_D3.8mm_W2.6mm_P2.50mm, symbol Device:C_Small
- removed RN401 (x2): 10K, Resistor_THT:R_Array_SIP9, symbol Device:R_Network08
- removed U303, U304: GAL22V10, Package_DIP:DIP-24_W7.62mm_Socket, symbol jrt-ICs:GAL22V10
Connections:
- no-connect marks 8 -> 2
Other:
- note removed: "addr_decode2.chp"
- note removed: "addr_decode3.chp"
- moved on the sheet: RN401, U301, U302

Commit message: Checkpoint in PCB layout.  Big change here is that address decoder gets A* inputs, not dA* inputs, because that's needed for the auto- vectoring interrupt controller.
Connections:
- net dA10 renamed A10
- net dA11 renamed A11
- net dA12 renamed A12
- net dA13 renamed A13
- net dA14 renamed A14
- net dA15 renamed A15
- net dA5 renamed A5
- net dA6 renamed A6
- net dA7 renamed A7
- net dA8 renamed A8
- net dA9 renamed A9

Commit message: Checkpoint with new layout.
Connections:
- net ~{HALT} is gone; now on net ~{IRQ}: RN401.5 (R4)
- net ~{IRQ}: no longer RN401.3 (R2)
- net ~{FIRQ}: no longer names the net of RN401.4 (R3)
- net ~{NMI}: no longer names the net of RN401.2 (R1)
- no-connect marks 2 -> 5
Changed lines of the file:
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@@
   (junction (at 245.11 81.28) (diameter 0) (color 0 0 0 0)
   )
+  (no_connect (at 234.95 113.03))
+  (no_connect (at 234.95 110.49))
   (no_connect (at 114.3 72.39))
+  (no_connect (at 234.95 107.95))
   (no_connect (at 114.3 149.86))
   (wire (pts (xy 139.7 137.16) (xy 151.13 137.16))
@@
     (stroke (width 0) (type default))
   )
-  (wire (pts (xy 223.52 110.49) (xy 234.95 110.49))
-    (stroke (width 0) (type default))
-  )
   (wire (pts (xy 106.68 124.46) (xy 114.3 124.46))
     (stroke (width 0) (type default))
@@
     )
   )
-  (global_label "~{HALT}" (shape input) (at 223.52 115.57 180) (fields_autoplaced)
-    (effects (font (size 1.27 1.27)) (justify right))
-    (property "Intersheetrefs" "${INTERSHEET_REFS}" (at 216.1994 115.57 0)
-      (effects (font (size 1.27 1.27)) (justify right) hide)
-    )
-  )
   (global_label "~{IO12SEL}" (shape output) (at 151.13 137.16 0) (fields_autoplaced)
     (effects (font (size 1.27 1.27)) (justify left))
@@
     )
   )
-  (global_label "~{FIRQ}" (shape input) (at 234.95 113.03 180) (fields_autoplaced)
-    (effects (font (size 1.27 1.27)) (justify right))
-    (property "Intersheetrefs" "${INTERSHEET_REFS}" (at 227.7503 113.03 0)
-      (effects (font (size 1.27 1.27)) (justify right) hide)
-    )
-  )
-  (global_label "~{IRQ}" (shape input) (at 223.52 110.49 180) (fields_autoplaced)
-    (effects (font (size 1.27 1.27)) (justify right))
-    (property "Intersheetrefs" "${INTERSHEET_REFS}" (at 217.4089 110.49 0)
+  (global_label "~{IRQ}" (shape input) (at 223.52 115.57 180) (fields_autoplaced)
+    (effects (font (size 1.27 1.27)) (justify right))
+    (property "Intersheetrefs" "${INTERSHEET_REFS}" (at 217.4089 115.57 0)
       (effects (font (size 1.27 1.27)) (justify right) hide)
     )
@@
       (effects (font (size 1.27 1.27)) (justify right) hide)
     )
-  )
-  (global_label "~{NMI}" (shape input) (at 234.95 107.95 180) (fields_autoplaced)
-    (effects (font (size 1.27 1.27)) (justify right))
-    (property "Intersheetrefs" "${INTERSHEET_REFS}" (at 228.6575 107.95 0)
-      (effects (font (size 1.27 1.27)) (justify right) hide)
-    )

Commit message: Move the ROM banker to the Address Decoder sheet and change its designation to U303.
Parts:
- added C203: 0.1µF, Capacitor_THT:C_Disc_D3.8mm_W2.6mm_P2.50mm, symbol Device:C_Small
- added U501: W65C21, Package_DIP:DIP-40_W15.24mm_Socket, symbol jrt-ICs:W65C21
Connections:
- net +5V: now also C203.1, U501.20 (VDD)
- net GND: now also C203.2, U501.1 (VSS)
- net ~{IO0SEL}: now also U501.23 (~{CS2})
- new net A0: U501.36 (RS0)
- new net A1: U501.35 (RS1)
- new net D0: U501.33 (D0)
- new net D1: U501.32 (D1)
- new net D2: U501.31 (D2)
- new net D3: U501.30 (D3)
- new net D4: U501.29 (D4)
- new net D5: U501.28 (D5)
- new net D6: U501.27 (D6)
- new net D7: U501.26 (D7)
- new net E: U501.25 (PHI2)
- new net FLASHWREN: U501.9 (PA7)
- new net RB0: U501.2 (PA0)
- new net RB1: U501.3 (PA1)
- new net RB2: U501.4 (PA2)
- new net RB3: U501.5 (PA3)
- new net RB4: U501.6 (PA4)
- new net RB5: U501.7 (PA5)
- new net R/~{W}: U501.21 (R/~{W})
- new net nA2: U501.22 (CS0)
- new net nA3: U501.24 (CS1)
- new net ~{RESET}: U501.34 (~{RESET})
- no-connect marks 5 -> 20
Other:
- moved on the sheet: C201, C202, RN401, U301, U302

Commit message: Move the RAM banker PIA to the decoder sheet and re-designate U304.
Parts:
- added C203: 0.1µF, Capacitor_THT:C_Disc_D3.8mm_W2.6mm_P2.50mm, symbol Device:C_Small
- added U501: W65C21, Package_DIP:DIP-40_W15.24mm_Socket, symbol jrt-ICs:W65C21
Connections:
- net +5V: now also C203.1, U501.20 (VDD)
- net A0: now also U501.36 (RS0)
- net A1: now also U501.35 (RS1)
- net D0: now also U501.33 (D0)
- net D1: now also U501.32 (D1)
- net D2: now also U501.31 (D2)
- net D3: now also U501.30 (D3)
- net D4: now also U501.29 (D4)
- net D5: now also U501.28 (D5)
- net D6: now also U501.27 (D6)
- net D7: now also U501.26 (D7)
- net E: now also U501.25 (PHI2)
- net GND: now also C203.2, U501.1 (VSS)
- net R/~{W}: now also U501.21 (R/~{W})
- net nA3: now also U501.24 (CS1)
- net ~{IO0SEL}: now also U501.23 (~{CS2})
- net ~{RESET}: now also U501.34 (~{RESET})
- new net A2: U501.22 (CS0)
- new net HRB0: U501.10 (PB0)
- new net HRB1: U501.11 (PB1)
- new net HRB2: U501.12 (PB2)
- new net HRB3: U501.13 (PB3)
- new net HRB4: U501.14 (PB4)
- new net HRB5: U501.15 (PB5)
- new net HRB6: U501.16 (PB6)
- new net HRB7: U501.17 (PB7)
- new net LRB0: U501.2 (PA0)
- new net LRB1: U501.3 (PA1)
- new net LRB2: U501.4 (PA2)
- new net LRB3: U501.5 (PA3)
- no-connect marks 20 -> 30

Commit message: New banked RAM layout: - The 2MB RAM group is now Low Banked RAM, and divided into 2   16K independently bankable regions back by 1MB each. - The 512KB RAM is now High Banked RAM. - Shuffle the Low and High banker PIAs.
Connections:
- net A2: now also U501.22 (CS0); no longer U501.22 (CS0)
- net FLASHWREN: now also U501.17 (PB7); no longer U501.9 (PA7)
- net HRB0: now also U501.2 (PA0); no longer U501.10 (PB0)
- net HRB1: now also U501.3 (PA1); no longer U501.11 (PB1)
- net HRB2: now also U501.4 (PA2); no longer U501.12 (PB2)
- net HRB3: now also U501.5 (PA3); no longer U501.13 (PB3)
- net HRB4: now also U501.6 (PA4); no longer U501.14 (PB4)
- net HRB5: now also U501.7 (PA5); no longer U501.15 (PB5)
- net RB0: now also U501.10 (PB0); no longer U501.2 (PA0)
- net RB1: now also U501.11 (PB1); no longer U501.3 (PA1)
- net RB2: now also U501.12 (PB2); no longer U501.4 (PA2)
- net RB3: now also U501.13 (PB3); no longer U501.5 (PA3)
- net RB4: now also U501.14 (PB4); no longer U501.6 (PA4)
- net RB5: now also U501.15 (PB5); no longer U501.7 (PA5)
- net nA2: now also U501.22 (CS0); no longer U501.22 (CS0)
- net LR0B4: now reaches U501.6 (PA4)
- net LR0B5: now reaches U501.7 (PA5)
- net HRB6: no longer names the net of U501.16 (PB6)
- net HRB7: no longer names the net of U501.17 (PB7)
- net LRB0 renamed LR0B0
- net LRB1 renamed LR0B1
- net LRB2 renamed LR0B2
- net LRB3 renamed LR0B3
- new net LR1B0: U501.10 (PB0)
- new net LR1B1: U501.11 (PB1)
- new net LR1B2: U501.12 (PB2)
- new net LR1B3: U501.13 (PB3)
- new net LR1B4: U501.14 (PB4)
- new net LR1B5: U501.15 (PB5)
- no-connect marks 30 -> 24
Other:
- note added: "High Memory Banker"
- note added: "Low Memory Banker"

Commit message: Add another high banked SRAM, for a total of 128 banks.
Connections:
- net HRB6: now reaches U501.8 (PA6)
- no-connect marks 24 -> 23
Changed lines of the file:
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@@
   (no_connect (at 34.544 61.976))
   (no_connect (at 108.712 99.06))
-  (no_connect (at 180.848 108.966))
   (no_connect (at 180.848 116.586))
   (no_connect (at 180.848 144.526))
@@
     )
   )
+  (global_label "HRB6" (shape output) (at 180.848 108.966 0) (fields_autoplaced)
+    (effects (font (size 1.27 1.27)) (justify left))
+    (property "Intersheetrefs" "${INTERSHEET_REFS}" (at 188.8338 108.966 0)
+      (effects (font (size 1.27 1.27)) (justify left) hide)
+    )
+  )
