File: design-files/pg09-system-addr-decode.kicad_sch (KiCad schematic)
At the start: 11 parts, among them U301 GAL22V10, U302 GAL22V10, U501 W65C21

Commit message: Add pull-down resistors to all bank selection signals to ensure that they won't be floating before the PIAs are initialized.
Parts:
- added R101: 10K, Resistor_THT:R_Axial_DIN0207_L6.3mm_D2.5mm_P7.62mm_Horizontal, symbol Device:R_Small
- added RN401 (x3): 10K, Resistor_THT:R_Array_SIP9, symbol Device:R_Network08
Connections:
- net GND: now also R101.2, RN401.1 (common), RN401.1 (common), RN401.1 (common)
- net HRB0: now also RN401.6 (R5)
- net HRB1: now also RN401.7 (R6)
- net HRB2: now also RN401.8 (R7)
- net HRB3: now also RN401.9 (R8)
- net HRB4: now also RN401.2 (R1)
- net HRB5: now also RN401.3 (R2)
- net HRB6: now also R101.1
- net LR0B0: now also RN401.2 (R1)
- net LR0B1: now also RN401.3 (R2)
- net LR0B2: now also RN401.4 (R3)
- net LR0B3: now also RN401.5 (R4)
- net LR0B4: now also RN401.6 (R5)
- net LR0B5: now also RN401.7 (R6)
- net LR1B0: now also RN401.8 (R7)
- net LR1B1: now also RN401.9 (R8)
- net LR1B2: now also RN401.2 (R1)
- net LR1B3: now also RN401.3 (R2)
- net LR1B4: now also RN401.4 (R3)
- net LR1B5: now also RN401.5 (R4)
- net RB0: now also RN401.4 (R3)
- net RB1: now also RN401.5 (R4)
- net RB2: now also RN401.6 (R5)
- net RB3: now also RN401.7 (R6)
- net RB4: now also RN401.8 (R7)
- net RB5: now also RN401.9 (R8)

Commit message: Overhaul how the "system registers" in IO0SEL work, paving the way to use a VIA for the interrupt enables (because that would also give us a timer).
Connections:
- net A2: now also U501.24 (CS1); no longer U501.22 (CS0)
- net nA2: now also U501.24 (CS1); no longer U501.22 (CS0)
- removed net nA3: U501.24 (CS1), U501.24 (CS1)
- new net nA3nA4: U501.22 (CS0), U501.22 (CS0)
Changed lines of the file:
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@@
     )
   )
-  (global_label "nA2" (shape input) (at 183.388 54.864 180) (fields_autoplaced)
-    (effects (font (size 1.27 1.27)) (justify right))
-    (property "Intersheetrefs" "${INTERSHEET_REFS}" (at 177.0351 54.864 0)
+  (global_label "nA3nA4" (shape input) (at 183.388 54.864 180) (fields_autoplaced)
+    (effects (font (size 1.27 1.27)) (justify right))
+    (property "Intersheetrefs" "${INTERSHEET_REFS}" (at 173.588 54.864 0)
       (effects (font (size 1.27 1.27)) (justify right) hide)
     )
@@
     )
   )
-  (global_label "nA3" (shape input) (at 192.278 57.404 180) (fields_autoplaced)
+  (global_label "nA2" (shape input) (at 192.278 57.404 180) (fields_autoplaced)
     (effects (font (size 1.27 1.27)) (justify right))
     (property "Intersheetrefs" "${INTERSHEET_REFS}" (at 185.9251 57.404 0)
@@
     )
   )
+  (global_label "nA3nA4" (shape input) (at 146.558 124.206 180) (fields_autoplaced)
+    (effects (font (size 1.27 1.27)) (justify right))
+    (property "Intersheetrefs" "${INTERSHEET_REFS}" (at 136.758 124.206 0)
+      (effects (font (size 1.27 1.27)) (justify right) hide)
+    )
+  )
   (global_label "LR1B4" (shape input) (at 259.588 89.789 180) (fields_autoplaced)
     (effects (font (size 1.27 1.27)) (justify right))
@@
     )
   )
-  (global_label "A2" (shape input) (at 146.558 124.206 180) (fields_autoplaced)
-    (effects (font (size 1.27 1.27)) (justify right))
-    (property "Intersheetrefs" "${INTERSHEET_REFS}" (at 141.3541 124.206 0)
-      (effects (font (size 1.27 1.27)) (justify right) hide)
-    )
-  )
   (global_label "~{IO6SEL}" (shape output) (at 71.374 54.356 0) (fields_autoplaced)
     (effects (font (size 1.27 1.27)) (justify left))
@@
     )
   )
-  (global_label "nA3" (shape input) (at 155.448 126.746 180) (fields_autoplaced)
-    (effects (font (size 1.27 1.27)) (justify right))
-    (property "Intersheetrefs" "${INTERSHEET_REFS}" (at 149.0951 126.746 0)
-      (effects (font (size 1.27 1.27)) (justify right) hide)
-    )
+  (global_label "A2" (shape input) (at 155.448 126.746 180) (fields_autoplaced)
+    (effects (font (size 1.27 1.27)) (justify right))
+    (property "Intersheetrefs" "${INTERSHEET_REFS}" (at 150.2441 126.746 0)
+      (effects (font (size 1.27 1.27)) (justify right) hide)
+    )

Commit message: Move the misc system register decoder to the address decoder sheet.
Parts:
- added C203: 0.1µF, Capacitor_THT:C_Disc_D3.8mm_W2.6mm_P2.50mm, symbol Device:C_Small
- added U412: 74AHC138, Package_DIP:DIP-16_W7.62mm_Socket, symbol 74xx:74LS138
Connections:
- net +5V: now also C203.1, U412.16 (VCC)
- net A0: now also U412.1 (A0)
- net A1: now also U412.2 (A1)
- net GND: now also C203.2, U412.8 (GND)
- net R/~{W}: now also U412.3 (A2)
- net ~{IO0SEL}: now also U412.4 (E1)
- new net A3: U412.6 (E3)
- new net A4: U412.5 (E2)
- new net ~{CLKSPD}: U412.11 (O4)
- new net ~{PSUCTL}: U412.15 (O0)
- new net ~{VBRH}: U412.13 (O2)
- new net ~{VBRL}: U412.12 (O3)
- no-connect marks 23 -> 27
Other:
- note added: "Misc. System register decoder"
- note added: "Read-only system registers"
- note added: "Write-only system registers"
- moved on the sheet: C201, C202, C203, RN401

Commit message: Change the PIA / VIA chips to S-variants.  Requires a diode on the IRQ line, since they have totem-pole outputs.
Parts:
- U501: value W65C21 -> W65C21S
Changed lines of the file:
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@@
   (symbol (lib_id "jrt-ICs:W65C21") (at 168.148 124.206 0) (unit 1)
     (in_bom yes) (on_board yes) (dnp no) (fields_autoplaced)
-    (property "Reference" "U501" (at 170.1039 87.376 0)
-      (effects (font (size 1.27 1.27)) (justify left))
-    )
-    (property "Value" "W65C21" (at 170.1039 89.916 0)
+    (property "Reference" "U501" (at 170.1039 87.63 0)
+      (effects (font (size 1.27 1.27)) (justify left))
+    )
+    (property "Value" "W65C21S" (at 170.1039 90.17 0)
       (effects (font (size 1.27 1.27)) (justify left))
     )
@@
   (symbol (lib_id "jrt-ICs:W65C21") (at 204.978 54.864 0) (unit 1)
     (in_bom yes) (on_board yes) (dnp no) (fields_autoplaced)
-    (property "Reference" "U501" (at 206.9339 18.034 0)
-      (effects (font (size 1.27 1.27)) (justify left))
-    )
-    (property "Value" "W65C21" (at 206.9339 20.574 0)
-      (effects (font (size 1.27 1.27)) (justify left))
-    )
+    (property "Reference" "U501" (at 206.9339 17.78 0)
+      (effects (font (size 1.27 1.27)) (justify left))
+    )
+    (property "Value" "W65C21S" (at 206.9339 20.32 0)
+      (effects (font (size 1.27 1.27)) (justify left))
+    )
