File: design-files/pg09-system-interrupts.kicad_sch (KiCad schematic)
At the start: 8 parts, among them Q401 2N7000, U401 W65C21, U402 GAL22V10, U403 GAL22V10, U404 GAL22V10

Commit message: Add text labels to address decoder and interrupt controller sheets.
Other:
- note added: "Interrupt Controller"
Changed lines of the file:
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@@
     (effects (font (size 1.27 1.27)) (justify left bottom))
+  )
+  (text "Interrupt Controller" (at 137.16 22.86 0)
+    (effects (font (size 2.54 2.54) (thickness 0.254) bold italic) (justify left bottom))
   )
   (text "intenc.chp" (at 148.59 29.21 0)

Commit message: Rework the INTMUX to have CS0, CS1, and /CS2, like the PIA.  Use the new nA2, along with A2 and A3 as additional chip-selects for these devices.
Connections:
- net A2: now also U404.10 (I10); no longer U401.22 (CS0), U401.24 (CS1), U404.11 (I11)
- net R/~{W}: now also U404.14 (IO1); no longer U404.13 (I12)
- net ~{IO0SEL}: now reaches U401.23 (~{CS2})
- net ~{IO0SEL}: now also U404.13 (I12); no longer U404.10 (I10)
- new net A3: U401.24 (CS1), U404.11 (I11)
- new net nA2: U401.22 (CS0)
- no-connect marks 11 -> 10
Changed lines of the file:
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@@
   (junction (at 255.27 83.82) (diameter 0) (color 0 0 0 0)
-  )
-  (junction (at 55.88 71.12) (diameter 0) (color 0 0 0 0)
   )
   (junction (at 247.65 78.74) (diameter 0) (color 0 0 0 0)
@@
   (no_connect (at 166.37 113.03))
   (no_connect (at 55.88 99.06))
-  (no_connect (at 227.33 76.2))
   (no_connect (at 55.88 96.52))
   (no_connect (at 81.28 60.96))
@@
     (stroke (width 0) (type default))
   )
-  (wire (pts (xy 49.53 71.12) (xy 55.88 71.12))
-    (stroke (width 0) (type default))
-  )
   (wire (pts (xy 116.84 55.88) (xy 116.84 83.82))
     (stroke (width 0) (type default))
@@
     (stroke (width 0) (type default))
   )
+  (wire (pts (xy 49.53 73.66) (xy 55.88 73.66))
+    (stroke (width 0) (type default))
+  )
   (wire (pts (xy 158.75 172.72) (xy 158.75 181.61))
     (stroke (width 0) (type default))
@@
     (stroke (width 0) (type default))
   )
+  (wire (pts (xy 196.85 99.06) (xy 201.93 99.06))
+    (stroke (width 0) (type default))
+  )
   (wire (pts (xy 109.22 143.51) (xy 167.64 143.51))
     (stroke (width 0) (type default))
@@
     (stroke (width 0) (type default))
   )
-  (wire (pts (xy 41.91 148.59) (xy 187.96 148.59))
-    (stroke (width 0) (type default))
-  )
   (wire (pts (xy 124.46 60.96) (xy 140.97 60.96))
     (stroke (width 0) (type default))
@@
     (stroke (width 0) (type default))
   )
-  (wire (pts (xy 187.96 148.59) (xy 187.96 99.06))
+  (wire (pts (xy 41.91 148.59) (xy 201.93 148.59))
+    (stroke (width 0) (type default))
+  )
+  (wire (pts (xy 201.93 148.59) (xy 201.93 104.14))
     (stroke (width 0) (type default))
   )
@@
     (stroke (width 0) (type default))
   )
-  (wire (pts (xy 55.88 71.12) (xy 55.88 73.66))
-    (stroke (width 0) (type default))
-  )
   (wire (pts (xy 133.35 58.42) (xy 140.97 58.42))
     (stroke (width 0) (type default))
@@
     (stroke (width 0) (type default))
   )
-  (wire (pts (xy 187.96 99.06) (xy 201.93 99.06))
-    (stroke (width 0) (type default))
-  )
   (wire (pts (xy 153.67 172.72) (xy 153.67 181.61))
     (stroke (width 0) (type default))
@@
   )
   (wire (pts (xy 123.19 43.18) (xy 123.19 63.5))
-    (stroke (width 0) (type default))
-  )
-  (wire (pts (xy 194.31 101.6) (xy 201.93 101.6))
     (stroke (width 0) (type default))
   )
@@
     )
   )
-  (global_label "A2" (shape input) (at 49.53 71.12 180) (fields_autoplaced)
-    (effects (font (size 1.27 1.27)) (justify right))
-    (property "Intersheetrefs" "${INTERSHEET_REFS}" (at 44.3261 71.12 0)
+  (global_label "nA2" (shape input) (at 55.88 71.12 180) (fields_autoplaced)
+    (effects (font (size 1.27 1.27)) (justify right))
+    (property "Intersheetrefs" "${INTERSHEET_REFS}" (at 49.5271 71.12 0)
+      (effects (font (size 1.27 1.27)) (justify right) hide)
+    )
+  )
+  (global_label "A2" (shape input) (at 196.85 99.06 180) (fields_autoplaced)
+    (effects (font (size 1.27 1.27)) (justify right))
+    (property "Intersheetrefs" "${INTERSHEET_REFS}" (at 191.6461 99.06 0)
       (effects (font (size 1.27 1.27)) (justify right) hide)
     )
@@
     )
   )
+  (global_label "~{IO0SEL}" (shape input) (at 41.91 76.2 180) (fields_autoplaced)
+    (effects (font (size 1.27 1.27)) (justify right))
+    (property "Intersheetrefs" "${INTERSHEET_REFS}" (at 32.4728 76.2 0)
+      (effects (font (size 1.27 1.27)) (justify right) hide)
+    )
+  )
   (global_label "~{IRQ14}" (shape input) (at 140.97 118.11 180) (fields_autoplaced)
     (effects (font (size 1.27 1.27)) (justify right))
@@
     )
   )
-  (global_label "A2" (shape input) (at 194.31 101.6 180) (fields_autoplaced)
-    (effects (font (size 1.27 1.27)) (justify right))
-    (property "Intersheetrefs" "${INTERSHEET_REFS}" (at 189.1061 101.6 0)
-      (effects (font (size 1.27 1.27)) (justify right) hide)
-    )
-  )
   (global_label "D2" (shape output) (at 232.41 93.98 0) (fields_autoplaced)
     (effects (font (size 1.27 1.27)) (justify left))
@@
     )
   )
+  (global_label "A3" (shape input) (at 201.93 101.6 180) (fields_autoplaced)
+    (effects (font (size 1.27 1.27)) (justify right))
+    (property "Intersheetrefs" "${INTERSHEET_REFS}" (at 196.7261 101.6 0)
+      (effects (font (size 1.27 1.27)) (justify right) hide)
+    )
+  )
   (global_label "~{IRQ10}" (shape input) (at 140.97 107.95 180) (fields_autoplaced)
     (effects (font (size 1.27 1.27)) (justify right))
@@
     )
   )
-  (global_label "R{slash}~{W}" (shape input) (at 201.93 104.14 180) (fields_autoplaced)
-    (effects (font (size 1.27 1.27)) (justify right))
-    (property "Intersheetrefs" "${INTERSHEET_REFS}" (at 194.9723 104.14 0)
-      (effects (font (size 1.27 1.27)) (justify right) hide)
-    )
+  (global_label "R{slash}~{W}" (shape input) (at 227.33 76.2 0) (fields_autoplaced)
+    (effects (font (size 1.27 1.27)) (justify left))
+    (property "Intersheetrefs" "${INTERSHEET_REFS}" (at 234.2877 76.2 0)
+      (effects (font (size 1.27 1.27)) (justify left) hide)
+    )
+  )
+  (global_label "A3" (shape input) (at 49.53 73.66 180) (fields_autoplaced)
+    (effects (font (size 1.27 1.27)) (justify right))
+    (property "Intersheetrefs" "${INTERSHEET_REFS}" (at 44.3261 73.66 0)
+      (effects (font (size 1.27 1.27)) (justify right) hide)
+    )

Commit message: Assign a bunch of footprints.
Parts:
- U401: footprint Package_DIP:DIP-40_W15.24mm -> Package_DIP:DIP-40_W15.24mm_Socket
- U402, U403, U404: footprint (none) -> Package_DIP:DIP-24_W7.62mm_Socket
Changed lines of the file:
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@@
       (effects (font (size 1.27 1.27)) (justify left))
     )
-    (property "Footprint" "Package_DIP:DIP-40_W15.24mm" (at 66.04 69.85 0)
+    (property "Footprint" "Package_DIP:DIP-40_W15.24mm_Socket" (at 66.04 69.85 0)
       (effects (font (size 1.27 1.27)) hide)
     )
@@
       (effects (font (size 1.27 1.27)) (justify left))
     )
-    (property "Footprint" "" (at 214.63 90.17 0)
+    (property "Footprint" "Package_DIP:DIP-24_W7.62mm_Socket" (at 214.63 90.17 0)
       (effects (font (size 1.27 1.27)) hide)
     )
@@
       (effects (font (size 1.27 1.27)) (justify left))
     )
-    (property "Footprint" "" (at 153.67 116.84 0)
+    (property "Footprint" "Package_DIP:DIP-24_W7.62mm_Socket" (at 153.67 116.84 0)
       (effects (font (size 1.27 1.27)) hide)
     )
@@
       (effects (font (size 1.27 1.27)) (justify left))
     )
-    (property "Footprint" "" (at 153.67 54.61 0)
-      (effects (font (size 1.27 1.27)) hide)
-    )
+    (property "Footprint" "Package_DIP:DIP-24_W7.62mm_Socket" (at 153.67 54.61 0)
+      (effects (font (size 1.27 1.27)) hide)
+    )

Commit message: Finish assigning footprints.
Parts:
- R401: footprint (none) -> Resistor_THT:R_Axial_DIN0207_L6.3mm_D2.5mm_P7.62mm_Horizontal
Changed lines of the file:
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@@
       (effects (font (size 1.27 1.27)) (justify left))
     )
-    (property "Footprint" "" (at 247.65 81.28 0)
+    (property "Footprint" "Resistor_THT:R_Axial_DIN0207_L6.3mm_D2.5mm_P7.62mm_Horizontal" (at 247.65 81.28 0)
       (effects (font (size 1.27 1.27)) hide)
     )

Commit message: Fix various errors and omissions discovered while working on the first cut of the PCB layout.
Parts:
- added C201, C202, C203 (x2): 0.1µF, Capacitor_THT:C_Disc_D6.0mm_W4.4mm_P5.00mm, symbol Device:C_Small
- renumbered RN1 to RN402
Connections:
- net +5V: now also C201.1, C202.1, C203.1, C203.1
- net GND: now also C201.2, C202.2, C203.2, C203.2
Changed lines of the file:
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@@
     (company "Copyright (c) 2022-2023 Jason R. Thorpe. See LICENSE.")
   )
+  (junction (at 233.68 139.7) (diameter 0) (color 0 0 0 0)
+  )
   (junction (at 255.27 83.82) (diameter 0) (color 0 0 0 0)
   )
+  (junction (at 243.84 134.62) (diameter 0) (color 0 0 0 0)
+  )
+  (junction (at 233.68 134.62) (diameter 0) (color 0 0 0 0)
+  )
+  (junction (at 223.52 134.62) (diameter 0) (color 0 0 0 0)
+  )
+  (junction (at 223.52 139.7) (diameter 0) (color 0 0 0 0)
+  )
   (junction (at 247.65 78.74) (diameter 0) (color 0 0 0 0)
+  )
+  (junction (at 243.84 139.7) (diameter 0) (color 0 0 0 0)
   )
   (no_connect (at 81.28 88.9))
@@
     (stroke (width 0) (type default))
   )
+  (wire (pts (xy 223.52 134.62) (xy 233.68 134.62))
+    (stroke (width 0) (type default))
+  )
   (wire (pts (xy 173.99 93.98) (xy 201.93 93.98))
     (stroke (width 0) (type default))
@@
     (stroke (width 0) (type default))
   )
+  (wire (pts (xy 223.52 139.7) (xy 233.68 139.7))
+    (stroke (width 0) (type default))
+  )
   (wire (pts (xy 143.51 172.72) (xy 143.51 181.61))
     (stroke (width 0) (type default))
@@
     (stroke (width 0) (type default))
   )
+  (wire (pts (xy 243.84 139.7) (xy 254 139.7))
+    (stroke (width 0) (type default))
+  )
+  (wire (pts (xy 233.68 139.7) (xy 243.84 139.7))
+    (stroke (width 0) (type default))
+  )
   (wire (pts (xy 81.28 81.28) (xy 107.95 81.28))
     (stroke (width 0) (type default))
@@
     (stroke (width 0) (type default))
   )
+  (wire (pts (xy 233.68 134.62) (xy 243.84 134.62))
+    (stroke (width 0) (type default))
+  )
   (wire (pts (xy 55.88 76.2) (xy 41.91 76.2))
     (stroke (width 0) (type default))
@@
   )
   (wire (pts (xy 171.45 110.49) (xy 166.37 110.49))
+    (stroke (width 0) (type default))
+  )
+  (wire (pts (xy 243.84 134.62) (xy 254 134.62))
     (stroke (width 0) (type default))
   )
@@
     )
   )
+  (symbol (lib_id "Device:C_Small") (at 223.52 137.16 0) (unit 1)
+    (in_bom yes) (on_board yes) (dnp no) (fields_autoplaced)
+    (property "Reference" "C201" (at 225.8441 136.3316 0)
+      (effects (font (size 1.27 1.27)) (justify left))
+    )
+    (property "Value" "0.1µF" (at 225.8441 138.8685 0)
+      (effects (font (size 1.27 1.27)) (justify left))
+    )
+    (property "Footprint" "Capacitor_THT:C_Disc_D6.0mm_W4.4mm_P5.00mm" (at 223.52 137.16 0)
+      (effects (font (size 1.27 1.27)) hide)
+    )
+    (property "Datasheet" "~" (at 223.52 137.16 0)
+      (effects (font (size 1.27 1.27)) hide)
+    )
+    (pin "1")
+    (pin "2")
+    (instances
+      (project "pg09-system"
+        (path "/44572023-3621-4b3a-bd53-c3b2b3f42871/4db01e9b-9f77-42a7-9351-8914253ebfe9"
+          (reference "C201") (unit 1)
+        )
+        (path "/44572023-3621-4b3a-bd53-c3b2b3f42871/c1ac9c41-410b-461b-8887-70fb93569524"
+          (reference "C301") (unit 1)
+        )
+        (path "/44572023-3621-4b3a-bd53-c3b2b3f42871/7138fc46-10d4-4cc4-afd5-54717dbe5db7"
+          (reference "C401") (unit 1)
+        )
+      )
+    )
+  )
   (symbol (lib_id "jrt-ICs:GAL22V10") (at 214.63 90.17 0) (unit 1)
     (in_bom yes) (on_board yes) (dnp no) (fields_autoplaced)
@@
     )
   )
+  (symbol (lib_id "Device:C_Small") (at 243.84 137.16 0) (unit 1)
+    (in_bom yes) (on_board yes) (dnp no) (fields_autoplaced)
+    (property "Reference" "C203" (at 246.1641 136.3316 0)
+      (effects (font (size 1.27 1.27)) (justify left))
+    )
+    (property "Value" "0.1µF" (at 246.1641 138.8685 0)
+      (effects (font (size 1.27 1.27)) (justify left))
+    )
+    (property "Footprint" "Capacitor_THT:C_Disc_D6.0mm_W4.4mm_P5.00mm" (at 243.84 137.16 0)
+      (effects (font (size 1.27 1.27)) hide)
+    )
+    (property "Datasheet" "~" (at 243.84 137.16 0)
+      (effects (font (size 1.27 1.27)) hide)
+    )
+    (pin "1")
+    (pin "2")
+    (instances
+      (project "pg09-system"
+        (path "/44572023-3621-4b3a-bd53-c3b2b3f42871/4db01e9b-9f77-42a7-9351-8914253ebfe9"
+          (reference "C203") (unit 1)
+        )
+        (path "/44572023-3621-4b3a-bd53-c3b2b3f42871/c1ac9c41-410b-461b-8887-70fb93569524"
+          (reference "C303") (unit 1)
+        )
+        (path "/44572023-3621-4b3a-bd53-c3b2b3f42871/7138fc46-10d4-4cc4-afd5-54717dbe5db7"
+          (reference "C403") (unit 1)
+        )
+      )
+    )
+  )
   (symbol (lib_id "power:GND") (at 153.67 73.66 0) (unit 1)
     (in_bom yes) (on_board yes) (dnp no) (fields_autoplaced)
@@
     )
   )
+  (symbol (lib_id "power:+5V") (at 223.52 134.62 0) (unit 1)
+    (in_bom yes) (on_board yes) (dnp no) (fields_autoplaced)
+    (property "Reference" "#PWR0214" (at 223.52 138.43 0)
+      (effects (font (size 1.27 1.27)) hide)
+    )
+    (property "Value" "+5V" (at 223.52 131.0442 0)
+      (effects (font (size 1.27 1.27)))
+    )
+    (property "Footprint" "" (at 223.52 134.62 0)
+      (effects (font (size 1.27 1.27)) hide)
+    )
+    (property "Datasheet" "" (at 223.52 134.62 0)
+      (effects (font (size 1.27 1.27)) hide)
+    )
+    (pin "1")
+    (instances
+      (project "pg09-system"
+        (path "/44572023-3621-4b3a-bd53-c3b2b3f42871/4db01e9b-9f77-42a7-9351-8914253ebfe9"
+          (reference "#PWR0214") (unit 1)
+        )
+        (path "/44572023-3621-4b3a-bd53-c3b2b3f42871/c1ac9c41-410b-461b-8887-70fb93569524"
+          (reference "#PWR0309") (unit 1)
+        )
+        (path "/44572023-3621-4b3a-bd53-c3b2b3f42871/7138fc46-10d4-4cc4-afd5-54717dbe5db7"
+          (reference "#PWR0410") (unit 1)
+        )
+      )
+    )
+  )
   (symbol (lib_id "power:+5V") (at 153.67 97.79 0) (unit 1)
     (in_bom yes) (on_board yes) (dnp no) (fields_autoplaced)
@@
     )
   )
+  (symbol (lib_id "Device:C_Small") (at 233.68 137.16 0) (unit 1)
+    (in_bom yes) (on_board yes) (dnp no) (fields_autoplaced)
+    (property "Reference" "C202" (at 236.0041 136.3316 0)
+      (effects (font (size 1.27 1.27)) (justify left))
+    )
+    (property "Value" "0.1µF" (at 236.0041 138.8685 0)
+      (effects (font (size 1.27 1.27)) (justify left))
+    )
+    (property "Footprint" "Capacitor_THT:C_Disc_D6.0mm_W4.4mm_P5.00mm" (at 233.68 137.16 0)
+      (effects (font (size 1.27 1.27)) hide)
+    )
+    (property "Datasheet" "~" (at 233.68 137.16 0)
+      (effects (font (size 1.27 1.27)) hide)
+    )
+    (pin "1")
+    (pin "2")
+    (instances
+      (project "pg09-system"
+        (path "/44572023-3621-4b3a-bd53-c3b2b3f42871/4db01e9b-9f77-42a7-9351-8914253ebfe9"
+          (reference "C202") (unit 1)
+        )
+        (path "/44572023-3621-4b3a-bd53-c3b2b3f42871/c1ac9c41-410b-461b-8887-70fb93569524"
+          (reference "C302") (unit 1)
+        )
+        (path "/44572023-3621-4b3a-bd53-c3b2b3f42871/7138fc46-10d4-4cc4-afd5-54717dbe5db7"
+          (reference "C402") (unit 1)
+        )
+      )
+    )
+  )
+  (symbol (lib_id "Device:C_Small") (at 254 137.16 0) (unit 1)
+    (in_bom yes) (on_board yes) (dnp no) (fields_autoplaced)
+    (property "Reference" "C203" (at 256.3241 136.3316 0)
+      (effects (font (size 1.27 1.27)) (justify left))
+    )
+    (property "Value" "0.1µF" (at 256.3241 138.8685 0)
+      (effects (font (size 1.27 1.27)) (justify left))
+    )
+    (property "Footprint" "Capacitor_THT:C_Disc_D6.0mm_W4.4mm_P5.00mm" (at 254 137.16 0)
+      (effects (font (size 1.27 1.27)) hide)
+    )
+    (property "Datasheet" "~" (at 254 137.16 0)
+      (effects (font (size 1.27 1.27)) hide)
+    )
+    (pin "1")
+    (pin "2")
+    (instances
+      (project "pg09-system"
+        (path "/44572023-3621-4b3a-bd53-c3b2b3f42871/4db01e9b-9f77-42a7-9351-8914253ebfe9"
+          (reference "C203") (unit 1)
+        )
+        (path "/44572023-3621-4b3a-bd53-c3b2b3f42871/c1ac9c41-410b-461b-8887-70fb93569524"
+          (reference "C304") (unit 1)
+        )
+        (path "/44572023-3621-4b3a-bd53-c3b2b3f42871/7138fc46-10d4-4cc4-afd5-54717dbe5db7"
+          (reference "C404") (unit 1)
+        )
+      )
+    )
+  )
+  (symbol (lib_id "power:GND") (at 223.52 139.7 0) (unit 1)
+    (in_bom yes) (on_board yes) (dnp no) (fields_autoplaced)
+    (property "Reference" "#PWR0216" (at 223.52 146.05 0)
+      (effects (font (size 1.27 1.27)) hide)
+    )
+    (property "Value" "GND" (at 223.52 144.1434 0)
+      (effects (font (size 1.27 1.27)))
+    )
+    (property "Footprint" "" (at 223.52 139.7 0)
+      (effects (font (size 1.27 1.27)) hide)
+    )
+    (property "Datasheet" "" (at 223.52 139.7 0)
+      (effects (font (size 1.27 1.27)) hide)
+    )
+    (pin "1")
+    (instances
+      (project "pg09-system"
+        (path "/44572023-3621-4b3a-bd53-c3b2b3f42871/4db01e9b-9f77-42a7-9351-8914253ebfe9"
+          (reference "#PWR0216") (unit 1)
+        )
+        (path "/44572023-3621-4b3a-bd53-c3b2b3f42871/c1ac9c41-410b-461b-8887-70fb93569524"
+          (reference "#PWR0310") (unit 1)
+        )
+        (path "/44572023-3621-4b3a-bd53-c3b2b3f42871/7138fc46-10d4-4cc4-afd5-54717dbe5db7"
+          (reference "#PWR0411") (unit 1)
+        )
+      )
+    )
+  )
   (symbol (lib_id "Device:R_Network08") (at 151.13 167.64 0) (unit 1)
     (in_bom yes) (on_board yes) (dnp no) (fields_autoplaced)
-    (property "Reference" "RN1" (at 161.29 167.259 0)
+    (property "Reference" "RN402" (at 161.29 167.259 0)
       (effects (font (size 1.27 1.27)) (justify left))
     )
@@
       (project "pg09-system"
         (path "/44572023-3621-4b3a-bd53-c3b2b3f42871/7138fc46-10d4-4cc4-afd5-54717dbe5db7"
-          (reference "RN1") (unit 1)
-        )
-      )
+          (reference "RN402") (unit 1)
+        )
+      )

Commit message: Specify a physically smaller bypass cap.
Parts:
- C201, C202, C203: footprint Capacitor_THT:C_Disc_D6.0mm_W4.4mm_P5.00mm -> Capacitor_THT:C_Disc_D3.8mm_W2.6mm_P2.50mm
Changed lines of the file:
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@@
       (effects (font (size 1.27 1.27)) (justify left))
     )
-    (property "Footprint" "Capacitor_THT:C_Disc_D6.0mm_W4.4mm_P5.00mm" (at 223.52 137.16 0)
+    (property "Footprint" "Capacitor_THT:C_Disc_D3.8mm_W2.6mm_P2.50mm" (at 223.52 137.16 0)
       (effects (font (size 1.27 1.27)) hide)
     )
@@
       (effects (font (size 1.27 1.27)) (justify left))
     )
-    (property "Footprint" "Capacitor_THT:C_Disc_D6.0mm_W4.4mm_P5.00mm" (at 243.84 137.16 0)
+    (property "Footprint" "Capacitor_THT:C_Disc_D3.8mm_W2.6mm_P2.50mm" (at 243.84 137.16 0)
       (effects (font (size 1.27 1.27)) hide)
     )
@@
       (effects (font (size 1.27 1.27)) (justify left))
     )
-    (property "Footprint" "Capacitor_THT:C_Disc_D6.0mm_W4.4mm_P5.00mm" (at 233.68 137.16 0)
+    (property "Footprint" "Capacitor_THT:C_Disc_D3.8mm_W2.6mm_P2.50mm" (at 233.68 137.16 0)
       (effects (font (size 1.27 1.27)) hide)
     )
@@
       (effects (font (size 1.27 1.27)) (justify left))
     )
-    (property "Footprint" "Capacitor_THT:C_Disc_D6.0mm_W4.4mm_P5.00mm" (at 254 137.16 0)
-      (effects (font (size 1.27 1.27)) hide)
-    )
+    (property "Footprint" "Capacitor_THT:C_Disc_D3.8mm_W2.6mm_P2.50mm" (at 254 137.16 0)
+      (effects (font (size 1.27 1.27)) hide)
+    )

Commit message: Integrate the auto-vectoring interrupt controller.
Parts:
- removed Q401: 2N7000, Package_TO_SOT_THT:TO-92_Inline, symbol Transistor_FET:2N7000
- removed R401: 10K, Resistor_THT:R_Axial_DIN0207_L6.3mm_D2.5mm_P7.62mm_Horizontal, symbol Device:R_Small
- added C203 (x3): 0.1µF, Capacitor_THT:C_Disc_D3.8mm_W2.6mm_P2.50mm, symbol Device:C_Small
- added U405, U406: 74AHC374, symbol 74xx:74AHC374
- added U407: 74AHC138, symbol 74xx:74LS138
Connections:
- net +5V: now also C203.1, C203.1, C203.1, U405.20 (VCC), U406.20 (VCC), U407.16 (VCC)
- net A0: now also U404.23 (IO10), U407.1 (A0)
- net A1: now also U404.22 (IO9), U407.3 (A2)
- net A2: now also U404.21 (IO8); no longer U404.10 (I10)
- net A3: now also U404.20 (IO7), U407.6 (E3); no longer U404.11 (I11)
- net D0: now also U406.3 (D0); no longer U404.23 (IO10)
- net D1: now also U406.4 (D1); no longer U404.22 (IO9)
- net D2: now also U406.7 (D2); no longer U404.21 (IO8)
- net D3: now also U406.8 (D3); no longer U404.20 (IO7)
- net D4: now also U406.13 (D4); no longer U404.19 (IO6)
- net D5: now also U405.14 (D5), U406.14 (D5); no longer U404.18 (IO5)
- net D6: now also U405.17 (D6), U406.17 (D6); no longer U404.17 (IO4)
- net D7: now also U405.18 (D7), U406.18 (D7); no longer U404.16 (IO3)
- net E: no longer U404.1 (I1/CLK)
- net GND: now also C203.2, C203.2, C203.2, U405.10 (GND), U405.13 (D4), U405.3 (D0), U405.4 (D1), U405.7 (D2), U405.8 (D3), U406.10 (GND), U407.8 (GND)
- net R/~{W}: no longer U404.14 (IO1)
- net nA2: now also U407.5 (E2)
- net ~{IO0SEL}: now also U407.4 (E1); no longer U404.13 (I12)
- net ~{IRQ}: now also U404.17 (IO4)
- net at U402.23 (IO10): now also U404.3 (I3); no longer U404.2 (I2)
- net at U402.22 (IO9): now also U404.4 (I4); no longer U404.3 (I3)
- net at U402.21 (IO8): now also U404.5 (I5); no longer U404.4 (I4)
- net at U402.20 (IO7): now also U404.6 (I6); no longer U404.5 (I5)
- net at U403.23 (IO10): now also U404.7 (I7); no longer U404.6 (I6)
- net at U403.22 (IO9): now also U404.8 (I8); no longer U404.7 (I7)
- net at U403.21 (IO8): now also U404.9 (I9); no longer U404.8 (I8)
- net at U403.20 (IO7): now also U404.10 (I10); no longer U404.9 (I9)
- new net: U406.11 (Cp), U407.15 (O0)
- new net: U405.11 (Cp), U407.14 (O1)
- new net A10: U406.6 (O2)
- new net A11: U406.9 (O3)
- new net A12: U406.12 (O4)
- new net A13: U406.15 (O5)
- new net A14: U406.16 (O6)
- new net A15: U406.19 (O7)
- new net A4: U404.19 (IO6)
- new net A5: U405.15 (O5)
- new net A6: U405.16 (O6)
- new net A7: U405.19 (O7)
- new net A8: U406.2 (O0)
- new net A9: U406.5 (O1)
- new net BS: U404.1 (I1/CLK)
- new net IVV: U404.18 (IO5)
- new net dA0: U404.11 (I11)
- new net ~{WR}: U407.2 (A1)
- new net ~{aINTC}: U404.2 (I2), U405.1 (OE), U406.1 (OE)
- no-connect marks 10 -> 25
Other:
- note added: "Auto-vector IRQ mux"
- note added: "IRQ Vector Base Register"
- note added: "intmux_av.chp"
- note removed: "intmux.chp"
- moved on the sheet: C201, C202, C203, RN401, RN402, U402, U403, U404

Commit message: WIP re-laying out PCB.
Parts:
- U405, U406: footprint (none) -> Package_DIP:DIP-20_W7.62mm_Socket
- U407: footprint (none) -> Package_DIP:DIP-16_W7.62mm_Socket
Changed lines of the file:
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@@
       (effects (font (size 1.27 1.27)) (justify left))
     )
-    (property "Footprint" "" (at 240.03 137.795 0)
+    (property "Footprint" "Package_DIP:DIP-20_W7.62mm_Socket" (at 240.03 137.795 0)
       (effects (font (size 1.27 1.27)) hide)
     )
@@
       (effects (font (size 1.27 1.27)) (justify left))
     )
-    (property "Footprint" "" (at 240.03 85.09 0)
+    (property "Footprint" "Package_DIP:DIP-20_W7.62mm_Socket" (at 240.03 85.09 0)
       (effects (font (size 1.27 1.27)) hide)
     )
@@
       (effects (font (size 1.27 1.27)) (justify left))
     )
-    (property "Footprint" "" (at 191.77 111.125 0)
-      (effects (font (size 1.27 1.27)) hide)
-    )
+    (property "Footprint" "Package_DIP:DIP-16_W7.62mm_Socket" (at 191.77 111.125 0)
+      (effects (font (size 1.27 1.27)) hide)
+    )
