File: design-files/pg09-system-interrupts.kicad_sch (KiCad schematic)
At the start: 16 parts, among them U401 W65C21, U402 GAL22V10, U403 GAL22V10, U404 GAL22V10, U405 74AHC374, U406 74AHC374, U407 74AHC138

Commit message: Re-work the interrupt controller to use discrete 74xx chips for mixing the enable signals and priority-encoding.
I made a major blunder in the INTENC GAL, and when I went to correct
it, it became clear that putting enable-mixing + priority encoding into
a single 22V10 wasn't going to fit.  At that point, the GAL was going
to be used either for priority encoding OR enable-mixing, and it just
didn't seem worth it.  So, INTENC goes away and is replaced by 74HC04s,
74HC00s, and 74HC148s.  The chip count kind of exploded here with 16
IRQs, but it fits on the board OK and the propagation delay for IRQ
signals doens't matter all that much.

Pay attention do how the 74HC148 is connected and look at the truth table
for that part carefully!
Parts:
- removed U402, U403: GAL22V10, Package_DIP:DIP-24_W7.62mm_Socket, symbol jrt-ICs:GAL22V10
- added C201, C202, C203 (x5): 0.1µF, Capacitor_THT:C_Disc_D3.8mm_W2.6mm_P2.50mm, symbol Device:C_Small
- added U402, U403, U404: 74HC04, Package_DIP:DIP-14_W7.62mm_Socket, symbol 74xx:74HC04
- added U405, U406, U407, U408: 74HC00, Package_DIP:DIP-14_W7.62mm_Socket, symbol 74xx:74HC00
- added U409, U410: 74HC148, Package_DIP:DIP-16_W7.62mm_Socket, symbol 74xx:74LS148
- renumbered U404 to U411, U407 to U412, U405 to U413, U406 to U414
Connections:
- net +5V: now also C201.1, C202.1, C203.1, C203.1, C203.1, C203.1, C203.1, U402.14 (VCC), U403.14 (VCC), U404.14 (VCC), U405.14 (VCC), U406.14 (VCC), U407.14 (VCC), U408.14 (VCC), U409.16 (VCC), U410.16 (VCC)
- net GND: now also C201.2, C202.2, C203.2, C203.2, C203.2, C203.2, C203.2, U402.7 (GND), U403.7 (GND), U404.11, U404.13, U404.7 (GND), U405.7 (GND), U406.7 (GND), U407.7 (GND), U408.7 (GND), U409.5 (EI), U409.8 (GND), U410.5 (EI), U410.8 (GND)
- net ~{IRQ0}: now also U402.1
- net ~{IRQ10}: now also U403.11
- net ~{IRQ11}: now also U403.13
- net ~{IRQ12}: now also U404.1
- net ~{IRQ13}: now also U404.3
- net ~{IRQ14}: now also U404.5
- net ~{IRQ15}: now also U404.9
- net ~{IRQ1}: now also U402.3
- net ~{IRQ2}: now also U402.5
- net ~{IRQ3}: now also U402.9
- net ~{IRQ4}: now also U402.11
- net ~{IRQ5}: now also U402.13
- net ~{IRQ6}: now also U403.1
- net ~{IRQ7}: now also U403.3
- net ~{IRQ8}: now also U403.5
- net ~{IRQ9}: now also U403.9
- net INT_E8: now reaches U401.10 (PB0)
- net INT_E8: now also U407.2
- net INT_E9: now reaches U401.11 (PB1)
- net INT_E9: now also U407.5
- net INT_E10: now reaches U401.12 (PB2)
- net INT_E10: now also U407.10
- net INT_E11: now reaches U401.13 (PB3)
- net INT_E11: now also U407.13
- net INT_E12: now reaches U401.14 (PB4)
- net INT_E12: now also U408.2
- net INT_E134: now reaches U401.15 (PB5)
- net INT_E14: now reaches U401.16 (PB6)
- net INT_E14: now also U408.10
- net INT_E15: now reaches U401.17 (PB7)
- net INT_E15: now also U408.13
- net INT_E0: now reaches U401.2 (PA0)
- net INT_E0: now also U405.2
- net INT_E1: now reaches U401.3 (PA1)
- net INT_E1: now also U405.5
- net INT_E2: now reaches U401.4 (PA2)
- net INT_E2: now also U405.10
- net INT_E3: now reaches U401.5 (PA3)
- net INT_E3: now also U405.13
- net INT_E4: now reaches U401.6 (PA4)
- net INT_E4: now also U406.2
- net INT_E5: now reaches U401.7 (PA5)
- net INT_E5: now also U406.5
- net INT_E6: now reaches U401.8 (PA6)
- net INT_E6: now also U406.10
- net INT_E7: now reaches U401.9 (PA7)
- net INT_E7: now also U406.13
- net INT_UA: now reaches U411.10 (I10)
- net INT_UA: now also U410.15 (EO)
- net INT_L2: now reaches U411.3 (I3)
- net INT_L2: now also U409.6 (S2)
- net INT_L1: now reaches U411.4 (I4)
- net INT_L1: now also U409.7 (S1)
- net INT_L0: now reaches U411.5 (I5)
- net INT_L0: now also U409.9 (S0)
- net INT_LA: now reaches U411.6 (I6)
- net INT_LA: now also U409.15 (EO)
- net INT_U2: now reaches U411.7 (I7)
- net INT_U2: now also U410.6 (S2)
- net INT_U1: now reaches U411.8 (I8)
- net INT_U1: now also U410.7 (S1)
- net INT_U0: now reaches U411.9 (I9)
- net INT_U0: now also U410.9 (S0)
- new net INT_0: U402.2, U405.1
- new net INT_1: U402.4, U405.4
- new net INT_10: U403.10, U407.9
- new net INT_11: U403.12, U407.12
- new net INT_12: U404.2, U408.1
- new net INT_13: U404.4, U408.4
- new net INT_14: U404.6, U408.9
- new net INT_15: U404.8, U408.12
- new net INT_2: U402.6, U405.9
- new net INT_3: U402.8, U405.12
- new net INT_4: U402.10, U406.1
- new net INT_5: U402.12, U406.4
- new net INT_6: U403.2, U406.9
- new net INT_7: U403.4, U406.12
- new net INT_8: U403.6, U407.1
- new net INT_9: U403.8, U407.4
- new net INT_E13: U408.5
- new net INT_O0: U405.3, U409.4 (I7)
- new net INT_O1: U405.6, U409.3 (I6)
- new net INT_O10: U407.8, U410.2 (I5)
- new net INT_O11: U407.11, U410.1 (I4)
- new net INT_O12: U408.3, U410.13 (I3)
- new net INT_O13: U408.6, U410.12 (I2)
- new net INT_O14: U408.8, U410.11 (I1)
- new net INT_O15: U408.11, U410.10 (IO)
- new net INT_O2: U405.8, U409.2 (I5)
- new net INT_O3: U405.11, U409.1 (I4)
- new net INT_O4: U406.3, U409.13 (I3)
- new net INT_O5: U406.6, U409.12 (I2)
- new net INT_O6: U406.8, U409.11 (I1)
- new net INT_O7: U406.11, U409.10 (IO)
- new net INT_O8: U407.3, U410.4 (I7)
- new net INT_O9: U407.6, U410.3 (I6)
Other:
- note removed: "intenc.chp"
- moved on the sheet: C201, C202, C203, RN401, RN402, U401, U411, U412, U413, U414

Commit message: Weakly pull-down the INT_Ex signals to GND so the NAND inputs don't float if the PIA isn't initialized or is initialized incorrectly.
Parts:
- added RN403, RN404: 10K, Resistor_THT:R_Array_SIP9, symbol Device:R_Network08
Connections:
- net GND: now also RN403.1 (common), RN404.1 (common)
- net INT_E0: now also RN403.2 (R1)
- net INT_E1: now also RN403.3 (R2)
- net INT_E10: now also RN404.4 (R3)
- net INT_E11: now also RN404.5 (R4)
- net INT_E12: now also RN404.6 (R5)
- net INT_E13: now also RN404.7 (R6)
- net INT_E14: now also RN404.8 (R7)
- net INT_E15: now also RN404.9 (R8)
- net INT_E2: now also RN403.4 (R3)
- net INT_E3: now also RN403.5 (R4)
- net INT_E4: now also RN403.6 (R5)
- net INT_E5: now also RN403.7 (R6)
- net INT_E6: now also RN403.8 (R7)
- net INT_E7: now also RN403.9 (R8)
- net INT_E8: now also RN404.2 (R1)
- net INT_E9: now also RN404.3 (R2)
Changed lines of the file:
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@@
     (effects (font (size 1.27 1.27)) (justify left bottom))
+  )
+  (label "INT_E15" (at 173.863 109.601 270) (fields_autoplaced)
+    (effects (font (size 1.27 1.27)) (justify right bottom))
   )
   (label "INT_E134" (at 59.309 63.881 0) (fields_autoplaced)
@@
     (effects (font (size 1.27 1.27)) (justify right bottom))
   )
+  (label "INT_E12" (at 166.243 109.601 270) (fields_autoplaced)
+    (effects (font (size 1.27 1.27)) (justify right bottom))
+  )
   (label "INT_E12" (at 106.68 60.579 180) (fields_autoplaced)
     (effects (font (size 1.27 1.27)) (justify right bottom))
@@
     (effects (font (size 1.27 1.27)) (justify left bottom))
   )
+  (label "INT_E6" (at 143.002 109.601 270) (fields_autoplaced)
+    (effects (font (size 1.27 1.27)) (justify right bottom))
+  )
   (label "INT_E9" (at 59.309 53.721 0) (fields_autoplaced)
     (effects (font (size 1.27 1.27)) (justify left bottom))
@@
     (effects (font (size 1.27 1.27)) (justify left bottom))
   )
+  (label "INT_E4" (at 137.922 109.601 270) (fields_autoplaced)
+    (effects (font (size 1.27 1.27)) (justify right bottom))
+  )
   (label "INT_O8" (at 182.118 48.387 180) (fields_autoplaced)
     (effects (font (size 1.27 1.27)) (justify right bottom))
@@
     (effects (font (size 1.27 1.27)) (justify left bottom))
   )
+  (label "INT_E14" (at 171.323 109.601 270) (fields_autoplaced)
+    (effects (font (size 1.27 1.27)) (justify right bottom))
+  )
   (label "INT_E10" (at 106.68 42.291 180) (fields_autoplaced)
     (effects (font (size 1.27 1.27)) (justify right bottom))
@@
     (effects (font (size 1.27 1.27)) (justify right bottom))
   )
+  (label "INT_E10" (at 161.163 109.601 270) (fields_autoplaced)
+    (effects (font (size 1.27 1.27)) (justify right bottom))
+  )
   (label "INT_L1" (at 231.775 34.29 180) (fields_autoplaced)
     (effects (font (size 1.27 1.27)) (justify right bottom))
@@
     (effects (font (size 1.27 1.27)) (justify right bottom))
   )
+  (label "INT_E9" (at 158.623 109.601 270) (fields_autoplaced)
+    (effects (font (size 1.27 1.27)) (justify right bottom))
+  )
   (label "INT_8" (at 106.68 18.923 180) (fields_autoplaced)
     (effects (font (size 1.27 1.27)) (justify right bottom))
@@
     (effects (font (size 1.27 1.27)) (justify left bottom))
   )
+  (label "INT_E8" (at 156.083 109.601 270) (fields_autoplaced)
+    (effects (font (size 1.27 1.27)) (justify right bottom))
+  )
   (label "INT_E9" (at 106.68 33.147 180) (fields_autoplaced)
     (effects (font (size 1.27 1.27)) (justify right bottom))
@@
     (effects (font (size 1.27 1.27)) (justify right bottom))
   )
+  (label "INT_E1" (at 130.302 109.601 270) (fields_autoplaced)
+    (effects (font (size 1.27 1.27)) (justify right bottom))
+  )
   (label "INT_E12" (at 59.309 61.341 0) (fields_autoplaced)
     (effects (font (size 1.27 1.27)) (justify left bottom))
@@
     (effects (font (size 1.27 1.27)) (justify left bottom))
   )
+  (label "INT_E0" (at 127.762 109.601 270) (fields_autoplaced)
+    (effects (font (size 1.27 1.27)) (justify right bottom))
+  )
   (label "INT_E4" (at 59.309 33.401 0) (fields_autoplaced)
     (effects (font (size 1.27 1.27)) (justify left bottom))
@@
     (effects (font (size 1.27 1.27)) (justify right bottom))
   )
+  (label "INT_E2" (at 132.842 109.601 270) (fields_autoplaced)
+    (effects (font (size 1.27 1.27)) (justify right bottom))
+  )
   (label "INT_2" (at 35.433 117.475 0) (fields_autoplaced)
     (effects (font (size 1.27 1.27)) (justify left bottom))
@@
     (effects (font (size 1.27 1.27)) (justify left bottom))
   )
+  (label "INT_E5" (at 140.462 109.601 270) (fields_autoplaced)
+    (effects (font (size 1.27 1.27)) (justify right bottom))
+  )
   (label "INT_10" (at 106.68 37.211 180) (fields_autoplaced)
     (effects (font (size 1.27 1.27)) (justify right bottom))
@@
     (effects (font (size 1.27 1.27)) (justify left bottom))
   )
+  (label "INT_E3" (at 135.382 109.601 270) (fields_autoplaced)
+    (effects (font (size 1.27 1.27)) (justify right bottom))
+  )
   (label "INT_13" (at 96.901 108.331 0) (fields_autoplaced)
     (effects (font (size 1.27 1.27)) (justify left bottom))
@@
     (effects (font (size 1.27 1.27)) (justify left bottom))
   )
+  (label "INT_E11" (at 163.703 109.601 270) (fields_autoplaced)
+    (effects (font (size 1.27 1.27)) (justify right bottom))
+  )
   (label "INT_0" (at 75.311 18.923 180) (fields_autoplaced)
     (effects (font (size 1.27 1.27)) (justify right bottom))
@@
     (effects (font (size 1.27 1.27)) (justify right bottom))
   )
+  (label "INT_E7" (at 145.542 109.601 270) (fields_autoplaced)
+    (effects (font (size 1.27 1.27)) (justify right bottom))
+  )
   (label "INT_E11" (at 106.68 51.435 180) (fields_autoplaced)
     (effects (font (size 1.27 1.27)) (justify right bottom))
@@
   )
   (label "INT_E6" (at 75.311 78.867 180) (fields_autoplaced)
+    (effects (font (size 1.27 1.27)) (justify right bottom))
+  )
+  (label "INT_E13" (at 168.783 109.601 270) (fields_autoplaced)
     (effects (font (size 1.27 1.27)) (justify right bottom))
   )
@@
     )
   )
+  (symbol (lib_id "Device:R_Network08") (at 166.243 104.521 0) (unit 1)
+    (in_bom yes) (on_board yes) (dnp no) (fields_autoplaced)
+    (property "Reference" "RN404" (at 176.403 104.14 0)
+      (effects (font (size 1.27 1.27)) (justify left))
+    )
+    (property "Value" "10K" (at 176.403 106.68 0)
+      (effects (font (size 1.27 1.27)) (justify left))
+    )
+    (property "Footprint" "Resistor_THT:R_Array_SIP9" (at 178.308 104.521 90)
+      (effects (font (size 1.27 1.27)) hide)
+    )
+    (property "Datasheet" "http://www.vishay.com/docs/31509/csc.pdf" (at 166.243 104.521 0)
+      (effects (font (size 1.27 1.27)) hide)
+    )
+    (pin "1")
+    (pin "2")
+    (pin "3")
+    (pin "4")
+    (pin "5")
+    (pin "6")
+    (pin "7")
+    (pin "8")
+    (pin "9")
+    (instances
+      (project "pg09-system"
+        (path "/44572023-3621-4b3a-bd53-c3b2b3f42871/7138fc46-10d4-4cc4-afd5-54717dbe5db7"
+          (reference "RN404") (unit 1)
+        )
+      )
+    )
+  )
   (symbol (lib_id "74xx:74HC04") (at 58.801 126.619 0) (unit 4)
     (in_bom yes) (on_board yes) (dnp no)
@@
     )
   )
+  (symbol (lib_id "Device:R_Network08") (at 137.922 104.521 0) (unit 1)
+    (in_bom yes) (on_board yes) (dnp no) (fields_autoplaced)
+    (property "Reference" "RN403" (at 148.082 104.14 0)
+      (effects (font (size 1.27 1.27)) (justify left))
+    )
+    (property "Value" "10K" (at 148.082 106.68 0)
+      (effects (font (size 1.27 1.27)) (justify left))
+    )
+    (property "Footprint" "Resistor_THT:R_Array_SIP9" (at 149.987 104.521 90)
+      (effects (font (size 1.27 1.27)) hide)
+    )
+    (property "Datasheet" "http://www.vishay.com/docs/31509/csc.pdf" (at 137.922 104.521 0)
+      (effects (font (size 1.27 1.27)) hide)
+    )
+    (pin "1")
+    (pin "2")
+    (pin "3")
+    (pin "4")
+    (pin "5")
+    (pin "6")
+    (pin "7")
+    (pin "8")
+    (pin "9")
+    (instances
+      (project "pg09-system"
+        (path "/44572023-3621-4b3a-bd53-c3b2b3f42871/7138fc46-10d4-4cc4-afd5-54717dbe5db7"
+          (reference "RN403") (unit 1)
+        )
+      )
+    )
+  )
   (symbol (lib_id "power:+5V") (at 250.444 64.77 0) (unit 1)
     (in_bom yes) (on_board yes) (dnp no) (fields_autoplaced)
@@
         )
       )
+    )
+  )
+  (symbol (lib_id "power:GND") (at 127.762 99.441 180) (unit 1)
+    (in_bom yes) (on_board yes) (dnp no) (fields_autoplaced)
+    (property "Reference" "#PWR0433" (at 127.762 93.091 0)
+      (effects (font (size 1.27 1.27)) hide)
+    )
+    (property "Value" "GND" (at 127.762 96.139 0)
+      (effects (font (size 1.27 1.27)))
+    )
+    (property "Footprint" "" (at 127.762 99.441 0)
+      (effects (font (size 1.27 1.27)) hide)
+    )
+    (property "Datasheet" "" (at 127.762 99.441 0)
+      (effects (font (size 1.27 1.27)) hide)
+    )
+    (pin "1")
+    (instances
+      (project "pg09-system"
+        (path "/44572023-3621-4b3a-bd53-c3b2b3f42871/7138fc46-10d4-4cc4-afd5-54717dbe5db7"
+          (reference "#PWR0433") (unit 1)
+        )
+      )
+    )
+  )
+  (symbol (lib_id "power:GND") (at 156.083 99.441 180) (unit 1)
+    (in_bom yes) (on_board yes) (dnp no) (fields_autoplaced)
+    (property "Reference" "#PWR0434" (at 156.083 93.091 0)
+      (effects (font (size 1.27 1.27)) hide)
+    )
+    (property "Value" "GND" (at 156.083 96.139 0)
+      (effects (font (size 1.27 1.27)))
+    )
+    (property "Footprint" "" (at 156.083 99.441 0)
+      (effects (font (size 1.27 1.27)) hide)
+    )
+    (property "Datasheet" "" (at 156.083 99.441 0)
+      (effects (font (size 1.27 1.27)) hide)
+    )
+    (pin "1")
+    (instances
+      (project "pg09-system"
+        (path "/44572023-3621-4b3a-bd53-c3b2b3f42871/7138fc46-10d4-4cc4-afd5-54717dbe5db7"
+          (reference "#PWR0434") (unit 1)
+        )
+      )

Commit message: Move the 74AHC05 from the UART sheet to the INTC sheet.
Parts:
- added C203: 0.1µF, Capacitor_THT:C_Disc_D3.8mm_W2.6mm_P2.50mm, symbol Device:C_Small
- added U703: 74AHC05, Package_DIP:DIP-14_W7.62mm_Socket, symbol 74xx:74LS05
Connections:
- net +5V: now also C203.1, U703.14 (VCC)
- net GND: now also C203.2, U703.11, U703.13, U703.7 (GND), U703.9
- net ~{IRQ3}: now also U703.2
- net ~{IRQ7}: now also U703.4
- new net INT3: U703.1
- new net INT7: U703.3
- no-connect marks 25 -> 28
Other:
- note added: "U415C is used on SPI SD sheet."
- moved on the sheet: RN401, RN402, RN403, RN404, U402G, U403G, U404G, U405E, U406E, U407E, U408E

Commit message: Move the 74AHC138 that strobes the VBR to the root sheet.  In a future commit, this is going to become a common part for other system registers.
Parts:
- removed C203: 0.1µF, Capacitor_THT:C_Disc_D3.8mm_W2.6mm_P2.50mm, symbol Device:C_Small
- removed U412: 74AHC138, Package_DIP:DIP-16_W7.62mm_Socket, symbol 74xx:74LS138
Connections:
- net ~{VBRL}: now reaches U414.11 (Cp)
- net ~{VBRL}: now also U413.11 (Cp)
- no-connect marks 28 -> 22
Other:
- moved on the sheet: C203

Commit message: Overhaul how the "system registers" in IO0SEL work, paving the way to use a VIA for the interrupt enables (because that would also give us a timer).
Connections:
- net nA2 is gone; now on net A4: U401.22 (CS0)
- net A3: no longer U401.24 (CS1)
- net A4: now also U401.24 (CS1)
- net ~{VBRL}: no longer U414.11 (Cp)
- new net ~{VBRH}: U414.11 (Cp)
Other:
- moved on the sheet: RN402, RN404, U703A, U703B, U703D, U703E, U703F

Commit message: Change the PIA / VIA chips to S-variants.  Requires a diode on the IRQ line, since they have totem-pole outputs.
Parts:
- U401: value W65C21 -> W65C21S
Changed lines of the file:
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@@
   (symbol (lib_id "jrt-ICs:W65C21") (at 46.609 53.721 0) (unit 1)
     (in_bom yes) (on_board yes) (dnp no) (fields_autoplaced)
-    (property "Reference" "U401" (at 48.5649 16.891 0)
+    (property "Reference" "U401" (at 48.5649 16.51 0)
       (effects (font (size 1.27 1.27)) (justify left))
     )
-    (property "Value" "W65C21" (at 48.5649 19.431 0)
+    (property "Value" "W65C21S" (at 48.5649 19.05 0)
       (effects (font (size 1.27 1.27)) (justify left))
     )
