File: design-files/pg09-system-uarts.kicad_sch (KiCad schematic)
At the start: 10 parts, among them Q701 2N7000, U701 W65C51, U702 16550, U703 74HC04, U704 Ali_Express_FTDI_Breakout, U705 Adafruit_FTDI_Friend, U706 Ali_Express_FTDI_Breakout, X701 1.8432MHz

Commit message: Assign a bunch of footprints.
Parts:
- U701: footprint Package_DIP:DIP-28_W15.24mm -> Package_DIP:DIP-28_W15.24mm_Socket
- U702: footprint Package_DIP:DIP-40_W15.24mm -> Package_DIP:DIP-40_W15.24mm_Socket
- U703: footprint (none) -> Package_DIP:DIP-14_W7.62mm_Socket
Changed lines of the file:
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@@
       (effects (font (size 1.27 1.27)))
     )
-    (property "Footprint" "" (at 229.87 41.91 0)
+    (property "Footprint" "Package_DIP:DIP-14_W7.62mm_Socket" (at 229.87 41.91 0)
       (effects (font (size 1.27 1.27)) hide)
     )
@@
       (effects (font (size 1.27 1.27)))
     )
-    (property "Footprint" "" (at 229.87 55.88 0)
+    (property "Footprint" "Package_DIP:DIP-14_W7.62mm_Socket" (at 229.87 55.88 0)
       (effects (font (size 1.27 1.27)) hide)
     )
@@
       (effects (font (size 1.27 1.27)))
     )
-    (property "Footprint" "" (at 229.87 27.94 0)
+    (property "Footprint" "Package_DIP:DIP-14_W7.62mm_Socket" (at 229.87 27.94 0)
       (effects (font (size 1.27 1.27)) hide)
     )
@@
       (effects (font (size 1.27 1.27)))
     )
-    (property "Footprint" "" (at 31.75 182.88 0)
+    (property "Footprint" "Package_DIP:DIP-14_W7.62mm_Socket" (at 31.75 182.88 0)
       (effects (font (size 1.27 1.27)) hide)
     )
@@
       (effects (font (size 1.27 1.27)))
     )
-    (property "Footprint" "" (at 229.87 68.58 0)
+    (property "Footprint" "Package_DIP:DIP-14_W7.62mm_Socket" (at 229.87 68.58 0)
       (effects (font (size 1.27 1.27)) hide)
     )
@@
       (effects (font (size 1.27 1.27)) (justify left))
     )
-    (property "Footprint" "" (at 254 33.02 0)
+    (property "Footprint" "Package_DIP:DIP-14_W7.62mm_Socket" (at 254 33.02 0)
       (effects (font (size 1.27 1.27)) hide)
     )
@@
       (effects (font (size 1.27 1.27)))
     )
-    (property "Footprint" "" (at 135.89 59.69 0)
+    (property "Footprint" "Package_DIP:DIP-14_W7.62mm_Socket" (at 135.89 59.69 0)
       (effects (font (size 1.27 1.27)) hide)
     )
@@
       (effects (font (size 1.27 1.27)) (justify left))
     )
-    (property "Footprint" "Package_DIP:DIP-28_W15.24mm" (at 86.36 50.8 0)
+    (property "Footprint" "Package_DIP:DIP-28_W15.24mm_Socket" (at 86.36 50.8 0)
       (effects (font (size 1.27 1.27)) hide)
     )
@@
       (effects (font (size 1.27 1.27)) (justify left))
     )
-    (property "Footprint" "Package_DIP:DIP-40_W15.24mm" (at 86.36 147.32 0)
+    (property "Footprint" "Package_DIP:DIP-40_W15.24mm_Socket" (at 86.36 147.32 0)
       (effects (font (size 1.27 1.27) italic) hide)
     )

Commit message: Finish assigning footprints.
Parts:
- R701, R702: footprint (none) -> Resistor_THT:R_Axial_DIN0207_L6.3mm_D2.5mm_P7.62mm_Horizontal
- U704, U706: footprint (none) -> jrt-Connectors:DIP-18_W10.16mm_Socket
Changed lines of the file:
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@@
       (effects (font (size 1.27 1.27)))
     )
-    (property "Footprint" "" (at 187.96 59.69 0)
+    (property "Footprint" "jrt-Connectors:DIP-18_W10.16mm_Socket" (at 187.96 59.69 0)
       (effects (font (size 1.27 1.27)) hide)
     )
@@
       (effects (font (size 1.27 1.27)) (justify left))
     )
-    (property "Footprint" "" (at 36.83 166.37 0)
+    (property "Footprint" "Resistor_THT:R_Axial_DIN0207_L6.3mm_D2.5mm_P7.62mm_Horizontal" (at 36.83 166.37 0)
       (effects (font (size 1.27 1.27)) hide)
     )
@@
       (effects (font (size 1.27 1.27)))
     )
-    (property "Footprint" "" (at 187.96 105.41 0)
+    (property "Footprint" "jrt-Connectors:DIP-18_W10.16mm_Socket" (at 187.96 105.41 0)
       (effects (font (size 1.27 1.27)) hide)
     )
@@
       (effects (font (size 1.27 1.27)) (justify left))
     )
-    (property "Footprint" "" (at 49.53 69.85 0)
-      (effects (font (size 1.27 1.27)) hide)
-    )
+    (property "Footprint" "Resistor_THT:R_Axial_DIN0207_L6.3mm_D2.5mm_P7.62mm_Horizontal" (at 49.53 69.85 0)
+      (effects (font (size 1.27 1.27)) hide)
+    )

Commit message: Fix various errors and omissions discovered while working on the first cut of the PCB layout.
Parts:
- added C201, C202, C203 (x2): 0.1µF, Capacitor_THT:C_Disc_D6.0mm_W4.4mm_P5.00mm, symbol Device:C_Small
Connections:
- net +5V: now also C201.1, C202.1, C203.1, C203.1
- net GND: now also C201.2, C202.2, C203.2, C203.2

Commit message: Correct footprint for FTDI breakout.
Parts:
- U704, U706: footprint jrt-Connectors:DIP-18_W10.16mm_Socket -> jrt-Connectors:Ali_Express_FTDI_Breakout
Changed lines of the file:
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@@
       (effects (font (size 1.27 1.27)))
     )
-    (property "Footprint" "jrt-Connectors:DIP-18_W10.16mm_Socket" (at 187.96 59.69 0)
+    (property "Footprint" "jrt-Connectors:Ali_Express_FTDI_Breakout" (at 187.96 59.69 0)
       (effects (font (size 1.27 1.27)) hide)
     )
@@
       (effects (font (size 1.27 1.27)))
     )
-    (property "Footprint" "jrt-Connectors:DIP-18_W10.16mm_Socket" (at 187.96 105.41 0)
-      (effects (font (size 1.27 1.27)) hide)
-    )
+    (property "Footprint" "jrt-Connectors:Ali_Express_FTDI_Breakout" (at 187.96 105.41 0)
+      (effects (font (size 1.27 1.27)) hide)
+    )

Commit message: Specify a physically smaller bypass cap.
Parts:
- C201, C202, C203: footprint Capacitor_THT:C_Disc_D6.0mm_W4.4mm_P5.00mm -> Capacitor_THT:C_Disc_D3.8mm_W2.6mm_P2.50mm
Changed lines of the file:
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@@
       (effects (font (size 1.27 1.27)) (justify left))
     )
-    (property "Footprint" "Capacitor_THT:C_Disc_D6.0mm_W4.4mm_P5.00mm" (at 257.81 125.73 0)
+    (property "Footprint" "Capacitor_THT:C_Disc_D3.8mm_W2.6mm_P2.50mm" (at 257.81 125.73 0)
       (effects (font (size 1.27 1.27)) hide)
     )
@@
       (effects (font (size 1.27 1.27)) (justify left))
     )
-    (property "Footprint" "Capacitor_THT:C_Disc_D6.0mm_W4.4mm_P5.00mm" (at 227.33 125.73 0)
+    (property "Footprint" "Capacitor_THT:C_Disc_D3.8mm_W2.6mm_P2.50mm" (at 227.33 125.73 0)
       (effects (font (size 1.27 1.27)) hide)
     )
@@
       (effects (font (size 1.27 1.27)) (justify left))
     )
-    (property "Footprint" "Capacitor_THT:C_Disc_D6.0mm_W4.4mm_P5.00mm" (at 247.65 125.73 0)
+    (property "Footprint" "Capacitor_THT:C_Disc_D3.8mm_W2.6mm_P2.50mm" (at 247.65 125.73 0)
       (effects (font (size 1.27 1.27)) hide)
     )
@@
       (effects (font (size 1.27 1.27)) (justify left))
     )
-    (property "Footprint" "Capacitor_THT:C_Disc_D6.0mm_W4.4mm_P5.00mm" (at 237.49 125.73 0)
-      (effects (font (size 1.27 1.27)) hide)
-    )
+    (property "Footprint" "Capacitor_THT:C_Disc_D3.8mm_W2.6mm_P2.50mm" (at 237.49 125.73 0)
+      (effects (font (size 1.27 1.27)) hide)
+    )

Commit message: Correct missing GND connection on the 2N7000 that pulls IRQ7 low for the 16550.
Connections:
- net GND: now also Q701.1 (S), R701.2
Changed lines of the file:
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@@
   (junction (at 227.33 128.27) (diameter 0) (color 0 0 0 0)
+  )
+  (junction (at 36.83 168.91) (diameter 0) (color 0 0 0 0)
   )
   (junction (at 111.76 124.46) (diameter 0) (color 0 0 0 0)
@@
         )
       )
+    )
+  )
+  (symbol (lib_id "power:GND") (at 36.83 168.91 0) (unit 1)
+    (in_bom yes) (on_board yes) (dnp no) (fields_autoplaced)
+    (property "Reference" "#PWR0718" (at 36.83 175.26 0)
+      (effects (font (size 1.27 1.27)) hide)
+    )
+    (property "Value" "GND" (at 36.83 173.99 0)
+      (effects (font (size 1.27 1.27)))
+    )
+    (property "Footprint" "" (at 36.83 168.91 0)
+      (effects (font (size 1.27 1.27)) hide)
+    )
+    (property "Datasheet" "" (at 36.83 168.91 0)
+      (effects (font (size 1.27 1.27)) hide)
+    )
+    (pin "1")
+    (instances
+      (project "pg09-system"
+        (path "/44572023-3621-4b3a-bd53-c3b2b3f42871/ac00d1d6-4857-42f9-90e1-ab396f3828b3"
+          (reference "#PWR0718") (unit 1)
+        )
+      )

Commit message: Oops, UARTs belong on IO1SEL, not IO11SEL!
Connections:
- net ~{IO11SEL} renamed ~{IO1SEL}
Changed lines of the file:
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@@
     )
   )
-  (global_label "~{IO11SEL}" (shape input) (at 60.96 147.32 180) (fields_autoplaced)
+  (global_label "~{IO1SEL}" (shape input) (at 60.96 147.32 180) (fields_autoplaced)
     (effects (font (size 1.27 1.27)) (justify right))
-    (property "Intersheetrefs" "${INTERSHEET_REFS}" (at 50.3133 147.32 0)
+    (property "Intersheetrefs" "${INTERSHEET_REFS}" (at 51.5228 147.32 0)
       (effects (font (size 1.27 1.27)) (justify right) hide)
     )
@@
     )
   )
-  (global_label "~{IO11SEL}" (shape input) (at 73.66 58.42 180) (fields_autoplaced)
+  (global_label "~{IO1SEL}" (shape input) (at 73.66 58.42 180) (fields_autoplaced)
     (effects (font (size 1.27 1.27)) (justify right))
-    (property "Intersheetrefs" "${INTERSHEET_REFS}" (at 63.0133 58.42 0)
+    (property "Intersheetrefs" "${INTERSHEET_REFS}" (at 64.2228 58.42 0)
       (effects (font (size 1.27 1.27)) (justify right) hide)
     )

Commit message: Replace the 74HC04 in the UART block with a 74HC14 -- we're going to use one of the inverters to de-bounce the NMI button.
Parts:
- removed U703: 74HC04, Package_DIP:DIP-14_W7.62mm_Socket, symbol 74xx:74HC04
- added U703: 74HC14, Package_DIP:DIP-14_W7.62mm_Socket, symbol 74xx:74HC14
Connections:
- net +5V: now also U703.14 (VCC)
- net GND: now also U703.11, U703.13, U703.5, U703.7 (GND), U703.9
- net ~{RESET}: now also U703.1
- net at U704.4 (~{CTS}): now also U703.4
- net at U702.35 (MR): now also U703.2
- net at R702.2, U701.26 (~{IRQ}): now also U703.3
