File: design-files/pg09-system-uarts.kicad_sch (KiCad schematic)
At the start: 14 parts, among them Q701 2N7000, U701 W65C51, U702 16550, U703 74HC14, U704 Ali_Express_FTDI_Breakout, U705 Adafruit_FTDI_Friend, U706 Ali_Express_FTDI_Breakout, X701 1.8432MHz

Commit message: Revert "Replace the 74HC04 in the UART block with a 74HC14 -- we're going to use"
This reverts commit c454c6436ca93ab385708a4f4269f39de4437bef.

Actually, this isn't needed at all -- I can essentially replicate the
reset circuit for this.
Parts:
- removed U703: 74HC14, Package_DIP:DIP-14_W7.62mm_Socket, symbol 74xx:74HC14
- added U703: 74HC04, Package_DIP:DIP-14_W7.62mm_Socket, symbol 74xx:74HC04
Connections:
- net +5V: now also U703.14 (VCC)
- net GND: now also U703.11, U703.13, U703.5, U703.7 (GND), U703.9
- net ~{RESET}: now also U703.1
- net at U704.4 (~{CTS}): now also U703.4
- net at R702.2, U701.26 (~{IRQ}): now also U703.3
- net at U702.35 (MR): now also U703.2

Commit message: Remove the FTDI module from the Data I/O UART, leaving only the FTDI header; we're out of space in the I/O area of the PCB.
Parts:
- removed U706: Ali_Express_FTDI_Breakout, jrt-Connectors:Ali_Express_FTDI_Breakout, symbol jrt-ICs:Ali_Express_FTDI_Breakout
Other:
- note removed: "Only install one of these FTDI modules. Both footprints provided for extra flexibility."
Changed lines of the file:
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@@
   (junction (at 60.96 142.24) (diameter 0) (color 0 0 0 0)
   )
-  (junction (at 148.59 128.27) (diameter 0) (color 0 0 0 0)
-  )
   (junction (at 49.53 73.66) (diameter 0) (color 0 0 0 0)
   )
@@
   (junction (at 111.76 121.92) (diameter 0) (color 0 0 0 0)
   )
-  (junction (at 151.13 154.94) (diameter 0) (color 0 0 0 0)
-  )
   (junction (at 227.33 123.19) (diameter 0) (color 0 0 0 0)
   )
@@
   )
   (junction (at 60.96 170.18) (diameter 0) (color 0 0 0 0)
-  )
-  (junction (at 149.86 152.4) (diameter 0) (color 0 0 0 0)
   )
   (no_connect (at 203.2 59.69))
@@
     (stroke (width 0) (type default))
   )
-  (wire (pts (xy 214.63 154.94) (xy 214.63 107.95))
-    (stroke (width 0) (type default))
-  )
   (wire (pts (xy 54.61 175.26) (xy 60.96 175.26))
     (stroke (width 0) (type default))
@@
     (stroke (width 0) (type default))
   )
-  (wire (pts (xy 149.86 152.4) (xy 213.36 152.4))
-    (stroke (width 0) (type default))
-  )
   (wire (pts (xy 39.37 182.88) (xy 60.96 182.88))
     (stroke (width 0) (type default))
@@
     (stroke (width 0) (type default))
   )
-  (wire (pts (xy 213.36 118.11) (xy 203.2 118.11))
-    (stroke (width 0) (type default))
-  )
   (wire (pts (xy 111.76 154.94) (xy 151.13 154.94))
     (stroke (width 0) (type default))
@@
     (stroke (width 0) (type default))
   )
-  (wire (pts (xy 148.59 128.27) (xy 148.59 105.41))
-    (stroke (width 0) (type default))
-  )
   (wire (pts (xy 63.5 55.88) (xy 73.66 55.88))
     (stroke (width 0) (type default))
@@
     (stroke (width 0) (type default))
   )
-  (wire (pts (xy 148.59 105.41) (xy 180.34 105.41))
-    (stroke (width 0) (type default))
-  )
   (wire (pts (xy 111.76 121.92) (xy 111.76 124.46))
     (stroke (width 0) (type default))
@@
     (stroke (width 0) (type default))
   )
-  (wire (pts (xy 213.36 152.4) (xy 213.36 118.11))
-    (stroke (width 0) (type default))
-  )
   (wire (pts (xy 222.25 27.94) (xy 222.25 41.91))
     (stroke (width 0) (type default))
@@
     (stroke (width 0) (type default))
   )
-  (wire (pts (xy 214.63 107.95) (xy 203.2 107.95))
-    (stroke (width 0) (type default))
-  )
   (wire (pts (xy 60.96 170.18) (xy 60.96 172.72))
     (stroke (width 0) (type default))
@@
   )
   (wire (pts (xy 180.34 125.73) (xy 177.8 125.73))
-    (stroke (width 0) (type default))
-  )
-  (wire (pts (xy 151.13 154.94) (xy 214.63 154.94))
     (stroke (width 0) (type default))
   )
@@
   (text "XXX Use one of the spare\ninverters and a diode instead?"
     (at 26.67 157.48 0)
-    (effects (font (size 1.27 1.27)) (justify left bottom))
-  )
-  (text "Only install one of these FTDI modules.\nBoth footprints provided for extra flexibility."
-    (at 167.64 147.32 0)
     (effects (font (size 1.27 1.27)) (justify left bottom))
   )
@@
         )
       )
-    )
-  )
-  (symbol (lib_id "jrt-ICs:Ali_Express_FTDI_Breakout") (at 191.77 107.95 0) (unit 1)
-    (in_bom yes) (on_board yes) (dnp no) (fields_autoplaced)
-    (property "Reference" "U706" (at 191.77 91.44 0)
-      (effects (font (size 1.27 1.27)))
-    )
-    (property "Value" "Ali_Express_FTDI_Breakout" (at 191.77 93.98 0)
-      (effects (font (size 1.27 1.27)))
-    )
-    (property "Footprint" "jrt-Connectors:Ali_Express_FTDI_Breakout" (at 187.96 105.41 0)
-      (effects (font (size 1.27 1.27)) hide)
-    )
-    (property "Datasheet" "" (at 187.96 105.41 0)
-      (effects (font (size 1.27 1.27)) hide)
-    )
-    (pin "1")
-    (pin "10")
-    (pin "11")
-    (pin "12")
-    (pin "13")
-    (pin "14")
-    (pin "15")
-    (pin "16")
-    (pin "17")
-    (pin "18")
-    (pin "2")
-    (pin "3")
-    (pin "4")
-    (pin "5")
-    (pin "6")
-    (pin "7")
-    (pin "8")
-    (pin "9")
-    (instances
-      (project "pg09-system"
-        (path "/44572023-3621-4b3a-bd53-c3b2b3f42871/ac00d1d6-4857-42f9-90e1-ab396f3828b3"
-          (reference "U706") (unit 1)
-        )
-      )

Commit message: Connect /CTS if the ACIA to ground.
Connections:
- net GND: now also U701.9 (~{CTS})
- no-connect marks 26 -> 25
Changed lines of the file:
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@@
   (no_connect (at 111.76 162.56))
   (no_connect (at 60.96 160.02))
-  (no_connect (at 99.06 33.02))
   (no_connect (at 203.2 52.07))
   (no_connect (at 203.2 69.85))
@@
         )
       )
+    )
+  )
+  (symbol (lib_id "power:GND") (at 99.06 33.02 90) (unit 1)
+    (in_bom yes) (on_board yes) (dnp no) (fields_autoplaced)
+    (property "Reference" "#PWR0719" (at 105.41 33.02 0)
+      (effects (font (size 1.27 1.27)) hide)
+    )
+    (property "Value" "GND" (at 102.87 33.655 90)
+      (effects (font (size 1.27 1.27)) (justify right))
+    )
+    (property "Footprint" "" (at 99.06 33.02 0)
+      (effects (font (size 1.27 1.27)) hide)
+    )
+    (property "Datasheet" "" (at 99.06 33.02 0)
+      (effects (font (size 1.27 1.27)) hide)
+    )
+    (pin "1")
+    (instances
+      (project "pg09-system"
+        (path "/44572023-3621-4b3a-bd53-c3b2b3f42871/ac00d1d6-4857-42f9-90e1-ab396f3828b3"
+          (reference "#PWR0719") (unit 1)
+        )
+      )

Commit message: Use a 74AHC05 hex inverter with open-drain outputs rather than discrete small-signal MOSFETs.  Share the gates and resistors between UART and SD SPI sheets.
Parts:
- removed Q701: 2N7000, Package_TO_SOT_THT:TO-92_Inline, symbol Transistor_FET:2N7000
- removed R701, R702: 10K, Resistor_THT:R_Axial_DIN0207_L6.3mm_D2.5mm_P7.62mm_Horizontal, symbol Device:R_Small
- removed unit 4 of U703
- added RN701: 10K, Resistor_THT:R_Array_SIP9, symbol Device:R_Network08_Split
- U703: value 74HC04 -> 74AHC05; symbol 74xx:74HC04 -> 74xx:74LS05
Connections:
- net +5V: now also RN701.1 (R1), RN701.1 (R1), RN701.1 (R1), RN701.1 (R1), RN701.1 (R1), RN701.1 (R1)
- net GND: no longer U703.5
- net ~{IRQ7}: now also U703.6, RN701.3 (R2.2)
- net at U703.4, U704.4 (~{CTS}): now also RN701.5 (R4.2)
- net at U702.30 (INTR): now also U703.5
- net at U702.35 (MR), U703.2: now also RN701.2 (R1.2)
- net at U701.26 (~{IRQ}), U703.3: now also RN701.4 (R3.2)
Other:
- note added: "RN701E, RN701F, and U703D are used on SPI SD sheet."
- note removed: "XXX Use one of the spare inverters and a diode instead?"
- moved on the sheet: C201, C202, C203, U703C, U703E, U703F

Commit message: Re-do the UARTs using a single TL16C2552 dual-UART in PLCC-44 package.
Parts:
- removed unit 3 of RN701
- removed unit 4 of RN701
- removed U701: W65C51, Package_DIP:DIP-28_W15.24mm_Socket, symbol jrt-ICs:W65C51
- removed U702: 16550, Package_DIP:DIP-40_W15.24mm_Socket, symbol Interface_UART:16550
- removed unit 3 of U703
- added unit 5 of RN701
- added unit 6 of RN701
- added U701: TL16C2552, Package_LCC:PLCC-44_THT-Socket, symbol jrt-ICs:TL16C2552
- added U702: 74AHC14, Package_DIP:DIP-14_W7.62mm_Socket, symbol 74xx:74HC14
- added unit 4 of U703
Connections:
- net +5V: now also RN701.1 (R1), RN701.1 (R1), U701.31 (~{RIB}), U701.33 (VCC), U701.43 (~{RIA}), U701.44 (VCC), U702.14 (VCC)
- net A0: now also U701.10 (A0)
- net A1: now also U701.14 (A1)
- net A2: now also U701.15 (A2)
- net D0: now also U701.2 (D0)
- net D1: now also U701.3 (D1)
- net D2: now also U701.4 (D2)
- net D3: now also U701.5 (D3)
- net D4: now also U701.6 (D4)
- net D5: now also U701.7 (D5)
- net D6: now also U701.8 (D6)
- net D7: now also U701.9 (D7)
- net GND: now also U701.12 (GND), U701.22 (GND), U701.28 (~{CTSB}), U701.29 (~{DSRB}), U701.30 (~{CDB}), U701.40 (~{CTSA}), U701.41 (~{DSRA}), U701.42 (~{CDA}), U702.11, U702.13, U702.3, U702.5, U702.7 (GND), U702.9, U703.9
- net nA3: now also U701.16 (CHSEL)
- net ~{IO1SEL}: now also U701.18 (~{CS})
- net ~{IRQ7}: now also U703.4
- net ~{RD}: now also U701.24 (~{IOR})
- net ~{RESET}: now also U702.1; no longer U703.1
- net ~{WR}: now also U701.20 (~{IOW})
- net at U704.10 (TXD): now also U701.39 (RXA)
- net at U704.14 (RXD): now also U701.38 (TXA)
- net at U704.4 (~{CTS}): now also U701.36 (~{RTSA}); no longer U703.4
- net ~{IRQ3}: now reaches RN701.2 (R1.2), U703.2
- net at U703.3: now also U701.17 (INTB)
- net at U705.2 (~{CTS}): now also U701.23 (~{RTSB})
- net at U705.4 (TX): now also U701.25 (RXB)
- net at U705.5 (RX): now also U701.26 (TXB)
- net at X701.8 (OUT): now also U701.11 (XIN)
- new net: U701.34 (INTA), U703.1
- new net RESETH: U701.21 (RESET), U702.2
- no-connect marks 25 -> 29
Other:
- note added: "RN701C, RN701D, and U703C are used on SPI SD sheet."
- note removed: "Automatic RTS/CTS flow control. When IRQ is asserted (low), the inverter de-asserts the CTS signal on the FTDI. When no IRQ is pending (high), the inverter asserts CTS on the FTDI."
- note removed: "RN701E, RN701F, and U703D are used on SPI SD sheet."
- moved on the sheet: C201, C202, C203, RN701A, RN701B, RN701G, RN701H, U703A, U703E, U703F, U704, U705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
