File: design-files/pg09-system-uarts.kicad_sch (KiCad schematic)
At the start: 11 parts, among them U701 TL16C2552, U702 74AHC14, U703 74AHC05, U704 Ali_Express_FTDI_Breakout, U705 Adafruit_FTDI_Friend, X701 1.8432MHz

Commit message: Use a now-free pin on the CLKSEL GAL to invert /RESET into an active-high RESETH signal that can be used all over the system.  Use RESETH with the 16550 UARTs and eliminate the 74HC14 Schmitt inverter that was used there. Saves a chip, and because if the reset circuit we're using, we don't need to use a Schmitt inverter.
Parts:
- removed C202: 0.1µF, Capacitor_THT:C_Disc_D3.8mm_W2.6mm_P2.50mm, symbol Device:C_Small
- removed U702: 74AHC14, Package_DIP:DIP-14_W7.62mm_Socket, symbol 74xx:74HC14
Connections:
- no-connect marks 29 -> 24
Other:
- moved on the sheet: C203

Commit message: Update some references on the UART sheet now that the Schmitt inverter is gone.
Parts:
- renumbered U704 to U702
Changed lines of the file:
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@@
         )
         (path "/44572023-3621-4b3a-bd53-c3b2b3f42871/ac00d1d6-4857-42f9-90e1-ab396f3828b3"
-          (reference "C704") (unit 1)
+          (reference "C703") (unit 1)
         )
       )
@@
   (symbol (lib_id "jrt-ICs:Ali_Express_FTDI_Breakout") (at 182.626 75.946 0) (unit 1)
     (in_bom yes) (on_board yes) (dnp no) (fields_autoplaced)
-    (property "Reference" "U704" (at 182.626 59.436 0)
+    (property "Reference" "U702" (at 182.626 59.436 0)
       (effects (font (size 1.27 1.27)))
     )
@@
       (project "pg09-system"
         (path "/44572023-3621-4b3a-bd53-c3b2b3f42871/ac00d1d6-4857-42f9-90e1-ab396f3828b3"
-          (reference "U704") (unit 1)
+          (reference "U702") (unit 1)
         )
       )
@@
         )
         (path "/44572023-3621-4b3a-bd53-c3b2b3f42871/ac00d1d6-4857-42f9-90e1-ab396f3828b3"
-          (reference "C703") (unit 1)
-        )
-      )
+          (reference "C702") (unit 1)
+        )
+      )

Commit message: Eliminate the resistor network on the UART sheet -- it's no longer needed to pull up the IRQ lines (interrupt controller sheet does that).  Just let the SPI sheet use its own discreet resistors.
Parts:
- removed RN701: 10K, Resistor_THT:R_Array_SIP9, symbol Device:R_Network08_Split
Connections:
- no-connect marks 24 -> 20
Other:
- note added: "U703C is used on SPI SD sheet."
- note removed: "RN701C, RN701D, and U703C are used on SPI SD sheet."

Commit message: Switch the oscillators to half-can.
Parts:
- X701: footprint Oscillator:Oscillator_DIP-14 -> Oscillator:Oscillator_DIP-8; symbol Oscillator:CXO_DIP14 -> Oscillator:CXO_DIP8
Connections:
- net +5V: now also X701.8 (Vcc); no longer X701.14 (Vcc)
- net GND: now also X701.4 (GND); no longer X701.7 (GND)
- net at U701.11 (XIN): now also X701.5 (OUT); no longer X701.8 (OUT)
Changed lines of the file:
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@@
     )
   )
-  (symbol (lib_id "Oscillator:CXO_DIP14") (at 38.1 97.536 0) (unit 1)
+  (symbol (lib_id "Oscillator:CXO_DIP8") (at 38.1 97.536 0) (unit 1)
     (in_bom yes) (on_board yes) (dnp no)
     (property "Reference" "X701" (at 44.45 87.376 0)
@@
       (effects (font (size 1.27 1.27)))
     )
-    (property "Footprint" "Oscillator:Oscillator_DIP-14" (at 49.53 106.426 0)
+    (property "Footprint" "Oscillator:Oscillator_DIP-8" (at 49.53 106.426 0)
       (effects (font (size 1.27 1.27)) hide)
     )
@@
     )
     (pin "1")
-    (pin "14")
-    (pin "7")
+    (pin "4")
+    (pin "5")
     (pin "8")
     (instances

Commit message: Move the 74AHC05 from the UART sheet to the INTC sheet.
Parts:
- removed C203: 0.1µF, Capacitor_THT:C_Disc_D3.8mm_W2.6mm_P2.50mm, symbol Device:C_Small
- removed U703: 74AHC05, Package_DIP:DIP-14_W7.62mm_Socket, symbol 74xx:74LS05
Connections:
- net INT3: now reaches U701.34 (INTA)
- net INT7: now reaches U701.17 (INTB)
- no-connect marks 20 -> 17
Other:
- note removed: "U703C is used on SPI SD sheet."
- moved on the sheet: C203
