File: design-files/pg09-system-spi-sdcard.kicad_sch (KiCad schematic)
At the start: 1 part, among them U1001 W65C22

Commit message: Move Reset to the main sheet.  Checkpoint SD Card SPI interface.
Parts:
- added C201, C202, C203: 0.1µF, Capacitor_THT:C_Disc_D3.8mm_W2.6mm_P2.50mm, symbol Device:C_Small
- added J1001: Adafruit MicroSD Card Breakout Board+, Connector_PinHeader_2.54mm:PinHeader_1x08_P2.54mm_Vertical, symbol Connector_Generic:Conn_01x08
- added Q701: 2N7000, Package_TO_SOT_THT:TO-92_Inline, symbol Transistor_FET:2N7000
- added R701 (x3): 10K, Resistor_THT:R_Axial_DIN0207_L6.3mm_D2.5mm_P7.62mm_Horizontal, symbol Device:R_Small
- added U1002: 74HC86, Package_DIP:DIP-14_W7.62mm_Socket, symbol 74xx:74HC86
- added U1003: 74HC164, Package_DIP:DIP-14_W7.62mm_Socket, symbol jrt-ICs:74LS164
- U1001: footprint Package_DIP:DIP-40_W15.24mm -> Package_DIP:DIP-40_W15.24mm_Socket
Connections:
- net +5V: now also C201.1, C202.1, C203.1, J1001.1 (Pin_1), R701.1, R701.1, U1002.14 (VCC), U1002.2, U1003.1 (A), U1003.14 (VCC)
- net GND: now also C201.2, C202.2, C203.2, J1001.3 (Pin_3), U1002.10, U1002.12, U1002.13, U1002.7 (GND), U1002.9, U1003.7 (GND)
- net ~{RESET}: now also U1003.9 (~{CLR})
- net at U1001.10 (PB0): now also U1003.3 (Qa)
- net at U1001.11 (PB1): now also U1003.4 (Qb)
- net at U1001.12 (PB2): now also U1003.5 (Qc)
- net at U1001.13 (PB3): now also U1003.6 (Qd)
- net at U1001.14 (PB4): now also U1003.10 (Qe)
- net at U1001.15 (PB5): now also U1003.11 (Qf)
- net at U1001.16 (PB6): now also U1003.12 (Qg)
- net at U1001.17 (PB7): now also U1003.13 (Qh)
- net at U1001.18 (CB1): now also U1002.1
- net at U1001.19 (CB2): now also U1002.5
- net SD_MOSI_INV: now reaches U1001.2 (PA0)
- net SD_MOSI_INV: now also U1002.4
- net at U1001.3 (PA1): now also Q701.2 (G), R701.1
- net SD_CD: now reaches U1001.39 (CA2)
- net SD_CD: now also U1001.4 (PA2), J1001.8 (Pin_8), R701.2
- new net: Q701.1 (S), R701.2
- new net SD_CS: J1001.7 (Pin_7), Q701.3 (D), R701.2
- new net SD_MISO: J1001.5 (Pin_5), U1003.2 (B)
- new net SD_MOSI: J1001.6 (Pin_6), U1002.6
- new net SD_SCK: J1001.4 (Pin_4), U1002.3, U1003.8 (CLK)
- no-connect marks 1 -> 10
Other:
- note added: "https://www.adafruit.com/product/254"

Commit message: Checkpoint SD card interface.  Need to add activity LED.
Parts:
- added H1001, H1002, H1003, H1004: MountingHole_Pad, MountingHole:MountingHole_2.2mm_M2_Pad_Via, symbol Mechanical:MountingHole_Pad
Connections:
- net GND: now also H1001.1, H1002.1, H1003.1, H1004.1
Changed lines of the file:
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@@
     (company "Copyright (c) 2022-2023 Jason R. Thorpe. See LICENSE.")
   )
+  (junction (at 196.088 130.048) (diameter 0) (color 0 0 0 0)
+  )
   (junction (at 57.658 176.276) (diameter 0) (color 0 0 0 0)
   )
@@
   (junction (at 109.855 174.625) (diameter 0) (color 0 0 0 0)
   )
+  (junction (at 192.532 116.84) (diameter 0) (color 0 0 0 0)
+  )
   (junction (at 134.62 94.488) (diameter 0) (color 0 0 0 0)
   )
   (junction (at 47.498 176.276) (diameter 0) (color 0 0 0 0)
+  )
+  (junction (at 192.532 123.19) (diameter 0) (color 0 0 0 0)
   )
   (junction (at 136.652 62.738) (diameter 0) (color 0 0 0 0)
@@
     (stroke (width 0) (type default))
   )
+  (wire (pts (xy 192.532 123.19) (xy 196.088 123.19))
+    (stroke (width 0) (type default))
+  )
+  (wire (pts (xy 192.532 116.84) (xy 192.532 123.19))
+    (stroke (width 0) (type default))
+  )
   (wire (pts (xy 86.36 103.378) (xy 103.886 103.378))
     (stroke (width 0) (type default))
@@
     (stroke (width 0) (type default))
   )
+  (wire (pts (xy 192.532 116.84) (xy 196.088 116.84))
+    (stroke (width 0) (type default))
+  )
   (wire (pts (xy 60.198 78.105) (xy 55.245 78.105))
     (stroke (width 0) (type default))
@@
     (stroke (width 0) (type default))
   )
+  (wire (pts (xy 196.088 109.982) (xy 192.532 109.982))
+    (stroke (width 0) (type default))
+  )
   (wire (pts (xy 136.144 99.568) (xy 136.144 142.748))
     (stroke (width 0) (type default))
@@
     (stroke (width 0) (type default))
   )
+  (wire (pts (xy 192.532 130.048) (xy 196.088 130.048))
+    (stroke (width 0) (type default))
+  )
   (wire (pts (xy 119.38 131.318) (xy 119.38 131.445))
     (stroke (width 0) (type default))
@@
     (stroke (width 0) (type default))
   )
+  (wire (pts (xy 192.532 109.982) (xy 192.532 116.84))
+    (stroke (width 0) (type default))
+  )
   (wire (pts (xy 58.928 105.918) (xy 60.96 105.918))
     (stroke (width 0) (type default))
@@
   )
   (wire (pts (xy 59.69 67.818) (xy 60.96 67.818))
+    (stroke (width 0) (type default))
+  )
+  (wire (pts (xy 192.532 123.19) (xy 192.532 130.048))
     (stroke (width 0) (type default))
   )
@@
         (path "/44572023-3621-4b3a-bd53-c3b2b3f42871/a9e9ad98-9eec-45f2-8e38-6db75be52ef6"
           (reference "U1002") (unit 4)
+        )
+      )
+    )
+  )
+  (symbol (lib_id "Mechanical:MountingHole_Pad") (at 196.088 127.508 0) (unit 1)
+    (in_bom yes) (on_board yes) (dnp no)
+    (property "Reference" "H1004" (at 199.39 126.873 0)
+      (effects (font (size 1.27 1.27)) (justify left))
+    )
+    (property "Value" "MountingHole_Pad" (at 208.026 128.778 0)
+      (effects (font (size 1.27 1.27)))
+    )
+    (property "Footprint" "MountingHole:MountingHole_2.2mm_M2_Pad_Via" (at 196.088 127.508 0)
+      (effects (font (size 1.27 1.27)) hide)
+    )
+    (property "Datasheet" "~" (at 196.088 127.508 0)
+      (effects (font (size 1.27 1.27)) hide)
+    )
+    (pin "1")
+    (instances
+      (project "pg09-system"
+        (path "/44572023-3621-4b3a-bd53-c3b2b3f42871/a9e9ad98-9eec-45f2-8e38-6db75be52ef6"
+          (reference "H1004") (unit 1)
         )
       )
@@
     )
   )
+  (symbol (lib_id "Mechanical:MountingHole_Pad") (at 196.088 120.65 0) (unit 1)
+    (in_bom yes) (on_board yes) (dnp no)
+    (property "Reference" "H1003" (at 199.39 120.015 0)
+      (effects (font (size 1.27 1.27)) (justify left))
+    )
+    (property "Value" "MountingHole_Pad" (at 208.026 121.92 0)
+      (effects (font (size 1.27 1.27)))
+    )
+    (property "Footprint" "MountingHole:MountingHole_2.2mm_M2_Pad_Via" (at 196.088 120.65 0)
+      (effects (font (size 1.27 1.27)) hide)
+    )
+    (property "Datasheet" "~" (at 196.088 120.65 0)
+      (effects (font (size 1.27 1.27)) hide)
+    )
+    (pin "1")
+    (instances
+      (project "pg09-system"
+        (path "/44572023-3621-4b3a-bd53-c3b2b3f42871/a9e9ad98-9eec-45f2-8e38-6db75be52ef6"
+          (reference "H1003") (unit 1)
+        )
+      )
+    )
+  )
+  (symbol (lib_id "Mechanical:MountingHole_Pad") (at 196.088 107.442 0) (unit 1)
+    (in_bom yes) (on_board yes) (dnp no)
+    (property "Reference" "H1001" (at 199.39 106.807 0)
+      (effects (font (size 1.27 1.27)) (justify left))
+    )
+    (property "Value" "MountingHole_Pad" (at 208.026 108.712 0)
+      (effects (font (size 1.27 1.27)))
+    )
+    (property "Footprint" "MountingHole:MountingHole_2.2mm_M2_Pad_Via" (at 196.088 107.442 0)
+      (effects (font (size 1.27 1.27)) hide)
+    )
+    (property "Datasheet" "~" (at 196.088 107.442 0)
+      (effects (font (size 1.27 1.27)) hide)
+    )
+    (pin "1")
+    (instances
+      (project "pg09-system"
+        (path "/44572023-3621-4b3a-bd53-c3b2b3f42871/a9e9ad98-9eec-45f2-8e38-6db75be52ef6"
+          (reference "H1001") (unit 1)
+        )
+      )
+    )
+  )
   (symbol (lib_id "power:GND") (at 114.046 118.618 0) (unit 1)
     (in_bom yes) (on_board yes) (dnp no) (fields_autoplaced)
@@
         (path "/44572023-3621-4b3a-bd53-c3b2b3f42871/a9e9ad98-9eec-45f2-8e38-6db75be52ef6"
           (reference "#PWR01015") (unit 1)
+        )
+      )
+    )
+  )
+  (symbol (lib_id "power:GND") (at 196.088 130.048 0) (unit 1)
+    (in_bom yes) (on_board yes) (dnp no) (fields_autoplaced)
+    (property "Reference" "#PWR01017" (at 196.088 136.398 0)
+      (effects (font (size 1.27 1.27)) hide)
+    )
+    (property "Value" "GND" (at 196.088 134.62 0)
+      (effects (font (size 1.27 1.27)))
+    )
+    (property "Footprint" "" (at 196.088 130.048 0)
+      (effects (font (size 1.27 1.27)) hide)
+    )
+    (property "Datasheet" "" (at 196.088 130.048 0)
+      (effects (font (size 1.27 1.27)) hide)
+    )
+    (pin "1")
+    (instances
+      (project "pg09-system"
+        (path "/44572023-3621-4b3a-bd53-c3b2b3f42871/a9e9ad98-9eec-45f2-8e38-6db75be52ef6"
+          (reference "#PWR01017") (unit 1)
         )
       )
@@
         )
       )
+    )
+  )
+  (symbol (lib_id "Mechanical:MountingHole_Pad") (at 196.088 114.3 0) (unit 1)
+    (in_bom yes) (on_board yes) (dnp no)
+    (property "Reference" "H1002" (at 199.39 113.665 0)
+      (effects (font (size 1.27 1.27)) (justify left))
+    )
+    (property "Value" "MountingHole_Pad" (at 208.026 115.57 0)
+      (effects (font (size 1.27 1.27)))
+    )
+    (property "Footprint" "MountingHole:MountingHole_2.2mm_M2_Pad_Via" (at 196.088 114.3 0)
+      (effects (font (size 1.27 1.27)) hide)
+    )
+    (property "Datasheet" "~" (at 196.088 114.3 0)
+      (effects (font (size 1.27 1.27)) hide)
+    )
+    (pin "1")
+    (instances
+      (project "pg09-system"
+        (path "/44572023-3621-4b3a-bd53-c3b2b3f42871/a9e9ad98-9eec-45f2-8e38-6db75be52ef6"
+          (reference "H1002") (unit 1)
+        )
+      )

Commit message: Add SD Card activity LED.
Parts:
- added D1001: SD Card, LED_THT:LED_D3.0mm, symbol Device:LED
- added R701: 1K, Resistor_THT:R_Axial_DIN0207_L6.3mm_D2.5mm_P7.62mm_Horizontal, symbol Device:R_Small
Connections:
- net GND: no longer U1002.10
- net SD_SCK: now also U1002.10
- net SD_LED+: now reaches U1002.8
- net SD_LED+: now also D1001.2 (A)
- net SD_CS renamed SD_LED-
- net SD_LED-: now also R701.2
- new net: D1001.1 (K), R701.1
Other:
- moved on the sheet: U1002C
Changed lines of the file:
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@@
   (junction (at 109.855 188.595) (diameter 0) (color 0 0 0 0)
   )
+  (junction (at 158.242 94.488) (diameter 0) (color 0 0 0 0)
+  )
+  (junction (at 193.802 62.738) (diameter 0) (color 0 0 0 0)
+  )
+  (junction (at 193.802 78.994) (diameter 0) (color 0 0 0 0)
+  )
   (junction (at 121.92 65.278) (diameter 0) (color 0 0 0 0)
   )
+  (junction (at 159.766 102.108) (diameter 0) (color 0 0 0 0)
+  )
   (junction (at 90.17 60.325) (diameter 0) (color 0 0 0 0)
   )
@@
   )
   (junction (at 47.498 181.356) (diameter 0) (color 0 0 0 0)
-  )
-  (junction (at 109.855 174.625) (diameter 0) (color 0 0 0 0)
   )
   (junction (at 192.532 116.84) (diameter 0) (color 0 0 0 0)
@@
     (stroke (width 0) (type default))
   )
-  (wire (pts (xy 109.855 169.545) (xy 109.855 174.625))
+  (wire (pts (xy 109.855 169.545) (xy 109.855 183.515))
+    (stroke (width 0) (type default))
+  )
+  (wire (pts (xy 190.5 62.738) (xy 193.802 62.738))
     (stroke (width 0) (type default))
   )
@@
     (stroke (width 0) (type default))
   )
+  (wire (pts (xy 193.802 71.882) (xy 193.802 70.358))
+    (stroke (width 0) (type default))
+  )
   (wire (pts (xy 86.36 103.378) (xy 103.886 103.378))
     (stroke (width 0) (type default))
@@
     (stroke (width 0) (type default))
   )
+  (wire (pts (xy 159.766 102.108) (xy 180.34 102.108))
+    (stroke (width 0) (type default))
+  )
   (wire (pts (xy 86.36 88.138) (xy 103.886 88.138))
     (stroke (width 0) (type default))
@@
     (stroke (width 0) (type default))
   )
+  (wire (pts (xy 193.802 78.994) (xy 159.766 78.994))
+    (stroke (width 0) (type default))
+  )
   (wire (pts (xy 134.62 128.778) (xy 134.62 94.488))
     (stroke (width 0) (type default))
@@
     (stroke (width 0) (type default))
   )
+  (wire (pts (xy 158.242 94.488) (xy 158.242 65.278))
+    (stroke (width 0) (type default))
+  )
   (wire (pts (xy 60.96 65.278) (xy 60.96 65.405))
     (stroke (width 0) (type default))
   )
+  (wire (pts (xy 159.766 78.994) (xy 159.766 102.108))
+    (stroke (width 0) (type default))
+  )
   (wire (pts (xy 86.36 65.278) (xy 98.044 65.278))
     (stroke (width 0) (type default))
   )
+  (wire (pts (xy 158.242 65.278) (xy 175.26 65.278))
+    (stroke (width 0) (type default))
+  )
   (wire (pts (xy 60.452 85.598) (xy 60.452 85.725))
     (stroke (width 0) (type default))
@@
     (stroke (width 0) (type default))
   )
+  (wire (pts (xy 158.242 94.488) (xy 180.34 94.488))
+    (stroke (width 0) (type default))
+  )
   (wire (pts (xy 90.17 60.325) (xy 90.17 140.208))
     (stroke (width 0) (type default))
@@
     (stroke (width 0) (type default))
   )
+  (wire (pts (xy 193.802 78.994) (xy 197.358 78.994))
+    (stroke (width 0) (type default))
+  )
   (wire (pts (xy 119.38 131.318) (xy 119.38 131.445))
     (stroke (width 0) (type default))
   )
-  (wire (pts (xy 156.464 102.108) (xy 180.34 102.108))
+  (wire (pts (xy 156.464 102.108) (xy 159.766 102.108))
     (stroke (width 0) (type default))
   )
@@
     (stroke (width 0) (type default))
   )
+  (wire (pts (xy 193.802 78.994) (xy 193.802 76.962))
+    (stroke (width 0) (type default))
+  )
   (wire (pts (xy 90.17 60.198) (xy 90.17 60.325))
     (stroke (width 0) (type default))
@@
     (stroke (width 0) (type default))
   )
-  (wire (pts (xy 134.62 94.488) (xy 180.34 94.488))
+  (wire (pts (xy 134.62 94.488) (xy 158.242 94.488))
     (stroke (width 0) (type default))
   )
@@
     (stroke (width 0) (type default))
   )
-  (wire (pts (xy 109.855 174.625) (xy 109.855 183.515))
-    (stroke (width 0) (type default))
-  )
   (wire (pts (xy 59.182 110.998) (xy 60.96 110.998))
     (stroke (width 0) (type default))
@@
   )
   (wire (pts (xy 60.706 93.345) (xy 52.07 93.345))
+    (stroke (width 0) (type default))
+  )
+  (wire (pts (xy 193.802 62.738) (xy 197.104 62.738))
     (stroke (width 0) (type default))
   )
@@
     )
   )
+  (global_label "SD_LED-" (shape input) (at 197.358 78.994 0) (fields_autoplaced)
+    (effects (font (size 1.27 1.27)) (justify left))
+    (property "Intersheetrefs" "${INTERSHEET_REFS}" (at 208.7304 78.994 0)
+      (effects (font (size 1.27 1.27)) (justify left) hide)
+    )
+  )
   (global_label "D0" (shape bidirectional) (at 60.96 60.325 180) (fields_autoplaced)
     (effects (font (size 1.27 1.27)) (justify right))
@@
     )
   )
+  (global_label "SD_LED+" (shape input) (at 197.104 62.738 0) (fields_autoplaced)
+    (effects (font (size 1.27 1.27)) (justify left))
+    (property "Intersheetrefs" "${INTERSHEET_REFS}" (at 208.4764 62.738 0)
+      (effects (font (size 1.27 1.27)) (justify left) hide)
+    )
+  )
   (global_label "A2" (shape input) (at 60.96 108.585 180) (fields_autoplaced)
     (effects (font (size 1.27 1.27)) (justify right))
@@
     )
   )
-  (symbol (lib_id "74xx:74HC86") (at 117.475 172.085 0) (unit 3)
-    (in_bom yes) (on_board yes) (dnp no) (fields_autoplaced)
-    (property "Reference" "U1002" (at 117.1702 163.83 0)
-      (effects (font (size 1.27 1.27)))
-    )
-    (property "Value" "74HC86" (at 117.1702 166.37 0)
-      (effects (font (size 1.27 1.27)))
-    )
-    (property "Footprint" "Package_DIP:DIP-14_W7.62mm_Socket" (at 117.475 172.085 0)
-      (effects (font (size 1.27 1.27)) hide)
-    )
-    (property "Datasheet" "http://www.ti.com/lit/gpn/sn74HC86" (at 117.475 172.085 0)
+  (symbol (lib_id "74xx:74HC86") (at 182.88 62.738 0) (unit 3)
+    (in_bom yes) (on_board yes) (dnp no) (fields_autoplaced)
+    (property "Reference" "U1002" (at 182.5752 54.483 0)
+      (effects (font (size 1.27 1.27)))
+    )
+    (property "Value" "74HC86" (at 182.5752 57.023 0)
+      (effects (font (size 1.27 1.27)))
+    )
+    (property "Footprint" "Package_DIP:DIP-14_W7.62mm_Socket" (at 182.88 62.738 0)
+      (effects (font (size 1.27 1.27)) hide)
+    )
+    (property "Datasheet" "http://www.ti.com/lit/gpn/sn74HC86" (at 182.88 62.738 0)
       (effects (font (size 1.27 1.27)) hide)
     )
@@
     )
   )
+  (symbol (lib_id "power:GND") (at 175.26 60.198 270) (unit 1)
+    (in_bom yes) (on_board yes) (dnp no) (fields_autoplaced)
+    (property "Reference" "#PWR01018" (at 168.91 60.198 0)
+      (effects (font (size 1.27 1.27)) hide)
+    )
+    (property "Value" "GND" (at 171.45 60.833 90)
+      (effects (font (size 1.27 1.27)) (justify right))
+    )
+    (property "Footprint" "" (at 175.26 60.198 0)
+      (effects (font (size 1.27 1.27)) hide)
+    )
+    (property "Datasheet" "" (at 175.26 60.198 0)
+      (effects (font (size 1.27 1.27)) hide)
+    )
+    (pin "1")
+    (instances
+      (project "pg09-system"
+        (path "/44572023-3621-4b3a-bd53-c3b2b3f42871/a9e9ad98-9eec-45f2-8e38-6db75be52ef6"
+          (reference "#PWR01018") (unit 1)
+        )
+      )
+    )
+  )
+  (symbol (lib_id "Device:LED") (at 193.802 66.548 90) (unit 1)
+    (in_bom yes) (on_board yes) (dnp no) (fields_autoplaced)
+    (property "Reference" "D1001" (at 196.85 67.5005 90)
+      (effects (font (size 1.27 1.27)) (justify right))
+    )
+    (property "Value" "SD Card" (at 196.85 70.0405 90)
+      (effects (font (size 1.27 1.27)) (justify right))
+    )
+    (property "Footprint" "LED_THT:LED_D3.0mm" (at 193.802 66.548 0)
+      (effects (font (size 1.27 1.27)) hide)
+    )
+    (property "Datasheet" "~" (at 193.802 66.548 0)
+      (effects (font (size 1.27 1.27)) hide)
+    )
+    (pin "1")
+    (pin "2")
+    (instances
+      (project "pg09-system"
+        (path "/44572023-3621-4b3a-bd53-c3b2b3f42871/a9e9ad98-9eec-45f2-8e38-6db75be52ef6"
+          (reference "D1001") (unit 1)
+        )
+      )
+    )
+  )
   (symbol (lib_id "jrt-ICs:74LS164") (at 114.046 97.028 0) (mirror y) (unit 1)
     (in_bom yes) (on_board yes) (dnp no)
@@
         )
       )
+    )
+  )
+  (symbol (lib_id "Device:R_Small") (at 193.802 74.422 0) (mirror y) (unit 1)
+    (in_bom yes) (on_board yes) (dnp no) (fields_autoplaced)
+    (property "Reference" "R701" (at 195.58 73.787 0)
+      (effects (font (size 1.27 1.27)) (justify right))
+    )
+    (property "Value" "1K" (at 195.58 76.327 0)
+      (effects (font (size 1.27 1.27)) (justify right))
+    )
+    (property "Footprint" "Resistor_THT:R_Axial_DIN0207_L6.3mm_D2.5mm_P7.62mm_Horizontal" (at 193.802 74.422 0)
+      (effects (font (size 1.27 1.27)) hide)
+    )
+    (property "Datasheet" "~" (at 193.802 74.422 0)
+      (effects (font (size 1.27 1.27)) hide)
+    )
+    (pin "1")
+    (pin "2")
+    (instances
+      (project "pg09-system"
+        (path "/44572023-3621-4b3a-bd53-c3b2b3f42871/ac00d1d6-4857-42f9-90e1-ab396f3828b3"
+          (reference "R701") (unit 1)
+        )
+        (path "/44572023-3621-4b3a-bd53-c3b2b3f42871/a9e9ad98-9eec-45f2-8e38-6db75be52ef6"
+          (reference "R1004") (unit 1)
+        )
+      )
