File: design-files/pg09-system-spi-sdcard.kicad_sch (KiCad schematic)
At the start: 17 parts, among them J1001 Adafruit MicroSD Card Breakou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, Q701 2N7000, U1001 W65C22, U1002 74HC86, U1003 74HC164

Commit message: Give the front panel LED its own current-limiting resistor.
Parts:
- added R701: 1K, Resistor_THT:R_Axial_DIN0207_L6.3mm_D2.5mm_P7.62mm_Horizontal, symbol Device:R_Small
Connections:
- net SD_LED-: now also R701.2; no longer J1001.7 (Pin_7), Q701.3 (D), R701.2, R701.2
- net at D1001.1 (K): now also R701.2; no longer R701.1
- new net SD_CS: J1001.7 (Pin_7), Q701.3 (D), R701.1, R701.1, R701.2
Other:
- moved on the sheet: D1001, R701
Changed lines of the file:
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@@
   (junction (at 158.242 94.488) (diameter 0) (color 0 0 0 0)
   )
+  (junction (at 184.15 75.184) (diameter 0) (color 0 0 0 0)
+  )
   (junction (at 193.802 62.738) (diameter 0) (color 0 0 0 0)
-  )
-  (junction (at 193.802 78.994) (diameter 0) (color 0 0 0 0)
   )
   (junction (at 121.92 65.278) (diameter 0) (color 0 0 0 0)
@@
     (stroke (width 0) (type default))
   )
+  (wire (pts (xy 197.358 81.28) (xy 197.358 75.184))
+    (stroke (width 0) (type default))
+  )
   (wire (pts (xy 192.532 116.84) (xy 192.532 123.19))
     (stroke (width 0) (type default))
   )
-  (wire (pts (xy 193.802 71.882) (xy 193.802 70.358))
+  (wire (pts (xy 193.802 71.628) (xy 193.802 75.184))
     (stroke (width 0) (type default))
   )
@@
     (stroke (width 0) (type default))
   )
+  (wire (pts (xy 184.15 75.184) (xy 159.766 75.184))
+    (stroke (width 0) (type default))
+  )
   (wire (pts (xy 159.766 102.108) (xy 180.34 102.108))
     (stroke (width 0) (type default))
@@
     (stroke (width 0) (type default))
   )
-  (wire (pts (xy 193.802 78.994) (xy 159.766 78.994))
-    (stroke (width 0) (type default))
-  )
   (wire (pts (xy 134.62 128.778) (xy 134.62 94.488))
     (stroke (width 0) (type default))
   )
+  (wire (pts (xy 191.77 75.184) (xy 193.802 75.184))
+    (stroke (width 0) (type default))
+  )
   (wire (pts (xy 192.532 116.84) (xy 196.088 116.84))
     (stroke (width 0) (type default))
@@
     (stroke (width 0) (type default))
   )
-  (wire (pts (xy 159.766 78.994) (xy 159.766 102.108))
+  (wire (pts (xy 159.766 75.184) (xy 159.766 102.108))
     (stroke (width 0) (type default))
   )
@@
     (stroke (width 0) (type default))
   )
+  (wire (pts (xy 193.802 64.008) (xy 193.802 62.738))
+    (stroke (width 0) (type default))
+  )
+  (wire (pts (xy 191.77 81.28) (xy 197.358 81.28))
+    (stroke (width 0) (type default))
+  )
   (wire (pts (xy 192.532 130.048) (xy 196.088 130.048))
     (stroke (width 0) (type default))
   )
-  (wire (pts (xy 193.802 78.994) (xy 197.358 78.994))
-    (stroke (width 0) (type default))
-  )
   (wire (pts (xy 119.38 131.318) (xy 119.38 131.445))
     (stroke (width 0) (type default))
@@
     (stroke (width 0) (type default))
   )
+  (wire (pts (xy 186.69 81.28) (xy 184.15 81.28))
+    (stroke (width 0) (type default))
+  )
   (wire (pts (xy 88.265 108.458) (xy 86.36 108.458))
     (stroke (width 0) (type default))
   )
-  (wire (pts (xy 193.802 78.994) (xy 193.802 76.962))
-    (stroke (width 0) (type default))
-  )
   (wire (pts (xy 90.17 60.198) (xy 90.17 60.325))
     (stroke (width 0) (type default))
@@
     (stroke (width 0) (type default))
   )
+  (wire (pts (xy 186.69 75.184) (xy 184.15 75.184))
+    (stroke (width 0) (type default))
+  )
   (wire (pts (xy 86.36 105.918) (xy 103.886 105.918))
     (stroke (width 0) (type default))
@@
   )
   (wire (pts (xy 86.36 100.838) (xy 103.886 100.838))
+    (stroke (width 0) (type default))
+  )
+  (wire (pts (xy 184.15 81.28) (xy 184.15 75.184))
     (stroke (width 0) (type default))
   )
@@
     )
   )
-  (global_label "SD_LED-" (shape input) (at 197.358 78.994 0) (fields_autoplaced)
+  (global_label "SD_LED-" (shape input) (at 197.358 75.184 0) (fields_autoplaced)
     (effects (font (size 1.27 1.27)) (justify left))
-    (property "Intersheetrefs" "${INTERSHEET_REFS}" (at 208.7304 78.994 0)
+    (property "Intersheetrefs" "${INTERSHEET_REFS}" (at 208.7304 75.184 0)
       (effects (font (size 1.27 1.27)) (justify left) hide)
     )
@@
     )
   )
-  (symbol (lib_id "Device:LED") (at 193.802 66.548 90) (unit 1)
-    (in_bom yes) (on_board yes) (dnp no) (fields_autoplaced)
-    (property "Reference" "D1001" (at 196.85 67.5005 90)
+  (symbol (lib_id "Device:LED") (at 193.802 67.818 90) (unit 1)
+    (in_bom yes) (on_board yes) (dnp no) (fields_autoplaced)
+    (property "Reference" "D1001" (at 196.85 68.7705 90)
       (effects (font (size 1.27 1.27)) (justify right))
     )
-    (property "Value" "SD Card" (at 196.85 70.0405 90)
+    (property "Value" "SD Card" (at 196.85 71.3105 90)
       (effects (font (size 1.27 1.27)) (justify right))
     )
-    (property "Footprint" "LED_THT:LED_D3.0mm" (at 193.802 66.548 0)
-      (effects (font (size 1.27 1.27)) hide)
-    )
-    (property "Datasheet" "~" (at 193.802 66.548 0)
+    (property "Footprint" "LED_THT:LED_D3.0mm" (at 193.802 67.818 0)
+      (effects (font (size 1.27 1.27)) hide)
+    )
+    (property "Datasheet" "~" (at 193.802 67.818 0)
       (effects (font (size 1.27 1.27)) hide)
     )
@@
     )
   )
-  (symbol (lib_id "Device:R_Small") (at 193.802 74.422 0) (mirror y) (unit 1)
-    (in_bom yes) (on_board yes) (dnp no) (fields_autoplaced)
-    (property "Reference" "R701" (at 195.58 73.787 0)
-      (effects (font (size 1.27 1.27)) (justify right))
-    )
-    (property "Value" "1K" (at 195.58 76.327 0)
-      (effects (font (size 1.27 1.27)) (justify right))
-    )
-    (property "Footprint" "Resistor_THT:R_Axial_DIN0207_L6.3mm_D2.5mm_P7.62mm_Horizontal" (at 193.802 74.422 0)
-      (effects (font (size 1.27 1.27)) hide)
-    )
-    (property "Datasheet" "~" (at 193.802 74.422 0)
+  (symbol (lib_id "Device:R_Small") (at 189.23 75.184 90) (mirror x) (unit 1)
+    (in_bom yes) (on_board yes) (dnp no) (fields_autoplaced)
+    (property "Reference" "R701" (at 189.23 70.866 90)
+      (effects (font (size 1.27 1.27)))
+    )
+    (property "Value" "1K" (at 189.23 73.406 90)
+      (effects (font (size 1.27 1.27)))
+    )
+    (property "Footprint" "Resistor_THT:R_Axial_DIN0207_L6.3mm_D2.5mm_P7.62mm_Horizontal" (at 189.23 75.184 0)
+      (effects (font (size 1.27 1.27)) hide)
+    )
+    (property "Datasheet" "~" (at 189.23 75.184 0)
       (effects (font (size 1.27 1.27)) hide)
     )
@@
         )
       )
+    )
+  )
+  (symbol (lib_id "Device:R_Small") (at 189.23 81.28 90) (mirror x) (unit 1)
+    (in_bom yes) (on_board yes) (dnp no) (fields_autoplaced)
+    (property "Reference" "R701" (at 189.23 76.962 90)
+      (effects (font (size 1.27 1.27)))
+    )
+    (property "Value" "1K" (at 189.23 79.502 90)
+      (effects (font (size 1.27 1.27)))
+    )
+    (property "Footprint" "Resistor_THT:R_Axial_DIN0207_L6.3mm_D2.5mm_P7.62mm_Horizontal" (at 189.23 81.28 0)
+      (effects (font (size 1.27 1.27)) hide)
+    )
+    (property "Datasheet" "~" (at 189.23 81.28 0)
+      (effects (font (size 1.27 1.27)) hide)
+    )
+    (pin "1")
+    (pin "2")
+    (instances
+      (project "pg09-system"
+        (path "/44572023-3621-4b3a-bd53-c3b2b3f42871/ac00d1d6-4857-42f9-90e1-ab396f3828b3"
+          (reference "R701") (unit 1)
+        )
+        (path "/44572023-3621-4b3a-bd53-c3b2b3f42871/a9e9ad98-9eec-45f2-8e38-6db75be52ef6"
+          (reference "R1005") (unit 1)
+        )
+      )
