File: design-files/pg09-system-spi-sdcard.kicad_sch (KiCad schematic)
At the start: 18 parts, among them J1001 Adafruit MicroSD Card Breakou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, Q701 2N7000, U1001 W65C22, U1002 74HC86, U1003 74HC164

Commit message: Use a 74AHC05 hex inverter with open-drain outputs rather than discrete small-signal MOSFETs.  Share the gates and resistors between UART and SD SPI sheets.
Parts:
- removed Q701: 2N7000, Package_TO_SOT_THT:TO-92_Inline, symbol Transistor_FET:2N7000
- removed R701 (x3): 10K, Resistor_THT:R_Axial_DIN0207_L6.3mm_D2.5mm_P7.62mm_Horizontal, symbol Device:R_Small
- added RN701 (x2): 10K, Resistor_THT:R_Array_SIP9, symbol Device:R_Network08_Split
- added U703: 74AHC05, Package_DIP:DIP-14_W7.62mm_Socket, symbol 74xx:74LS05
Connections:
- net +5V: now also RN701.1 (R1), RN701.1 (R1)
- net SD_CD: now also RN701.5 (R4.2)
- net SD_CS: now also RN701.5 (R4.2), U703.8
- net at U1001.3 (PA1): now also U703.9
Other:
- note added: "Spare gates and resistors from UART sheet."
