File: design-files/pg09-system-spi-sdcard.kicad_sch (KiCad schematic)
At the start: 17 parts, among them J1001 Adafruit MicroSD Card Breakou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, U1001 W65C22, U1002 74HC86, U1003 74HC164, U703 74AHC05

Commit message: Eliminate the resistor network on the UART sheet -- it's no longer needed to pull up the IRQ lines (interrupt controller sheet does that).  Just let the SPI sheet use its own discreet resistors.
Parts:
- removed RN701 (x2): 10K, Resistor_THT:R_Array_SIP9, symbol Device:R_Network08_Split
- added R101 (x2): 10K, Resistor_THT:R_Axial_DIN0207_L6.3mm_D2.5mm_P7.62mm_Horizontal, symbol Device:R_Small
Connections:
- net +5V: now also R101.2, R101.2
- net SD_CD: now also R101.1
- net SD_CS: now also R101.1
Changed lines of the file:
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@@
     )
   )
-  (symbol (lib_id "power:+5V") (at 156.464 53.213 0) (unit 1)
-    (in_bom yes) (on_board yes) (dnp no) (fields_autoplaced)
-    (property "Reference" "#PWR01013" (at 156.464 57.023 0)
-      (effects (font (size 1.27 1.27)) hide)
-    )
-    (property "Value" "+5V" (at 156.464 48.895 0)
-      (effects (font (size 1.27 1.27)))
-    )
-    (property "Footprint" "" (at 156.464 53.213 0)
-      (effects (font (size 1.27 1.27)) hide)
-    )
-    (property "Datasheet" "" (at 156.464 53.213 0)
+  (symbol (lib_id "power:+5V") (at 156.464 55.753 0) (unit 1)
+    (in_bom yes) (on_board yes) (dnp no) (fields_autoplaced)
+    (property "Reference" "#PWR01013" (at 156.464 59.563 0)
+      (effects (font (size 1.27 1.27)) hide)
+    )
+    (property "Value" "+5V" (at 156.464 51.435 0)
+      (effects (font (size 1.27 1.27)))
+    )
+    (property "Footprint" "" (at 156.464 55.753 0)
+      (effects (font (size 1.27 1.27)) hide)
+    )
+    (property "Datasheet" "" (at 156.464 55.753 0)
       (effects (font (size 1.27 1.27)) hide)
     )
@@
     )
   )
-  (symbol (lib_id "Device:R_Network08_Split") (at 156.464 57.023 0) (unit 4)
-    (in_bom yes) (on_board yes) (dnp no) (fields_autoplaced)
-    (property "Reference" "RN701" (at 158.369 56.388 0)
-      (effects (font (size 1.27 1.27)) (justify left))
-    )
-    (property "Value" "10K" (at 158.369 58.928 0)
-      (effects (font (size 1.27 1.27)) (justify left))
-    )
-    (property "Footprint" "Resistor_THT:R_Array_SIP9" (at 154.432 57.023 90)
-      (effects (font (size 1.27 1.27)) hide)
-    )
-    (property "Datasheet" "http://www.vishay.com/docs/31509/csc.pdf" (at 156.464 57.023 0)
-      (effects (font (size 1.27 1.27)) hide)
-    )
-    (pin "1")
-    (pin "2")
-    (pin "3")
-    (pin "4")
-    (pin "5")
-    (pin "6")
-    (pin "7")
-    (pin "8")
-    (pin "9")
-    (instances
-      (project "pg09-system"
-        (path "/44572023-3621-4b3a-bd53-c3b2b3f42871/ac00d1d6-4857-42f9-90e1-ab396f3828b3"
-          (reference "RN701") (unit 4)
-        )
-        (path "/44572023-3621-4b3a-bd53-c3b2b3f42871/a9e9ad98-9eec-45f2-8e38-6db75be52ef6"
-          (reference "RN701") (unit 4)
-        )
-      )
-    )
-  )
   (symbol (lib_id "Mechanical:MountingHole_Pad") (at 196.088 107.442 0) (unit 1)
     (in_bom yes) (on_board yes) (dnp no)
@@
     )
   )
+  (symbol (lib_id "Device:R_Small") (at 121.92 55.118 180) (unit 1)
+    (in_bom yes) (on_board yes) (dnp no) (fields_autoplaced)
+    (property "Reference" "R101" (at 124.079 54.483 0)
+      (effects (font (size 1.27 1.27)) (justify right))
+    )
+    (property "Value" "10K" (at 124.079 57.023 0)
+      (effects (font (size 1.27 1.27)) (justify right))
+    )
+    (property "Footprint" "Resistor_THT:R_Axial_DIN0207_L6.3mm_D2.5mm_P7.62mm_Horizontal" (at 121.92 55.118 0)
+      (effects (font (size 1.27 1.27)) hide)
+    )
+    (property "Datasheet" "~" (at 121.92 55.118 0)
+      (effects (font (size 1.27 1.27)) hide)
+    )
+    (pin "1")
+    (pin "2")
+    (instances
+      (project "pg09-system"
+        (path "/44572023-3621-4b3a-bd53-c3b2b3f42871"
+          (reference "R101") (unit 1)
+        )
+        (path "/44572023-3621-4b3a-bd53-c3b2b3f42871/a9e9ad98-9eec-45f2-8e38-6db75be52ef6"
+          (reference "R1001") (unit 1)
+        )
+      )
+    )
+  )
   (symbol (lib_id "power:GND") (at 114.046 118.618 0) (unit 1)
     (in_bom yes) (on_board yes) (dnp no) (fields_autoplaced)
@@
         (path "/44572023-3621-4b3a-bd53-c3b2b3f42871/a9e9ad98-9eec-45f2-8e38-6db75be52ef6"
           (reference "#PWR01015") (unit 1)
-        )
-      )
-    )
-  )
-  (symbol (lib_id "Device:R_Network08_Split") (at 121.92 53.848 0) (unit 4)
-    (in_bom yes) (on_board yes) (dnp no) (fields_autoplaced)
-    (property "Reference" "RN701" (at 123.825 53.213 0)
-      (effects (font (size 1.27 1.27)) (justify left))
-    )
-    (property "Value" "10K" (at 123.825 55.753 0)
-      (effects (font (size 1.27 1.27)) (justify left))
-    )
-    (property "Footprint" "Resistor_THT:R_Array_SIP9" (at 119.888 53.848 90)
-      (effects (font (size 1.27 1.27)) hide)
-    )
-    (property "Datasheet" "http://www.vishay.com/docs/31509/csc.pdf" (at 121.92 53.848 0)
-      (effects (font (size 1.27 1.27)) hide)
-    )
-    (pin "1")
-    (pin "2")
-    (pin "3")
-    (pin "4")
-    (pin "5")
-    (pin "6")
-    (pin "7")
-    (pin "8")
-    (pin "9")
-    (instances
-      (project "pg09-system"
-        (path "/44572023-3621-4b3a-bd53-c3b2b3f42871/ac00d1d6-4857-42f9-90e1-ab396f3828b3"
-          (reference "RN701") (unit 4)
-        )
-        (path "/44572023-3621-4b3a-bd53-c3b2b3f42871/a9e9ad98-9eec-45f2-8e38-6db75be52ef6"
-          (reference "RN701") (unit 3)
         )
       )
@@
     )
   )
-  (symbol (lib_id "power:+5V") (at 121.92 50.038 0) (unit 1)
-    (in_bom yes) (on_board yes) (dnp no) (fields_autoplaced)
-    (property "Reference" "#PWR01014" (at 121.92 53.848 0)
-      (effects (font (size 1.27 1.27)) hide)
-    )
-    (property "Value" "+5V" (at 121.92 45.72 0)
-      (effects (font (size 1.27 1.27)))
-    )
-    (property "Footprint" "" (at 121.92 50.038 0)
-      (effects (font (size 1.27 1.27)) hide)
-    )
-    (property "Datasheet" "" (at 121.92 50.038 0)
+  (symbol (lib_id "power:+5V") (at 121.92 52.578 0) (unit 1)
+    (in_bom yes) (on_board yes) (dnp no) (fields_autoplaced)
+    (property "Reference" "#PWR01014" (at 121.92 56.388 0)
+      (effects (font (size 1.27 1.27)) hide)
+    )
+    (property "Value" "+5V" (at 121.92 48.26 0)
+      (effects (font (size 1.27 1.27)))
+    )
+    (property "Footprint" "" (at 121.92 52.578 0)
+      (effects (font (size 1.27 1.27)) hide)
+    )
+    (property "Datasheet" "" (at 121.92 52.578 0)
       (effects (font (size 1.27 1.27)) hide)
     )
@@
         )
       )
+    )
+  )
+  (symbol (lib_id "Device:R_Small") (at 156.464 58.293 180) (unit 1)
+    (in_bom yes) (on_board yes) (dnp no) (fields_autoplaced)
+    (property "Reference" "R101" (at 158.623 57.658 0)
+      (effects (font (size 1.27 1.27)) (justify right))
+    )
+    (property "Value" "10K" (at 158.623 60.198 0)
+      (effects (font (size 1.27 1.27)) (justify right))
+    )
+    (property "Footprint" "Resistor_THT:R_Axial_DIN0207_L6.3mm_D2.5mm_P7.62mm_Horizontal" (at 156.464 58.293 0)
+      (effects (font (size 1.27 1.27)) hide)
+    )
+    (property "Datasheet" "~" (at 156.464 58.293 0)
+      (effects (font (size 1.27 1.27)) hide)
+    )
+    (pin "1")
+    (pin "2")
+    (instances
+      (project "pg09-system"
+        (path "/44572023-3621-4b3a-bd53-c3b2b3f42871"
+          (reference "R101") (unit 1)
+        )
+        (path "/44572023-3621-4b3a-bd53-c3b2b3f42871/a9e9ad98-9eec-45f2-8e38-6db75be52ef6"
+          (reference "R1002") (unit 1)
+        )
+      )

Commit message: Move the 74AHC05 from the UART sheet to the INTC sheet.
Other:
- note added: "Spare gate from INTC sheet."
- note removed: "Spare gates and resistors from UART sheet."
Changed lines of the file:
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@@
     (effects (font (size 1.27 1.27)) (justify left bottom))
   )
-  (text "Spare gates and resistors from UART sheet." (at 124.968 46.355 0)
+  (text "Spare gate from INTC sheet." (at 130.937 47.752 0)
     (effects (font (size 1.27 1.27) italic) (justify left bottom))
   )
@@
         )
         (path "/44572023-3621-4b3a-bd53-c3b2b3f42871/a9e9ad98-9eec-45f2-8e38-6db75be52ef6"
-          (reference "U703") (unit 3)
+          (reference "U415") (unit 3)
         )
       )

Commit message: Change the PIA / VIA chips to S-variants.  Requires a diode on the IRQ line, since they have totem-pole outputs.
Parts:
- added D101: 1N4148, Diode_THT:D_DO-35_SOD27_P7.62mm_Horizontal, symbol Diode:1N4148
- U1001: value W65C22 -> W65C22S
Connections:
- net ~{IRQ0}: now also D101.2 (A); no longer U1001.21 (~{IRQ})
- new net: D101.1 (K), U1001.21 (~{IRQ})
Changed lines of the file:
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@@
     )
   )
-  (global_label "~{IRQ0}" (shape output) (at 60.96 118.618 180) (fields_autoplaced)
-    (effects (font (size 1.27 1.27)) (justify right))
-    (property "Intersheetrefs" "${INTERSHEET_REFS}" (at 53.6394 118.618 0)
+  (global_label "~{IRQ0}" (shape output) (at 53.34 118.618 180) (fields_autoplaced)
+    (effects (font (size 1.27 1.27)) (justify right))
+    (property "Intersheetrefs" "${INTERSHEET_REFS}" (at 46.0194 118.618 0)
       (effects (font (size 1.27 1.27)) (justify right) hide)
     )
@@
   (symbol (lib_id "jrt-ICs:W65C22") (at 73.66 89.408 0) (unit 1)
     (in_bom yes) (on_board yes) (dnp no) (fields_autoplaced)
-    (property "Reference" "U1001" (at 75.6159 53.213 0)
-      (effects (font (size 1.27 1.27)) (justify left))
-    )
-    (property "Value" "W65C22" (at 75.6159 55.753 0)
+    (property "Reference" "U1001" (at 75.6159 53.34 0)
+      (effects (font (size 1.27 1.27)) (justify left))
+    )
+    (property "Value" "W65C22S" (at 75.6159 55.88 0)
       (effects (font (size 1.27 1.27)) (justify left))
     )
@@
         )
       )
+    )
+  )
+  (symbol (lib_id "Diode:1N4148") (at 57.15 118.618 180) (unit 1)
+    (in_bom yes) (on_board yes) (dnp no)
+    (property "Reference" "D101" (at 60.325 121.539 0)
+      (effects (font (size 1.27 1.27)) (justify left))
+    )
+    (property "Value" "1N4148" (at 57.15 123.571 0)
+      (effects (font (size 1.27 1.27)))
+    )
+    (property "Footprint" "Diode_THT:D_DO-35_SOD27_P7.62mm_Horizontal" (at 57.15 118.618 0)
+      (effects (font (size 1.27 1.27)) hide)
+    )
+    (property "Datasheet" "https://assets.nexperia.com/documents/data-sheet/1N4148_1N4448.pdf" (at 57.15 118.618 0)
+      (effects (font (size 1.27 1.27)) hide)
+    )
+    (property "Sim.Device" "D" (at 57.15 118.618 0)
+      (effects (font (size 1.27 1.27)) hide)
+    )
+    (property "Sim.Pins" "1=K 2=A" (at 57.15 118.618 0)
+      (effects (font (size 1.27 1.27)) hide)
+    )
+    (pin "1")
+    (pin "2")
+    (instances
+      (project "pg09-system"
+        (path "/44572023-3621-4b3a-bd53-c3b2b3f42871"
+          (reference "D101") (unit 1)
+        )
+        (path "/44572023-3621-4b3a-bd53-c3b2b3f42871/a9e9ad98-9eec-45f2-8e38-6db75be52ef6"
+          (reference "D1002") (unit 1)
+        )
+      )
