File: design-files/pg09-system-psu.kicad_sch (KiCad schematic)
At the start: 3 parts, among them J1 ATX-24, J802 Power Switch

Commit message: Add an Adafruit Metro Mini to act as a PSU controller.
Parts:
- added J803: PSU-CTRL console, Connector_PinHeader_2.54mm:PinHeader_1x03_P2.54mm_Vertical, symbol Connector:Conn_01x03_Pin
- added SW201: SW_Push, Button_Switch_THT:SW_PUSH_6mm, symbol Switch:SW_Push
- added U801: Adafruit_Metro_Mini, Package_DIP:DIP-28_W15.24mm_Socket, symbol jrt-Arduino:Adafruit_Metro_Mini
- J802: value Power Switch -> #PS_ON
Connections:
- net GND: now also J803.3 (Pin_3), SW201.2, U801.5 (GND), U801.6 (GND)
- net at J1.16 (PS_ON#), J802.1 (Pin_1): now also U801.23 (D8)
- net at J1.9 (+5VSB): now also U801.4 (5V)
- new net: J803.1 (Pin_1), U801.16 (D1)
- new net: J803.2 (Pin_2), U801.15 (D0)
- new net: SW201.1, U801.17 (D2)
- new net PSU_CTRL_D0: U801.19 (D4)
- new net PSU_CTRL_D1: U801.20 (D5)
- new net ~{PSU_CTRL_WR}: U801.18 (D3)
- new net ~{RESET}: U801.27 (D12)
- no-connect marks 5 -> 21
Other:
- note added: "GND"
- note added: "Rx"
- note added: "Tx"
- moved on the sheet: C801, J1, J802

Commit message: Add +12v / -12v rails for the expansion interface.
Connections:
- net +12V: now reaches J1.10 (+12V), J1.11 (+12V)
- net -12V: now reaches J1.14 (-12V)
- no-connect marks 21 -> 19
Changed lines of the file:
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@@
   )
   (no_connect (at 146.685 97.155))
-  (no_connect (at 154.94 46.355))
   (no_connect (at 154.305 116.205))
   (no_connect (at 133.985 135.255))
-  (no_connect (at 154.94 61.595))
   (no_connect (at 133.985 127.635))
   (no_connect (at 133.985 125.095))
@@
     (stroke (width 0) (type default))
   )
-  (wire (pts (xy 154.94 51.435) (xy 163.195 51.435))
+  (wire (pts (xy 154.94 51.435) (xy 165.735 51.435))
     (stroke (width 0) (type default))
   )
@@
     (stroke (width 0) (type default))
   )
-  (wire (pts (xy 163.195 73.025) (xy 149.225 73.025))
+  (wire (pts (xy 165.735 73.025) (xy 149.225 73.025))
     (stroke (width 0) (type default))
   )
@@
     (stroke (width 0) (type default))
   )
-  (wire (pts (xy 163.195 51.435) (xy 163.195 73.025))
+  (wire (pts (xy 165.735 51.435) (xy 165.735 73.025))
     (stroke (width 0) (type default))
   )
@@
         (path "/44572023-3621-4b3a-bd53-c3b2b3f42871/91a9a724-fdbf-449f-802f-4b411bd73828"
           (reference "#PWR0805") (unit 1)
+        )
+      )
+    )
+  )
+  (symbol (lib_id "power:+12V") (at 154.94 46.355 270) (unit 1)
+    (in_bom yes) (on_board yes) (dnp no) (fields_autoplaced)
+    (property "Reference" "#PWR0806" (at 151.13 46.355 0)
+      (effects (font (size 1.27 1.27)) hide)
+    )
+    (property "Value" "+12V" (at 158.75 46.99 90)
+      (effects (font (size 1.27 1.27)) (justify left))
+    )
+    (property "Footprint" "" (at 154.94 46.355 0)
+      (effects (font (size 1.27 1.27)) hide)
+    )
+    (property "Datasheet" "" (at 154.94 46.355 0)
+      (effects (font (size 1.27 1.27)) hide)
+    )
+    (pin "1")
+    (instances
+      (project "pg09-system"
+        (path "/44572023-3621-4b3a-bd53-c3b2b3f42871/91a9a724-fdbf-449f-802f-4b411bd73828"
+          (reference "#PWR0806") (unit 1)
         )
       )
@@
         )
       )
+    )
+  )
+  (symbol (lib_id "power:-12V") (at 154.94 61.595 270) (unit 1)
+    (in_bom yes) (on_board yes) (dnp no) (fields_autoplaced)
+    (property "Reference" "#PWR0807" (at 157.48 61.595 0)
+      (effects (font (size 1.27 1.27)) hide)
+    )
+    (property "Value" "-12V" (at 158.75 62.23 90)
+      (effects (font (size 1.27 1.27)) (justify left))
+    )
+    (property "Footprint" "" (at 154.94 61.595 0)
+      (effects (font (size 1.27 1.27)) hide)
+    )
+    (property "Datasheet" "" (at 154.94 61.595 0)
+      (effects (font (size 1.27 1.27)) hide)
+    )
+    (pin "1")
+    (instances
+      (project "pg09-system"
+        (path "/44572023-3621-4b3a-bd53-c3b2b3f42871/91a9a724-fdbf-449f-802f-4b411bd73828"
+          (reference "#PWR0807") (unit 1)
+        )
+      )

Commit message: Name the Power button.
Parts:
- SW201: value SW_Push -> Power
Changed lines of the file:
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@@
       (effects (font (size 1.27 1.27)))
     )
-    (property "Value" "SW_Push" (at 188.595 127.9961 0)
+    (property "Value" "Power" (at 188.595 127.9961 0)
       (effects (font (size 1.27 1.27)))
     )

Commit message: Checkpoint: no more unconnected items.
Connections:
- net +5VSB: now reaches J1.9 (+5VSB), U801.4 (5V)
- net +3V3: now reaches J1.1 (+3.3V), J1.12 (+3.3V), J1.13 (+3.3V), J1.2 (+3.3V)
- no-connect marks 19 -> 18
Changed lines of the file:
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@@
     (company "Copyright (c) 2022-2023 Jason R. Thorpe. See LICENSE.")
+  )
+  (junction (at 165.735 73.025) (diameter 0) (color 0 0 0 0)
   )
   (junction (at 142.875 147.955) (diameter 0) (color 0 0 0 0)
@@
   (no_connect (at 154.305 118.745))
   (no_connect (at 133.985 113.665))
-  (no_connect (at 154.94 53.975))
   (no_connect (at 133.985 120.015))
   (no_connect (at 139.065 97.155))
@@
   )
   (wire (pts (xy 154.94 51.435) (xy 165.735 51.435))
+    (stroke (width 0) (type default))
+  )
+  (wire (pts (xy 165.735 73.025) (xy 168.275 73.025))
     (stroke (width 0) (type default))
   )
@@
     )
   )
+  (global_label "+5VSB" (shape output) (at 168.275 73.025 0) (fields_autoplaced)
+    (effects (font (size 1.27 1.27)) (justify left))
+    (property "Intersheetrefs" "${INTERSHEET_REFS}" (at 177.5308 73.025 0)
+      (effects (font (size 1.27 1.27)) (justify left) hide)
+    )
+  )
   (global_label "PSU_CTRL_D1" (shape input) (at 175.26 114.935 0) (fields_autoplaced)
     (effects (font (size 1.27 1.27)) (justify left))
@@
     )
   )
+  (symbol (lib_id "power:+3V3") (at 154.94 53.975 270) (unit 1)
+    (in_bom yes) (on_board yes) (dnp no) (fields_autoplaced)
+    (property "Reference" "#PWR0808" (at 151.13 53.975 0)
+      (effects (font (size 1.27 1.27)) hide)
+    )
+    (property "Value" "+3V3" (at 158.75 54.61 90)
+      (effects (font (size 1.27 1.27)) (justify left))
+    )
+    (property "Footprint" "" (at 154.94 53.975 0)
+      (effects (font (size 1.27 1.27)) hide)
+    )
+    (property "Datasheet" "" (at 154.94 53.975 0)
+      (effects (font (size 1.27 1.27)) hide)
+    )
+    (pin "1")
+    (instances
+      (project "pg09-system"
+        (path "/44572023-3621-4b3a-bd53-c3b2b3f42871/91a9a724-fdbf-449f-802f-4b411bd73828"
+          (reference "#PWR0808") (unit 1)
+        )
+      )
+    )
+  )

Commit message: Add 470uF caps to the +12V, -12V, and +3V3 rails.  Increase the cap on the +5V rail to 2700uF.
Parts:
- added C802, C803, C804: 470µF 50V, Capacitor_THT:CP_Radial_D12.5mm_P5.00mm, symbol Device:C_Polarized_US
- C801: value 470µF 50V -> 2700µF 50V; footprint Capacitor_THT:CP_Radial_D12.5mm_P5.00mm -> Capacitor_THT:CP_Radial_D18.0mm_P7.50mm; Mouser 871-B41888C6477M -> 871-B41888C6278M
Connections:
- net +12V: now also C802.1
- net +3V3: now also C804.1
- net -12V: now also C803.2
- net GND: now also C802.2, C803.1, C804.2
- net ~{PWRBUT}: now reaches SW201.1, U801.17 (D2)
Other:
- moved on the sheet: SW201

Commit message: Add Mouser part # for ATX PSU connector.
Parts:
- J1: Mouser (none) -> 538-39-28-1243
Changed lines of the file:
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@@
+      (effects (font (size 1.27 1.27)) hide)
+    )
+    (property "Mouser" "538-39-28-1243" (at 142.24 51.435 0)
+      (effects (font (size 1.27 1.27)) hide)
+    )
+    (property "Field5" "" (at 142.24 51.435 0)
       (effects (font (size 1.27 1.27)) hide)
     )

Commit message: Add Power LED.  Tweak UART interface connectors.
Parts:
- added D1001: Power, LED_THT:LED_D3.0mm, symbol Device:LED
- added R701 (x2): 1K, Resistor_THT:R_Axial_DIN0207_L6.3mm_D2.5mm_P7.62mm_Horizontal, symbol Device:R_Small
Connections:
- net GND: now also R701.1, R701.1
- net PWR_LED+: now reaches U801.28 (D13)
- net PWR_LED+: now also D1001.2 (A)
- new net: D1001.1 (K), R701.2
- new net PWR_LED-: R701.2
- no-connect marks 18 -> 17

Commit message: Use physically smaller caps in the PSU.
Parts:
- C801: value 2700µF 50V -> 4700µF 16V; footprint Capacitor_THT:CP_Radial_D18.0mm_P7.50mm -> Capacitor_THT:CP_Radial_D12.5mm_P5.00mm; Mouser 871-B41888C6278M -> 667-EEU-FR1C472L
- C802, C803, C804: value 470µF 50V -> 470µF 25V; footprint Capacitor_THT:CP_Radial_D12.5mm_P5.00mm -> Capacitor_THT:CP_Radial_D10.0mm_P5.00mm; Mouser 871-B41888C6477M -> 232-25ZLH470MEFC10X1
Changed lines of the file:
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@@
       (effects (font (size 1.27 1.27)) (justify left))
     )
-    (property "Value" "470µF 50V" (at 203.2 51.435 0)
-      (effects (font (size 1.27 1.27)) (justify left))
-    )
-    (property "Footprint" "Capacitor_THT:CP_Radial_D12.5mm_P5.00mm" (at 199.39 50.165 0)
+    (property "Value" "470µF 25V" (at 203.2 51.435 0)
+      (effects (font (size 1.27 1.27)) (justify left))
+    )
+    (property "Footprint" "Capacitor_THT:CP_Radial_D10.0mm_P5.00mm" (at 199.39 50.165 0)
       (effects (font (size 1.27 1.27)) hide)
     )
@@
       (effects (font (size 1.27 1.27)) hide)
     )
-    (property "Mouser" "871-B41888C6477M" (at 199.39 50.165 0)
+    (property "Mouser" "232-25ZLH470MEFC10X1" (at 199.39 50.165 0)
       (effects (font (size 1.27 1.27)) hide)
     )
@@
       (effects (font (size 1.27 1.27)) (justify left))
     )
-    (property "Value" "470µF 50V" (at 203.2 43.815 0)
-      (effects (font (size 1.27 1.27)) (justify left))
-    )
-    (property "Footprint" "Capacitor_THT:CP_Radial_D12.5mm_P5.00mm" (at 199.39 42.545 0)
+    (property "Value" "470µF 25V" (at 203.2 43.815 0)
+      (effects (font (size 1.27 1.27)) (justify left))
+    )
+    (property "Footprint" "Capacitor_THT:CP_Radial_D10.0mm_P5.00mm" (at 199.39 42.545 0)
       (effects (font (size 1.27 1.27)) hide)
     )
@@
       (effects (font (size 1.27 1.27)) hide)
     )
-    (property "Mouser" "871-B41888C6477M" (at 199.39 42.545 0)
+    (property "Mouser" "232-25ZLH470MEFC10X1" (at 199.39 42.545 0)
       (effects (font (size 1.27 1.27)) hide)
     )
@@
       (effects (font (size 1.27 1.27)) (justify left))
     )
-    (property "Value" "2700µF 50V" (at 177.8 53.975 0)
-      (effects (font (size 1.27 1.27)) (justify left))
-    )
-    (property "Footprint" "Capacitor_THT:CP_Radial_D18.0mm_P7.50mm" (at 173.99 52.705 0)
+    (property "Value" "4700µF 16V" (at 177.8 53.975 0)
+      (effects (font (size 1.27 1.27)) (justify left))
+    )
+    (property "Footprint" "Capacitor_THT:CP_Radial_D12.5mm_P5.00mm" (at 173.99 52.705 0)
       (effects (font (size 1.27 1.27)) hide)
     )
@@
       (effects (font (size 1.27 1.27)) hide)
     )
-    (property "Mouser" "871-B41888C6278M" (at 173.99 52.705 0)
+    (property "Mouser" "667-EEU-FR1C472L" (at 173.99 52.705 0)
+      (effects (font (size 1.27 1.27)) hide)
+    )
+    (property "Field5" "" (at 173.99 52.705 0)
       (effects (font (size 1.27 1.27)) hide)
     )
@@
   (symbol (lib_id "Device:C_Polarized_US") (at 219.075 42.545 0) (unit 1)
     (in_bom yes) (on_board yes) (dnp no) (fields_autoplaced)
-    (property "Reference" "C804" (at 222.885 41.275 0)
-      (effects (font (size 1.27 1.27)) (justify left))
-    )
-    (property "Value" "470µF 50V" (at 222.885 43.815 0)
-      (effects (font (size 1.27 1.27)) (justify left))
-    )
-    (property "Footprint" "Capacitor_THT:CP_Radial_D12.5mm_P5.00mm" (at 219.075 42.545 0)
+    (property "Reference" "C804" (at 222.25 41.275 0)
+      (effects (font (size 1.27 1.27)) (justify left))
+    )
+    (property "Value" "470µF 25V" (at 222.25 43.815 0)
+      (effects (font (size 1.27 1.27)) (justify left))
+    )
+    (property "Footprint" "Capacitor_THT:CP_Radial_D10.0mm_P5.00mm" (at 219.075 42.545 0)
       (effects (font (size 1.27 1.27)) hide)
     )
@@
       (effects (font (size 1.27 1.27)) hide)
     )
-    (property "Mouser" "871-B41888C6477M" (at 219.075 42.545 0)
-      (effects (font (size 1.27 1.27)) hide)
-    )
+    (property "Mouser" "232-25ZLH470MEFC10X1" (at 219.075 42.545 0)
+      (effects (font (size 1.27 1.27)) hide)
+    )
