File: design-files/pg09-system-psu.kicad_sch (KiCad schematic)
At the start: 12 parts, among them J1 ATX-24, J802 #PS_ON, J803 PSU-CTRL console, SW201 Power, U801 Adafruit_Metro_Mini

Commit message: Disconnect the PSU controller from the ROM banker PIA and instead give it its own register (offset $11) in IO0SEL.  Use a '138 to decode the address and generate the write strobe for it.
Parts:
- added C203: 0.1µF, Capacitor_THT:C_Disc_D3.8mm_W2.6mm_P2.50mm, symbol Device:C_Small
- added U802: 74AHC138, Package_DIP:DIP-16_W7.62mm_Socket, symbol 74xx:74LS138
Connections:
- net +5V: now also C203.1, U802.16 (VCC)
- net GND: now also C203.2, U802.8 (GND)
- net ~{PSU_CTRL_WR}: now also U802.11 (O4)
- net PSU_CTRL_D0 renamed D0
- net PSU_CTRL_D1 renamed D1
- new net A0: U802.3 (A2)
- new net A1: U802.4 (E1)
- new net A2: U802.2 (A1)
- new net A4: U802.6 (E3)
- new net ~{IO0SEL}: U802.5 (E2)
- new net ~{WR}: U802.1 (A0)
- no-connect marks 17 -> 24
