File: design-files/pg09-system-psu.kicad_sch (KiCad schematic)
At the start: 14 parts, among them J1 ATX-24, J802 #PS_ON, J803 PSU-CTRL console, SW201 Power, U801 Adafruit_Metro_Mini, U802 74AHC138

Commit message: Overhaul how the "system registers" in IO0SEL work, paving the way to use a VIA for the interrupt enables (because that would also give us a timer).
Parts:
- removed U802: 74AHC138, Package_DIP:DIP-16_W7.62mm_Socket, symbol 74xx:74LS138
- added U414: 74AHC374, Package_DIP:DIP-20_W7.62mm_Socket, symbol 74xx:74AHC374
Connections:
- net +5V: now also U414.20 (VCC)
- net D0: now also U414.3 (D0); no longer U801.19 (D4)
- net D1: now also U414.4 (D1); no longer U801.20 (D5)
- net GND: now also U414.1 (OE), U414.10 (GND)
- net ~{PSU_CTRL_WR} renamed ~{PSUCTL}
- net ~{PSUCTL}: now also U414.11 (Cp)
- new net D2: U414.7 (D2)
- new net D3: U414.8 (D3)
- new net D4: U414.13 (D4)
- new net D5: U414.14 (D5)
- new net D6: U414.17 (D6)
- new net D7: U414.18 (D7)
- new net PSU_CTRL_D0: U414.2 (O0), U801.20 (D5)
- new net PSU_CTRL_D1: U414.5 (O1), U801.19 (D4)
- no-connect marks 24 -> 23
