File: design-files/pg09-system-ram.kicad_sch (KiCad schematic)
At the start: 16 parts, among them U501 W65C21, U602 AS6C4008-55PCN, U603 74AHC138, U604 AS6C4008-55PCN, U605 AS6C4008-55PCN, U606 AS6C4008-55PCN, U607 AS6C4008-55PCN, U608 AS6C6264-55PCN

Commit message: Assign a bunch of footprints.
Parts:
- C201, C202, C203: footprint (none) -> Capacitor_THT:C_Disc_D6.0mm_W4.4mm_P5.00mm
- U501: footprint Package_DIP:DIP-40_W15.24mm -> Package_DIP:DIP-40_W15.24mm_Socket
- U602, U604, U605, U606, U607: footprint Package_DIP:DIP-32_W15.24mm -> Package_DIP:DIP-32_W15.24mm_Socket
- U603: footprint (none) -> Package_DIP:DIP-16_W7.62mm_Socket
- U608: footprint Package_DIP:DIP-28_W15.24mm -> Package_DIP:DIP-28_W15.24mm_Socket
Changed lines of the file:
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@@
       (effects (font (size 1.27 1.27)) (justify left))
     )
-    (property "Footprint" "" (at 64.77 173.99 0)
+    (property "Footprint" "Capacitor_THT:C_Disc_D6.0mm_W4.4mm_P5.00mm" (at 64.77 173.99 0)
       (effects (font (size 1.27 1.27)) hide)
     )
@@
       (effects (font (size 1.27 1.27)) (justify left))
     )
-    (property "Footprint" "" (at 74.93 173.99 0)
+    (property "Footprint" "Capacitor_THT:C_Disc_D6.0mm_W4.4mm_P5.00mm" (at 74.93 173.99 0)
       (effects (font (size 1.27 1.27)) hide)
     )
@@
       (effects (font (size 1.27 1.27)) (justify left))
     )
-    (property "Footprint" "Package_DIP:DIP-32_W15.24mm" (at 144.78 44.45 0)
+    (property "Footprint" "Package_DIP:DIP-32_W15.24mm_Socket" (at 144.78 44.45 0)
       (effects (font (size 1.27 1.27)) hide)
     )
@@
       (effects (font (size 1.27 1.27)) (justify left))
     )
-    (property "Footprint" "" (at 83.82 125.73 0)
+    (property "Footprint" "Package_DIP:DIP-16_W7.62mm_Socket" (at 83.82 125.73 0)
       (effects (font (size 1.27 1.27)) hide)
     )
@@
       (effects (font (size 1.27 1.27)) (justify left))
     )
-    (property "Footprint" "Package_DIP:DIP-32_W15.24mm" (at 205.74 121.92 0)
+    (property "Footprint" "Package_DIP:DIP-32_W15.24mm_Socket" (at 205.74 121.92 0)
       (effects (font (size 1.27 1.27)) hide)
     )
@@
       (effects (font (size 1.27 1.27)) (justify left))
     )
-    (property "Footprint" "Package_DIP:DIP-32_W15.24mm" (at 144.78 121.92 0)
+    (property "Footprint" "Package_DIP:DIP-32_W15.24mm_Socket" (at 144.78 121.92 0)
       (effects (font (size 1.27 1.27)) hide)
     )
@@
       (effects (font (size 1.27 1.27)) (justify left))
     )
-    (property "Footprint" "" (at 95.25 173.99 0)
+    (property "Footprint" "Capacitor_THT:C_Disc_D6.0mm_W4.4mm_P5.00mm" (at 95.25 173.99 0)
       (effects (font (size 1.27 1.27)) hide)
     )
@@
       (effects (font (size 1.27 1.27)) (justify left))
     )
-    (property "Footprint" "" (at 44.45 173.99 0)
+    (property "Footprint" "Capacitor_THT:C_Disc_D6.0mm_W4.4mm_P5.00mm" (at 44.45 173.99 0)
       (effects (font (size 1.27 1.27)) hide)
     )
@@
       (effects (font (size 1.27 1.27)) (justify left))
     )
-    (property "Footprint" "" (at 105.41 173.99 0)
+    (property "Footprint" "Capacitor_THT:C_Disc_D6.0mm_W4.4mm_P5.00mm" (at 105.41 173.99 0)
       (effects (font (size 1.27 1.27)) hide)
     )
@@
       (effects (font (size 1.27 1.27)) (justify left))
     )
-    (property "Footprint" "Package_DIP:DIP-32_W15.24mm" (at 205.74 44.45 0)
+    (property "Footprint" "Package_DIP:DIP-32_W15.24mm_Socket" (at 205.74 44.45 0)
       (effects (font (size 1.27 1.27)) hide)
     )
@@
       (effects (font (size 1.27 1.27)) (justify left))
     )
-    (property "Footprint" "Package_DIP:DIP-40_W15.24mm" (at 41.91 91.44 0)
+    (property "Footprint" "Package_DIP:DIP-40_W15.24mm_Socket" (at 41.91 91.44 0)
       (effects (font (size 1.27 1.27)) hide)
     )
@@
       (effects (font (size 1.27 1.27)) (justify left))
     )
-    (property "Footprint" "" (at 85.09 173.99 0)
+    (property "Footprint" "Capacitor_THT:C_Disc_D6.0mm_W4.4mm_P5.00mm" (at 85.09 173.99 0)
       (effects (font (size 1.27 1.27)) hide)
     )
@@
       (effects (font (size 1.27 1.27)) (justify left))
     )
-    (property "Footprint" "" (at 34.29 173.99 0)
+    (property "Footprint" "Capacitor_THT:C_Disc_D6.0mm_W4.4mm_P5.00mm" (at 34.29 173.99 0)
       (effects (font (size 1.27 1.27)) hide)
     )
@@
       (effects (font (size 1.27 1.27)) (justify left))
     )
-    (property "Footprint" "Package_DIP:DIP-28_W15.24mm" (at 254 88.9 0)
+    (property "Footprint" "Package_DIP:DIP-28_W15.24mm_Socket" (at 254 88.9 0)
       (effects (font (size 1.27 1.27)) hide)
     )
@@
       (effects (font (size 1.27 1.27)) (justify left))
     )
-    (property "Footprint" "" (at 54.61 173.99 0)
+    (property "Footprint" "Capacitor_THT:C_Disc_D6.0mm_W4.4mm_P5.00mm" (at 54.61 173.99 0)
       (effects (font (size 1.27 1.27)) hide)
     )
@@
       (effects (font (size 1.27 1.27)) (justify left))
     )
-    (property "Footprint" "Package_DIP:DIP-32_W15.24mm" (at 83.82 44.45 0)
-      (effects (font (size 1.27 1.27)) hide)
-    )
+    (property "Footprint" "Package_DIP:DIP-32_W15.24mm_Socket" (at 83.82 44.45 0)
+      (effects (font (size 1.27 1.27)) hide)
+    )

Commit message: Specify a physically smaller bypass cap.
Parts:
- C201, C202, C203: footprint Capacitor_THT:C_Disc_D6.0mm_W4.4mm_P5.00mm -> Capacitor_THT:C_Disc_D3.8mm_W2.6mm_P2.50mm
Changed lines of the file:
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@@
       (effects (font (size 1.27 1.27)) (justify left))
     )
-    (property "Footprint" "Capacitor_THT:C_Disc_D6.0mm_W4.4mm_P5.00mm" (at 64.77 173.99 0)
+    (property "Footprint" "Capacitor_THT:C_Disc_D3.8mm_W2.6mm_P2.50mm" (at 64.77 173.99 0)
       (effects (font (size 1.27 1.27)) hide)
     )
@@
       (effects (font (size 1.27 1.27)) (justify left))
     )
-    (property "Footprint" "Capacitor_THT:C_Disc_D6.0mm_W4.4mm_P5.00mm" (at 74.93 173.99 0)
+    (property "Footprint" "Capacitor_THT:C_Disc_D3.8mm_W2.6mm_P2.50mm" (at 74.93 173.99 0)
       (effects (font (size 1.27 1.27)) hide)
     )
@@
       (effects (font (size 1.27 1.27)) (justify left))
     )
-    (property "Footprint" "Capacitor_THT:C_Disc_D6.0mm_W4.4mm_P5.00mm" (at 95.25 173.99 0)
+    (property "Footprint" "Capacitor_THT:C_Disc_D3.8mm_W2.6mm_P2.50mm" (at 95.25 173.99 0)
       (effects (font (size 1.27 1.27)) hide)
     )
@@
       (effects (font (size 1.27 1.27)) (justify left))
     )
-    (property "Footprint" "Capacitor_THT:C_Disc_D6.0mm_W4.4mm_P5.00mm" (at 44.45 173.99 0)
+    (property "Footprint" "Capacitor_THT:C_Disc_D3.8mm_W2.6mm_P2.50mm" (at 44.45 173.99 0)
       (effects (font (size 1.27 1.27)) hide)
     )
@@
       (effects (font (size 1.27 1.27)) (justify left))
     )
-    (property "Footprint" "Capacitor_THT:C_Disc_D6.0mm_W4.4mm_P5.00mm" (at 105.41 173.99 0)
+    (property "Footprint" "Capacitor_THT:C_Disc_D3.8mm_W2.6mm_P2.50mm" (at 105.41 173.99 0)
       (effects (font (size 1.27 1.27)) hide)
     )
@@
       (effects (font (size 1.27 1.27)) (justify left))
     )
-    (property "Footprint" "Capacitor_THT:C_Disc_D6.0mm_W4.4mm_P5.00mm" (at 85.09 173.99 0)
+    (property "Footprint" "Capacitor_THT:C_Disc_D3.8mm_W2.6mm_P2.50mm" (at 85.09 173.99 0)
       (effects (font (size 1.27 1.27)) hide)
     )
@@
       (effects (font (size 1.27 1.27)) (justify left))
     )
-    (property "Footprint" "Capacitor_THT:C_Disc_D6.0mm_W4.4mm_P5.00mm" (at 34.29 173.99 0)
+    (property "Footprint" "Capacitor_THT:C_Disc_D3.8mm_W2.6mm_P2.50mm" (at 34.29 173.99 0)
       (effects (font (size 1.27 1.27)) hide)
     )
@@
       (effects (font (size 1.27 1.27)) (justify left))
     )
-    (property "Footprint" "Capacitor_THT:C_Disc_D6.0mm_W4.4mm_P5.00mm" (at 54.61 173.99 0)
-      (effects (font (size 1.27 1.27)) hide)
-    )
+    (property "Footprint" "Capacitor_THT:C_Disc_D3.8mm_W2.6mm_P2.50mm" (at 54.61 173.99 0)
+      (effects (font (size 1.27 1.27)) hide)
+    )

Commit message: Change U603 (the high banked RAM mux) from '138 to a '139 so it can also be used for the low banked RAM.
Parts:
- added unit 3 of U603
- added unit 2 of U603
- U603: value 74AHC138 -> 74AHC139; symbol 74xx:74LS138 -> 74xx:74LS139
Connections:
- net +5V: now also U603.13 (A1), U603.14 (A0), U603.15 (E), U603.16 (VCC); no longer U603.16 (VCC), U603.6 (E3)
- net GND: now also U603.8 (GND); no longer U603.3 (A2), U603.8 (GND)
- net ~{HBRAMSEL}: now also U603.1 (E); no longer U603.4 (E1), U603.5 (E2)
- net at U604.22 (CE#): now also U603.4 (O0); no longer U603.15 (O0)
- net at U501.16 (PB6): now also U603.3 (A1); no longer U603.1 (A0)
- net at U607.22 (CE#): now also U603.7 (O3); no longer U603.12 (O3)
- net at U606.22 (CE#): now also U603.6 (O2); no longer U603.13 (O2)
- net at U605.22 (CE#): now also U603.5 (O1); no longer U603.14 (O1)
Other:
- moved on the sheet: C201, C202, C203

Commit message: Move the RAM banker PIA to the decoder sheet and re-designate U304.
Parts:
- removed C203: 0.1µF, Capacitor_THT:C_Disc_D3.8mm_W2.6mm_P2.50mm, symbol Device:C_Small
- removed U501: W65C21, Package_DIP:DIP-40_W15.24mm_Socket, symbol jrt-ICs:W65C21
Connections:
- net HRB5: now reaches U604.1 (A18), U605.1 (A18), U606.1 (A18), U607.1 (A18)
- net HRB3: now reaches U604.2 (A16), U605.2 (A16), U606.2 (A16), U607.2 (A16)
- net HRB0: now reaches U604.28 (A13), U605.28 (A13), U606.28 (A13), U607.28 (A13)
- net HRB1: now reaches U604.3 (A14), U605.3 (A14), U606.3 (A14), U607.3 (A14)
- net HRB4: now reaches U604.30 (A17), U605.30 (A17), U606.30 (A17), U607.30 (A17)
- net HRB2: now reaches U604.31 (A15), U605.31 (A15), U606.31 (A15), U607.31 (A15)
- net HRB7: now reaches U603.2 (A0)
- net HRB6: now reaches U603.3 (A1)
- net LRB0: now reaches U602.31 (A15)
- net LRB1: now reaches U602.2 (A16)
- net LRB2: now reaches U602.30 (A17)
- net LRB3: now reaches U602.1 (A18)
- no-connect marks 14 -> 4

Commit message: Re-designate RAM components.
Parts:
- renumbered U603 to U601, U608 to U602, U604 to U603, U605 to U604, U606 to U605, U607 to U606, U602 to U607
Changed lines of the file:
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@@
   (symbol (lib_id "74xx:74LS139") (at 33.782 156.972 0) (unit 3)
     (in_bom yes) (on_board yes) (dnp no)
-    (property "Reference" "U603" (at 35.052 145.034 0)
+    (property "Reference" "U601" (at 35.052 145.034 0)
       (effects (font (size 1.27 1.27)) (justify left))
     )
@@
       (project "pg09-system"
         (path "/44572023-3621-4b3a-bd53-c3b2b3f42871/c22548cb-3a32-4ecf-b2c4-e43fd96dc369"
-          (reference "U603") (unit 3)
+          (reference "U601") (unit 3)
         )
       )
@@
   (symbol (lib_id "Memory_RAM:AS6C4008-55PCN") (at 144.78 46.99 0) (unit 1)
     (in_bom yes) (on_board yes) (dnp no) (fields_autoplaced)
-    (property "Reference" "U604" (at 146.7359 17.78 0)
+    (property "Reference" "U603" (at 146.7359 17.78 0)
       (effects (font (size 1.27 1.27)) (justify left))
     )
@@
       (project "pg09-system"
         (path "/44572023-3621-4b3a-bd53-c3b2b3f42871/c22548cb-3a32-4ecf-b2c4-e43fd96dc369"
-          (reference "U604") (unit 1)
+          (reference "U603") (unit 1)
         )
       )
@@
   (symbol (lib_id "74xx:74LS139") (at 83.82 120.65 0) (unit 1)
     (in_bom yes) (on_board yes) (dnp no)
-    (property "Reference" "U603" (at 79.502 111.506 0)
+    (property "Reference" "U601" (at 79.502 111.506 0)
       (effects (font (size 1.27 1.27)) (justify left))
     )
@@
       (project "pg09-system"
         (path "/44572023-3621-4b3a-bd53-c3b2b3f42871/c22548cb-3a32-4ecf-b2c4-e43fd96dc369"
-          (reference "U603") (unit 1)
+          (reference "U601") (unit 1)
         )
       )
@@
   (symbol (lib_id "Memory_RAM:AS6C4008-55PCN") (at 205.74 124.46 0) (unit 1)
     (in_bom yes) (on_board yes) (dnp no) (fields_autoplaced)
-    (property "Reference" "U607" (at 207.6959 95.25 0)
+    (property "Reference" "U606" (at 207.6959 95.25 0)
       (effects (font (size 1.27 1.27)) (justify left))
     )
@@
       (project "pg09-system"
         (path "/44572023-3621-4b3a-bd53-c3b2b3f42871/c22548cb-3a32-4ecf-b2c4-e43fd96dc369"
-          (reference "U607") (unit 1)
+          (reference "U606") (unit 1)
         )
       )
@@
   (symbol (lib_id "Memory_RAM:AS6C4008-55PCN") (at 144.78 124.46 0) (unit 1)
     (in_bom yes) (on_board yes) (dnp no) (fields_autoplaced)
-    (property "Reference" "U606" (at 146.7359 95.25 0)
+    (property "Reference" "U605" (at 146.7359 95.25 0)
       (effects (font (size 1.27 1.27)) (justify left))
     )
@@
       (project "pg09-system"
         (path "/44572023-3621-4b3a-bd53-c3b2b3f42871/c22548cb-3a32-4ecf-b2c4-e43fd96dc369"
-          (reference "U606") (unit 1)
+          (reference "U605") (unit 1)
         )
       )
@@
   (symbol (lib_id "Memory_RAM:AS6C4008-55PCN") (at 205.74 46.99 0) (unit 1)
     (in_bom yes) (on_board yes) (dnp no) (fields_autoplaced)
-    (property "Reference" "U605" (at 207.6959 17.78 0)
+    (property "Reference" "U604" (at 207.6959 17.78 0)
       (effects (font (size 1.27 1.27)) (justify left))
     )
@@
       (project "pg09-system"
         (path "/44572023-3621-4b3a-bd53-c3b2b3f42871/c22548cb-3a32-4ecf-b2c4-e43fd96dc369"
-          (reference "U605") (unit 1)
+          (reference "U604") (unit 1)
         )
       )
@@
   (symbol (lib_id "jrt-ICs:AS6C6264") (at 254 81.28 0) (unit 1)
     (in_bom yes) (on_board yes) (dnp no) (fields_autoplaced)
-    (property "Reference" "U608" (at 255.9559 59.69 0)
+    (property "Reference" "U602" (at 255.9559 59.69 0)
       (effects (font (size 1.27 1.27)) (justify left))
     )
@@
       (project "pg09-system"
         (path "/44572023-3621-4b3a-bd53-c3b2b3f42871/c22548cb-3a32-4ecf-b2c4-e43fd96dc369"
-          (reference "U608") (unit 1)
+          (reference "U602") (unit 1)
         )
       )
@@
   (symbol (lib_id "Memory_RAM:AS6C4008-55PCN") (at 83.82 46.99 0) (unit 1)
     (in_bom yes) (on_board yes) (dnp no) (fields_autoplaced)
-    (property "Reference" "U602" (at 85.7759 17.78 0)
+    (property "Reference" "U607" (at 85.7759 17.78 0)
       (effects (font (size 1.27 1.27)) (justify left))
     )
@@
       (project "pg09-system"
         (path "/44572023-3621-4b3a-bd53-c3b2b3f42871/c22548cb-3a32-4ecf-b2c4-e43fd96dc369"
-          (reference "U602") (unit 1)
+          (reference "U607") (unit 1)
         )
       )
@@
   (symbol (lib_id "74xx:74LS139") (at 73.152 156.21 0) (unit 2)
     (in_bom yes) (on_board yes) (dnp no)
-    (property "Reference" "U603" (at 68.834 147.066 0)
+    (property "Reference" "U601" (at 68.834 147.066 0)
       (effects (font (size 1.27 1.27)) (justify left))
     )
@@
       (project "pg09-system"
         (path "/44572023-3621-4b3a-bd53-c3b2b3f42871/c22548cb-3a32-4ecf-b2c4-e43fd96dc369"
-          (reference "U603") (unit 2)
-        )
-      )
+          (reference "U601") (unit 2)
+        )
+      )

Commit message: New banked RAM layout: - The 2MB RAM group is now Low Banked RAM, and divided into 2   16K independently bankable regions back by 1MB each. - The 512KB RAM is now High Banked RAM. - Shuffle the Low and High banker PIAs.
Connections:
- net HRB6 is gone; now on net A14: U601.3 (A1)
- net HRB7 is gone; now on net A13: U601.2 (A0)
- net LRB0 is gone; now on net HRB2: U607.31 (A15)
- net LRB1 is gone; now on net HRB3: U607.2 (A16)
- net LRB2 is gone; now on net HRB4: U607.30 (A17)
- net LRB3 is gone; now on net HRB5: U607.1 (A18)
- net A13: no longer U607.28 (A13)
- net A14: no longer U607.3 (A14)
- net A15: now also U601.1 (E); no longer U607.22 (CE#)
- net HRB0: now also U607.28 (A13); no longer U603.28 (A13), U604.28 (A13), U605.28 (A13), U606.28 (A13)
- net HRB1: now also U607.3 (A14); no longer U603.3 (A14), U604.3 (A14), U605.3 (A14), U606.3 (A14)
- net HRB2: no longer U603.31 (A15), U604.31 (A15), U605.31 (A15), U606.31 (A15)
- net HRB3: no longer U603.2 (A16), U604.2 (A16), U605.2 (A16), U606.2 (A16)
- net HRB4: no longer U603.30 (A17), U604.30 (A17), U605.30 (A17), U606.30 (A17)
- net HRB5: no longer U603.1 (A18), U604.1 (A18), U605.1 (A18), U606.1 (A18)
- net ~{HBRAMSEL}: now also U607.22 (CE#); no longer U601.1 (E)
- new net LR0B0: U603.28 (A13), U604.28 (A13)
- new net LR0B1: U603.3 (A14), U604.3 (A14)
- new net LR0B2: U603.31 (A15), U604.31 (A15)
- new net LR0B3: U603.2 (A16), U604.2 (A16)
- new net LR0B4: U603.30 (A17), U604.30 (A17)
- new net LR0B5: U603.1 (A18), U604.1 (A18)
- new net LR1B0: U605.28 (A13), U606.28 (A13)
- new net LR1B1: U605.3 (A14), U606.3 (A14)
- new net LR1B2: U605.31 (A15), U606.31 (A15)
- new net LR1B3: U605.2 (A16), U606.2 (A16)
- new net LR1B4: U605.30 (A17), U606.30 (A17)
- new net LR1B5: U605.1 (A18), U606.1 (A18)
Other:
- note added: "Low Banked RAM 0"
- note added: "Low Banked RAM 1"
- note removed: "Low Banked RAM"
- moved on the sheet: C201, C202, C203, U601A, U601B, U601C, U602, U603, U604, U605, U606, U607

Commit message: Add another high banked SRAM, for a total of 128 banks.
Parts:
- added C203: 0.1µF, Capacitor_THT:C_Disc_D3.8mm_W2.6mm_P2.50mm, symbol Device:C_Small
- added U608: AS6C4008-55PCN, Package_DIP:DIP-32_W15.24mm_Socket, symbol Memory_RAM:AS6C4008-55PCN
Connections:
- net +5V: now also C203.1, U608.32 (VCC); no longer U601.13 (A1), U601.14 (A0), U601.15 (E)
- net A0: now also U608.12 (A0)
- net A1: now also U608.11 (A1)
- net A10: now also U608.23 (A10)
- net A11: now also U608.25 (A11)
- net A12: now also U608.4 (A12)
- net A2: now also U608.10 (A2)
- net A3: now also U608.9 (A3)
- net A4: now also U608.8 (A4)
- net A5: now also U608.7 (A5)
- net A6: now also U608.6 (A6)
- net A7: now also U608.5 (A7)
- net A8: now also U608.27 (A8)
- net A9: now also U608.26 (A9)
- net D0: now also U608.13 (DQ0)
- net D1: now also U608.14 (DQ1)
- net D2: now also U608.15 (DQ2)
- net D3: now also U608.17 (DQ3)
- net D4: now also U608.18 (DQ4)
- net D5: now also U608.19 (DQ5)
- net D6: now also U608.20 (DQ6)
- net D7: now also U608.21 (DQ7)
- net GND: now also U601.14 (A0), C203.2, U608.16 (VSS)
- net HRB0: now also U608.28 (A13)
- net HRB1: now also U608.3 (A14)
- net HRB2: now also U608.31 (A15)
- net HRB3: now also U608.2 (A16)
- net HRB4: now also U608.30 (A17)
- net HRB5: now also U608.1 (A18)
- net ~{HBRAMSEL}: now also U601.15 (E); no longer U607.22 (CE#)
- net ~{RD}: now also U608.24 (OE#)
- net ~{WR}: now also U608.29 (WE#)
- net at U601.11 (O1): now also U608.22 (CE#)
- net at U601.12 (O0): now also U607.22 (CE#)
- new net HRB6: U601.13 (A1)
- no-connect marks 4 -> 2
Other:
- note added: "Low Banked RAM 0 (0-16K)"
- note added: "Low Banked RAM 1 (16K-32K)"
- note removed: "Low Banked RAM 0"
- note removed: "Low Banked RAM 1"

Commit message: Correct wiring mistake on High Banked RAM decoder: HRB6 needs to be connected to the A0 input.
Connections:
- net GND: now also U601.13 (A1); no longer U601.14 (A0)
- net HRB6: now also U601.14 (A0); no longer U601.13 (A1)
Changed lines of the file:
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@@
     )
   )
-  (global_label "HRB6" (shape input) (at 202.946 94.488 180) (fields_autoplaced)
-    (effects (font (size 1.27 1.27)) (justify right))
-    (property "Intersheetrefs" "${INTERSHEET_REFS}" (at 194.9602 94.488 0)
+  (global_label "HRB6" (shape input) (at 202.946 97.028 180) (fields_autoplaced)
+    (effects (font (size 1.27 1.27)) (justify right))
+    (property "Intersheetrefs" "${INTERSHEET_REFS}" (at 194.9602 97.028 0)
       (effects (font (size 1.27 1.27)) (justify right) hide)
     )
@@
     )
   )
-  (symbol (lib_id "power:GND") (at 202.946 97.028 270) (unit 1)
-    (in_bom yes) (on_board yes) (dnp no) (fields_autoplaced)
-    (property "Reference" "#PWR0502" (at 196.596 97.028 0)
-      (effects (font (size 1.27 1.27)) hide)
-    )
-    (property "Value" "GND" (at 199.39 97.663 90)
+  (symbol (lib_id "power:GND") (at 202.946 94.488 270) (unit 1)
+    (in_bom yes) (on_board yes) (dnp no) (fields_autoplaced)
+    (property "Reference" "#PWR0502" (at 196.596 94.488 0)
+      (effects (font (size 1.27 1.27)) hide)
+    )
+    (property "Value" "GND" (at 199.39 95.123 90)
       (effects (font (size 1.27 1.27)) (justify right))
     )
-    (property "Footprint" "" (at 202.946 97.028 0)
-      (effects (font (size 1.27 1.27)) hide)
-    )
-    (property "Datasheet" "" (at 202.946 97.028 0)
-      (effects (font (size 1.27 1.27)) hide)
-    )
+    (property "Footprint" "" (at 202.946 94.488 0)
+      (effects (font (size 1.27 1.27)) hide)
+    )
+    (property "Datasheet" "" (at 202.946 94.488 0)
+      (effects (font (size 1.27 1.27)) hide)
+    )
