File: design-files/pg09-system-ram.kicad_sch (KiCad schematic)
At the start: 16 parts, among them U601 74AHC139, U602 AS6C6264-55PCN, U603 AS6C4008-55PCN, U604 AS6C4008-55PCN, U605 AS6C4008-55PCN, U606 AS6C4008-55PCN, U607 AS6C4008-55PCN, U608 AS6C4008-55PCN

Commit message: Re-work low banked RAM so that not all SRAM chips have to be installed.
Parts:
- added C203 (x2): 0.1µF, Capacitor_THT:C_Disc_D3.8mm_W2.6mm_P2.50mm, symbol Device:C_Small
- added U502 (x2): 74AHC157, Package_DIP:DIP-16_W7.62mm_Socket, symbol 74xx:74LS157
Connections:
- net +5V: now also C203.1, C203.1, U502.16 (VCC), U502.16 (VCC)
- net A13: now also U603.28 (A13), U604.28 (A13), U605.28 (A13), U606.28 (A13); no longer U601.2 (A0)
- net A14: now also U603.3 (A14), U604.3 (A14), U605.3 (A14), U606.3 (A14), U502.1 (S), U502.1 (S); no longer U601.3 (A1)
- net GND: now also C203.2, C203.2, U502.10 (I1c), U502.11 (I0c), U502.13 (I1d), U502.14 (I0d), U502.15 (E), U502.15 (E), U502.8 (GND), U502.8 (GND)
- net LR0B0: now also U502.2 (I0a); no longer U603.28 (A13), U604.28 (A13)
- net LR0B1: now also U502.5 (I0b); no longer U603.3 (A14), U604.3 (A14)
- net LR0B2: now also U502.11 (I0c); no longer U603.31 (A15), U604.31 (A15)
- net LR0B3: now also U502.14 (I0d); no longer U603.2 (A16), U604.2 (A16)
- net LR0B4: now also U502.2 (I0a); no longer U603.30 (A17), U604.30 (A17)
- net LR0B5: now also U502.5 (I0b); no longer U603.1 (A18), U604.1 (A18)
- net LR1B0: now also U502.3 (I1a); no longer U605.28 (A13), U606.28 (A13)
- net LR1B1: now also U502.6 (I1b); no longer U605.3 (A14), U606.3 (A14)
- net LR1B2: now also U502.10 (I1c); no longer U605.31 (A15), U606.31 (A15)
- net LR1B3: now also U502.13 (I1d); no longer U605.2 (A16), U606.2 (A16)
- net LR1B4: now also U502.3 (I1a); no longer U605.30 (A17), U606.30 (A17)
- net LR1B5: now also U502.6 (I1b); no longer U605.1 (A18), U606.1 (A18)
- new net: U502.4 (Za), U601.2 (A0)
- new net: U502.7 (Zb), U601.3 (A1)
- new net LRBS0: U502.4 (Za), U603.31 (A15), U604.31 (A15), U605.31 (A15), U606.31 (A15)
- new net LRBS1: U502.7 (Zb), U603.2 (A16), U604.2 (A16), U605.2 (A16), U606.2 (A16)
- new net LRBS2: U502.9 (Zc), U603.30 (A17), U604.30 (A17), U605.30 (A17), U606.30 (A17)
- new net LRBS3: U502.12 (Zd), U603.1 (A18), U604.1 (A18), U605.1 (A18), U606.1 (A18)
- no-connect marks 2 -> 4
Other:
- note added: "Low Banked RAM"
- note removed: "Low Banked RAM 0 (0-16K)"
- note removed: "Low Banked RAM 1 (16K-32K)"
- company: Copyright (c) 2022-2023 Jason R. Thorpe. See LICENSE. -> Copyright (c) 2022-2024 Jason R. Thorpe. See LICENSE.
- moved on the sheet: C201, C202, C203, U601A, U601B, U601C, U602, U603, U604, U605, U606, U607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
