File: design-files/pg09-system-clock.kicad_sch (KiCad schematic)
At the start: 18 parts, among them J201 Clock Speed, Q201 2N7000, SW201 Reset, U201 CD74ACT109, U202 CD74ACT163, U203 DS1813, U204 GAL22V10, X201 ACO-32.000MHz

Commit message: Move Reset to the main sheet.  Checkpoint SD Card SPI interface.
Parts:
- removed R203: 3K3, Resistor_THT:R_Axial_DIN0207_L6.3mm_D2.5mm_P7.62mm_Horizontal, symbol Device:R_Small
- removed SW201: Reset, Button_Switch_THT:SW_PUSH_6mm, symbol Switch:SW_Push
- removed U203: DS1813, Package_TO_SOT_THT:TO-92_Inline, symbol jrt-ICs:DS1813
Other:
- note removed: "Reset Generator"
Changed lines of the file:
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@@
   (junction (at 219.075 113.03) (diameter 0) (color 0 0 0 0)
   )
-  (junction (at 69.85 158.115) (diameter 0) (color 0 0 0 0)
-  )
-  (junction (at 69.85 168.275) (diameter 0) (color 0 0 0 0)
-  )
   (junction (at 172.72 79.375) (diameter 0) (color 0 0 0 0)
   )
-  (junction (at 57.15 149.225) (diameter 0) (color 0 0 0 0)
-  )
   (junction (at 83.185 79.375) (diameter 0) (color 0 0 0 0)
   )
@@
   )
   (junction (at 219.075 107.95) (diameter 0) (color 0 0 0 0)
-  )
-  (junction (at 80.01 168.275) (diameter 0) (color 0 0 0 0)
   )
   (junction (at 172.72 74.295) (diameter 0) (color 0 0 0 0)
@@
   (no_connect (at 132.08 125.095))
   (no_connect (at 132.08 122.555))
-  (wire (pts (xy 57.15 149.225) (xy 62.23 149.225))
-    (stroke (width 0) (type default))
-  )
   (wire (pts (xy 113.03 130.175) (xy 114.935 130.175))
     (stroke (width 0) (type default))
@@
     (stroke (width 0) (type default))
   )
-  (wire (pts (xy 80.01 168.275) (xy 83.82 168.275))
-    (stroke (width 0) (type default))
-  )
-  (wire (pts (xy 57.15 154.305) (xy 57.15 158.115))
-    (stroke (width 0) (type default))
-  )
   (wire (pts (xy 114.935 86.995) (xy 131.445 86.995))
     (stroke (width 0) (type default))
@@
     (stroke (width 0) (type default))
   )
-  (wire (pts (xy 69.85 158.115) (xy 69.85 168.275))
-    (stroke (width 0) (type default))
-  )
   (wire (pts (xy 173.99 76.835) (xy 173.99 81.915))
     (stroke (width 0) (type default))
@@
     (stroke (width 0) (type default))
   )
-  (wire (pts (xy 80.01 149.225) (xy 80.01 168.275))
-    (stroke (width 0) (type default))
-  )
   (wire (pts (xy 114.935 130.175) (xy 132.08 130.175))
     (stroke (width 0) (type default))
@@
     (stroke (width 0) (type default))
   )
-  (wire (pts (xy 57.15 158.115) (xy 69.85 158.115))
-    (stroke (width 0) (type default))
-  )
   (wire (pts (xy 172.72 74.295) (xy 172.72 79.375))
     (stroke (width 0) (type default))
@@
     (stroke (width 0) (type default))
   )
-  (wire (pts (xy 77.47 149.225) (xy 80.01 149.225))
-    (stroke (width 0) (type default))
-  )
   (wire (pts (xy 100.33 130.175) (xy 100.33 132.715))
     (stroke (width 0) (type default))
@@
   )
   (wire (pts (xy 114.935 79.375) (xy 131.445 79.375))
-    (stroke (width 0) (type default))
-  )
-  (wire (pts (xy 62.23 168.275) (xy 69.85 168.275))
     (stroke (width 0) (type default))
   )
@@
     (at 95.25 142.875 0)
     (effects (font (size 1.27 1.27)) (justify left bottom))
-  )
-  (text "Reset Generator" (at 53.975 140.335 0)
-    (effects (font (size 2.54 2.54) (thickness 0.254) bold italic) (justify left bottom))
   )
   (global_label "CLK_4MHz" (shape input) (at 116.205 66.675 0) (fields_autoplaced)
@@
     (property "Intersheetrefs" "${INTERSHEET_REFS}" (at 166.6753 79.375 0)
       (effects (font (size 1.27 1.27)) (justify left) hide)
-    )
-  )
-  (global_label "~{RESET}" (shape output) (at 62.23 168.275 180) (fields_autoplaced)
-    (effects (font (size 1.27 1.27)) (justify right))
-    (property "Intersheetrefs" "${INTERSHEET_REFS}" (at 54.0717 168.1956 0)
-      (effects (font (size 1.27 1.27)) (justify right) hide)
     )
   )
@@
     )
   )
-  (symbol (lib_id "jrt-ICs:DS1813") (at 69.85 150.495 0) (unit 1)
-    (in_bom yes) (on_board yes) (dnp no) (fields_autoplaced)
-    (property "Reference" "U203" (at 69.85 141.766 0)
-      (effects (font (size 1.27 1.27)))
-    )
-    (property "Value" "DS1813" (at 69.85 144.3029 0)
-      (effects (font (size 1.27 1.27)))
-    )
-    (property "Footprint" "Package_TO_SOT_THT:TO-92_Inline" (at 69.85 170.815 0)
-      (effects (font (size 1.27 1.27)) hide)
-    )
-    (property "Datasheet" "https://www.analog.com/media/en/technical-documentation/data-sheets/DS1813.pdf" (at 69.85 173.355 0)
-      (effects (font (size 1.27 1.27)) hide)
-    )
-    (pin "1")
-    (pin "2")
-    (pin "3")
-    (instances
-      (project "pg09-system"
-        (path "/44572023-3621-4b3a-bd53-c3b2b3f42871/4db01e9b-9f77-42a7-9351-8914253ebfe9"
-          (reference "U203") (unit 1)
-        )
-      )
-    )
-  )
   (symbol (lib_id "Device:R_Small") (at 227.33 88.265 180) (unit 1)
     (in_bom yes) (on_board yes) (dnp no)
@@
         (path "/44572023-3621-4b3a-bd53-c3b2b3f42871/4db01e9b-9f77-42a7-9351-8914253ebfe9"
           (reference "#PWR0211") (unit 1)
-        )
-      )
-    )
-  )
-  (symbol (lib_id "Switch:SW_Push") (at 74.93 168.275 0) (unit 1)
-    (in_bom yes) (on_board yes) (dnp no)
-    (property "Reference" "SW201" (at 74.93 161.6542 0)
-      (effects (font (size 1.27 1.27)))
-    )
-    (property "Value" "Reset" (at 74.93 164.1911 0)
-      (effects (font (size 1.27 1.27)))
-    )
-    (property "Footprint" "Button_Switch_THT:SW_PUSH_6mm" (at 74.93 163.195 0)
-      (effects (font (size 1.27 1.27)) hide)
-    )
-    (property "Datasheet" "~" (at 74.93 163.195 0)
-      (effects (font (size 1.27 1.27)) hide)
-    )
-    (pin "1")
-    (pin "2")
-    (instances
-      (project "pg09-system"
-        (path "/44572023-3621-4b3a-bd53-c3b2b3f42871/4db01e9b-9f77-42a7-9351-8914253ebfe9"
-          (reference "SW201") (unit 1)
         )
       )
@@
         (path "/44572023-3621-4b3a-bd53-c3b2b3f42871/4db01e9b-9f77-42a7-9351-8914253ebfe9"
           (reference "J201") (unit 1)
-        )
-      )
-    )
-  )
-  (symbol (lib_id "power:GND") (at 83.82 168.275 0) (unit 1)
-    (in_bom yes) (on_board yes) (dnp no) (fields_autoplaced)
-    (property "Reference" "#PWR0219" (at 83.82 174.625 0)
-      (effects (font (size 1.27 1.27)) hide)
-    )
-    (property "Value" "GND" (at 83.82 172.7184 0)
-      (effects (font (size 1.27 1.27)))
-    )
-    (property "Footprint" "" (at 83.82 168.275 0)
-      (effects (font (size 1.27 1.27)) hide)
-    )
-    (property "Datasheet" "" (at 83.82 168.275 0)
-      (effects (font (size 1.27 1.27)) hide)
-    )
-    (pin "1")
-    (instances
-      (project "pg09-system"
-        (path "/44572023-3621-4b3a-bd53-c3b2b3f42871/4db01e9b-9f77-42a7-9351-8914253ebfe9"
-          (reference "#PWR0219") (unit 1)
         )
       )
@@
     )
   )
-  (symbol (lib_id "Device:R_Small") (at 57.15 151.765 180) (unit 1)
-    (in_bom yes) (on_board yes) (dnp no)
-    (property "Reference" "R203" (at 50.8 150.495 0)
-      (effects (font (size 1.27 1.27)) (justify right))
-    )
-    (property "Value" "3K3" (at 52.07 153.035 0)
-      (effects (font (size 1.27 1.27)) (justify right))
-    )
-    (property "Footprint" "Resistor_THT:R_Axial_DIN0207_L6.3mm_D2.5mm_P7.62mm_Horizontal" (at 57.15 151.765 0)
-      (effects (font (size 1.27 1.27)) hide)
-    )
-    (property "Datasheet" "~" (at 57.15 151.765 0)
-      (effects (font (size 1.27 1.27)) hide)
-    )
-    (pin "1")
-    (pin "2")
-    (instances
-      (project "pg09-system"
-        (path "/44572023-3621-4b3a-bd53-c3b2b3f42871/4db01e9b-9f77-42a7-9351-8914253ebfe9"
-          (reference "R203") (unit 1)
-        )
-      )
-    )
-  )
   (symbol (lib_id "power:GND") (at 234.95 90.805 0) (unit 1)
     (in_bom yes) (on_board yes) (dnp no) (fields_autoplaced)
@@
         )
       )
-    )
-  )
-  (symbol (lib_id "power:+5V") (at 57.15 149.225 0) (unit 1)
-    (in_bom yes) (on_board yes) (dnp no) (fields_autoplaced)
-    (property "Reference" "#PWR0218" (at 57.15 153.035 0)
-      (effects (font (size 1.27 1.27)) hide)
-    )
-    (property "Value" "+5V" (at 57.15 145.6492 0)
-      (effects (font (size 1.27 1.27)))
-    )
-    (property "Footprint" "" (at 57.15 149.225 0)
-      (effects (font (size 1.27 1.27)) hide)
-    )
-    (property "Datasheet" "" (at 57.15 149.225 0)
-      (effects (font (size 1.27 1.27)) hide)
-    )
-    (pin "1")
-    (instances
-      (project "pg09-system"
-        (path "/44572023-3621-4b3a-bd53-c3b2b3f42871/4db01e9b-9f77-42a7-9351-8914253ebfe9"
-          (reference "#PWR0218") (unit 1)
-        )
-      )

Commit message: Remove CPU_E and the associated circuitry -- measurements on a prototype indicate that it's not necessary.
Parts:
- removed Q201: 2N7000, Package_TO_SOT_THT:TO-92_Inline, symbol Transistor_FET:2N7000
- removed R201: 150, Resistor_THT:R_Axial_DIN0207_L6.3mm_D2.5mm_P7.62mm_Horizontal, symbol Device:R_Small
- removed R202: 3K3, Resistor_THT:R_Axial_DIN0207_L6.3mm_D2.5mm_P7.62mm_Horizontal, symbol Device:R_Small
- removed R204, R205: 100, Resistor_THT:R_Axial_DIN0207_L6.3mm_D2.5mm_P7.62mm_Horizontal, symbol Device:R_Small
Connections:
- net E: now also U201.10 (Q)
- net Q: now also U201.13 (~{K}), U201.14 (J), U201.6 (Q)
Other:
- note removed: "Series resistors to tamp down over- and under-shoot of E and Q signals. Values may need adjustment."

Commit message: Re-arrange CLKSEL pins for board layout reasons.
Connections:
- net D0: now also U204.21 (IO8); no longer U204.23 (IO10)
- net D1: now also U204.20 (IO7); no longer U204.22 (IO9)
- net D2: now also U204.19 (IO6); no longer U204.21 (IO8)
- net D3: now also U204.18 (IO5); no longer U204.20 (IO7)
- net D4: now also U204.17 (IO4); no longer U204.19 (IO6)
- net D5: now also U204.16 (IO3); no longer U204.18 (IO5)
- net D6: now also U204.15 (IO2); no longer U204.17 (IO4)
- net D7: now also U204.14 (IO1); no longer U204.16 (IO3)
- net E: now also U204.13 (I12); no longer U204.1 (I1/CLK)
- net at U201.12 (C), U201.4 (C): now also U204.23 (IO10); no longer U204.14 (IO1)

Commit message: Move the PHI2/E input to the CLKSEL GAL up to pin 22, again, for board layout reasons.
Connections:
- net E: now also U204.22 (IO9); no longer U204.13 (I12)
Changed lines of the file:
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@@
   (junction (at 219.075 107.95) (diameter 0) (color 0 0 0 0)
   )
+  (no_connect (at 131.572 102.362))
   (no_connect (at 108.585 89.535))
   (no_connect (at 131.572 74.422))
   (no_connect (at 108.585 84.455))
-  (no_connect (at 156.972 94.742))
   (no_connect (at 191.77 81.915))
   (no_connect (at 132.08 125.095))
@@
     (stroke (width 0) (type default))
   )
+  (wire (pts (xy 156.972 94.742) (xy 161.29 94.742))
+    (stroke (width 0) (type default))
+  )
   (wire (pts (xy 219.075 113.03) (xy 229.235 113.03))
     (stroke (width 0) (type default))
@@
     )
   )
-  (global_label "E" (shape input) (at 131.572 102.362 180) (fields_autoplaced)
-    (effects (font (size 1.27 1.27)) (justify right))
-    (property "Intersheetrefs" "${INTERSHEET_REFS}" (at 127.5172 102.362 0)
-      (effects (font (size 1.27 1.27)) (justify right) hide)
-    )
-  )
+  (global_label "E" (shape input) (at 161.29 94.742 0) (fields_autoplaced)
+    (effects (font (size 1.27 1.27)) (justify left))
+    (property "Intersheetrefs" "${INTERSHEET_REFS}" (at 165.3448 94.742 0)
+      (effects (font (size 1.27 1.27)) (justify left) hide)
+    )
+  )

Commit message: Pull-up /RESET on RN201.
Connections:
- net ~{RESET}: now reaches RN201.5 (R4)
- no-connect marks 7 -> 6
Other:
- note added: "Reset and NMI buttons on main sheet rely on these pull-ups here."
Changed lines of the file:
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@@
   (junction (at 114.935 79.375) (diameter 0) (color 0 0 0 0)
   )
-  (junction (at 113.665 127.635) (diameter 0) (color 0 0 0 0)
+  (junction (at 114.935 130.048) (diameter 0) (color 0 0 0 0)
   )
   (junction (at 83.185 89.535) (diameter 0) (color 0 0 0 0)
@@
   (junction (at 116.205 81.915) (diameter 0) (color 0 0 0 0)
   )
-  (junction (at 114.935 130.175) (diameter 0) (color 0 0 0 0)
-  )
   (junction (at 229.235 113.03) (diameter 0) (color 0 0 0 0)
   )
@@
   (junction (at 229.235 107.95) (diameter 0) (color 0 0 0 0)
   )
-  (junction (at 116.205 132.715) (diameter 0) (color 0 0 0 0)
-  )
   (junction (at 100.33 132.715) (diameter 0) (color 0 0 0 0)
   )
@@
   (junction (at 208.915 113.03) (diameter 0) (color 0 0 0 0)
   )
+  (junction (at 113.665 127.508) (diameter 0) (color 0 0 0 0)
+  )
   (junction (at 113.665 76.835) (diameter 0) (color 0 0 0 0)
+  )
+  (junction (at 116.205 132.588) (diameter 0) (color 0 0 0 0)
   )
   (junction (at 83.185 81.915) (diameter 0) (color 0 0 0 0)
@@
   (no_connect (at 108.585 84.455))
   (no_connect (at 191.77 81.915))
-  (no_connect (at 132.08 125.095))
-  (no_connect (at 132.08 122.555))
+  (no_connect (at 132.08 124.968))
   (wire (pts (xy 113.03 130.175) (xy 114.935 130.175))
     (stroke (width 0) (type default))
@@
     (stroke (width 0) (type default))
   )
+  (wire (pts (xy 125.476 122.428) (xy 132.08 122.428))
+    (stroke (width 0) (type default))
+  )
   (wire (pts (xy 228.6 76.835) (xy 228.6 66.802))
     (stroke (width 0) (type default))
@@
     (stroke (width 0) (type default))
   )
-  (wire (pts (xy 125.73 117.475) (xy 132.08 117.475))
+  (wire (pts (xy 125.73 117.348) (xy 132.08 117.348))
     (stroke (width 0) (type default))
   )
@@
     (stroke (width 0) (type default))
   )
+  (wire (pts (xy 113.665 127.508) (xy 113.665 127.635))
+    (stroke (width 0) (type default))
+  )
   (wire (pts (xy 113.665 59.055) (xy 113.665 76.835))
     (stroke (width 0) (type default))
@@
     (stroke (width 0) (type default))
   )
-  (wire (pts (xy 114.935 130.175) (xy 132.08 130.175))
+  (wire (pts (xy 114.935 130.048) (xy 132.08 130.048))
     (stroke (width 0) (type default))
   )
@@
     (stroke (width 0) (type default))
   )
+  (wire (pts (xy 116.205 132.588) (xy 116.205 132.715))
+    (stroke (width 0) (type default))
+  )
   (wire (pts (xy 219.075 113.03) (xy 229.235 113.03))
     (stroke (width 0) (type default))
   )
-  (wire (pts (xy 116.205 89.662) (xy 116.205 132.715))
-    (stroke (width 0) (type default))
-  )
-  (wire (pts (xy 114.935 87.122) (xy 114.935 130.175))
+  (wire (pts (xy 116.205 89.662) (xy 116.205 132.588))
+    (stroke (width 0) (type default))
+  )
+  (wire (pts (xy 114.935 87.122) (xy 114.935 130.048))
     (stroke (width 0) (type default))
   )
@@
     (stroke (width 0) (type default))
   )
+  (wire (pts (xy 114.935 130.048) (xy 114.935 130.175))
+    (stroke (width 0) (type default))
+  )
   (wire (pts (xy 83.185 81.915) (xy 83.185 84.455))
     (stroke (width 0) (type default))
@@
     (stroke (width 0) (type default))
   )
-  (wire (pts (xy 113.665 84.582) (xy 113.665 127.635))
+  (wire (pts (xy 113.665 84.582) (xy 113.665 127.508))
+    (stroke (width 0) (type default))
+  )
+  (wire (pts (xy 132.08 119.888) (xy 132.08 120.015))
     (stroke (width 0) (type default))
   )
@@
     (stroke (width 0) (type default))
   )
-  (wire (pts (xy 113.665 127.635) (xy 132.08 127.635))
+  (wire (pts (xy 113.665 127.508) (xy 132.08 127.508))
     (stroke (width 0) (type default))
   )
@@
     (stroke (width 0) (type default))
   )
-  (wire (pts (xy 116.205 132.715) (xy 132.08 132.715))
+  (wire (pts (xy 116.205 132.588) (xy 132.08 132.588))
     (stroke (width 0) (type default))
   )
@@
   (text "4MHz" (at 98.425 128.27 0)
     (effects (font (size 1.27 1.27)) (justify right bottom))
+  )
+  (text "Reset and NMI buttons on main\nsheet rely on these pull-ups here."
+    (at 141.478 123.444 0)
+    (effects (font (size 1.27 1.27)) (justify left bottom))
   )
   (text "2MHz" (at 98.425 130.81 0)
@@
     )
   )
+  (global_label "~{RESET}" (shape input) (at 125.476 122.428 180) (fields_autoplaced)
+    (effects (font (size 1.27 1.27)) (justify right))
+    (property "Intersheetrefs" "${INTERSHEET_REFS}" (at 116.8251 122.428 0)
+      (effects (font (size 1.27 1.27)) (justify right) hide)
+    )
+  )
   (global_label "D4" (shape output) (at 156.972 82.042 0) (fields_autoplaced)
     (effects (font (size 1.27 1.27)) (justify left))
@@
     )
   )
-  (global_label "~{FIRQ}" (shape input) (at 125.73 117.475 180) (fields_autoplaced)
+  (global_label "~{FIRQ}" (shape input) (at 125.73 117.348 180) (fields_autoplaced)
     (effects (font (size 1.27 1.27)) (justify right))
-    (property "Intersheetrefs" "${INTERSHEET_REFS}" (at 118.5303 117.475 0)
+    (property "Intersheetrefs" "${INTERSHEET_REFS}" (at 118.5303 117.348 0)
       (effects (font (size 1.27 1.27)) (justify right) hide)
     )
@@
     )
   )
-  (global_label "~{NMI}" (shape input) (at 132.08 114.935 180) (fields_autoplaced)
+  (global_label "~{NMI}" (shape input) (at 132.08 114.808 180) (fields_autoplaced)
     (effects (font (size 1.27 1.27)) (justify right))
-    (property "Intersheetrefs" "${INTERSHEET_REFS}" (at 125.7875 114.935 0)
+    (property "Intersheetrefs" "${INTERSHEET_REFS}" (at 125.7875 114.808 0)
       (effects (font (size 1.27 1.27)) (justify right) hide)
     )
@@
     )
   )
-  (symbol (lib_id "Device:R_Network08") (at 137.16 125.095 270) (unit 1)
-    (in_bom yes) (on_board yes) (dnp no) (fields_autoplaced)
-    (property "Reference" "RN201" (at 136.906 109.855 90)
-      (effects (font (size 1.27 1.27)))
-    )
-    (property "Value" "10K" (at 136.906 112.395 90)
-      (effects (font (size 1.27 1.27)))
-    )
-    (property "Footprint" "Resistor_THT:R_Array_SIP9" (at 137.16 137.16 90)
-      (effects (font (size 1.27 1.27)) hide)
-    )
-    (property "Datasheet" "http://www.vishay.com/docs/31509/csc.pdf" (at 137.16 125.095 0)
+  (symbol (lib_id "Device:R_Network08") (at 137.16 124.968 270) (unit 1)
+    (in_bom yes) (on_board yes) (dnp no) (fields_autoplaced)
+    (property "Reference" "RN201" (at 136.906 109.728 90)
+      (effects (font (size 1.27 1.27)))
+    )
+    (property "Value" "10K" (at 136.906 112.268 90)
+      (effects (font (size 1.27 1.27)))
+    )
+    (property "Footprint" "Resistor_THT:R_Array_SIP9" (at 137.16 137.033 90)
+      (effects (font (size 1.27 1.27)) hide)
+    )
+    (property "Datasheet" "http://www.vishay.com/docs/31509/csc.pdf" (at 137.16 124.968 0)
       (effects (font (size 1.27 1.27)) hide)
     )
@@
     )
   )
-  (symbol (lib_id "power:+5V") (at 142.24 114.935 270) (unit 1)
-    (in_bom yes) (on_board yes) (dnp no) (fields_autoplaced)
-    (property "Reference" "#PWR0221" (at 138.43 114.935 0)
-      (effects (font (size 1.27 1.27)) hide)
-    )
-    (property "Value" "+5V" (at 146.05 115.57 90)
-      (effects (font (size 1.27 1.27)) (justify left))
-    )
-    (property "Footprint" "" (at 142.24 114.935 0)
-      (effects (font (size 1.27 1.27)) hide)
-    )
-    (property "Datasheet" "" (at 142.24 114.935 0)
-      (effects (font (size 1.27 1.27)) hide)
-    )
+  (symbol (lib_id "power:+5V") (at 142.24 114.808 270) (unit 1)
+    (in_bom yes) (on_board yes) (dnp no) (fields_autoplaced)
+    (property "Reference" "#PWR0221" (at 138.43 114.808 0)
+      (effects (font (size 1.27 1.27)) hide)
+    )
+    (property "Value" "+5V" (at 146.05 115.443 90)
+      (effects (font (size 1.27 1.27)) (justify left))
+    )
+    (property "Footprint" "" (at 142.24 114.808 0)
+      (effects (font (size 1.27 1.27)) hide)
+    )
+    (property "Datasheet" "" (at 142.24 114.808 0)
+      (effects (font (size 1.27 1.27)) hide)
+    )

Commit message: Tweak the reset and NMI circuits -- no pull-ups on those signals needed; the DS1813 has us covered.  Add power-on-reset delay of ~0.5 seconds.
Connections:
- net ~{NMI} is gone; now on net ~{FIRQ}: RN201.2 (R1)
- net ~{FIRQ}: no longer RN201.3 (R2)
- net ~{HALT}: now also RN201.3 (R2); no longer RN201.4 (R3)
- net ~{RESET}: no longer names the net of RN201.5 (R4)
- no-connect marks 6 -> 8
Other:
- note removed: "Reset and NMI buttons on main sheet rely on these pull-ups here."
Changed lines of the file:
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@@
   (no_connect (at 108.585 84.455))
   (no_connect (at 191.77 81.915))
+  (no_connect (at 132.08 122.428))
   (no_connect (at 132.08 124.968))
+  (no_connect (at 132.08 119.888))
   (wire (pts (xy 113.03 130.175) (xy 114.935 130.175))
     (stroke (width 0) (type default))
@@
     (stroke (width 0) (type default))
   )
-  (wire (pts (xy 125.476 122.428) (xy 132.08 122.428))
-    (stroke (width 0) (type default))
-  )
   (wire (pts (xy 228.6 76.835) (xy 228.6 66.802))
     (stroke (width 0) (type default))
@@
   )
   (wire (pts (xy 113.665 84.582) (xy 113.665 127.508))
-    (stroke (width 0) (type default))
-  )
-  (wire (pts (xy 132.08 119.888) (xy 132.08 120.015))
     (stroke (width 0) (type default))
   )
@@
   (text "4MHz" (at 98.425 128.27 0)
     (effects (font (size 1.27 1.27)) (justify right bottom))
-  )
-  (text "Reset and NMI buttons on main\nsheet rely on these pull-ups here."
-    (at 141.478 123.444 0)
-    (effects (font (size 1.27 1.27)) (justify left bottom))
   )
   (text "2MHz" (at 98.425 130.81 0)
@@
     )
   )
-  (global_label "~{RESET}" (shape input) (at 125.476 122.428 180) (fields_autoplaced)
-    (effects (font (size 1.27 1.27)) (justify right))
-    (property "Intersheetrefs" "${INTERSHEET_REFS}" (at 116.8251 122.428 0)
-      (effects (font (size 1.27 1.27)) (justify right) hide)
-    )
-  )
   (global_label "D4" (shape output) (at 156.972 82.042 0) (fields_autoplaced)
     (effects (font (size 1.27 1.27)) (justify left))
@@
     )
   )
-  (global_label "~{FIRQ}" (shape input) (at 125.73 117.348 180) (fields_autoplaced)
-    (effects (font (size 1.27 1.27)) (justify right))
-    (property "Intersheetrefs" "${INTERSHEET_REFS}" (at 118.5303 117.348 0)
+  (global_label "~{FIRQ}" (shape input) (at 132.08 114.808 180) (fields_autoplaced)
+    (effects (font (size 1.27 1.27)) (justify right))
+    (property "Intersheetrefs" "${INTERSHEET_REFS}" (at 124.8803 114.808 0)
       (effects (font (size 1.27 1.27)) (justify right) hide)
     )
@@
     )
   )
-  (global_label "~{HALT}" (shape input) (at 132.08 120.015 180) (fields_autoplaced)
-    (effects (font (size 1.27 1.27)) (justify right))
-    (property "Intersheetrefs" "${INTERSHEET_REFS}" (at 124.7594 120.015 0)
-      (effects (font (size 1.27 1.27)) (justify right) hide)
-    )
-  )
-  (global_label "~{NMI}" (shape input) (at 132.08 114.808 180) (fields_autoplaced)
-    (effects (font (size 1.27 1.27)) (justify right))
-    (property "Intersheetrefs" "${INTERSHEET_REFS}" (at 125.7875 114.808 0)
-      (effects (font (size 1.27 1.27)) (justify right) hide)
-    )
+  (global_label "~{HALT}" (shape input) (at 125.73 117.348 180) (fields_autoplaced)
+    (effects (font (size 1.27 1.27)) (justify right))
+    (property "Intersheetrefs" "${INTERSHEET_REFS}" (at 118.4094 117.348 0)
+      (effects (font (size 1.27 1.27)) (justify right) hide)
+    )

Commit message: Re-do the UARTs using a single TL16C2552 dual-UART in PLCC-44 package.
Parts:
- X201: value ACO-32.000MHz -> ACO-32.0000MHz
Changed lines of the file:
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@@
   (symbol (lib_id "Oscillator:ACO-xxxMHz") (at 69.215 97.155 0) (unit 1)
     (in_bom yes) (on_board yes) (dnp no) (fields_autoplaced)
-    (property "Reference" "X201" (at 63.373 96.3203 0)
+    (property "Reference" "X201" (at 62.23 96.52 0)
       (effects (font (size 1.27 1.27)) (justify right))
     )
-    (property "Value" "ACO-32.000MHz" (at 63.373 98.8572 0)
+    (property "Value" "ACO-32.0000MHz" (at 62.23 99.06 0)
       (effects (font (size 1.27 1.27)) (justify right))
     )
