File: design-files/pg09-system-clock.kicad_sch (KiCad schematic)
At the start: 10 parts, among them J201 Clock Speed, U201 CD74ACT109, U202 CD74ACT163, U204 GAL22V10, X201 ACO-32.0000MHz

Commit message: Change the CLKSEL GAL to use /RD rather than R/W + E.  Frees up a pin to use for other purposes in a separate change.
Connections:
- net E: no longer U204.22 (IO9)
- net R/~{W} renamed ~{RD}
- no-connect marks 7 -> 8
Changed lines of the file:
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@@
   (junction (at 219.075 107.95) (diameter 0) (color 0 0 0 0)
   )
+  (no_connect (at 156.972 94.742))
   (no_connect (at 131.572 102.362))
   (no_connect (at 98.171 89.535))
@@
     (stroke (width 0) (type default))
   )
-  (wire (pts (xy 156.972 94.742) (xy 161.29 94.742))
-    (stroke (width 0) (type default))
-  )
   (wire (pts (xy 116.205 132.588) (xy 116.205 132.715))
     (stroke (width 0) (type default))
@@
     )
   )
-  (global_label "E" (shape input) (at 161.29 94.742 0) (fields_autoplaced)
-    (effects (font (size 1.27 1.27)) (justify left))
-    (property "Intersheetrefs" "${INTERSHEET_REFS}" (at 165.3448 94.742 0)
-      (effects (font (size 1.27 1.27)) (justify left) hide)
-    )
-  )
   (global_label "E" (shape output) (at 231.14 66.802 0) (fields_autoplaced)
     (effects (font (size 1.27 1.27)) (justify left))
@@
     )
   )
-  (global_label "R{slash}~{W}" (shape input) (at 123.19 99.822 180) (fields_autoplaced)
+  (global_label "~{RD}" (shape input) (at 123.19 99.822 180) (fields_autoplaced)
     (effects (font (size 1.27 1.27)) (justify right))
-    (property "Intersheetrefs" "${INTERSHEET_REFS}" (at 116.2323 99.822 0)
+    (property "Intersheetrefs" "${INTERSHEET_REFS}" (at 117.7442 99.822 0)
       (effects (font (size 1.27 1.27)) (justify right) hide)
     )

Commit message: Use a now-free pin on the CLKSEL GAL to invert /RESET into an active-high RESETH signal that can be used all over the system.  Use RESETH with the 16550 UARTs and eliminate the 74HC14 Schmitt inverter that was used there. Saves a chip, and because if the reset circuit we're using, we don't need to use a Schmitt inverter.
Connections:
- net ~{RESET}: now reaches U204.13 (I12)
- net RESETH: now reaches U204.22 (IO9)
- no-connect marks 8 -> 6
Changed lines of the file:
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@@
   (junction (at 219.075 107.95) (diameter 0) (color 0 0 0 0)
   )
-  (no_connect (at 156.972 94.742))
-  (no_connect (at 131.572 102.362))
   (no_connect (at 98.171 89.535))
   (no_connect (at 131.572 74.422))
@@
     (stroke (width 0) (type default))
   )
+  (wire (pts (xy 156.972 94.742) (xy 161.29 94.742))
+    (stroke (width 0) (type default))
+  )
   (wire (pts (xy 142.748 69.215) (xy 144.145 69.215))
     (stroke (width 0) (type default))
@@
     )
   )
+  (global_label "~{RESET}" (shape input) (at 131.572 102.362 180) (fields_autoplaced)
+    (effects (font (size 1.27 1.27)) (justify right))
+    (property "Intersheetrefs" "${INTERSHEET_REFS}" (at 122.9211 102.362 0)
+      (effects (font (size 1.27 1.27)) (justify right) hide)
+    )
+  )
   (global_label "D1" (shape output) (at 161.29 89.662 0) (fields_autoplaced)
     (effects (font (size 1.27 1.27)) (justify left))
@@
       (effects (font (size 1.27 1.27)) (justify left) hide)
     )
+  )
+  (global_label "RESETH" (shape output) (at 161.29 94.742 0) (fields_autoplaced)
+    (effects (font (size 1.27 1.27)) (justify left))
+    (property "Intersheetrefs" "${INTERSHEET_REFS}" (at 171.2714 94.742 0)
+      (effects (font (size 1.27 1.27)) (justify left) hide)
+    )

Commit message: Switch the oscillators to half-can.
Parts:
- X201: value ACO-32.0000MHz -> 32.0000MHz; footprint Oscillator:Oscillator_DIP-14 -> Oscillator:Oscillator_DIP-8; symbol Oscillator:ACO-xxxMHz -> Oscillator:CXO_DIP8
Connections:
- net +5V: now also X201.8 (Vcc); no longer X201.14 (Vcc)
- net GND: now also X201.4 (GND); no longer X201.7 (GND)
- net at U202.2 (CP): now also X201.5 (OUT); no longer X201.8 (OUT)
- no-connect marks 6 -> 7
Changed lines of the file:
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@@
   (junction (at 219.075 107.95) (diameter 0) (color 0 0 0 0)
   )
+  (no_connect (at 51.181 97.155))
   (no_connect (at 98.171 89.535))
   (no_connect (at 131.572 74.422))
@@
     )
   )
-  (symbol (lib_id "Oscillator:ACO-xxxMHz") (at 58.801 97.155 0) (unit 1)
-    (in_bom yes) (on_board yes) (dnp no) (fields_autoplaced)
-    (property "Reference" "X201" (at 51.816 96.52 0)
+  (symbol (lib_id "Oscillator:CXO_DIP8") (at 58.801 97.155 0) (unit 1)
+    (in_bom yes) (on_board yes) (dnp no)
+    (property "Reference" "X201" (at 48.387 96.52 0)
       (effects (font (size 1.27 1.27)) (justify right))
     )
-    (property "Value" "ACO-32.0000MHz" (at 51.816 99.06 0)
+    (property "Value" "32.0000MHz" (at 51.816 99.06 0)
       (effects (font (size 1.27 1.27)) (justify right))
     )
-    (property "Footprint" "Oscillator:Oscillator_DIP-14" (at 70.231 106.045 0)
-      (effects (font (size 1.27 1.27)) hide)
-    )
-    (property "Datasheet" "http://www.conwin.com/datasheets/cx/cx030.pdf" (at 56.261 97.155 0)
-      (effects (font (size 1.27 1.27)) hide)
-    )
-    (pin "1")
-    (pin "14")
-    (pin "7")
+    (property "Footprint" "Oscillator:Oscillator_DIP-8" (at 70.231 106.045 0)
+      (effects (font (size 1.27 1.27)) hide)
+    )
+    (property "Datasheet" "http://cdn-reichelt.de/documents/datenblatt/B400/OSZI.pdf" (at 56.261 97.155 0)
+      (effects (font (size 1.27 1.27)) hide)
+    )
+    (pin "1")
+    (pin "4")
+    (pin "5")
     (pin "8")
     (instances

Commit message: Overhaul how the "system registers" in IO0SEL work, paving the way to use a VIA for the interrupt enables (because that would also give us a timer).
Connections:
- net nA0 is gone; now on net ~{RD}: U204.9 (I9)
- net ~{IO0SEL} is gone; now on net ~{RESET}: U204.10 (I10)
- net ~{RD}: no longer U204.11 (I11)
- net ~{RESET}: no longer U204.13 (I12)
- net ~{WR}: now reaches RN201.4 (R3)
- net ~{FLASHWR}: now reaches RN201.5 (R4)
- net A4 renamed ~{CLKSPD}
Changed lines of the file:
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@@
   )
   (no_connect (at 51.181 97.155))
+  (no_connect (at 131.572 102.362))
   (no_connect (at 98.171 89.535))
   (no_connect (at 131.572 74.422))
+  (no_connect (at 131.572 99.822))
   (no_connect (at 191.77 81.915))
-  (no_connect (at 132.08 122.428))
   (no_connect (at 132.08 124.968))
-  (no_connect (at 132.08 119.888))
   (wire (pts (xy 113.03 130.175) (xy 114.935 130.175))
     (stroke (width 0) (type default))
@@
     (stroke (width 0) (type default))
   )
-  (wire (pts (xy 125.73 117.348) (xy 132.08 117.348))
+  (wire (pts (xy 125.984 117.348) (xy 132.08 117.348))
     (stroke (width 0) (type default))
   )
@@
     (stroke (width 0) (type default))
   )
+  (wire (pts (xy 127.508 122.428) (xy 132.08 122.428))
+    (stroke (width 0) (type default))
+  )
   (wire (pts (xy 194.31 93.345) (xy 194.31 79.375))
     (stroke (width 0) (type default))
@@
     (stroke (width 0) (type default))
   )
-  (wire (pts (xy 123.19 94.742) (xy 131.572 94.742))
+  (wire (pts (xy 121.92 94.742) (xy 131.572 94.742))
     (stroke (width 0) (type default))
   )
@@
   )
   (wire (pts (xy 66.421 97.155) (xy 72.771 97.155))
-    (stroke (width 0) (type default))
-  )
-  (wire (pts (xy 123.19 99.822) (xy 131.572 99.822))
     (stroke (width 0) (type default))
   )
@@
     )
   )
+  (global_label "~{WR}" (shape input) (at 132.08 119.888 180) (fields_autoplaced)
+    (effects (font (size 1.27 1.27)) (justify right))
+    (property "Intersheetrefs" "${INTERSHEET_REFS}" (at 126.4528 119.888 0)
+      (effects (font (size 1.27 1.27)) (justify right) hide)
+    )
+  )
   (global_label "CLK_16MHz" (shape input) (at 103.251 59.055 0) (fields_autoplaced)
     (effects (font (size 1.27 1.27)) (justify left))
@@
     )
   )
-  (global_label "~{IO0SEL}" (shape input) (at 131.572 97.282 180) (fields_autoplaced)
-    (effects (font (size 1.27 1.27)) (justify right))
-    (property "Intersheetrefs" "${INTERSHEET_REFS}" (at 122.1348 97.282 0)
-      (effects (font (size 1.27 1.27)) (justify right) hide)
-    )
-  )
   (global_label "E" (shape output) (at 231.14 66.802 0) (fields_autoplaced)
     (effects (font (size 1.27 1.27)) (justify left))
@@
     )
   )
-  (global_label "nA0" (shape input) (at 123.19 94.742 180) (fields_autoplaced)
-    (effects (font (size 1.27 1.27)) (justify right))
-    (property "Intersheetrefs" "${INTERSHEET_REFS}" (at 116.8371 94.742 0)
-      (effects (font (size 1.27 1.27)) (justify right) hide)
-    )
-  )
   (global_label "D4" (shape output) (at 156.972 82.042 0) (fields_autoplaced)
     (effects (font (size 1.27 1.27)) (justify left))
@@
     )
   )
-  (global_label "~{RESET}" (shape input) (at 131.572 102.362 180) (fields_autoplaced)
-    (effects (font (size 1.27 1.27)) (justify right))
-    (property "Intersheetrefs" "${INTERSHEET_REFS}" (at 122.9211 102.362 0)
+  (global_label "~{RESET}" (shape input) (at 131.572 97.282 180) (fields_autoplaced)
+    (effects (font (size 1.27 1.27)) (justify right))
+    (property "Intersheetrefs" "${INTERSHEET_REFS}" (at 122.9211 97.282 0)
       (effects (font (size 1.27 1.27)) (justify right) hide)
     )
@@
     )
   )
+  (global_label "~{FLASHWR}" (shape input) (at 127.508 122.428 180) (fields_autoplaced)
+    (effects (font (size 1.27 1.27)) (justify right))
+    (property "Intersheetrefs" "${INTERSHEET_REFS}" (at 116.1355 122.428 0)
+      (effects (font (size 1.27 1.27)) (justify right) hide)
+    )
+  )
   (global_label "Q" (shape output) (at 231.14 59.69 0) (fields_autoplaced)
     (effects (font (size 1.27 1.27)) (justify left))
@@
     )
   )
-  (global_label "~{RD}" (shape input) (at 123.19 99.822 180) (fields_autoplaced)
-    (effects (font (size 1.27 1.27)) (justify right))
-    (property "Intersheetrefs" "${INTERSHEET_REFS}" (at 117.7442 99.822 0)
+  (global_label "~{RD}" (shape input) (at 121.92 94.742 180) (fields_autoplaced)
+    (effects (font (size 1.27 1.27)) (justify right))
+    (property "Intersheetrefs" "${INTERSHEET_REFS}" (at 116.4742 94.742 0)
       (effects (font (size 1.27 1.27)) (justify right) hide)
     )
@@
     )
   )
-  (global_label "A4" (shape input) (at 131.572 92.202 180) (fields_autoplaced)
-    (effects (font (size 1.27 1.27)) (justify right))
-    (property "Intersheetrefs" "${INTERSHEET_REFS}" (at 126.3681 92.202 0)
+  (global_label "~{CLKSPD}" (shape input) (at 131.572 92.202 180) (fields_autoplaced)
+    (effects (font (size 1.27 1.27)) (justify right))
+    (property "Intersheetrefs" "${INTERSHEET_REFS}" (at 121.3486 92.202 0)
       (effects (font (size 1.27 1.27)) (justify right) hide)
     )
@@
     )
   )
-  (global_label "~{HALT}" (shape input) (at 125.73 117.348 180) (fields_autoplaced)
-    (effects (font (size 1.27 1.27)) (justify right))
-    (property "Intersheetrefs" "${INTERSHEET_REFS}" (at 118.4094 117.348 0)
-      (effects (font (size 1.27 1.27)) (justify right) hide)
-    )
+  (global_label "~{HALT}" (shape input) (at 125.984 117.348 180) (fields_autoplaced)
+    (effects (font (size 1.27 1.27)) (justify right))
+    (property "Intersheetrefs" "${INTERSHEET_REFS}" (at 118.6634 117.348 0)
+      (effects (font (size 1.27 1.27)) (justify right) hide)
+    )
