File: design-files/pg09-system-expansion.kicad_sch (KiCad schematic)
At the start: 1 part, among them J901 Expansion 1

Commit message: Add enough of the expanion interface to start being able to fiddle with the PCB layout.
Parts:
- added J902: Expansion 1 ext, Connector_PinHeader_2.54mm:PinHeader_2x08_P2.54mm_Vertical, symbol Connector_Generic:Conn_02x08_Odd_Even
- added J903: Expansion 2, Connector_PinHeader_2.54mm:PinHeader_2x20_P2.54mm_Vertical, symbol Connector_Generic:Conn_02x20_Odd_Even
- added J904: Expansion 2 ext, Connector_PinHeader_2.54mm:PinHeader_2x08_P2.54mm_Vertical, symbol Connector_Generic:Conn_02x08_Odd_Even
Connections:
- net ~{IRQ3} is gone; now on net ~{IRQ8}: J901.26 (Pin_26)
- net +5V: now also J903.2 (Pin_2)
- net A0: now also J903.1 (Pin_1)
- net A1: now also J903.3 (Pin_3)
- net A2: now also J903.5 (Pin_5)
- net A3: now also J903.7 (Pin_7)
- net A4: now also J903.9 (Pin_9)
- net D0: now also J903.4 (Pin_4)
- net D1: now also J903.6 (Pin_6)
- net D2: now also J903.8 (Pin_8)
- net D3: now also J903.10 (Pin_10)
- net D4: now also J903.12 (Pin_12)
- net D5: now also J903.14 (Pin_14)
- net D6: now also J903.16 (Pin_16)
- net D7: now also J903.18 (Pin_18)
- net E: now also J901.19 (Pin_19), J903.19 (Pin_19); no longer J901.17 (Pin_17)
- net GND: now also J901.17 (Pin_17), J901.21 (Pin_21), J902.1 (Pin_1), J902.2 (Pin_2), J902.5 (Pin_5), J902.6 (Pin_6), J903.17 (Pin_17), J903.21 (Pin_21), J903.39 (Pin_39), J904.1 (Pin_1), J904.2 (Pin_2), J904.5 (Pin_5), J904.6 (Pin_6)
- net R/~{W}: now also J903.11 (Pin_11)
- net ~{IO10SEL}: now also J901.27 (Pin_27), J903.27 (Pin_27); no longer J901.23 (Pin_23)
- net ~{IO11SEL}: now also J901.29 (Pin_29), J903.29 (Pin_29); no longer J901.25 (Pin_25)
- net ~{IO12SEL}: now also J901.31 (Pin_31), J903.31 (Pin_31); no longer J901.27 (Pin_27)
- net ~{IO13SEL}: now also J901.33 (Pin_33), J903.33 (Pin_33); no longer J901.29 (Pin_29)
- net ~{IO14SEL}: now also J901.35 (Pin_35), J903.35 (Pin_35); no longer J901.31 (Pin_31)
- net ~{IO15SEL}: now also J901.37 (Pin_37), J903.37 (Pin_37); no longer J901.33 (Pin_33)
- net ~{IO8SEL}: now also J901.23 (Pin_23), J903.23 (Pin_23); no longer J901.19 (Pin_19)
- net ~{IO9SEL}: now also J901.25 (Pin_25), J903.25 (Pin_25); no longer J901.21 (Pin_21)
- net ~{IRQ10}: now also J901.30 (Pin_30), J903.30 (Pin_30); no longer J901.32 (Pin_32)
- net ~{IRQ11}: now also J901.32 (Pin_32), J903.32 (Pin_32); no longer J901.34 (Pin_34)
- net ~{IRQ8}: now also J903.26 (Pin_26); no longer J901.28 (Pin_28)
- net ~{IRQ9}: now also J901.28 (Pin_28), J903.28 (Pin_28); no longer J901.30 (Pin_30)
- net ~{RD}: now also J903.13 (Pin_13)
- net ~{WR}: now also J903.15 (Pin_15)
- net ~{IRQ13}: now reaches J901.36 (Pin_36)
- net ~{IRQ13}: now also J903.36 (Pin_36)
- net ~{IRQ14}: now reaches J901.38 (Pin_38)
- net ~{IRQ14}: now also J903.38 (Pin_38)
- net ~{IRQ15}: now reaches J901.40 (Pin_40)
- net ~{IRQ15}: now also J903.40 (Pin_40)
- net ~{IRQ0} renamed ~{IRQ4}
- net ~{IRQ4}: now also J903.20 (Pin_20)
- net ~{IRQ1} renamed ~{IRQ5}
- net ~{IRQ5}: now also J903.22 (Pin_22)
- net ~{IRQ2} renamed ~{IRQ6}
- net ~{IRQ6}: now also J903.24 (Pin_24)
- new net EXP1_AUDIO_L: J902.3 (Pin_3)
- new net EXP1_AUDIO_R: J902.4 (Pin_4)
- new net EXP2_AUDIO_L: J904.3 (Pin_3)
- new net EXP2_AUDIO_R: J904.4 (Pin_4)
- new net ~{IRQ12}: J901.34 (Pin_34), J903.34 (Pin_34)
- no-connect marks 2 -> 20

Commit message: Add +12v / -12v rails for the expansion interface.
Connections:
- net +12V: now reaches J904.15 (Pin_15)
- net +12V: now also J902.15 (Pin_15)
- net -12V: now reaches J904.16 (Pin_16)
- net -12V: now also J902.16 (Pin_16)
- no-connect marks 20 -> 16
Changed lines of the file:
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@@
   (no_connect (at 91.44 143.51))
   (no_connect (at 146.685 140.97))
-  (no_connect (at 133.985 146.05))
-  (no_connect (at 146.685 146.05))
   (no_connect (at 146.685 138.43))
   (no_connect (at 78.74 140.97))
@@
   (no_connect (at 146.685 143.51))
   (no_connect (at 133.985 140.97))
-  (no_connect (at 91.44 146.05))
   (no_connect (at 91.44 138.43))
   (no_connect (at 133.985 138.43))
   (no_connect (at 78.74 135.89))
-  (no_connect (at 78.74 146.05))
   (no_connect (at 78.74 138.43))
   (no_connect (at 133.985 143.51))
@@
     )
   )
+  (symbol (lib_id "power:+12V") (at 133.985 146.05 90) (unit 1)
+    (in_bom yes) (on_board yes) (dnp no) (fields_autoplaced)
+    (property "Reference" "#PWR0919" (at 137.795 146.05 0)
+      (effects (font (size 1.27 1.27)) hide)
+    )
+    (property "Value" "+12V" (at 130.175 146.685 90)
+      (effects (font (size 1.27 1.27)) (justify left))
+    )
+    (property "Footprint" "" (at 133.985 146.05 0)
+      (effects (font (size 1.27 1.27)) hide)
+    )
+    (property "Datasheet" "" (at 133.985 146.05 0)
+      (effects (font (size 1.27 1.27)) hide)
+    )
+    (pin "1")
+    (instances
+      (project "pg09-system"
+        (path "/44572023-3621-4b3a-bd53-c3b2b3f42871/f2ee21e0-2cfa-4d23-9aa0-c0fb39e3aeb3"
+          (reference "#PWR0919") (unit 1)
+        )
+      )
+    )
+  )
   (symbol (lib_id "power:GND") (at 78.74 133.35 270) (unit 1)
     (in_bom yes) (on_board yes) (dnp no) (fields_autoplaced)
@@
         (path "/44572023-3621-4b3a-bd53-c3b2b3f42871/f2ee21e0-2cfa-4d23-9aa0-c0fb39e3aeb3"
           (reference "#PWR0902") (unit 1)
+        )
+      )
+    )
+  )
+  (symbol (lib_id "power:-12V") (at 146.685 146.05 270) (unit 1)
+    (in_bom yes) (on_board yes) (dnp no) (fields_autoplaced)
+    (property "Reference" "#PWR0920" (at 149.225 146.05 0)
+      (effects (font (size 1.27 1.27)) hide)
+    )
+    (property "Value" "-12V" (at 150.495 146.685 90)
+      (effects (font (size 1.27 1.27)) (justify left))
+    )
+    (property "Footprint" "" (at 146.685 146.05 0)
+      (effects (font (size 1.27 1.27)) hide)
+    )
+    (property "Datasheet" "" (at 146.685 146.05 0)
+      (effects (font (size 1.27 1.27)) hide)
+    )
+    (pin "1")
+    (instances
+      (project "pg09-system"
+        (path "/44572023-3621-4b3a-bd53-c3b2b3f42871/f2ee21e0-2cfa-4d23-9aa0-c0fb39e3aeb3"
+          (reference "#PWR0920") (unit 1)
         )
       )
@@
         (path "/44572023-3621-4b3a-bd53-c3b2b3f42871/f2ee21e0-2cfa-4d23-9aa0-c0fb39e3aeb3"
           (reference "#PWR0905") (unit 1)
+        )
+      )
+    )
+  )
+  (symbol (lib_id "power:+12V") (at 78.74 146.05 90) (unit 1)
+    (in_bom yes) (on_board yes) (dnp no) (fields_autoplaced)
+    (property "Reference" "#PWR0917" (at 82.55 146.05 0)
+      (effects (font (size 1.27 1.27)) hide)
+    )
+    (property "Value" "+12V" (at 74.93 146.685 90)
+      (effects (font (size 1.27 1.27)) (justify left))
+    )
+    (property "Footprint" "" (at 78.74 146.05 0)
+      (effects (font (size 1.27 1.27)) hide)
+    )
+    (property "Datasheet" "" (at 78.74 146.05 0)
+      (effects (font (size 1.27 1.27)) hide)
+    )
+    (pin "1")
+    (instances
+      (project "pg09-system"
+        (path "/44572023-3621-4b3a-bd53-c3b2b3f42871/f2ee21e0-2cfa-4d23-9aa0-c0fb39e3aeb3"
+          (reference "#PWR0917") (unit 1)
         )
       )
@@
         )
       )
+    )
+  )
+  (symbol (lib_id "power:-12V") (at 91.44 146.05 270) (unit 1)
+    (in_bom yes) (on_board yes) (dnp no) (fields_autoplaced)
+    (property "Reference" "#PWR0918" (at 93.98 146.05 0)
+      (effects (font (size 1.27 1.27)) hide)
+    )
+    (property "Value" "-12V" (at 95.25 146.685 90)
+      (effects (font (size 1.27 1.27)) (justify left))
+    )
+    (property "Footprint" "" (at 91.44 146.05 0)
+      (effects (font (size 1.27 1.27)) hide)
+    )
+    (property "Datasheet" "" (at 91.44 146.05 0)
+      (effects (font (size 1.27 1.27)) hide)
+    )
+    (pin "1")
+    (instances
+      (project "pg09-system"
+        (path "/44572023-3621-4b3a-bd53-c3b2b3f42871/f2ee21e0-2cfa-4d23-9aa0-c0fb39e3aeb3"
+          (reference "#PWR0918") (unit 1)
+        )
+      )

Commit message: Checkpoint on expansion connectors.
Parts:
- added J905: Expansion 3, Connector_PinHeader_2.54mm:PinHeader_2x20_P2.54mm_Vertical, symbol Connector_Generic:Conn_02x20_Odd_Even
- added J906: Expansion 3 ext, Connector_PinHeader_2.54mm:PinHeader_2x08_P2.54mm_Vertical, symbol Connector_Generic:Conn_02x08_Odd_Even
- added J907: Expansion 4, Connector_PinHeader_2.54mm:PinHeader_2x20_P2.54mm_Vertical, symbol Connector_Generic:Conn_02x20_Odd_Even
- added J908: Expansion 4 ext, Connector_PinHeader_2.54mm:PinHeader_2x08_P2.54mm_Vertical, symbol Connector_Generic:Conn_02x08_Odd_Even
Connections:
- net +12V: now also J906.15 (Pin_15), J908.15 (Pin_15)
- net +5V: now also J905.2 (Pin_2), J907.2 (Pin_2)
- net -12V: now also J906.16 (Pin_16), J908.16 (Pin_16)
- net A0: now also J905.1 (Pin_1), J907.1 (Pin_1)
- net A1: now also J905.3 (Pin_3), J907.3 (Pin_3)
- net A2: now also J905.5 (Pin_5), J907.5 (Pin_5)
- net A3: now also J905.7 (Pin_7), J907.7 (Pin_7)
- net A4: now also J905.9 (Pin_9), J907.9 (Pin_9)
- net D0: now also J905.4 (Pin_4), J907.4 (Pin_4)
- net D1: now also J905.6 (Pin_6), J907.6 (Pin_6)
- net D2: now also J905.8 (Pin_8), J907.8 (Pin_8)
- net D3: now also J905.10 (Pin_10), J907.10 (Pin_10)
- net D4: now also J905.12 (Pin_12), J907.12 (Pin_12)
- net D5: now also J905.14 (Pin_14), J907.14 (Pin_14)
- net D6: now also J905.16 (Pin_16), J907.16 (Pin_16)
- net D7: now also J905.18 (Pin_18), J907.18 (Pin_18)
- net E: now also J905.19 (Pin_19), J907.19 (Pin_19)
- net GND: now also J905.17 (Pin_17), J905.21 (Pin_21), J906.1 (Pin_1), J906.2 (Pin_2), J906.5 (Pin_5), J906.6 (Pin_6), J907.17 (Pin_17), J907.21 (Pin_21), J908.1 (Pin_1), J908.2 (Pin_2), J908.5 (Pin_5), J908.6 (Pin_6); no longer J901.39 (Pin_39), J903.39 (Pin_39)
- net R/~{W}: now also J905.11 (Pin_11), J907.11 (Pin_11)
- net ~{IO10SEL}: now also J905.27 (Pin_27), J907.27 (Pin_27)
- net ~{IO11SEL}: now also J905.29 (Pin_29), J907.29 (Pin_29)
- net ~{IO12SEL}: now also J905.31 (Pin_31), J907.31 (Pin_31)
- net ~{IO13SEL}: now also J905.33 (Pin_33), J907.33 (Pin_33)
- net ~{IO14SEL}: now also J905.35 (Pin_35), J907.35 (Pin_35)
- net ~{IO15SEL}: now also J905.37 (Pin_37), J907.37 (Pin_37)
- net ~{IO8SEL}: now also J905.23 (Pin_23), J907.23 (Pin_23)
- net ~{IO9SEL}: now also J905.25 (Pin_25), J907.25 (Pin_25)
- net ~{IRQ10}: now also J905.30 (Pin_30), J907.30 (Pin_30)
- net ~{IRQ11}: now also J905.32 (Pin_32), J907.32 (Pin_32)
- net ~{IRQ12}: now also J905.34 (Pin_34), J907.34 (Pin_34)
- net ~{IRQ13}: now also J905.36 (Pin_36), J907.36 (Pin_36)
- net ~{IRQ14}: now also J905.38 (Pin_38), J907.38 (Pin_38)
- net ~{IRQ15}: now also J905.40 (Pin_40), J907.40 (Pin_40)
- net ~{IRQ4}: now also J905.20 (Pin_20), J907.20 (Pin_20)
- net ~{IRQ5}: now also J905.22 (Pin_22), J907.22 (Pin_22)
- net ~{IRQ6}: now also J905.24 (Pin_24), J907.24 (Pin_24)
- net ~{IRQ8}: now also J905.26 (Pin_26), J907.26 (Pin_26)
- net ~{IRQ9}: now also J905.28 (Pin_28), J907.28 (Pin_28)
- net ~{RD}: now also J905.13 (Pin_13), J907.13 (Pin_13)
- net ~{WR}: now also J905.15 (Pin_15), J907.15 (Pin_15)
- new net EXP3_AUDIO_L: J906.3 (Pin_3)
- new net EXP3_AUDIO_R: J906.4 (Pin_4)
- new net EXP4_AUDIO_L: J908.3 (Pin_3)
- new net EXP4_AUDIO_R: J908.4 (Pin_4)
- new net ~{RESET}: J901.39 (Pin_39), J903.39 (Pin_39), J905.39 (Pin_39), J907.39 (Pin_39)
- no-connect marks 16 -> 32
Other:
- moved on the sheet: J901, J902, J903, J904

Commit message: Tweaks to the expansion interface.
Connections:
- net E: now also J901.17 (Pin_17), J903.17 (Pin_17), J905.17 (Pin_17), J907.17 (Pin_17); no longer J901.19 (Pin_19), J903.19 (Pin_19), J905.19 (Pin_19), J907.19 (Pin_19)
- net EXP1_AUDIO_L: now also J902.1 (Pin_1); no longer J902.3 (Pin_3)
- net EXP1_AUDIO_R: now also J902.2 (Pin_2); no longer J902.4 (Pin_4)
- net EXP2_AUDIO_L: now also J904.1 (Pin_1); no longer J904.3 (Pin_3)
- net EXP2_AUDIO_R: now also J904.2 (Pin_2); no longer J904.4 (Pin_4)
- net EXP3_AUDIO_L: now also J906.1 (Pin_1); no longer J906.3 (Pin_3)
- net EXP3_AUDIO_R: now also J906.2 (Pin_2); no longer J906.4 (Pin_4)
- net EXP4_AUDIO_L: now also J908.1 (Pin_1); no longer J908.3 (Pin_3)
- net EXP4_AUDIO_R: now also J908.2 (Pin_2); no longer J908.4 (Pin_4)
- net GND: now also J901.39 (Pin_39), J903.39 (Pin_39), J905.39 (Pin_39), J907.39 (Pin_39); no longer J901.17 (Pin_17), J901.21 (Pin_21), J902.1 (Pin_1), J902.2 (Pin_2), J902.5 (Pin_5), J902.6 (Pin_6), J903.17 (Pin_17), J903.21 (Pin_21), J904.1 (Pin_1), J904.2 (Pin_2), J904.5 (Pin_5), J904.6 (Pin_6), J905.17 (Pin_17), J905.21 (Pin_21), J906.1 (Pin_1), J906.2 (Pin_2), J906.5 (Pin_5), J906.6 (Pin_6), J907.17 (Pin_17), J907.21 (Pin_21), J908.1 (Pin_1), J908.2 (Pin_2), J908.5 (Pin_5), J908.6 (Pin_6)
- net ~{RESET}: now also J901.19 (Pin_19), J903.19 (Pin_19), J905.19 (Pin_19), J907.19 (Pin_19); no longer J901.39 (Pin_39), J903.39 (Pin_39), J905.39 (Pin_39), J907.39 (Pin_39)
- new net ~{HALT}: J901.21 (Pin_21), J903.21 (Pin_21), J905.21 (Pin_21), J907.21 (Pin_21)
- no-connect marks 32 -> 48

Commit message: IRQ12 is reserved for keyboard, IRQ15 is reserved for video.  Take them off of the expansion interface.
Connections:
- removed net ~{IRQ12}: J901.34 (Pin_34), J903.34 (Pin_34), J905.34 (Pin_34), J907.34 (Pin_34)
- removed net ~{IRQ15}: J901.40 (Pin_40), J903.40 (Pin_40), J905.40 (Pin_40), J907.40 (Pin_40)
- no-connect marks 48 -> 56
